File: Schematics/RESHA/pg_11.kicad_sch (KiCad schematic)
At the start: 0 parts

Commit message: Add the RESHA backplane pins, as an approximation
Parts:
- added GB1, GB10, GB100, GB101, GB102, GB1020, GB103, GB1039, GB104, GB1040, GB105, GB106, GB107, GB108, GB109, GB11, GB110, GB111, GB112, GB113, GB1136, GB114, GB115, GB116, GB117, GB118, GB119, GB12, GB121, GB122, GB123, GB124, GB125, GB126, GB127, GB128, GB129, GB13, GB130, GB131, GB132, GB133, GB134, GB135, GB137, GB14, GB141, GB142, GB143, GB144, GB145, GB146, GB147, GB148, GB149, GB15, GB150, GB16, GB17, GB18, GB19, GB2, GB20, GB200, GB201, GB203, GB2039, GB204, GB2040, GB206, GB207, GB21, GB2136, GB22, GB23, GB24, GB25, GB26, GB27, GB28, GB29, GB30, GB31, GB32, GB33, GB34, GB35, GB36, GB37, GB38, GB4, GB41, GB42, GB43, GB44, GB45, GB46, GB47, GB48, GB49, GB5, GB50, GB51, GB52, GB53, GB54, GB55, GB56, GB57, GB58, GB59, GB6, GB60, GB61, GB62, GB63, GB64, GB65, GB66, GB67, GB68, GB69, GB70, GB71, GB72, GB73, GB76, GB77, GB78, GB79, GB8, GB80, GB81, GB82, GB83, GB84, GB85, GB86, GB87, GB88, GB89, GB9, GB90, GB91, GB92, GB93, GB94, GB95, GB96, GB97, GB98, GB99: GB, symbol r1000:GB
Connections:
- new net +5V: GB10.1, GB100.1, GB119.1, GB20.1, GB2039.1, GB2040.1, GB29.1, GB30.1, GB49.1, GB50.1, GB61.1, GB62.1, GB79.1, GB80.1, GB9.1, GB99.1
- new net B_CLAMP~: GB73.1
- new net B_CLK_2X: GB148.1
- new net B_CLK_MARGIN: GB36.1
- new net B_CLK~2X: GB147.1
- new net B_CONS_CTS: GB41.1
- new net B_CONS_DCD: GB37.1
- new net B_CONS_DSR: GB38.1
- new net B_CONS_DTR_TTL: GB45.1
- new net B_CONS_RTS_TTL: GB44.1
- new net B_CONS_RXD: GB42.1
- new net B_CONS_TXD_TTL: GB43.1
- new net B_CPU_RUNNING: GB64.1
- new net B_DCH_ACTIVE: GB71.1
- new net B_EXT_A09: GB16.1
- new net B_EXT_A10: GB17.1
- new net B_EXT_A11: GB18.1
- new net B_EXT_D0: GB28.1
- new net B_EXT_D1: GB27.1
- new net B_EXT_D2: GB26.1
- new net B_EXT_D3: GB25.1
- new net B_EXT_D4: GB24.1
- new net B_EXT_D5: GB23.1
- new net B_EXT_D6: GB22.1
- new net B_EXT_D7: GB21.1
- new net B_EXT_ID0: GB204.1
- new net B_EXT_ID1: GB203.1
- new net B_EXT_ID2: GB15.1
- new net B_EXT_~WR: GB32.1
- new net B_EXT~CS: GB33.1
- new net B_EXT~LEVEL1: GB34.1
- new net B_EXT~LEVEL6: GB35.1
- new net B_EXT~RD: GB31.1
- new net B_FP_LED0: GB57.1
- new net B_FP_LED1: GB59.1
- new net B_FP_LED2: GB60.1
- new net B_FP_LED3: GB63.1
- new net B_FP_SWITCH: GB72.1
- new net B_IOP_EPO: GB13.1
- new net B_IOP_HALT: GB68.1
- new net B_IOP_RUNNING: GB67.1
- new net B_M12V: GB58.1
- new net B_MARGIN_HI: GB11.1
- new net B_MARGIN_LO: GB14.1
- new net B_MODEM_CTS: GB48.1
- new net B_MODEM_DCD: GB46.1
- new net B_MODEM_DSR: GB47.1
- new net B_MODEM_DTR_TTL: GB56.1
- new net B_MODEM_RTS_TTL: GB55.1
- new net B_MODEM_RXD: GB51.1
- new net B_MODEM_TXD_TTL: GB52.1
- new net B_P12V: GB65.1, GB66.1
- new net B_PS0_ADJUST: GB4.1
- new net B_PS0_ENABLE: GB5.1
- new net B_PS0~ACFAIL: GB6.1
- new net B_PWR_MARGIN: GB12.1
- new net B_RESET: GB127.1
- new net B_RESET~: GB8.1
- new net B_TEMP_REF: GB206.1
- new net B_TEMP_SENSE: GB207.1
- new net GND: GB1.1, GB1020.1, GB1039.1, GB1040.1, GB109.1, GB110.1, GB129.1, GB130.1, GB149.1, GB150.1, GB19.1, GB2.1, GB53.1, GB54.1, GB69.1, GB70.1, GB89.1, GB90.1
- new net UNI_A00~: GB121.1
- new net UNI_A01~: GB122.1
- new net UNI_A02~: GB118.1
- new net UNI_A03~: GB141.1
- new net UNI_A04~: GB137.1
- new net UNI_A05~: GB142.1
- new net UNI_A06~: GB1136.1
- new net UNI_A07~: GB134.1
- new net UNI_A08~: GB133.1
- new net UNI_A09~: GB2136.1
- new net UNI_A10~: GB135.1
- new net UNI_A11~: GB132.1
- new net UNI_A12~: GB113.1
- new net UNI_A13~: GB128.1
- new net UNI_A14~: GB131.1
- new net UNI_A15~: GB114.1
- new net UNI_A16~: GB116.1
- new net UNI_A17~: GB115.1
- new net UNI_A18~: GB77.1
- new net UNI_A19~: GB76.1
- new net UNI_ACL~: GB200.1
- new net UNI_BBSY~: GB144.1
- new net UNI_BGI4: GB107.1
- new net UNI_BGI5: GB108.1
- new net UNI_BGI6: GB111.1
- new net UNI_BGI7: GB112.1
- new net UNI_C0~: GB126.1
- new net UNI_C1~: GB117.1
- new net UNI_D00~: GB96.1
- new net UNI_D01~: GB95.1
- new net UNI_D02~: GB98.1
- new net UNI_D03~: GB97.1
- new net UNI_D04~: GB93.1
- new net UNI_D05~: GB94.1
- new net UNI_D06~: GB101.1
- new net UNI_D07~: GB92.1
- new net UNI_D08~: GB91.1
- new net UNI_D09~: GB88.1
- new net UNI_D10~: GB87.1
- new net UNI_D11~: GB85.1
- new net UNI_D12~: GB86.1
- new net UNI_D13~: GB84.1
- new net UNI_D14~: GB83.1
- new net UNI_D15~: GB82.1
- new net UNI_DCLO~: GB201.1
- new net UNI_DR4~: GB103.1
- new net UNI_DR5~: GB104.1
- new net UNI_DR6~: GB105.1
- new net UNI_DR7~: GB106.1
- new net UNI_INIT~: GB102.1
- new net UNI_INTR~: GB125.1
- new net UNI_MSYN~: GB123.1
- new net UNI_NPG1: GB143.1
- new net UNI_NPR~: GB145.1
- new net UNI_PA~: GB78.1
- new net UNI_PB~: GB81.1
- new net UNI_SACK~: GB146.1
- new net UNI_SSYN~: GB124.1
Other:
- title: RESHA 11 -> BACK PANEL CONNECTIONS
