File: Schematics/VAL/pg_56.kicad_sch (KiCad schematic)
At the start: 12 parts, among them U5801 2167, U5802 2167, U5803 2167, U5804 2167, U5805 2167, U5806 2167, U5807 2167, U5808 2167, U5809 93S48, U5810 93S48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

Commit message: Use backplane clocks
Connections:
- net WCS.B1.A0 renamed WCS.A0
- net WCS.B1.A1 renamed WCS.A1
- net WCS.B1.A10 renamed WCS.A10
- net WCS.B1.A11 renamed WCS.A11
- net WCS.B1.A12 renamed WCS.A12
- net WCS.B1.A13 renamed WCS.A13
- net WCS.B1.A2 renamed WCS.A2
- net WCS.B1.A3 renamed WCS.A3
- net WCS.B1.A4 renamed WCS.A4
- net WCS.B1.A5 renamed WCS.A5
- net WCS.B1.A6 renamed WCS.A6
- net WCS.B1.A7 renamed WCS.A7
- net WCS.B1.A8 renamed WCS.A8
- net WCS.B1.A9 renamed WCS.A9

Commit message: Use megacomponents for register file and writable control store
Parts:
- removed U5802, U5803, U5804, U5805, U5806, U5807, U5808: 2167, symbol r1000:2167
- U5801: value 2167 -> XWCSRAM; symbol r1000:2167 -> r1000:XWCSRAM; Location I24 -> x99; Name WCS20 -> WCS4
Connections:
- net WCS.WE~1 is gone; now on net UIR.ALU_FUNC3: U5801.9 (D4)
- net PD: no longer U5801.11 (CS)
- net UIR.ALU_FUNC0: now also U5801.3 (D1)
- net UIR.ALU_FUNC1: now also U5801.5 (D2)
- net UIR.ALU_FUNC2: now also U5801.7 (D3)
- net UIR.ALU_FUNC4: now also U5801.11 (D5)
- net UIR.C_SOURCE: now also U5801.13 (D6)
- net UIR.M_B_SRC1: now also U5801.1 (D0); no longer U5801.12 (D)
- net UIR.P: now also U5801.15 (D7)
- net WCS.A0: now also U5801.17 (A0); no longer U5801.1 (A0)
- net WCS.A1: now also U5801.18 (A1); no longer U5801.2 (A1)
- net WCS.A10: now also U5801.27 (A10); no longer U5801.16 (A10)
- net WCS.A11: now also U5801.28 (A11); no longer U5801.17 (A11)
- net WCS.A12: now also U5801.29 (A12); no longer U5801.18 (A12)
- net WCS.A13: now also U5801.30 (A13); no longer U5801.19 (A13)
- net WCS.A2: now also U5801.19 (A2); no longer U5801.3 (A2)
- net WCS.A3: now also U5801.20 (A3); no longer U5801.4 (A3)
- net WCS.A4: now also U5801.21 (A4); no longer U5801.5 (A4)
- net WCS.A5: now also U5801.22 (A5); no longer U5801.6 (A5)
- net WCS.A6: now also U5801.23 (A6); no longer U5801.7 (A6)
- net WCS.A7: now also U5801.24 (A7); no longer U5801.13 (A7)
- net WCS.A8: now also U5801.25 (A8); no longer U5801.14 (A8)
- net WCS.A9: now also U5801.26 (A9); no longer U5801.15 (A9)
- net WCS.D32: now also U5801.2 (Q0); no longer U5801.8 (Q)
- net WCS.D33: now also U5801.4 (Q1)
- net WCS.D34: now also U5801.6 (Q2)
- net WCS.D35: now also U5801.8 (Q3)
- net WCS.D36: now also U5801.10 (Q4)
- net WCS.D37: now also U5801.12 (Q5)
- net WCS.D38: now also U5801.14 (Q6)
- net WCS.P: now also U5801.16 (Q7)
- new net WCS.WE~: U5801.31 (WE)

Commit message: Use megacomponents
Parts:
- removed U5801: XWCSRAM, symbol r1000:XWCSRAM

Commit message: WCS parity checking, updated XPAR64 symbol.
Parts:
- removed U5809, U5810, U5811, U5812: 93S48, symbol r1000:93S48
Connections:
- no-connect marks 4 -> 0
