File: Schematics/VAL/pg_64.kicad_sch (KiCad schematic)
At the start: 64 parts

Commit message: KiCad 6
Parts:
- GB1, GB10, GB100, GB109, GB110, GB119, GB120, GB129, GB130, GB139, GB140, GB149, GB150, GB151, GB152, GB159, GB160, GB169, GB170, GB179, GB180, GB189, GB19, GB190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: value GB -> (none)

Commit message: Recover from KiCad-6 munging
Parts:
- GB1, GB10, GB100, GB109, GB110, GB119, GB120, GB129, GB130, GB139, GB140, GB149, GB150, GB151, GB152, GB159, GB160, GB169, GB170, GB179, GB180, GB189, GB19, GB190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: value (none) -> GB
