File: Schematics/VAL/VAL.kicad_sch (KiCad schematic)
At the start: 2 parts

Commit message: Fix XPAR64 parity mode
Parts:
- U101, U102: value (none) -> ~
Changed lines of the file:
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@@
   (wire (pts (xy 566.42 241.3) (xy 566.42 243.84) ) (stroke (width 0) (type default) ) )
   (wire (pts (xy 566.42 259.08) (xy 566.42 261.62) ) (stroke (width 0) (type default) ) )
-  (symbol (lib_id "r1000:PU") (at 566.42 241.3 0) (unit 1) (in_bom yes) (on_board yes) (property "Reference" "#PWR0102" (id 0) (at 566.42 241.3 0) (effects (font (size 1.27 1.27) ) hide ) ) (property "Value" "" (id 1) (at 566.42 241.3 0) (effects (font (size 1.27 1.27) ) hide ) ) (property "Footprint" "" (id 2) (at 566.42 241.3 0) (effects (font (size 1.27 1.27) ) hide ) ) (property "Datasheet" "" (id 3) (at 566.42 241.3 0) (effects (font (size 1.27 1.27) ) hide ) ) (pin "1" ) )
-  (symbol (lib_id "r1000:Pull_Down") (at 566.42 259.08 0) (unit 1) (in_bom yes) (on_board yes) (property "Reference" "U102" (id 0) (at 566.42 259.08 0) (effects (font (size 1.27 1.27) ) ) ) (property "Value" "" (id 1) (at 566.42 255.27 0) (effects (font (size 2.54 2.54) ) ) ) (property "Footprint" "" (id 2) (at 566.42 259.08 0) (effects (font (size 1.27 1.27) ) hide ) ) (property "Datasheet" "" (id 3) (at 566.42 259.08 0) (effects (font (size 1.27 1.27) ) hide ) ) (pin "1" ) )
-  (symbol (lib_id "r1000:Pull_Up") (at 566.42 243.84 0) (unit 1) (in_bom yes) (on_board yes) (property "Reference" "U101" (id 0) (at 566.42 243.84 0) (effects (font (size 1.27 1.27) ) ) ) (property "Value" "" (id 1) (at 566.42 247.65 0) (effects (font (size 2.54 2.54) ) ) ) (property "Footprint" "" (id 2) (at 566.42 243.84 0) (effects (font (size 1.27 1.27) ) hide ) ) (property "Datasheet" "" (id 3) (at 566.42 243.84 0) (effects (font (size 1.27 1.27) ) hide ) ) (pin "1" ) )
-  (symbol (lib_id "r1000:PD") (at 566.42 261.62 0) (unit 1) (in_bom no) (on_board yes) (property "Reference" "#PWR0101" (id 0) (at 566.42 261.62 0) (effects (font (size 1.27 1.27) ) hide ) ) (property "Value" "" (id 1) (at 566.42 261.62 0) (effects (font (size 1.27 1.27) ) hide ) ) (property "Footprint" "" (id 2) (at 566.42 261.62 0) (effects (font (size 1.27 1.27) ) hide ) ) (property "Datasheet" "" (id 3) (at 566.42 261.62 0) (effects (font (size 1.27 1.27) ) hide ) ) (pin "1" ) )
+  (symbol (lib_id "r1000:PU") (at 566.42 241.3 0) (unit 1) (in_bom yes) (on_board yes) (property "Reference" "#PWR0102" (id 0) (at 566.42 241.3 0) (effects (font (size 1.27 1.27) ) hide ) ) (property "Value" "~" (id 1) (at 566.42 241.3 0) (effects (font (size 1.27 1.27) ) hide ) ) (property "Footprint" "" (id 2) (at 566.42 241.3 0) (effects (font (size 1.27 1.27) ) hide ) ) (property "Datasheet" "" (id 3) (at 566.42 241.3 0) (effects (font (size 1.27 1.27) ) hide ) ) (pin "1" ) )
+  (symbol (lib_id "r1000:Pull_Down") (at 566.42 259.08 0) (unit 1) (in_bom yes) (on_board yes) (property "Reference" "U102" (id 0) (at 566.42 259.08 0) (effects (font (size 1.27 1.27) ) ) ) (property "Value" "~" (id 1) (at 566.42 255.27 0) (effects (font (size 2.54 2.54) ) ) ) (property "Footprint" "" (id 2) (at 566.42 259.08 0) (effects (font (size 1.27 1.27) ) hide ) ) (property "Datasheet" "" (id 3) (at 566.42 259.08 0) (effects (font (size 1.27 1.27) ) hide ) ) (pin "1" ) )
+  (symbol (lib_id "r1000:Pull_Up") (at 566.42 243.84 0) (unit 1) (in_bom yes) (on_board yes) (property "Reference" "U101" (id 0) (at 566.42 243.84 0) (effects (font (size 1.27 1.27) ) ) ) (property "Value" "~" (id 1) (at 566.42 247.65 0) (effects (font (size 2.54 2.54) ) ) ) (property "Footprint" "" (id 2) (at 566.42 243.84 0) (effects (font (size 1.27 1.27) ) hide ) ) (property "Datasheet" "" (id 3) (at 566.42 243.84 0) (effects (font (size 1.27 1.27) ) hide ) ) (pin "1" ) )
+  (symbol (lib_id "r1000:PD") (at 566.42 261.62 0) (unit 1) (in_bom no) (on_board yes) (property "Reference" "#PWR0101" (id 0) (at 566.42 261.62 0) (effects (font (size 1.27 1.27) ) hide ) ) (property "Value" "~" (id 1) (at 566.42 261.62 0) (effects (font (size 1.27 1.27) ) hide ) ) (property "Footprint" "" (id 2) (at 566.42 261.62 0) (effects (font (size 1.27 1.27) ) hide ) ) (property "Datasheet" "" (id 3) (at 566.42 261.62 0) (effects (font (size 1.27 1.27) ) hide ) ) (pin "1" ) )
   (text "Board: VAL Branch: megacomp2" (at 7.62 370.84 0) (effects (font (size 7.62 7.62) (thickness 1.27) bold ) (justify left bottom) ) )
   (sheet_instances

Commit message: Use "bidirectional" as intended.
Parts:
- U101, U102: value ~ -> (none)
Changed lines of the file:
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@@
   (wire (pts (xy 566.42 241.3) (xy 566.42 243.84) ) (stroke (width 0) (type default) ) )
   (wire (pts (xy 566.42 259.08) (xy 566.42 261.62) ) (stroke (width 0) (type default) ) )
-  (symbol (lib_id "r1000:PU") (at 566.42 241.3 0) (unit 1) (in_bom yes) (on_board yes) (property "Reference" "#PWR0102" (id 0) (at 566.42 241.3 0) (effects (font (size 1.27 1.27) ) hide ) ) (property "Value" "~" (id 1) (at 566.42 241.3 0) (effects (font (size 1.27 1.27) ) hide ) ) (property "Footprint" "" (id 2) (at 566.42 241.3 0) (effects (font (size 1.27 1.27) ) hide ) ) (property "Datasheet" "" (id 3) (at 566.42 241.3 0) (effects (font (size 1.27 1.27) ) hide ) ) (pin "1" ) )
-  (symbol (lib_id "r1000:Pull_Down") (at 566.42 259.08 0) (unit 1) (in_bom yes) (on_board yes) (property "Reference" "U102" (id 0) (at 566.42 259.08 0) (effects (font (size 1.27 1.27) ) ) ) (property "Value" "~" (id 1) (at 566.42 255.27 0) (effects (font (size 2.54 2.54) ) ) ) (property "Footprint" "" (id 2) (at 566.42 259.08 0) (effects (font (size 1.27 1.27) ) hide ) ) (property "Datasheet" "" (id 3) (at 566.42 259.08 0) (effects (font (size 1.27 1.27) ) hide ) ) (pin "1" ) )
-  (symbol (lib_id "r1000:Pull_Up") (at 566.42 243.84 0) (unit 1) (in_bom yes) (on_board yes) (property "Reference" "U101" (id 0) (at 566.42 243.84 0) (effects (font (size 1.27 1.27) ) ) ) (property "Value" "~" (id 1) (at 566.42 247.65 0) (effects (font (size 2.54 2.54) ) ) ) (property "Footprint" "" (id 2) (at 566.42 243.84 0) (effects (font (size 1.27 1.27) ) hide ) ) (property "Datasheet" "" (id 3) (at 566.42 243.84 0) (effects (font (size 1.27 1.27) ) hide ) ) (pin "1" ) )
-  (symbol (lib_id "r1000:PD") (at 566.42 261.62 0) (unit 1) (in_bom no) (on_board yes) (property "Reference" "#PWR0101" (id 0) (at 566.42 261.62 0) (effects (font (size 1.27 1.27) ) hide ) ) (property "Value" "~" (id 1) (at 566.42 261.62 0) (effects (font (size 1.27 1.27) ) hide ) ) (property "Footprint" "" (id 2) (at 566.42 261.62 0) (effects (font (size 1.27 1.27) ) hide ) ) (property "Datasheet" "" (id 3) (at 566.42 261.62 0) (effects (font (size 1.27 1.27) ) hide ) ) (pin "1" ) )
+  (symbol (lib_id "r1000:PU") (at 566.42 241.3 0) (unit 1) (in_bom yes) (on_board yes) (property "Reference" "#PWR0102" (id 0) (at 566.42 241.3 0) (effects (font (size 1.27 1.27) ) hide ) ) (property "Value" "" (id 1) (at 566.42 241.3 0) (effects (font (size 1.27 1.27) ) hide ) ) (property "Footprint" "" (id 2) (at 566.42 241.3 0) (effects (font (size 1.27 1.27) ) hide ) ) (property "Datasheet" "" (id 3) (at 566.42 241.3 0) (effects (font (size 1.27 1.27) ) hide ) ) (pin "1" ) )
+  (symbol (lib_id "r1000:Pull_Down") (at 566.42 259.08 0) (unit 1) (in_bom yes) (on_board yes) (property "Reference" "U102" (id 0) (at 566.42 259.08 0) (effects (font (size 1.27 1.27) ) ) ) (property "Value" "" (id 1) (at 566.42 255.27 0) (effects (font (size 2.54 2.54) ) ) ) (property "Footprint" "" (id 2) (at 566.42 259.08 0) (effects (font (size 1.27 1.27) ) hide ) ) (property "Datasheet" "" (id 3) (at 566.42 259.08 0) (effects (font (size 1.27 1.27) ) hide ) ) (pin "1" ) )
+  (symbol (lib_id "r1000:Pull_Up") (at 566.42 243.84 0) (unit 1) (in_bom yes) (on_board yes) (property "Reference" "U101" (id 0) (at 566.42 243.84 0) (effects (font (size 1.27 1.27) ) ) ) (property "Value" "" (id 1) (at 566.42 247.65 0) (effects (font (size 2.54 2.54) ) ) ) (property "Footprint" "" (id 2) (at 566.42 243.84 0) (effects (font (size 1.27 1.27) ) hide ) ) (property "Datasheet" "" (id 3) (at 566.42 243.84 0) (effects (font (size 1.27 1.27) ) hide ) ) (pin "1" ) )
+  (symbol (lib_id "r1000:PD") (at 566.42 261.62 0) (unit 1) (in_bom no) (on_board yes) (property "Reference" "#PWR0101" (id 0) (at 566.42 261.62 0) (effects (font (size 1.27 1.27) ) hide ) ) (property "Value" "" (id 1) (at 566.42 261.62 0) (effects (font (size 1.27 1.27) ) hide ) ) (property "Footprint" "" (id 2) (at 566.42 261.62 0) (effects (font (size 1.27 1.27) ) hide ) ) (property "Datasheet" "" (id 3) (at 566.42 261.62 0) (effects (font (size 1.27 1.27) ) hide ) ) (pin "1" ) )
   (text "Board: VAL Branch: megacomp2" (at 7.62 370.84 0) (effects (font (size 7.62 7.62) (thickness 1.27) bold ) (justify left bottom) ) )
   (sheet_instances

Commit message: Snapshot
Parts:
- U101, U102: value (none) -> ~
Other:
- note added: "REGISTER FILE B PARITY <6>"
- note added: "WRITE DATA REGISTER - PARITY BITS <6>"
- note removed: "REGISTER FILE B PARITY"
- note removed: "WRITE DATA REGISTER - PARITY BITS"
Changed lines of the file:
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@@
   (wire (pts (xy 566.42 241.3) (xy 566.42 243.84) ) (stroke (width 0) (type default) ) )
   (wire (pts (xy 566.42 259.08) (xy 566.42 261.62) ) (stroke (width 0) (type default) ) )
-  (symbol (lib_id "r1000:PU") (at 566.42 241.3 0) (unit 1) (in_bom yes) (on_board yes) (property "Reference" "#PWR0102" (id 0) (at 566.42 241.3 0) (effects (font (size 1.27 1.27) ) hide ) ) (property "Value" "" (id 1) (at 566.42 241.3 0) (effects (font (size 1.27 1.27) ) hide ) ) (property "Footprint" "" (id 2) (at 566.42 241.3 0) (effects (font (size 1.27 1.27) ) hide ) ) (property "Datasheet" "" (id 3) (at 566.42 241.3 0) (effects (font (size 1.27 1.27) ) hide ) ) (pin "1" ) )
-  (symbol (lib_id "r1000:Pull_Down") (at 566.42 259.08 0) (unit 1) (in_bom yes) (on_board yes) (property "Reference" "U102" (id 0) (at 566.42 259.08 0) (effects (font (size 1.27 1.27) ) ) ) (property "Value" "" (id 1) (at 566.42 255.27 0) (effects (font (size 2.54 2.54) ) ) ) (property "Footprint" "" (id 2) (at 566.42 259.08 0) (effects (font (size 1.27 1.27) ) hide ) ) (property "Datasheet" "" (id 3) (at 566.42 259.08 0) (effects (font (size 1.27 1.27) ) hide ) ) (pin "1" ) )
-  (symbol (lib_id "r1000:Pull_Up") (at 566.42 243.84 0) (unit 1) (in_bom yes) (on_board yes) (property "Reference" "U101" (id 0) (at 566.42 243.84 0) (effects (font (size 1.27 1.27) ) ) ) (property "Value" "" (id 1) (at 566.42 247.65 0) (effects (font (size 2.54 2.54) ) ) ) (property "Footprint" "" (id 2) (at 566.42 243.84 0) (effects (font (size 1.27 1.27) ) hide ) ) (property "Datasheet" "" (id 3) (at 566.42 243.84 0) (effects (font (size 1.27 1.27) ) hide ) ) (pin "1" ) )
-  (symbol (lib_id "r1000:PD") (at 566.42 261.62 0) (unit 1) (in_bom no) (on_board yes) (property "Reference" "#PWR0101" (id 0) (at 566.42 261.62 0) (effects (font (size 1.27 1.27) ) hide ) ) (property "Value" "" (id 1) (at 566.42 261.62 0) (effects (font (size 1.27 1.27) ) hide ) ) (property "Footprint" "" (id 2) (at 566.42 261.62 0) (effects (font (size 1.27 1.27) ) hide ) ) (property "Datasheet" "" (id 3) (at 566.42 261.62 0) (effects (font (size 1.27 1.27) ) hide ) ) (pin "1" ) )
+  (symbol (lib_id "r1000:PU") (at 566.42 241.3 0) (unit 1) (in_bom yes) (on_board yes) (property "Reference" "#PWR0102" (id 0) (at 566.42 241.3 0) (effects (font (size 1.27 1.27) ) hide ) ) (property "Value" "~" (id 1) (at 566.42 241.3 0) (effects (font (size 1.27 1.27) ) hide ) ) (property "Footprint" "" (id 2) (at 566.42 241.3 0) (effects (font (size 1.27 1.27) ) hide ) ) (property "Datasheet" "" (id 3) (at 566.42 241.3 0) (effects (font (size 1.27 1.27) ) hide ) ) (pin "1" ) )
+  (symbol (lib_id "r1000:Pull_Down") (at 566.42 259.08 0) (unit 1) (in_bom yes) (on_board yes) (property "Reference" "U102" (id 0) (at 566.42 259.08 0) (effects (font (size 1.27 1.27) ) ) ) (property "Value" "~" (id 1) (at 566.42 255.27 0) (effects (font (size 2.54 2.54) ) ) ) (property "Footprint" "" (id 2) (at 566.42 259.08 0) (effects (font (size 1.27 1.27) ) hide ) ) (property "Datasheet" "" (id 3) (at 566.42 259.08 0) (effects (font (size 1.27 1.27) ) hide ) ) (pin "1" ) )
+  (symbol (lib_id "r1000:Pull_Up") (at 566.42 243.84 0) (unit 1) (in_bom yes) (on_board yes) (property "Reference" "U101" (id 0) (at 566.42 243.84 0) (effects (font (size 1.27 1.27) ) ) ) (property "Value" "~" (id 1) (at 566.42 247.65 0) (effects (font (size 2.54 2.54) ) ) ) (property "Footprint" "" (id 2) (at 566.42 243.84 0) (effects (font (size 1.27 1.27) ) hide ) ) (property "Datasheet" "" (id 3) (at 566.42 243.84 0) (effects (font (size 1.27 1.27) ) hide ) ) (pin "1" ) )
+  (symbol (lib_id "r1000:PD") (at 566.42 261.62 0) (unit 1) (in_bom no) (on_board yes) (property "Reference" "#PWR0101" (id 0) (at 566.42 261.62 0) (effects (font (size 1.27 1.27) ) hide ) ) (property "Value" "~" (id 1) (at 566.42 261.62 0) (effects (font (size 1.27 1.27) ) hide ) ) (property "Footprint" "" (id 2) (at 566.42 261.62 0) (effects (font (size 1.27 1.27) ) hide ) ) (property "Datasheet" "" (id 3) (at 566.42 261.62 0) (effects (font (size 1.27 1.27) ) hide ) ) (pin "1" ) )
   (text "Board: VAL Branch: megacomp2" (at 7.62 370.84 0) (effects (font (size 7.62 7.62) (thickness 1.27) bold ) (justify left bottom) ) )
   (sheet_instances
@@
   (sheet (at 12.70 119.38) (size 20.32 5.08) (property "Sheet name" "Page 14" (id 0) (at 35.56 124.46 0) (effects (font (size 2.54 2.54) ) (justify left bottom) ) ) (property "Sheet file" "pg_14.kicad_sch" (id 1) (at 35.56 121.92 0) (effects (justify left bottom) hide ) ) )
   (text "WRITE DATA REGISTER - REGISTER ARRAY" (at 53.34 124.46 0) (effects (font (size 2.54 2.54) ) (justify left bottom) ) )
-  (sheet (at 12.70 127.00) (size 20.32 5.08) (property "Sheet name" "Page 15" (id 0) (at 35.56 132.08 0) (effects (font (size 2.54 2.54) ) (justify left bottom) ) ) (property "Sheet file" "pg_15.kicad_sch" (id 1) (at 35.56 129.54 0) (effects (justify left bottom) hide ) ) )
-  (text "WRITE DATA REGISTER - PARITY BITS" (at 53.34 132.08 0) (effects (font (size 2.54 2.54) ) (justify left bottom) ) )
+  (sheet (at 12.70 127.00) (size 20.32 5.08) (property "Sheet name" "Page 15" (id 0) (at 35.56 132.08 0) (effects (font (size 2.54 2.54) ) (justify left bottom) ) ) (property "Sheet file" "pg_15.kicad_sch" (id 1) (at 35.56 129.54 0) (effects (justify left bottom) hide ) ) (fill (color 192 192 192 1.0) ) )
+  (text "WRITE DATA REGISTER - PARITY BITS <6>" (at 53.34 132.08 0) (effects (font (size 2.54 2.54) ) (justify left bottom) ) )
   (sheet (at 12.70 134.62) (size 20.32 5.08) (property "Sheet name" "Page 16" (id 0) (at 35.56 139.70 0) (effects (font (size 2.54 2.54) ) (justify left bottom) ) ) (property "Sheet file" "pg_16.kicad_sch" (id 1) (at 35.56 137.16 0) (effects (justify left bottom) hide ) ) )
   (text "SHIFT MUX - MOST SIGNIFICANT BITS" (at 53.34 139.70 0) (effects (font (size 2.54 2.54) ) (justify left bottom) ) )
@@
   (sheet (at 12.70 165.10) (size 20.32 5.08) (property "Sheet name" "Page 20" (id 0) (at 35.56 170.18 0) (effects (font (size 2.54 2.54) ) (justify left bottom) ) ) (property "Sheet file" "pg_20.kicad_sch" (id 1) (at 35.56 167.64 0) (effects (justify left bottom) hide ) ) )
   (text "REGISTER FILE B - RAM ARRAY" (at 53.34 170.18 0) (effects (font (size 2.54 2.54) ) (justify left bottom) ) )
-  (sheet (at 12.70 172.72) (size 20.32 5.08) (property "Sheet name" "Page 21" (id 0) (at 35.56 177.80 0) (effects (font (size 2.54 2.54) ) (justify left bottom) ) ) (property "Sheet file" "pg_21.kicad_sch" (id 1) (at 35.56 175.26 0) (effects (justify left bottom) hide ) ) )
-  (text "REGISTER FILE B PARITY" (at 53.34 177.80 0) (effects (font (size 2.54 2.54) ) (justify left bottom) ) )
+  (sheet (at 12.70 172.72) (size 20.32 5.08) (property "Sheet name" "Page 21" (id 0) (at 35.56 177.80 0) (effects (font (size 2.54 2.54) ) (justify left bottom) ) ) (property "Sheet file" "pg_21.kicad_sch" (id 1) (at 35.56 175.26 0) (effects (justify left bottom) hide ) ) (fill (color 192 192 192 1.0) ) )
+  (text "REGISTER FILE B PARITY <6>" (at 53.34 177.80 0) (effects (font (size 2.54 2.54) ) (justify left bottom) ) )
   (sheet (at 12.70 180.34) (size 20.32 5.08) (property "Sheet name" "Page 22" (id 0) (at 35.56 185.42 0) (effects (font (size 2.54 2.54) ) (justify left bottom) ) ) (property "Sheet file" "pg_22.kicad_sch" (id 1) (at 35.56 182.88 0) (effects (justify left bottom) hide ) ) )
   (text "C BUS DRIVER" (at 53.34 185.42 0) (effects (font (size 2.54 2.54) ) (justify left bottom) ) )

Commit message: Polish
Parts:
- U101, U102: value ~ -> (none)
Changed lines of the file:
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@@
   (wire (pts (xy 566.42 241.3) (xy 566.42 243.84) ) (stroke (width 0) (type default) ) )
   (wire (pts (xy 566.42 259.08) (xy 566.42 261.62) ) (stroke (width 0) (type default) ) )
-  (symbol (lib_id "r1000:PU") (at 566.42 241.3 0) (unit 1) (in_bom yes) (on_board yes) (property "Reference" "#PWR0102" (id 0) (at 566.42 241.3 0) (effects (font (size 1.27 1.27) ) hide ) ) (property "Value" "~" (id 1) (at 566.42 241.3 0) (effects (font (size 1.27 1.27) ) hide ) ) (property "Footprint" "" (id 2) (at 566.42 241.3 0) (effects (font (size 1.27 1.27) ) hide ) ) (property "Datasheet" "" (id 3) (at 566.42 241.3 0) (effects (font (size 1.27 1.27) ) hide ) ) (pin "1" ) )
-  (symbol (lib_id "r1000:Pull_Down") (at 566.42 259.08 0) (unit 1) (in_bom yes) (on_board yes) (property "Reference" "U102" (id 0) (at 566.42 259.08 0) (effects (font (size 1.27 1.27) ) ) ) (property "Value" "~" (id 1) (at 566.42 255.27 0) (effects (font (size 2.54 2.54) ) ) ) (property "Footprint" "" (id 2) (at 566.42 259.08 0) (effects (font (size 1.27 1.27) ) hide ) ) (property "Datasheet" "" (id 3) (at 566.42 259.08 0) (effects (font (size 1.27 1.27) ) hide ) ) (pin "1" ) )
-  (symbol (lib_id "r1000:Pull_Up") (at 566.42 243.84 0) (unit 1) (in_bom yes) (on_board yes) (property "Reference" "U101" (id 0) (at 566.42 243.84 0) (effects (font (size 1.27 1.27) ) ) ) (property "Value" "~" (id 1) (at 566.42 247.65 0) (effects (font (size 2.54 2.54) ) ) ) (property "Footprint" "" (id 2) (at 566.42 243.84 0) (effects (font (size 1.27 1.27) ) hide ) ) (property "Datasheet" "" (id 3) (at 566.42 243.84 0) (effects (font (size 1.27 1.27) ) hide ) ) (pin "1" ) )
-  (symbol (lib_id "r1000:PD") (at 566.42 261.62 0) (unit 1) (in_bom no) (on_board yes) (property "Reference" "#PWR0101" (id 0) (at 566.42 261.62 0) (effects (font (size 1.27 1.27) ) hide ) ) (property "Value" "~" (id 1) (at 566.42 261.62 0) (effects (font (size 1.27 1.27) ) hide ) ) (property "Footprint" "" (id 2) (at 566.42 261.62 0) (effects (font (size 1.27 1.27) ) hide ) ) (property "Datasheet" "" (id 3) (at 566.42 261.62 0) (effects (font (size 1.27 1.27) ) hide ) ) (pin "1" ) )
+  (symbol (lib_id "r1000:PU") (at 566.42 241.3 0) (unit 1) (in_bom yes) (on_board yes) (property "Reference" "#PWR0102" (id 0) (at 566.42 241.3 0) (effects (font (size 1.27 1.27) ) hide ) ) (property "Value" "" (id 1) (at 566.42 241.3 0) (effects (font (size 1.27 1.27) ) hide ) ) (property "Footprint" "" (id 2) (at 566.42 241.3 0) (effects (font (size 1.27 1.27) ) hide ) ) (property "Datasheet" "" (id 3) (at 566.42 241.3 0) (effects (font (size 1.27 1.27) ) hide ) ) (pin "1" ) )
+  (symbol (lib_id "r1000:Pull_Down") (at 566.42 259.08 0) (unit 1) (in_bom yes) (on_board yes) (property "Reference" "U102" (id 0) (at 566.42 259.08 0) (effects (font (size 1.27 1.27) ) ) ) (property "Value" "" (id 1) (at 566.42 255.27 0) (effects (font (size 2.54 2.54) ) ) ) (property "Footprint" "" (id 2) (at 566.42 259.08 0) (effects (font (size 1.27 1.27) ) hide ) ) (property "Datasheet" "" (id 3) (at 566.42 259.08 0) (effects (font (size 1.27 1.27) ) hide ) ) (pin "1" ) )
+  (symbol (lib_id "r1000:Pull_Up") (at 566.42 243.84 0) (unit 1) (in_bom yes) (on_board yes) (property "Reference" "U101" (id 0) (at 566.42 243.84 0) (effects (font (size 1.27 1.27) ) ) ) (property "Value" "" (id 1) (at 566.42 247.65 0) (effects (font (size 2.54 2.54) ) ) ) (property "Footprint" "" (id 2) (at 566.42 243.84 0) (effects (font (size 1.27 1.27) ) hide ) ) (property "Datasheet" "" (id 3) (at 566.42 243.84 0) (effects (font (size 1.27 1.27) ) hide ) ) (pin "1" ) )
+  (symbol (lib_id "r1000:PD") (at 566.42 261.62 0) (unit 1) (in_bom no) (on_board yes) (property "Reference" "#PWR0101" (id 0) (at 566.42 261.62 0) (effects (font (size 1.27 1.27) ) hide ) ) (property "Value" "" (id 1) (at 566.42 261.62 0) (effects (font (size 1.27 1.27) ) hide ) ) (property "Footprint" "" (id 2) (at 566.42 261.62 0) (effects (font (size 1.27 1.27) ) hide ) ) (property "Datasheet" "" (id 3) (at 566.42 261.62 0) (effects (font (size 1.27 1.27) ) hide ) ) (pin "1" ) )
   (text "Board: VAL Branch: megacomp2" (at 7.62 370.84 0) (effects (font (size 7.62 7.62) (thickness 1.27) bold ) (justify left bottom) ) )
   (sheet_instances
