File: Schematics/VAL/pg_16.kicad_sch (KiCad schematic)
At the start: 19 parts, among them U1801 F257, U1802 F257, U1803 F257, U1804 F257, U1805 F257, U1806 F257, U1807 F257, U1808 F257, U1809 F257, U1810 F257, U1811 F257, U1812 F257, U1813 F257, U1814 F257, U1815 F257, U1816 F257, U1817 F08, U1818 F08, U1819 F244

Commit message: Update VAL and use larger components
Parts:
- removed U1802, U1803, U1804, U1805, U1806, U1807, U1808, U1809, U1810, U1811, U1812, U1813, U1814, U1815, U1816: F257, symbol r1000:F257
- added U1820: XMUX32, symbol r1000:XMUX32
- U1801: value F257 -> XMUX32; symbol r1000:F257 -> r1000:XMUX32; Location C39 -> x99
Connections:
- net ALU.D0: now also U1801.1 (A0), U1820.69 (B16); no longer U1801.2 (A0)
- net ALU.D1: now also U1801.3 (A1), U1820.1 (A0), U1820.71 (B17); no longer U1801.5 (A1)
- net ALU.D10: now also U1801.15 (A10), U1820.14 (A9), U1820.89 (B26)
- net ALU.D11: now also U1801.16 (A11), U1820.15 (A10), U1820.91 (B27)
- net ALU.D12: now also U1801.17 (A12), U1820.16 (A11), U1820.93 (B28)
- net ALU.D13: now also U1801.18 (A13), U1820.17 (A12), U1820.95 (B29)
- net ALU.D14: now also U1801.19 (A14), U1820.18 (A13), U1820.97 (B30)
- net ALU.D15: now also U1801.20 (A15), U1820.19 (A14), U1820.99 (B31)
- net ALU.D16: now also U1801.21 (A16), U1820.20 (A15)
- net ALU.D17: now also U1801.22 (A17), U1820.21 (A16)
- net ALU.D18: now also U1801.23 (A18), U1820.22 (A17)
- net ALU.D19: now also U1801.24 (A19), U1820.23 (A18)
- net ALU.D2: now also U1801.5 (A2), U1820.3 (A1), U1820.73 (B18); no longer U1801.11 (A2)
- net ALU.D20: now also U1801.25 (A20), U1820.24 (A19)
- net ALU.D21: now also U1801.26 (A21), U1820.25 (A20)
- net ALU.D22: now also U1801.27 (A22), U1820.26 (A21)
- net ALU.D23: now also U1801.28 (A23), U1820.27 (A22)
- net ALU.D24: now also U1801.29 (A24), U1820.28 (A23)
- net ALU.D25: now also U1801.30 (A25), U1820.29 (A24)
- net ALU.D26: now also U1801.31 (A26), U1820.30 (A25)
- net ALU.D27: now also U1801.32 (A27), U1820.31 (A26)
- net ALU.D28: now also U1801.33 (A28), U1820.32 (A27)
- net ALU.D29: now also U1801.34 (A29), U1820.33 (A28)
- net ALU.D3: now also U1801.7 (A3), U1820.5 (A2), U1820.75 (B19); no longer U1801.14 (A3)
- net ALU.D30: now also U1801.35 (A30), U1820.34 (A29)
- net ALU.D31: now also U1801.36 (A31), U1820.35 (A30)
- net ALU.D32: now also U1820.36 (A31)
- net ALU.D4: now also U1801.9 (A4), U1820.7 (A3), U1820.77 (B20)
- net ALU.D5: now also U1801.10 (A5), U1820.79 (B21), U1820.9 (A4)
- net ALU.D6: now also U1801.11 (A6), U1820.10 (A5), U1820.81 (B22)
- net ALU.D7: now also U1801.12 (A7), U1820.11 (A6), U1820.83 (B23)
- net ALU.D8: now also U1801.13 (A8), U1820.12 (A7), U1820.85 (B24)
- net ALU.D9: now also U1801.14 (A9), U1820.13 (A8), U1820.87 (B25)
- net C.D0: now also U1801.38 (Y0), U1820.38 (Y0); no longer U1801.4 (Y0)
- net C.D1: now also U1801.40 (Y1), U1820.40 (Y1); no longer U1801.7 (Y1)
- net C.D10: now also U1801.58 (Y10), U1820.58 (Y10)
- net C.D11: now also U1801.60 (Y11), U1820.60 (Y11)
- net C.D12: now also U1801.62 (Y12), U1820.62 (Y12)
- net C.D13: now also U1801.64 (Y13), U1820.64 (Y13)
- net C.D14: now also U1801.66 (Y14), U1820.66 (Y14)
- net C.D15: now also U1801.68 (Y15), U1820.68 (Y15)
- net C.D16: now also U1801.70 (Y16), U1820.70 (Y16)
- net C.D17: now also U1801.72 (Y17), U1820.72 (Y17)
- net C.D18: now also U1801.74 (Y18), U1820.74 (Y18)
- net C.D19: now also U1801.76 (Y19), U1820.76 (Y19)
- net C.D2: now also U1801.42 (Y2), U1820.42 (Y2); no longer U1801.9 (Y2)
- net C.D20: now also U1801.78 (Y20), U1820.78 (Y20)
- net C.D21: now also U1801.80 (Y21), U1820.80 (Y21)
- net C.D22: now also U1801.82 (Y22), U1820.82 (Y22)
- net C.D23: now also U1801.84 (Y23), U1820.84 (Y23)
- net C.D24: now also U1801.86 (Y24), U1820.86 (Y24)
- net C.D25: now also U1801.88 (Y25), U1820.88 (Y25)
- net C.D26: now also U1801.90 (Y26), U1820.90 (Y26)
- net C.D27: now also U1801.92 (Y27), U1820.92 (Y27)
- net C.D28: now also U1801.94 (Y28), U1820.94 (Y28)
- net C.D29: now also U1801.96 (Y29), U1820.96 (Y29)
- net C.D3: now also U1801.44 (Y3), U1820.44 (Y3); no longer U1801.12 (Y3)
- net C.D30: now also U1801.98 (Y30), U1820.98 (Y30)
- net C.D31: now also U1801.100 (Y31), U1820.100 (Y31)
- net C.D4: now also U1801.46 (Y4), U1820.46 (Y4)
- net C.D5: now also U1801.48 (Y5), U1820.48 (Y5)
- net C.D6: now also U1801.50 (Y6), U1820.50 (Y6)
- net C.D7: now also U1801.52 (Y7), U1820.52 (Y7)
- net C.D8: now also U1801.54 (Y8), U1820.54 (Y8)
- net C.D9: now also U1801.56 (Y9), U1820.56 (Y9)
- net C_MUX.OE0~.B0: now also U1820.8 (OE)
- net C_MUX.OE0~.B1: now also U1801.8 (OE); no longer U1801.15 (OE)
- net C_MUX.SEL1.B0: now also U1801.4 (S), U1820.4 (S); no longer U1801.1 (S)
- net PU: now also U1820.37 (B0), U1820.39 (B1), U1820.41 (B2), U1820.43 (B3), U1820.45 (B4), U1820.47 (B5), U1820.49 (B6), U1820.51 (B7), U1820.53 (B8), U1820.55 (B9), U1820.57 (B10), U1820.59 (B11), U1820.61 (B12), U1820.63 (B13), U1820.65 (B14), U1820.67 (B15)
- net WDR.D0: now also U1801.37 (B0); no longer U1801.3 (B0)
- net WDR.D1: now also U1801.39 (B1); no longer U1801.6 (B1)
- net WDR.D10: now also U1801.57 (B10)
- net WDR.D11: now also U1801.59 (B11)
- net WDR.D12: now also U1801.61 (B12)
- net WDR.D13: now also U1801.63 (B13)
- net WDR.D14: now also U1801.65 (B14)
- net WDR.D15: now also U1801.67 (B15)
- net WDR.D16: now also U1801.69 (B16)
- net WDR.D17: now also U1801.71 (B17)
- net WDR.D18: now also U1801.73 (B18)
- net WDR.D19: now also U1801.75 (B19)
- net WDR.D2: now also U1801.41 (B2); no longer U1801.10 (B2)
- net WDR.D20: now also U1801.77 (B20)
- net WDR.D21: now also U1801.79 (B21)
- net WDR.D22: now also U1801.81 (B22)
- net WDR.D23: now also U1801.83 (B23)
- net WDR.D24: now also U1801.85 (B24)
- net WDR.D25: now also U1801.87 (B25)
- net WDR.D26: now also U1801.89 (B26)
- net WDR.D27: now also U1801.91 (B27)
- net WDR.D28: now also U1801.93 (B28)
- net WDR.D29: now also U1801.95 (B29)
- net WDR.D3: now also U1801.43 (B3); no longer U1801.13 (B3)
- net WDR.D30: now also U1801.97 (B30)
- net WDR.D31: now also U1801.99 (B31)
- net WDR.D4: now also U1801.45 (B4)
- net WDR.D5: now also U1801.47 (B5)
- net WDR.D6: now also U1801.49 (B6)
- net WDR.D7: now also U1801.51 (B7)
- net WDR.D8: now also U1801.53 (B8)
- net WDR.D9: now also U1801.55 (B9)
- new net PD: U1801.6 (E), U1820.6 (E)
- no-connect marks 0 -> 2

Commit message: KiCad 6
Parts:
- U1801, U1820: value XMUX32 -> (none)
- U1817, U1818: value F08 -> (none)
- U1819: value F244 -> (none)

Commit message: Recover from KiCad-6 munging
Parts:
- U1801, U1820: value (none) -> XMUX32
- U1817, U1818: value (none) -> F08
- U1819: value (none) -> F244

Commit message: Snapshot
Other:
- moved on the sheet: U1817, U1818, U1819

Commit message: Megacomp the multiplier
Parts:
- removed U1817, U1818: F08, symbol r1000:F08
- removed U1819: F244, symbol r1000:F244
- removed U1820: XMUX32, symbol r1000:XMUX32
- added U1802, U1803, U1804, U1805, U1806, U1807, U1808: XFBUF32, symbol r1000:XFBUF32
- U1801: value XMUX32 -> XFBUF32; symbol r1000:XMUX32 -> r1000:XFBUF32; Name SMUX1 -> SMUX10
Connections:
- net ALU.D0: now also U1802.3 (I0), U1805.35 (I16); no longer U1801.1 (A0)
- net ALU.D1: now also U1802.5 (I1), U1804.3 (I0), U1805.37 (I17); no longer U1801.3 (A1)
- net ALU.D10: now also U1802.23 (I10), U1804.21 (I9), U1805.55 (I26); no longer U1801.15 (A10)
- net ALU.D11: now also U1802.25 (I11), U1804.23 (I10), U1805.57 (I27); no longer U1801.16 (A11)
- net ALU.D12: now also U1802.27 (I12), U1804.25 (I11), U1805.59 (I28); no longer U1801.17 (A12)
- net ALU.D13: now also U1802.29 (I13), U1804.27 (I12), U1805.61 (I29); no longer U1801.18 (A13)
- net ALU.D14: now also U1802.31 (I14), U1804.29 (I13), U1805.63 (I30); no longer U1801.19 (A14)
- net ALU.D15: now also U1802.33 (I15), U1804.31 (I14), U1805.65 (I31); no longer U1801.20 (A15)
- net ALU.D16: now also U1802.35 (I16), U1804.33 (I15), U1807.3 (I0); no longer U1801.21 (A16)
- net ALU.D17: now also U1802.37 (I17), U1804.35 (I16), U1807.5 (I1); no longer U1801.22 (A17)
- net ALU.D18: now also U1802.39 (I18), U1804.37 (I17), U1807.7 (I2); no longer U1801.23 (A18)
- net ALU.D19: now also U1802.41 (I19), U1804.39 (I18), U1807.9 (I3); no longer U1801.24 (A19)
- net ALU.D2: now also U1802.7 (I2), U1804.5 (I1), U1805.39 (I18); no longer U1801.5 (A2)
- net ALU.D20: now also U1802.43 (I20), U1804.41 (I19), U1807.11 (I4); no longer U1801.25 (A20)
- net ALU.D21: now also U1802.45 (I21), U1804.43 (I20), U1807.13 (I5); no longer U1801.26 (A21)
- net ALU.D22: now also U1802.47 (I22), U1804.45 (I21), U1807.15 (I6); no longer U1801.27 (A22)
- net ALU.D23: now also U1802.49 (I23), U1804.47 (I22), U1807.17 (I7); no longer U1801.28 (A23)
- net ALU.D24: now also U1802.51 (I24), U1804.49 (I23), U1807.19 (I8); no longer U1801.29 (A24)
- net ALU.D25: now also U1802.53 (I25), U1804.51 (I24), U1807.21 (I9); no longer U1801.30 (A25)
- net ALU.D26: now also U1802.55 (I26), U1804.53 (I25), U1807.23 (I10); no longer U1801.31 (A26)
- net ALU.D27: now also U1802.57 (I27), U1804.55 (I26), U1807.25 (I11); no longer U1801.32 (A27)
- net ALU.D28: now also U1802.59 (I28), U1804.57 (I27), U1807.27 (I12); no longer U1801.33 (A28)
- net ALU.D29: now also U1802.61 (I29), U1804.59 (I28), U1807.29 (I13); no longer U1801.34 (A29)
- net ALU.D3: now also U1802.9 (I3), U1804.7 (I2), U1805.41 (I19); no longer U1801.7 (A3)
- net ALU.D30: now also U1802.63 (I30), U1804.61 (I29), U1807.31 (I14); no longer U1801.35 (A30)
- net ALU.D31: now also U1802.65 (I31), U1804.63 (I30), U1807.33 (I15); no longer U1801.36 (A31)
- net ALU.D32: now also U1803.3 (I0), U1804.65 (I31), U1807.35 (I16)
- net ALU.D4: now also U1802.11 (I4), U1804.9 (I3), U1805.43 (I20); no longer U1801.9 (A4)
- net ALU.D5: now also U1802.13 (I5), U1804.11 (I4), U1805.45 (I21); no longer U1801.10 (A5)
- net ALU.D6: now also U1802.15 (I6), U1804.13 (I5), U1805.47 (I22); no longer U1801.11 (A6)
- net ALU.D7: now also U1802.17 (I7), U1804.15 (I6), U1805.49 (I23); no longer U1801.12 (A7)
- net ALU.D8: now also U1802.19 (I8), U1804.17 (I7), U1805.51 (I24); no longer U1801.13 (A8)
- net ALU.D9: now also U1802.21 (I9), U1804.19 (I8), U1805.53 (I25); no longer U1801.14 (A9)
- net C.D0: now also U1802.4 (Y0), U1804.4 (Y0), U1805.4 (Y0), U1806.4 (Y0); no longer U1801.38 (Y0)
- net C.D1: now also U1802.6 (Y1), U1804.6 (Y1), U1805.6 (Y1), U1806.6 (Y1); no longer U1801.40 (Y1)
- net C.D10: now also U1802.24 (Y10), U1804.24 (Y10), U1805.24 (Y10), U1806.24 (Y10); no longer U1801.58 (Y10)
- net C.D11: now also U1802.26 (Y11), U1804.26 (Y11), U1805.26 (Y11), U1806.26 (Y11); no longer U1801.60 (Y11)
- net C.D12: now also U1802.28 (Y12), U1804.28 (Y12), U1805.28 (Y12), U1806.28 (Y12); no longer U1801.62 (Y12)
- net C.D13: now also U1802.30 (Y13), U1804.30 (Y13), U1805.30 (Y13), U1806.30 (Y13); no longer U1801.64 (Y13)
- net C.D14: now also U1802.32 (Y14), U1804.32 (Y14), U1805.32 (Y14), U1806.32 (Y14); no longer U1801.66 (Y14)
- net C.D15: now also U1802.34 (Y15), U1804.34 (Y15), U1805.34 (Y15), U1806.34 (Y15); no longer U1801.68 (Y15)
- net C.D16: now also U1802.36 (Y16), U1804.36 (Y16), U1805.36 (Y16), U1806.36 (Y16); no longer U1801.70 (Y16)
- net C.D17: now also U1802.38 (Y17), U1804.38 (Y17), U1805.38 (Y17), U1806.38 (Y17); no longer U1801.72 (Y17)
- net C.D18: now also U1802.40 (Y18), U1804.40 (Y18), U1805.40 (Y18), U1806.40 (Y18); no longer U1801.74 (Y18)
- net C.D19: now also U1802.42 (Y19), U1804.42 (Y19), U1805.42 (Y19), U1806.42 (Y19); no longer U1801.76 (Y19)
- net C.D2: now also U1802.8 (Y2), U1804.8 (Y2), U1805.8 (Y2), U1806.8 (Y2); no longer U1801.42 (Y2)
- net C.D20: now also U1802.44 (Y20), U1804.44 (Y20), U1805.44 (Y20), U1806.44 (Y20); no longer U1801.78 (Y20)
- net C.D21: now also U1802.46 (Y21), U1804.46 (Y21), U1805.46 (Y21), U1806.46 (Y21); no longer U1801.80 (Y21)
- net C.D22: now also U1802.48 (Y22), U1804.48 (Y22), U1805.48 (Y22), U1806.48 (Y22); no longer U1801.82 (Y22)
- net C.D23: now also U1802.50 (Y23), U1804.50 (Y23), U1805.50 (Y23), U1806.50 (Y23); no longer U1801.84 (Y23)
- net C.D24: now also U1802.52 (Y24), U1804.52 (Y24), U1805.52 (Y24), U1806.52 (Y24); no longer U1801.86 (Y24)
- net C.D25: now also U1802.54 (Y25), U1804.54 (Y25), U1805.54 (Y25), U1806.54 (Y25); no longer U1801.88 (Y25)
- net C.D26: now also U1802.56 (Y26), U1804.56 (Y26), U1805.56 (Y26), U1806.56 (Y26); no longer U1801.90 (Y26)
- net C.D27: now also U1802.58 (Y27), U1804.58 (Y27), U1805.58 (Y27), U1806.58 (Y27); no longer U1801.92 (Y27)
- net C.D28: now also U1802.60 (Y28), U1804.60 (Y28), U1805.60 (Y28), U1806.60 (Y28); no longer U1801.94 (Y28)
- net C.D29: now also U1802.62 (Y29), U1804.62 (Y29), U1805.62 (Y29), U1806.62 (Y29); no longer U1801.96 (Y29)
- net C.D3: now also U1802.10 (Y3), U1804.10 (Y3), U1805.10 (Y3), U1806.10 (Y3); no longer U1801.44 (Y3)
- net C.D30: now also U1802.64 (Y30), U1804.64 (Y30), U1805.64 (Y30), U1806.64 (Y30); no longer U1801.98 (Y30)
- net C.D31: now also U1802.66 (Y31), U1804.66 (Y31), U1805.66 (Y31), U1806.66 (Y31); no longer U1801.100 (Y31)
- net C.D4: now also U1802.12 (Y4), U1804.12 (Y4), U1805.12 (Y4), U1806.12 (Y4); no longer U1801.46 (Y4)
- net C.D5: now also U1802.14 (Y5), U1804.14 (Y5), U1805.14 (Y5), U1806.14 (Y5); no longer U1801.48 (Y5)
- net C.D6: now also U1802.16 (Y6), U1804.16 (Y6), U1805.16 (Y6), U1806.16 (Y6); no longer U1801.50 (Y6)
- net C.D7: now also U1802.18 (Y7), U1804.18 (Y7), U1805.18 (Y7), U1806.18 (Y7); no longer U1801.52 (Y7)
- net C.D8: now also U1802.20 (Y8), U1804.20 (Y8), U1805.20 (Y8), U1806.20 (Y8); no longer U1801.54 (Y8)
- net C.D9: now also U1802.22 (Y9), U1804.22 (Y9), U1805.22 (Y9), U1806.22 (Y9); no longer U1801.56 (Y9)
- net PU: now also U1801.65 (I31), U1805.11 (I4), U1805.13 (I5), U1805.15 (I6), U1805.17 (I7), U1805.19 (I8), U1805.21 (I9), U1805.23 (I10), U1805.25 (I11), U1805.27 (I12), U1805.29 (I13), U1805.3 (I0), U1805.31 (I14), U1805.33 (I15), U1805.5 (I1), U1805.7 (I2), U1805.9 (I3)
- net WDR.D0: now also U1806.3 (I0); no longer U1801.37 (B0)
- net WDR.D1: now also U1806.5 (I1); no longer U1801.39 (B1)
- net WDR.D10: now also U1806.23 (I10); no longer U1801.57 (B10)
- net WDR.D11: now also U1806.25 (I11); no longer U1801.59 (B11)
- net WDR.D12: now also U1806.27 (I12); no longer U1801.61 (B12)
- net WDR.D13: now also U1806.29 (I13); no longer U1801.63 (B13)
- net WDR.D14: now also U1806.31 (I14); no longer U1801.65 (B14)
- net WDR.D15: now also U1806.33 (I15); no longer U1801.67 (B15)
- net WDR.D16: now also U1806.35 (I16); no longer U1801.69 (B16)
- net WDR.D17: now also U1806.37 (I17); no longer U1801.71 (B17)
- net WDR.D18: now also U1806.39 (I18); no longer U1801.73 (B18)
- net WDR.D19: now also U1806.41 (I19); no longer U1801.75 (B19)
- net WDR.D2: now also U1806.7 (I2); no longer U1801.41 (B2)
- net WDR.D20: now also U1806.43 (I20); no longer U1801.77 (B20)
- net WDR.D21: now also U1806.45 (I21); no longer U1801.79 (B21)
- net WDR.D22: now also U1806.47 (I22); no longer U1801.81 (B22)
- net WDR.D23: now also U1806.49 (I23); no longer U1801.83 (B23)
- net WDR.D24: now also U1806.51 (I24); no longer U1801.85 (B24)
- net WDR.D25: now also U1806.53 (I25); no longer U1801.87 (B25)
- net WDR.D26: now also U1806.55 (I26); no longer U1801.89 (B26)
- net WDR.D27: now also U1806.57 (I27); no longer U1801.91 (B27)
- net WDR.D28: now also U1806.59 (I28); no longer U1801.93 (B28)
- net WDR.D29: now also U1806.61 (I29); no longer U1801.95 (B29)
- net WDR.D3: now also U1806.9 (I3); no longer U1801.43 (B3)
- net WDR.D30: now also U1806.63 (I30); no longer U1801.97 (B30)
- net WDR.D31: now also U1806.65 (I31); no longer U1801.99 (B31)
- net WDR.D4: now also U1806.11 (I4); no longer U1801.45 (B4)
- net WDR.D5: now also U1806.13 (I5); no longer U1801.47 (B5)
- net WDR.D6: now also U1806.15 (I6); no longer U1801.49 (B6)
- net WDR.D7: now also U1806.17 (I7); no longer U1801.51 (B7)
- net WDR.D8: now also U1806.19 (I8); no longer U1801.53 (B8)
- net WDR.D9: now also U1806.21 (I9); no longer U1801.55 (B9)
- net CSEL_1_0: now reaches U1801.2 (OE)
- net C_MUX.OE0~.B1 renamed C.D34
- net C.D34: now also U1803.8 (Y2), U1807.8 (Y2), U1808.8 (Y2)
- net C_MUX.SEL1.B0 renamed C.D32
- net C.D32: now also U1803.4 (Y0), U1807.4 (Y0), U1808.4 (Y0)
- net PD renamed C.D33
- net C.D33: now also U1803.6 (Y1), U1807.6 (Y1), U1808.6 (Y1)
- new net ALU.D33: U1801.3 (I0), U1803.5 (I1), U1807.37 (I17)
- new net ALU.D34: U1801.5 (I1), U1803.7 (I2), U1807.39 (I18)
- new net ALU.D35: U1801.7 (I2), U1803.9 (I3), U1807.41 (I19)
- new net ALU.D36: U1801.9 (I3), U1803.11 (I4), U1807.43 (I20)
- new net ALU.D37: U1801.11 (I4), U1803.13 (I5), U1807.45 (I21)
- new net ALU.D38: U1801.13 (I5), U1803.15 (I6), U1807.47 (I22)
- new net ALU.D39: U1801.15 (I6), U1803.17 (I7), U1807.49 (I23)
- new net ALU.D40: U1801.17 (I7), U1803.19 (I8), U1807.51 (I24)
- new net ALU.D41: U1801.19 (I8), U1803.21 (I9), U1807.53 (I25)
- new net ALU.D42: U1801.21 (I9), U1803.23 (I10), U1807.55 (I26)
- new net ALU.D43: U1801.23 (I10), U1803.25 (I11), U1807.57 (I27)
- new net ALU.D44: U1801.25 (I11), U1803.27 (I12), U1807.59 (I28)
- new net ALU.D45: U1801.27 (I12), U1803.29 (I13), U1807.61 (I29)
- new net ALU.D46: U1801.29 (I13), U1803.31 (I14), U1807.63 (I30)
- new net ALU.D47: U1801.31 (I14), U1803.33 (I15), U1807.65 (I31)
- new net ALU.D48: U1801.33 (I15), U1803.35 (I16)
- new net ALU.D49: U1801.35 (I16), U1803.37 (I17)
- new net ALU.D50: U1801.37 (I17), U1803.39 (I18)
- new net ALU.D51: U1801.39 (I18), U1803.41 (I19)
- new net ALU.D52: U1801.41 (I19), U1803.43 (I20)
- new net ALU.D53: U1801.43 (I20), U1803.45 (I21)
- new net ALU.D54: U1801.45 (I21), U1803.47 (I22)
- new net ALU.D55: U1801.47 (I22), U1803.49 (I23)
- new net ALU.D56: U1801.49 (I23), U1803.51 (I24)
- new net ALU.D57: U1801.51 (I24), U1803.53 (I25)
- new net ALU.D58: U1801.53 (I25), U1803.55 (I26)
- new net ALU.D59: U1801.55 (I26), U1803.57 (I27)
- new net ALU.D60: U1801.57 (I27), U1803.59 (I28)
- new net ALU.D61: U1801.59 (I28), U1803.61 (I29)
- new net ALU.D62: U1801.61 (I29), U1803.63 (I30)
- new net ALU.D63: U1801.63 (I30), U1803.65 (I31)
- new net C.D35: U1801.10 (Y3), U1803.10 (Y3), U1807.10 (Y3), U1808.10 (Y3)
- new net C.D36: U1801.12 (Y4), U1803.12 (Y4), U1807.12 (Y4), U1808.12 (Y4)
- new net C.D37: U1801.14 (Y5), U1803.14 (Y5), U1807.14 (Y5), U1808.14 (Y5)
- new net C.D38: U1801.16 (Y6), U1803.16 (Y6), U1807.16 (Y6), U1808.16 (Y6)
- new net C.D39: U1801.18 (Y7), U1803.18 (Y7), U1807.18 (Y7), U1808.18 (Y7)
- new net C.D40: U1801.20 (Y8), U1803.20 (Y8), U1807.20 (Y8), U1808.20 (Y8)
- new net C.D41: U1801.22 (Y9), U1803.22 (Y9), U1807.22 (Y9), U1808.22 (Y9)
- new net C.D42: U1801.24 (Y10), U1803.24 (Y10), U1807.24 (Y10), U1808.24 (Y10)
- new net C.D43: U1801.26 (Y11), U1803.26 (Y11), U1807.26 (Y11), U1808.26 (Y11)
- new net C.D44: U1801.28 (Y12), U1803.28 (Y12), U1807.28 (Y12), U1808.28 (Y12)
- new net C.D45: U1801.30 (Y13), U1803.30 (Y13), U1807.30 (Y13), U1808.30 (Y13)
- new net C.D46: U1801.32 (Y14), U1803.32 (Y14), U1807.32 (Y14), U1808.32 (Y14)
- new net C.D47: U1801.34 (Y15), U1803.34 (Y15), U1807.34 (Y15), U1808.34 (Y15)
- new net C.D48: U1801.36 (Y16), U1803.36 (Y16), U1807.36 (Y16), U1808.36 (Y16)
- new net C.D49: U1801.38 (Y17), U1803.38 (Y17), U1807.38 (Y17), U1808.38 (Y17)
- new net C.D50: U1801.40 (Y18), U1803.40 (Y18), U1807.40 (Y18), U1808.40 (Y18)
- new net C.D51: U1801.42 (Y19), U1803.42 (Y19), U1807.42 (Y19), U1808.42 (Y19)
- new net C.D52: U1801.44 (Y20), U1803.44 (Y20), U1807.44 (Y20), U1808.44 (Y20)
- new net C.D53: U1801.46 (Y21), U1803.46 (Y21), U1807.46 (Y21), U1808.46 (Y21)
- new net C.D54: U1801.48 (Y22), U1803.48 (Y22), U1807.48 (Y22), U1808.48 (Y22)
- new net C.D55: U1801.50 (Y23), U1803.50 (Y23), U1807.50 (Y23), U1808.50 (Y23)
- new net C.D56: U1801.52 (Y24), U1803.52 (Y24), U1807.52 (Y24), U1808.52 (Y24)
- new net C.D57: U1801.54 (Y25), U1803.54 (Y25), U1807.54 (Y25), U1808.54 (Y25)
- new net C.D58: U1801.56 (Y26), U1803.56 (Y26), U1807.56 (Y26), U1808.56 (Y26)
- new net C.D59: U1801.58 (Y27), U1803.58 (Y27), U1807.58 (Y27), U1808.58 (Y27)
- new net C.D60: U1801.60 (Y28), U1803.60 (Y28), U1807.60 (Y28), U1808.60 (Y28)
- new net C.D61: U1801.62 (Y29), U1803.62 (Y29), U1807.62 (Y29), U1808.62 (Y29)
- new net C.D62: U1801.64 (Y30), U1803.64 (Y30), U1807.64 (Y30), U1808.64 (Y30)
- new net C.D63: U1801.66 (Y31), U1803.66 (Y31), U1807.66 (Y31), U1808.66 (Y31)
- new net CSEL_0_0: U1804.2 (OE)
- new net CSEL_0_1: U1805.2 (OE)
- new net CSEL_0_2: U1802.2 (OE)
- new net CSEL_0_3: U1806.2 (OE)
- new net CSEL_1_1: U1807.2 (OE)
- new net CSEL_1_2: U1803.2 (OE)
- new net CSEL_1_3: U1808.2 (OE)
- new net WDR.D32: U1808.3 (I0)
- new net WDR.D33: U1808.5 (I1)
- new net WDR.D34: U1808.7 (I2)
- new net WDR.D35: U1808.9 (I3)
- new net WDR.D36: U1808.11 (I4)
- new net WDR.D37: U1808.13 (I5)
- new net WDR.D38: U1808.15 (I6)
- new net WDR.D39: U1808.17 (I7)
- new net WDR.D40: U1808.19 (I8)
- new net WDR.D41: U1808.21 (I9)
- new net WDR.D42: U1808.23 (I10)
- new net WDR.D43: U1808.25 (I11)
- new net WDR.D44: U1808.27 (I12)
- new net WDR.D45: U1808.29 (I13)
- new net WDR.D46: U1808.31 (I14)
- new net WDR.D47: U1808.33 (I15)
- new net WDR.D48: U1808.35 (I16)
- new net WDR.D49: U1808.37 (I17)
- new net WDR.D50: U1808.39 (I18)
- new net WDR.D51: U1808.41 (I19)
- new net WDR.D52: U1808.43 (I20)
- new net WDR.D53: U1808.45 (I21)
- new net WDR.D54: U1808.47 (I22)
- new net WDR.D55: U1808.49 (I23)
- new net WDR.D56: U1808.51 (I24)
- new net WDR.D57: U1808.53 (I25)
- new net WDR.D58: U1808.55 (I26)
- new net WDR.D59: U1808.57 (I27)
- new net WDR.D60: U1808.59 (I28)
- new net WDR.D61: U1808.61 (I29)
- new net WDR.D62: U1808.63 (I30)
- new net WDR.D63: U1808.65 (I31)
- no-connect marks 2 -> 8
