File: Schematics/VAL/pg_11.kicad_sch (KiCad schematic)
At the start: 11 parts, among them U1301 F148, U1302 F148, U1303 F148, U1304 F148, U1305 F148, U1306 F148, U1307 F148, U1308 F148, U1309 F151, U1310 F151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

Commit message: Speed up VAL board
Parts:
- removed U1301, U1302, U1303, U1304, U1305, U1306, U1307, U1308: F148, symbol r1000:F148
- removed U1309, U1310, U1311: F151, symbol r1000:F151
Connections:
- no-connect marks 19 -> 0
