File: Schematics/VAL/pg_27.kicad_sch (KiCad schematic)
At the start: 4 parts, among them U2901 25S558, U2902 25S558, U2903 25S558, U2904 25S558

Commit message: KiCad 6
Parts:
- U2901, U2902, U2903, U2904: value 25S558 -> (none)

Commit message: Recover from KiCad-6 munging
Parts:
- U2901, U2902, U2903, U2904: value (none) -> 25S558

Commit message: Align to grid
Parts:
- removed U2901, U2902, U2903, U2904: 25S558, symbol r1000:25S558
- added U (x4): (no value), symbol r1000:25S558
Connections:
- net AHI_BLOW.D0: now also U.23 (Y0)
- net AHI_BLOW.D1: now also U.24 (Y1)
- net AHI_BLOW.D10: now also U.34 (Y10)
- net AHI_BLOW.D11: now also U.35 (Y11)
- net AHI_BLOW.D12: now also U.36 (Y12)
- net AHI_BLOW.D13: now also U.37 (Y13)
- net AHI_BLOW.D14: now also U.38 (Y14)
- net AHI_BLOW.D15: now also U.39 (Y15)
- net AHI_BLOW.D2: now also U.25 (Y2)
- net AHI_BLOW.D3: now also U.26 (Y3)
- net AHI_BLOW.D4: now also U.27 (Y4)
- net AHI_BLOW.D5: now also U.28 (Y5)
- net AHI_BLOW.D6: now also U.29 (Y6)
- net AHI_BLOW.D7: now also U.31 (Y7)
- net AHI_BLOW.D8: now also U.32 (Y8)
- net AHI_BLOW.D9: now also U.33 (Y9)
- net ALOW_BHI.D0: now also U.23 (Y0)
- net ALOW_BHI.D1: now also U.24 (Y1)
- net ALOW_BHI.D10: now also U.34 (Y10)
- net ALOW_BHI.D11: now also U.35 (Y11)
- net ALOW_BHI.D12: now also U.36 (Y12)
- net ALOW_BHI.D13: now also U.37 (Y13)
- net ALOW_BHI.D14: now also U.38 (Y14)
- net ALOW_BHI.D15: now also U.39 (Y15)
- net ALOW_BHI.D2: now also U.25 (Y2)
- net ALOW_BHI.D3: now also U.26 (Y3)
- net ALOW_BHI.D4: now also U.27 (Y4)
- net ALOW_BHI.D5: now also U.28 (Y5)
- net ALOW_BHI.D6: now also U.29 (Y6)
- net ALOW_BHI.D7: now also U.31 (Y7)
- net ALOW_BHI.D8: now also U.32 (Y8)
- net ALOW_BHI.D9: now also U.33 (Y9)
- net A_QUARTER.D0: now also U.8 (A0), U.8 (A0)
- net A_QUARTER.D1: now also U.7 (A1), U.7 (A1)
- net A_QUARTER.D10: now also U.6 (A2), U.6 (A2)
- net A_QUARTER.D11: now also U.5 (A3), U.5 (A3)
- net A_QUARTER.D12: now also U.4 (A4), U.4 (A4)
- net A_QUARTER.D13: now also U.3 (A5), U.3 (A5)
- net A_QUARTER.D14: now also U.2 (A6), U.2 (A6)
- net A_QUARTER.D15: now also U.1 (A7), U.1 (A7)
- net A_QUARTER.D2: now also U.6 (A2), U.6 (A2)
- net A_QUARTER.D3: now also U.5 (A3), U.5 (A3)
- net A_QUARTER.D4: now also U.4 (A4), U.4 (A4)
- net A_QUARTER.D5: now also U.3 (A5), U.3 (A5)
- net A_QUARTER.D6: now also U.2 (A6), U.2 (A6)
- net A_QUARTER.D7: now also U.1 (A7), U.1 (A7)
- net A_QUARTER.D8: now also U.8 (A0), U.8 (A0)
- net A_QUARTER.D9: now also U.7 (A1), U.7 (A1)
- net BHI_ALOW.D0: now also U.32 (Y8)
- net BHI_ALOW.D1: now also U.33 (Y9)
- net BHI_ALOW.D10: now also U.25 (Y2)
- net BHI_ALOW.D11: now also U.26 (Y3)
- net BHI_ALOW.D12: now also U.27 (Y4)
- net BHI_ALOW.D13: now also U.28 (Y5)
- net BHI_ALOW.D14: now also U.29 (Y6)
- net BHI_ALOW.D15: now also U.31 (Y7)
- net BHI_ALOW.D2: now also U.34 (Y10)
- net BHI_ALOW.D3: now also U.35 (Y11)
- net BHI_ALOW.D4: now also U.36 (Y12)
- net BHI_ALOW.D5: now also U.37 (Y13)
- net BHI_ALOW.D6: now also U.38 (Y14)
- net BHI_ALOW.D7: now also U.39 (Y15)
- net BHI_ALOW.D8: now also U.23 (Y0)
- net BHI_ALOW.D9: now also U.24 (Y1)
- net B_QUARTER.D0: now also U.19 (B0), U.19 (B0)
- net B_QUARTER.D1: now also U.18 (B1), U.18 (B1)
- net B_QUARTER.D10: now also U.17 (B2), U.17 (B2)
- net B_QUARTER.D11: now also U.16 (B3), U.16 (B3)
- net B_QUARTER.D12: now also U.15 (B4), U.15 (B4)
- net B_QUARTER.D13: now also U.14 (B5), U.14 (B5)
- net B_QUARTER.D14: now also U.13 (B6), U.13 (B6)
- net B_QUARTER.D15: now also U.12 (B7), U.12 (B7)
- net B_QUARTER.D2: now also U.17 (B2), U.17 (B2)
- net B_QUARTER.D3: now also U.16 (B3), U.16 (B3)
- net B_QUARTER.D4: now also U.15 (B4), U.15 (B4)
- net B_QUARTER.D5: now also U.14 (B5), U.14 (B5)
- net B_QUARTER.D6: now also U.13 (B6), U.13 (B6)
- net B_QUARTER.D7: now also U.12 (B7), U.12 (B7)
- net B_QUARTER.D8: now also U.19 (B0), U.19 (B0)
- net B_QUARTER.D9: now also U.18 (B1), U.18 (B1)
- net LSBYTE.D0: now also U.32 (Y8)
- net LSBYTE.D1: now also U.33 (Y9)
- net LSBYTE.D2: now also U.34 (Y10)
- net LSBYTE.D3: now also U.35 (Y11)
- net LSBYTE.D4: now also U.36 (Y12)
- net LSBYTE.D5: now also U.37 (Y13)
- net LSBYTE.D6: now also U.38 (Y14)
- net LSBYTE.D7: now also U.39 (Y15)
- net MULT_OUT.D0: now also U.23 (Y0)
- net MULT_OUT.D1: now also U.24 (Y1)
- net MULT_OUT.D2: now also U.25 (Y2)
- net MULT_OUT.D3: now also U.26 (Y3)
- net MULT_OUT.D4: now also U.27 (Y4)
- net MULT_OUT.D5: now also U.28 (Y5)
- net MULT_OUT.D6: now also U.29 (Y6)
- net MULT_OUT.D7: now also U.31 (Y7)
- net PD: now also U.11 (RU), U.11 (RU), U.11 (RU), U.11 (RU), U.20 (BM), U.20 (BM), U.20 (BM), U.20 (BM), U.21 (OE), U.21 (OE), U.21 (OE), U.21 (OE), U.40 (AM), U.40 (AM), U.40 (AM), U.40 (AM), U.9 (RS), U.9 (RS), U.9 (RS), U.9 (RS)

Commit message: Snapshot
Parts:
- removed U (x4): (no value), symbol r1000:25S558
Connections:
- no-connect marks 4 -> 0
