File: Schematics/VAL/pg_29.kicad_sch (KiCad schematic)
At the start: 32 parts, among them U3101 F04, U3102 F04, U3103 F04, U3104 F04, U3105 F04, U3106 F04, U3107 F04, U3108 F04, U3109 F04, U3110 F04, U3111 F04, U3112 F04, U3113 F04, U3114 F04, U3115 F04, U3116 F04, U3117 F04, U3118 F04, U3119 F04, U3120 F04, U3121 F04, U3122 F04, U3123 F04, U3124 F04, U3125 F04, U3126 F04, U3127 F04, U3128 F04, U3129 F04, U3130 F04, U3131 F04, U3132 F04

Commit message: Align to grid
Parts:
- removed U3101, U3102, U3103, U3104, U3105, U3106, U3107, U3108, U3109, U3110, U3111, U3112, U3113, U3114, U3115, U3116, U3117, U3118, U3119, U3120, U3121, U3122, U3123, U3124, U3125, U3126, U3127, U3128, U3129, U3130, U3131, U3132: F04, symbol r1000:F04
- added U (x32): (no value), symbol r1000:F04
Connections:
- net CPA.D0: now also U.1 (D0)
- net CPA.D1: now also U.1 (D0)
- net CPA.D10: now also U.1 (D0)
- net CPA.D11: now also U.1 (D0)
- net CPA.D12: now also U.1 (D0)
- net CPA.D13: now also U.1 (D0)
- net CPA.D14: now also U.1 (D0)
- net CPA.D15: now also U.1 (D0)
- net CPA.D16: now also U.1 (D0)
- net CPA.D17: now also U.1 (D0)
- net CPA.D18: now also U.1 (D0)
- net CPA.D19: now also U.1 (D0)
- net CPA.D2: now also U.1 (D0)
- net CPA.D20: now also U.1 (D0)
- net CPA.D21: now also U.1 (D0)
- net CPA.D22: now also U.1 (D0)
- net CPA.D23: now also U.1 (D0)
- net CPA.D3: now also U.1 (D0)
- net CPA.D4: now also U.1 (D0)
- net CPA.D5: now also U.1 (D0)
- net CPA.D6: now also U.1 (D0)
- net CPA.D7: now also U.1 (D0)
- net CPA.D8: now also U.1 (D0)
- net CPA.D9: now also U.1 (D0)
- net LSBYTE.D0: now also U.1 (D0)
- net LSBYTE.D1: now also U.1 (D0)
- net LSBYTE.D2: now also U.1 (D0)
- net LSBYTE.D3: now also U.1 (D0)
- net LSBYTE.D4: now also U.1 (D0)
- net LSBYTE.D5: now also U.1 (D0)
- net LSBYTE.D6: now also U.1 (D0)
- net LSBYTE.D7: now also U.1 (D0)
- net PRODUCT.D0: now also U.2 (Q)
- net PRODUCT.D1: now also U.2 (Q)
- net PRODUCT.D10: now also U.2 (Q)
- net PRODUCT.D11: now also U.2 (Q)
- net PRODUCT.D12: now also U.2 (Q)
- net PRODUCT.D13: now also U.2 (Q)
- net PRODUCT.D14: now also U.2 (Q)
- net PRODUCT.D15: now also U.2 (Q)
- net PRODUCT.D16: now also U.2 (Q)
- net PRODUCT.D17: now also U.2 (Q)
- net PRODUCT.D18: now also U.2 (Q)
- net PRODUCT.D19: now also U.2 (Q)
- net PRODUCT.D2: now also U.2 (Q)
- net PRODUCT.D20: now also U.2 (Q)
- net PRODUCT.D21: now also U.2 (Q)
- net PRODUCT.D22: now also U.2 (Q)
- net PRODUCT.D23: now also U.2 (Q)
- net PRODUCT.D24: now also U.2 (Q)
- net PRODUCT.D25: now also U.2 (Q)
- net PRODUCT.D26: now also U.2 (Q)
- net PRODUCT.D27: now also U.2 (Q)
- net PRODUCT.D28: now also U.2 (Q)
- net PRODUCT.D29: now also U.2 (Q)
- net PRODUCT.D3: now also U.2 (Q)
- net PRODUCT.D30: now also U.2 (Q)
- net PRODUCT.D31: now also U.2 (Q)
- net PRODUCT.D4: now also U.2 (Q)
- net PRODUCT.D5: now also U.2 (Q)
- net PRODUCT.D6: now also U.2 (Q)
- net PRODUCT.D7: now also U.2 (Q)
- net PRODUCT.D8: now also U.2 (Q)
- net PRODUCT.D9: now also U.2 (Q)

Commit message: Snapshot
Parts:
- removed U (x32): (no value), symbol r1000:F04
