File: Schematics/TYP/TYP.kicad_sch (KiCad schematic)
At the start: 2 parts, among them U101 Pull_Up, U102 Pull_Down

Commit message: New diff'able format
Other:
- sheet Page 0 renamed Page 00
- sheet Page 1 renamed Page 01
- sheet Page 2 renamed Page 02
- sheet Page 3 renamed Page 03
- sheet Page 4 renamed Page 04
- sheet Page 5 renamed Page 05
- sheet Page 6 renamed Page 06
- sheet Page 7 renamed Page 07
- sheet Page 8 renamed Page 08
- sheet Page 9 renamed Page 09
- note added: "A LATCH"
- note added: "ADDRESS BUS DRIVERS"
- note added: "ADDRESS BUS PARITY - PARITY"
- note added: "ALU ARRAY - LEAST SIGNIFICANT BITS"
- note added: "ALU ARRAY - MOST SIGNIFICANT BITS"
- note added: "B LATCH"
- note added: "BUS CONTROL"
- note added: "Board: TYP Branch: main"
- note added: "C BUS DRIVER"
- note added: "C BUS SOURCE <6>"
- note added: "C SOURCE CONTROL"
- note added: "C SOURCE MUX"
- note added: "CHECKER LOGIC <6>"
- note added: "CLASS CHECK LOGIC"
- note added: "CLOCK GENERATION - FREE RUNNING CLOCKS"
- note added: "CLOCK GENERATION - RAM WRITE ENABLES"
- note added: "CLOCK GENERATION - STATE CLOCKS"
- note added: "CONDITION LOGIC"
- note added: "COUNTER LOGIC"
- note added: "DIAG & CONTROL SYSTEM <6>"
- note added: "DIAGNOSTIC PROCESSOR - 8051 AND NOVRAM"
- note added: "DIAGNOSTIC PROCESSOR - FINITE STATE MACHINE"
- note added: "DIAGNOSTIC PROCESSOR - PULLUPS & PARITY REGISTER"
- note added: "FIU DRIVER AND RECEIVER"
- note added: "FIU DRIVER AND RECEIVER - PARITY"
- note added: "LOOP COUNTER CONTROL"
- note added: "LOOP COUNTER LOGIC - ZERO DRIVERS"
- note added: "OF KIND CONDITION LOGIC"
- note added: "POWER AND GROUND FINGERS - & BYPASS CAPACITORS <6>"
- note added: "PRIVACY CHECK LOGIC"
- note added: "REGISTER FILE <6>"
- note added: "REGISTER FILE A - RAM ARRAY"
- note added: "REGISTER FILE A PARITY"
- note added: "REGISTER FILE B - RAM ARRAY"
- note added: "REGISTER FILE B PARITY"
- note added: "REGISTER FILE CONTROL"
- note added: "REGISTER FILE CONTROL - A ADDRESS GENERATION"
- note added: "REGISTER FILE CONTROL - B ADDRESS GENERATION"
- note added: "REGISTER FILE CONTROL - C ADDRESS GENERATION"
- note added: "REGISTER FILE CONTROL - CSA ADRESS GENERATION"
- note added: "TYPE BOARD <6>"
- note added: "TYPE BOARD MICROCODE <6>"
- note added: "TYPE DRIVER AND RECEIVER"
- note added: "TYPE DRIVERS AND RECEIVERS - PARITY"
- note added: "WRITABLE CONTROL STORE - CSA CONTROL"
- note added: "WRITABLE CONTROL STORE - LOOP REGISTER PRE-DECODE"
- note added: "WRITABLE CONTROL STORE - MICRO INSTRUCTION REGISTER"
- note added: "WRITABLE CONTROL STORE - WCS ADDRESS GENERATION"
- note added: "WRITABLE CONTROL STORE - WCS BITS 0 TO 15"
- note added: "WRITABLE CONTROL STORE - WCS BITS 16 TO 31"
- note added: "WRITABLE CONTROL STORE - WCS BITS 32 TO 45"
- note added: "WRITABLE CONTROL STORE - WCS PARITY"
- note added: "WRITE DATA REGISTER - INPUT BUFFER"
- note added: "WRITE DATA REGISTER - PARITY BITS"
- note added: "WRITE DATA REGISTER - REGISTER ARRAY"
- note removed: "00: TYPE BOARD MICROCODE 01: TYPE BOARD 02: TYPE BOARD 03: C BUS SOURCE 04: REGISTER FILE 05: CHECKER LOGIC 06: DIAG & CONTROL SYSTEM 07: DIAG & CONTROL SYSTEM 08: DIAG & CONTROL SYSTEM 09: DIAG & CONTROL SYSTEM 10: COUNTER LOGIC 11: LOOP COUNTER LOGIC - ZERO DRIVERS 12: WRITE DATA REGISTER - INPUT BUFFER 13: WRITE DATA REGISTER - REGISTER ARRAY 14: WRITE DATA REGISTER - PARITY BITS 15: C SOURCE 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"
- moved on the sheet: U101, U102

Commit message: Unduplicate signals
Other:
- note added: "Board: TYP Branch: optimized"
- note removed: "Board: TYP Branch: main"
Changed lines of the file:
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@@
   (symbol (lib_id "r1000:Pull_Down") (at 566.42 259.08 0) (unit 1) (in_bom yes) (on_board yes) (property "Reference" "U102" (id 0) (at 566.42 259.08 0) ) (property "Value" "Pull_Down" (id 1) (at 566.42 255.27 0) (effects (font (size 2.54 2.54) ) ) ) (property "Footprint" "" (id 2) (at 566.42 259.08 0) (effects (font (size 1.27 1.27) ) hide ) ) (property "Datasheet" "" (id 3) (at 566.42 259.08 0) (effects (font (size 1.27 1.27) ) hide ) ) (pin "1" ) )
   (symbol (lib_id "r1000:PU") (at 566.42 241.3 0) (unit 1) (in_bom yes) (on_board yes) (property "Reference" "#PWR0101" (id 0) (at 566.42 241.3 0) (effects (font (size 1.27 1.27) ) hide ) ) (property "Value" "PU" (id 1) (at 566.42 241.3 0) (effects (font (size 1.27 1.27) ) hide ) ) (property "Footprint" "" (id 2) (at 566.42 241.3 0) (effects (font (size 1.27 1.27) ) hide ) ) (property "Datasheet" "" (id 3) (at 566.42 241.3 0) (effects (font (size 1.27 1.27) ) hide ) ) (pin "1" ) )
-  (text "Board: TYP Branch: main" (at 7.62 370.84 0) (effects (font (size 7.62 7.62) (thickness 1.27) bold ) (justify left bottom) ) )
+  (text "Board: TYP Branch: optimized" (at 7.62 370.84 0) (effects (font (size 7.62 7.62) (thickness 1.27) bold ) (justify left bottom) ) )
   (sheet_instances
     (path "/" (page "00") )

Commit message: Snapshot
Other:
- note added: "Board: TYP Branch: megacomp2"
- note removed: "Board: TYP Branch: optimized"
Changed lines of the file:
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@@
   (symbol (lib_id "r1000:Pull_Down") (at 566.42 259.08 0) (unit 1) (in_bom yes) (on_board yes) (property "Reference" "U102" (id 0) (at 566.42 259.08 0) ) (property "Value" "Pull_Down" (id 1) (at 566.42 255.27 0) (effects (font (size 2.54 2.54) ) ) ) (property "Footprint" "" (id 2) (at 566.42 259.08 0) (effects (font (size 1.27 1.27) ) hide ) ) (property "Datasheet" "" (id 3) (at 566.42 259.08 0) (effects (font (size 1.27 1.27) ) hide ) ) (pin "1" ) )
   (symbol (lib_id "r1000:PU") (at 566.42 241.3 0) (unit 1) (in_bom yes) (on_board yes) (property "Reference" "#PWR0101" (id 0) (at 566.42 241.3 0) (effects (font (size 1.27 1.27) ) hide ) ) (property "Value" "PU" (id 1) (at 566.42 241.3 0) (effects (font (size 1.27 1.27) ) hide ) ) (property "Footprint" "" (id 2) (at 566.42 241.3 0) (effects (font (size 1.27 1.27) ) hide ) ) (property "Datasheet" "" (id 3) (at 566.42 241.3 0) (effects (font (size 1.27 1.27) ) hide ) ) (pin "1" ) )
-  (text "Board: TYP Branch: optimized" (at 7.62 370.84 0) (effects (font (size 7.62 7.62) (thickness 1.27) bold ) (justify left bottom) ) )
+  (text "Board: TYP Branch: megacomp2" (at 7.62 370.84 0) (effects (font (size 7.62 7.62) (thickness 1.27) bold ) (justify left bottom) ) )
   (sheet_instances
     (path "/" (page "00") )

Commit message: Use XWCSRAM
Other:
- note added: "WRITABLE CONTROL STORE - WCS BITS 16 TO 31 <6>"
- note added: "WRITABLE CONTROL STORE - WCS BITS 32 TO 45 <6>"
- note removed: "WRITABLE CONTROL STORE - WCS BITS 16 TO 31"
- note removed: "WRITABLE CONTROL STORE - WCS BITS 32 TO 45"
Changed lines of the file:
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@@
   (sheet (at 266.70 50.80) (size 20.32 5.08) (property "Sheet name" "Page 50" (id 0) (at 289.56 55.88 0) (effects (font (size 2.54 2.54) ) (justify left bottom) ) ) (property "Sheet file" "pg_50.kicad_sch" (id 1) (at 289.56 53.34 0) (effects (justify left bottom) hide ) ) )
   (text "WRITABLE CONTROL STORE - WCS BITS 0 TO 15" (at 307.34 55.88 0) (effects (font (size 2.54 2.54) ) (justify left bottom) ) )
-  (sheet (at 266.70 58.42) (size 20.32 5.08) (property "Sheet name" "Page 51" (id 0) (at 289.56 63.50 0) (effects (font (size 2.54 2.54) ) (justify left bottom) ) ) (property "Sheet file" "pg_51.kicad_sch" (id 1) (at 289.56 60.96 0) (effects (justify left bottom) hide ) ) )
-  (text "WRITABLE CONTROL STORE - WCS BITS 16 TO 31" (at 307.34 63.50 0) (effects (font (size 2.54 2.54) ) (justify left bottom) ) )
-  (sheet (at 266.70 66.04) (size 20.32 5.08) (property "Sheet name" "Page 52" (id 0) (at 289.56 71.12 0) (effects (font (size 2.54 2.54) ) (justify left bottom) ) ) (property "Sheet file" "pg_52.kicad_sch" (id 1) (at 289.56 68.58 0) (effects (justify left bottom) hide ) ) )
-  (text "WRITABLE CONTROL STORE - WCS BITS 32 TO 45" (at 307.34 71.12 0) (effects (font (size 2.54 2.54) ) (justify left bottom) ) )
+  (sheet (at 266.70 58.42) (size 20.32 5.08) (property "Sheet name" "Page 51" (id 0) (at 289.56 63.50 0) (effects (font (size 2.54 2.54) ) (justify left bottom) ) ) (property "Sheet file" "pg_51.kicad_sch" (id 1) (at 289.56 60.96 0) (effects (justify left bottom) hide ) ) (fill (color 192 192 192 1.0) ) )
+  (text "WRITABLE CONTROL STORE - WCS BITS 16 TO 31 <6>" (at 307.34 63.50 0) (effects (font (size 2.54 2.54) ) (justify left bottom) ) )
+  (sheet (at 266.70 66.04) (size 20.32 5.08) (property "Sheet name" "Page 52" (id 0) (at 289.56 71.12 0) (effects (font (size 2.54 2.54) ) (justify left bottom) ) ) (property "Sheet file" "pg_52.kicad_sch" (id 1) (at 289.56 68.58 0) (effects (justify left bottom) hide ) ) (fill (color 192 192 192 1.0) ) )
+  (text "WRITABLE CONTROL STORE - WCS BITS 32 TO 45 <6>" (at 307.34 71.12 0) (effects (font (size 2.54 2.54) ) (justify left bottom) ) )
   (sheet (at 266.70 73.66) (size 20.32 5.08) (property "Sheet name" "Page 53" (id 0) (at 289.56 78.74 0) (effects (font (size 2.54 2.54) ) (justify left bottom) ) ) (property "Sheet file" "pg_53.kicad_sch" (id 1) (at 289.56 76.20 0) (effects (justify left bottom) hide ) ) )
   (text "WRITABLE CONTROL STORE - WCS PARITY" (at 307.34 78.74 0) (effects (font (size 2.54 2.54) ) (justify left bottom) ) )

Commit message: Megacomp'ing TYP
Other:
- note added: "WRITE DATA REGISTER - PARITY BITS <6>"
- note removed: "WRITE DATA REGISTER - PARITY BITS"
Changed lines of the file:
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@@
   (sheet (at 12.70 111.76) (size 20.32 5.08) (property "Sheet name" "Page 13" (id 0) (at 35.56 116.84 0) (effects (font (size 2.54 2.54) ) (justify left bottom) ) ) (property "Sheet file" "pg_13.kicad_sch" (id 1) (at 35.56 114.30 0) (effects (justify left bottom) hide ) ) )
   (text "WRITE DATA REGISTER - REGISTER ARRAY" (at 53.34 116.84 0) (effects (font (size 2.54 2.54) ) (justify left bottom) ) )
-  (sheet (at 12.70 119.38) (size 20.32 5.08) (property "Sheet name" "Page 14" (id 0) (at 35.56 124.46 0) (effects (font (size 2.54 2.54) ) (justify left bottom) ) ) (property "Sheet file" "pg_14.kicad_sch" (id 1) (at 35.56 121.92 0) (effects (justify left bottom) hide ) ) )
-  (text "WRITE DATA REGISTER - PARITY BITS" (at 53.34 124.46 0) (effects (font (size 2.54 2.54) ) (justify left bottom) ) )
+  (sheet (at 12.70 119.38) (size 20.32 5.08) (property "Sheet name" "Page 14" (id 0) (at 35.56 124.46 0) (effects (font (size 2.54 2.54) ) (justify left bottom) ) ) (property "Sheet file" "pg_14.kicad_sch" (id 1) (at 35.56 121.92 0) (effects (justify left bottom) hide ) ) (fill (color 192 192 192 1.0) ) )
+  (text "WRITE DATA REGISTER - PARITY BITS <6>" (at 53.34 124.46 0) (effects (font (size 2.54 2.54) ) (justify left bottom) ) )
   (sheet (at 12.70 127.00) (size 20.32 5.08) (property "Sheet name" "Page 15" (id 0) (at 35.56 132.08 0) (effects (font (size 2.54 2.54) ) (justify left bottom) ) ) (property "Sheet file" "pg_15.kicad_sch" (id 1) (at 35.56 129.54 0) (effects (justify left bottom) hide ) ) )
   (text "C SOURCE MUX" (at 53.34 132.08 0) (effects (font (size 2.54 2.54) ) (justify left bottom) ) )

Commit message: More polishing
Other:
- note added: "ALU ARRAY - LEAST SIGNIFICANT BITS <6>"
- note removed: "ALU ARRAY - LEAST SIGNIFICANT BITS"
Changed lines of the file:
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@@
   (sheet (at 12.70 226.06) (size 20.32 5.08) (property "Sheet name" "Page 28" (id 0) (at 35.56 231.14 0) (effects (font (size 2.54 2.54) ) (justify left bottom) ) ) (property "Sheet file" "pg_28.kicad_sch" (id 1) (at 35.56 228.60 0) (effects (justify left bottom) hide ) ) )
   (text "ALU ARRAY - MOST SIGNIFICANT BITS" (at 53.34 231.14 0) (effects (font (size 2.54 2.54) ) (justify left bottom) ) )
-  (sheet (at 12.70 233.68) (size 20.32 5.08) (property "Sheet name" "Page 29" (id 0) (at 35.56 238.76 0) (effects (font (size 2.54 2.54) ) (justify left bottom) ) ) (property "Sheet file" "pg_29.kicad_sch" (id 1) (at 35.56 236.22 0) (effects (justify left bottom) hide ) ) )
-  (text "ALU ARRAY - LEAST SIGNIFICANT BITS" (at 53.34 238.76 0) (effects (font (size 2.54 2.54) ) (justify left bottom) ) )
+  (sheet (at 12.70 233.68) (size 20.32 5.08) (property "Sheet name" "Page 29" (id 0) (at 35.56 238.76 0) (effects (font (size 2.54 2.54) ) (justify left bottom) ) ) (property "Sheet file" "pg_29.kicad_sch" (id 1) (at 35.56 236.22 0) (effects (justify left bottom) hide ) ) (fill (color 192 192 192 1.0) ) )
+  (text "ALU ARRAY - LEAST SIGNIFICANT BITS <6>" (at 53.34 238.76 0) (effects (font (size 2.54 2.54) ) (justify left bottom) ) )
   (sheet (at 12.70 241.30) (size 20.32 5.08) (property "Sheet name" "Page 30" (id 0) (at 35.56 246.38 0) (effects (font (size 2.54 2.54) ) (justify left bottom) ) ) (property "Sheet file" "pg_30.kicad_sch" (id 1) (at 35.56 243.84 0) (effects (justify left bottom) hide ) ) )
   (text "CONDITION LOGIC" (at 53.34 246.38 0) (effects (font (size 2.54 2.54) ) (justify left bottom) ) )

Commit message: KiCad 6
Parts:
- U101: value Pull_Up -> (none)
- U102: value Pull_Down -> (none)
Changed lines of the file:
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@@
   (wire (pts (xy 566.42 259.08) (xy 566.42 261.62) ) (stroke (width 0) (type default) (color 0 0 0 0) ) )
   (wire (pts (xy 566.42 241.3) (xy 566.42 243.84) ) (stroke (width 0) (type default) (color 0 0 0 0) ) )
-  (symbol (lib_id "r1000:PD") (at 566.42 261.62 0) (unit 1) (in_bom no) (on_board yes) (property "Reference" "#PWR0102" (id 0) (at 566.42 261.62 0) (effects (font (size 1.27 1.27) ) hide ) ) (property "Value" "PD" (id 1) (at 566.42 261.62 0) (effects (font (size 1.27 1.27) ) hide ) ) (property "Footprint" "" (id 2) (at 566.42 261.62 0) (effects (font (size 1.27 1.27) ) hide ) ) (property "Datasheet" "" (id 3) (at 566.42 261.62 0) (effects (font (size 1.27 1.27) ) hide ) ) (pin "1" ) )
-  (symbol (lib_id "r1000:Pull_Up") (at 566.42 243.84 0) (unit 1) (in_bom yes) (on_board yes) (property "Reference" "U101" (id 0) (at 566.42 243.84 0) ) (property "Value" "Pull_Up" (id 1) (at 566.42 247.65 0) (effects (font (size 2.54 2.54) ) ) ) (property "Footprint" "" (id 2) (at 566.42 243.84 0) (effects (font (size 1.27 1.27) ) hide ) ) (property "Datasheet" "" (id 3) (at 566.42 243.84 0) (effects (font (size 1.27 1.27) ) hide ) ) (pin "1" ) )
-  (symbol (lib_id "r1000:Pull_Down") (at 566.42 259.08 0) (unit 1) (in_bom yes) (on_board yes) (property "Reference" "U102" (id 0) (at 566.42 259.08 0) ) (property "Value" "Pull_Down" (id 1) (at 566.42 255.27 0) (effects (font (size 2.54 2.54) ) ) ) (property "Footprint" "" (id 2) (at 566.42 259.08 0) (effects (font (size 1.27 1.27) ) hide ) ) (property "Datasheet" "" (id 3) (at 566.42 259.08 0) (effects (font (size 1.27 1.27) ) hide ) ) (pin "1" ) )
-  (symbol (lib_id "r1000:PU") (at 566.42 241.3 0) (unit 1) (in_bom yes) (on_board yes) (property "Reference" "#PWR0101" (id 0) (at 566.42 241.3 0) (effects (font (size 1.27 1.27) ) hide ) ) (property "Value" "PU" (id 1) (at 566.42 241.3 0) (effects (font (size 1.27 1.27) ) hide ) ) (property "Footprint" "" (id 2) (at 566.42 241.3 0) (effects (font (size 1.27 1.27) ) hide ) ) (property "Datasheet" "" (id 3) (at 566.42 241.3 0) (effects (font (size 1.27 1.27) ) hide ) ) (pin "1" ) )
+  (symbol (lib_id "r1000:PD") (at 566.42 261.62 0) (unit 1) (in_bom no) (on_board yes) (property "Reference" "#PWR0102" (id 0) (at 566.42 261.62 0) (effects (font (size 1.27 1.27) ) hide ) ) (property "Value" "" (id 1) (at 566.42 261.62 0) (effects (font (size 1.27 1.27) ) hide ) ) (property "Footprint" "" (id 2) (at 566.42 261.62 0) (effects (font (size 1.27 1.27) ) hide ) ) (property "Datasheet" "" (id 3) (at 566.42 261.62 0) (effects (font (size 1.27 1.27) ) hide ) ) (pin "1" ) )
+  (symbol (lib_id "r1000:Pull_Up") (at 566.42 243.84 0) (unit 1) (in_bom yes) (on_board yes) (property "Reference" "U101" (id 0) (at 566.42 243.84 0) ) (property "Value" "" (id 1) (at 566.42 247.65 0) (effects (font (size 2.54 2.54) ) ) ) (property "Footprint" "" (id 2) (at 566.42 243.84 0) (effects (font (size 1.27 1.27) ) hide ) ) (property "Datasheet" "" (id 3) (at 566.42 243.84 0) (effects (font (size 1.27 1.27) ) hide ) ) (pin "1" ) )
+  (symbol (lib_id "r1000:Pull_Down") (at 566.42 259.08 0) (unit 1) (in_bom yes) (on_board yes) (property "Reference" "U102" (id 0) (at 566.42 259.08 0) ) (property "Value" "" (id 1) (at 566.42 255.27 0) (effects (font (size 2.54 2.54) ) ) ) (property "Footprint" "" (id 2) (at 566.42 259.08 0) (effects (font (size 1.27 1.27) ) hide ) ) (property "Datasheet" "" (id 3) (at 566.42 259.08 0) (effects (font (size 1.27 1.27) ) hide ) ) (pin "1" ) )
+  (symbol (lib_id "r1000:PU") (at 566.42 241.3 0) (unit 1) (in_bom yes) (on_board yes) (property "Reference" "#PWR0101" (id 0) (at 566.42 241.3 0) (effects (font (size 1.27 1.27) ) hide ) ) (property "Value" "" (id 1) (at 566.42 241.3 0) (effects (font (size 1.27 1.27) ) hide ) ) (property "Footprint" "" (id 2) (at 566.42 241.3 0) (effects (font (size 1.27 1.27) ) hide ) ) (property "Datasheet" "" (id 3) (at 566.42 241.3 0) (effects (font (size 1.27 1.27) ) hide ) ) (pin "1" ) )
   (text "Board: TYP Branch: megacomp2" (at 7.62 370.84 0) (effects (font (size 7.62 7.62) (thickness 1.27) bold ) (justify left bottom) ) )
   (sheet_instances
