File: Schematics/TYP/pg_33.kicad_sch (KiCad schematic)
At the start: 5 parts, among them U3501 XPAR64, U3509 F240, U3510 F240, U3511 F244, U3512 F521

Commit message: Snapshot
Connections:
- net B.PCHK0: now also U3510.2 (I0); no longer U3510.8 (I3)
- net B.PCHK1: now also U3510.4 (I1); no longer U3510.6 (I2)
- net B.PCHK2: now also U3510.6 (I2); no longer U3510.4 (I1)
- net B.PCHK3: now also U3510.8 (I3); no longer U3510.2 (I0)
- net B.PCHK4: now also U3510.11 (I4); no longer U3510.17 (I7)
- net B.PCHK5: now also U3510.13 (I5); no longer U3510.15 (I6)
- net B.PCHK6: now also U3510.15 (I6); no longer U3510.13 (I5)
- net B.PCHK7: now also U3510.17 (I7); no longer U3510.11 (I4)
- net T.TYPE.P0: now also U3510.18 (Y0); no longer U3510.12 (Y3)
- net T.TYPE.P1: now also U3510.16 (Y1); no longer U3510.14 (Y2)
- net T.TYPE.P2: now also U3510.14 (Y2); no longer U3510.16 (Y1)
- net T.TYPE.P3: now also U3510.12 (Y3); no longer U3510.18 (Y0)
- net T.TYPE.P4: now also U3510.9 (Y4); no longer U3510.3 (Y7)
- net T.TYPE.P5: now also U3510.7 (Y5); no longer U3510.5 (Y6)
- net T.TYPE.P6: now also U3510.5 (Y6); no longer U3510.7 (Y5)
- net T.TYPE.P7: now also U3510.3 (Y7); no longer U3510.9 (Y4)
Changed lines of the file:
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@@
   (label "B.PCHK6" (at 154.94 66.04 0) (effects (font (size 2.54 2.54) ) (justify left bottom) ) )
   (label "B.PCHK7" (at 154.94 71.12 0) (effects (font (size 2.54 2.54) ) (justify left bottom) ) )
-  (label "B.PCHK3" (at 236.22 132.08 0) (effects (font (size 2.54 2.54) ) (justify left bottom) ) )
-  (label "B.PCHK2" (at 236.22 137.16 0) (effects (font (size 2.54 2.54) ) (justify left bottom) ) )
-  (label "B.PCHK1" (at 236.22 142.24 0) (effects (font (size 2.54 2.54) ) (justify left bottom) ) )
-  (label "B.PCHK0" (at 236.22 147.32 0) (effects (font (size 2.54 2.54) ) (justify left bottom) ) )
-  (label "B.PCHK7" (at 236.22 152.4 0) (effects (font (size 2.54 2.54) ) (justify left bottom) ) )
-  (label "B.PCHK6" (at 236.22 157.48 0) (effects (font (size 2.54 2.54) ) (justify left bottom) ) )
-  (label "B.PCHK5" (at 236.22 162.56 0) (effects (font (size 2.54 2.54) ) (justify left bottom) ) )
-  (label "B.PCHK4" (at 236.22 167.64 0) (effects (font (size 2.54 2.54) ) (justify left bottom) ) )
+  (label "B.PCHK0" (at 236.22 132.08 0) (effects (font (size 2.54 2.54) ) (justify left bottom) ) )
+  (label "B.PCHK1" (at 236.22 137.16 0) (effects (font (size 2.54 2.54) ) (justify left bottom) ) )
+  (label "B.PCHK2" (at 236.22 142.24 0) (effects (font (size 2.54 2.54) ) (justify left bottom) ) )
+  (label "B.PCHK3" (at 236.22 147.32 0) (effects (font (size 2.54 2.54) ) (justify left bottom) ) )
+  (label "B.PCHK4" (at 236.22 152.4 0) (effects (font (size 2.54 2.54) ) (justify left bottom) ) )
+  (label "B.PCHK5" (at 236.22 157.48 0) (effects (font (size 2.54 2.54) ) (justify left bottom) ) )
+  (label "B.PCHK6" (at 236.22 162.56 0) (effects (font (size 2.54 2.54) ) (justify left bottom) ) )
+  (label "B.PCHK7" (at 236.22 167.64 0) (effects (font (size 2.54 2.54) ) (justify left bottom) ) )
   (global_label "TYPE_DRV.OE~" (shape input) (at 264.16 114.3 180) (fields_autoplaced) (effects (font (size 2.54 2.54) ) (justify right) ) (property "Intersheet References" "${INTERSHEET_REFS}" (id 0) (at 233.2083 114.1413 0) (effects (font (size 1.905 1.905) ) (justify right) ) ) )
   (junction (at 271.78 114.3) (diameter 0) (color 0 0 0 0) )
   (symbol (lib_id "r1000:F240") (at 274.32 165.1 0) (unit 1) (in_bom yes) (on_board yes) (property "Reference" "U3510" (id 0) (at 276.86 160.02 0) (effects (font (size 1.27 1.27) ) ) ) (property "Value" "F240" (id 1) (at 270.51 172.72 0) (effects (font (size 2.54 2.54) ) (justify left) ) ) (property "Footprint" "" (id 2) (at 275.59 166.37 0) (effects (font (size 1.27 1.27) ) hide ) ) (property "Datasheet" "" (id 3) (at 275.59 166.37 0) (effects (font (size 1.27 1.27) ) hide ) ) (property "Location" "A20" (id 4) (at 273.05 165.1 0) (effects (font (size 2.54 2.54) ) (justify left) ) ) (property "Name" "TPDR1" (id 5) (at 275.59 180.34 0) (effects (font (size 2.54 2.54) ) (justify bottom) ) ) (pin "1") (pin "11") (pin "12") (pin "13") (pin "14") (pin "15") (pin "16") (pin "17") (pin "18") (pin "19") (pin "2") (pin "3") (pin "4") (pin "5") (pin "6") (pin "7") (pin "8") (pin "9") )
-  (label "T.TYPE.P3" (at 299.72 132.08 0) (effects (font (size 2.54 2.54) ) (justify left bottom) ) )
-  (label "T.TYPE.P2" (at 299.72 137.16 0) (effects (font (size 2.54 2.54) ) (justify left bottom) ) )
-  (label "T.TYPE.P1" (at 299.72 142.24 0) (effects (font (size 2.54 2.54) ) (justify left bottom) ) )
-  (label "T.TYPE.P0" (at 299.72 147.32 0) (effects (font (size 2.54 2.54) ) (justify left bottom) ) )
-  (label "T.TYPE.P7" (at 299.72 152.4 0) (effects (font (size 2.54 2.54) ) (justify left bottom) ) )
-  (label "T.TYPE.P6" (at 299.72 157.48 0) (effects (font (size 2.54 2.54) ) (justify left bottom) ) )
-  (label "T.TYPE.P5" (at 299.72 162.56 0) (effects (font (size 2.54 2.54) ) (justify left bottom) ) )
-  (label "T.TYPE.P4" (at 299.72 167.64 0) (effects (font (size 2.54 2.54) ) (justify left bottom) ) )
+  (label "T.TYPE.P0" (at 299.72 132.08 0) (effects (font (size 2.54 2.54) ) (justify left bottom) ) )
+  (label "T.TYPE.P1" (at 299.72 137.16 0) (effects (font (size 2.54 2.54) ) (justify left bottom) ) )
+  (label "T.TYPE.P2" (at 299.72 142.24 0) (effects (font (size 2.54 2.54) ) (justify left bottom) ) )
+  (label "T.TYPE.P3" (at 299.72 147.32 0) (effects (font (size 2.54 2.54) ) (justify left bottom) ) )
+  (label "T.TYPE.P4" (at 299.72 152.4 0) (effects (font (size 2.54 2.54) ) (justify left bottom) ) )
+  (label "T.TYPE.P5" (at 299.72 157.48 0) (effects (font (size 2.54 2.54) ) (justify left bottom) ) )
+  (label "T.TYPE.P6" (at 299.72 162.56 0) (effects (font (size 2.54 2.54) ) (justify left bottom) ) )
+  (label "T.TYPE.P7" (at 299.72 167.64 0) (effects (font (size 2.54 2.54) ) (justify left bottom) ) )
   (global_label "B_ADR.P[0..7]" (shape input) (at 318.0315 203.2 180) (fields_autoplaced) (effects (font (size 2.54 2.54) ) (justify right) ) (property "Intersheet References" "${INTERSHEET_REFS}" (id 0) (at 287.0798 203.0413 0) (effects (font (size 1.905 1.905) ) (justify right) ) ) )
   (global_label "T.TYPE.P[0..7]" (shape input) (at 322.58 68.58 180) (fields_autoplaced) (effects (font (size 2.54 2.54) ) (justify right) ) (property "Intersheet References" "${INTERSHEET_REFS}" (id 0) (at 291.2654 68.4213 0) (effects (font (size 1.905 1.905) ) (justify right) ) ) )
