File: Schematics/TYP/pg_59.kicad_sch (KiCad schematic)
At the start: 24 parts, among them U6101 PA019, U6102 PA018, U6103 PA017, U6104 F374, U6105 F374, U6106 F374, U6107 F37, U6108 F138, U6109 PA013, U6110 F10, U6112 F374, U6113 F158, U6114 F04, U6116 F04, U6117 F04, U6118 F04, U6119 F04, U6120 PA014, U6121 PA015, U6122 PA016, U6123 F374, U6124 F374, U6125 F374

Commit message: Update symbols from library
Parts:
- removed GB53: GB, symbol r1000:GB
- removed U6101: PA019, symbol r1000:PAxxx
- removed U6102: PA018, symbol r1000:PAxxx
- removed U6103: PA017, symbol r1000:PAxxx
- removed U6104, U6105, U6106, U6112, U6123, U6124, U6125: F374, symbol r1000:F374
- removed U6107: F37, symbol r1000:F37
- removed U6108: F138, symbol r1000:F138
- removed U6109: PA013, symbol r1000:PAxxx
- removed U6110: F10, symbol r1000:F10
- removed U6113: F158, symbol r1000:F158
- removed U6114, U6116, U6117, U6118, U6119: F04, symbol r1000:F04
- removed U6120: PA014, symbol r1000:PAxxx
- removed U6121: PA015, symbol r1000:PAxxx
- removed U6122: PA016, symbol r1000:PAxxx
- added U: (no value), symbol r1000:F37
- added U (x7): (no value), symbol r1000:PAxxx
- added U (x7): (no value), symbol r1000:F374
- added U (x5): (no value), symbol r1000:F04
- added U: (no value), symbol r1000:F138
- added U: (no value), symbol r1000:F10
- added U: (no value), symbol r1000:F158
- added U: (no value), symbol r1000:GB
Connections:
- net ACS.DIAG_OFF~: now also U.15 (Q5)
- net ADR.DIAG_OFF~: now also U.16 (Q6)
- net A_L.DIAG_OFF~: now also U.5 (Q1)
- net A_O.DIAG_ON~: now also U.9 (Q3)
- net BANK_SELECT~: now also U.2 (D1), U.3 (D2), U.6 (Q2)
- net BCS.DIAG_OFF~: now also U.16 (Q6)
- net B_L.DIAG_OFF~: now also U.9 (Q3)
- net B_O.DIAG_ON: now also U.2 (Q0)
- net CLK.2X.B0: now also U.11 (CLK), U.11 (CLK), U.11 (CLK), U.11 (CLK), U.11 (CLK), U.11 (CLK)
- net CM.DIAG_ON~: now also U.2 (Q0)
- net COND.DIAG.EN~: now also U.15 (Q5)
- net CSA.DIAG.EN~: now also U.5 (Q1)
- net CSA.DIAG0: now also U.6 (Q2)
- net CSA.DIAG1: now also U.9 (Q3)
- net CSA.DIAG2: now also U.12 (Q4)
- net CTR_OVF~: now also U.1 (S)
- net C_B.DIAG_ON~: now also U.5 (Q1)
- net DIAG.CMD0: now also U.19 (A0)
- net DIAG.CMD1: now also U.18 (A1)
- net DIAG.CMD2: now also U.17 (A2)
- net DIAG.CMD3: now also U.16 (A3)
- net DIAG.CMD4: now also U.5 (A4)
- net DIAG.CMD5: now also U.4 (A5), U.4 (A5), U.4 (A5), U.4 (A5), U.4 (A5), U.4 (A5)
- net DIAG.CMD6: now also U.3 (A6), U.3 (A6), U.3 (A6), U.3 (A6), U.3 (A6), U.3 (A6)
- net DIAG.CMD7: now also U.2 (A7), U.2 (A7), U.2 (A7), U.2 (A7), U.2 (A7), U.2 (A7)
- net DIAG.HUA0: now also U.19 (A0), U.19 (A0), U.19 (A0), U.19 (A0), U.19 (A0), U.19 (A0), U.2 (Q0)
- net DIAG.HUA1: now also U.18 (A1), U.18 (A1), U.18 (A1), U.18 (A1), U.18 (A1), U.18 (A1), U.5 (Q1)
- net DIAG.HUA2: now also U.17 (A2), U.17 (A2), U.17 (A2), U.17 (A2), U.17 (A2), U.17 (A2), U.6 (Q2)
- net DIAG.HUA3: now also U.16 (A3), U.16 (A3), U.16 (A3), U.16 (A3), U.16 (A3), U.16 (A3), U.9 (Q3)
- net DIAG.HUA4: now also U.12 (Q4), U.5 (A4), U.5 (A4), U.5 (A4), U.5 (A4), U.5 (A4), U.5 (A4)
- net DIAG.NO_STOP: now also U.12 (Q4)
- net DIAG.NSTATE0: now also U.4 (A5), U.4 (Y0)
- net DIAG.NSTATE1: now also U.3 (A6), U.7 (Y1)
- net DIAG.NSTATE2: now also U.2 (A7), U.9 (Y2)
- net DIAG.NSTATE3: now also U.1 (A8), U.12 (Y3)
- net DIAG.STATE1: now also U.15 (Q5), U.6 (B1)
- net DIAG.STATE2: now also U.10 (B2), U.16 (Q6)
- net DIAG.STATE3: now also U.13 (B3), U.19 (Q7)
- net DIAG.WDR.EN: now also U.19 (Q7)
- net DIAG.WDR.S0~: now also U.19 (Q7)
- net DIAG.WDR.S1~: now also U.16 (Q6)
- net DIAG_CNTR.EN~: now also U.9 (Q3)
- net DIAG_CNTR.LD~: now also U.12 (Q4)
- net DIAG_MODE: now also U.1 (D0), U.12 (Q4)
- net DIAG_MODE.B0: now also U.2 (Q)
- net DIAG_MODE.B1: now also U.2 (Q)
- net DIAG_MODE~: now also U.1 (D0), U.1 (D0), U.1 (D0), U.2 (Q)
- net DIAG_STOP: now also U.2 (Q0)
- net DIAG_UADR.SEL: now also U.3 (Q)
- net DIAG_WRITE0: now also U.2 (Q0)
- net DIAG_WRITE1: now also U.5 (Q1)
- net FIU.DIAG_ON~: now also U.12 (Q4)
- net FORCE_SP_H1~: now also U.6 (Q2)
- net FREEZE: now also U.15 (E)
- net FREEZE.EN: now also U.15 (Q5)
- net FSM_DONE~: now also U.15 (Q5)
- net H1: now also U.1 (A8), U.1 (A8), U.1 (A8), U.1 (A8), U.1 (A8), U.1 (A8)
- net LOOP.DIAG.CT~: now also U.5 (Q1)
- net LOOP.DIAG.EN: now also U.6 (Q2)
- net LOOP.DIAG.LD~: now also U.2 (Q0)
- net NEW_CMD~: now also U.1 (D0)
- net NOVRAM.CS~: now also U.9 (Q3)
- net NOV_STORE.D~: now also U.10 (Y5_)
- net PAREG.SEL0: now also U.16 (Q6)
- net PAREG.SEL1: now also U.19 (Q7)
- net PD: now also U.1 (OE), U.1 (OE), U.1 (OE), U.1 (OE), U.1 (OE), U.1 (OE), U.1 (OE), U.14 (A3), U.15 (OE), U.15 (OE), U.15 (OE), U.15 (OE), U.15 (OE), U.15 (OE), U.15 (OE), U.2 (A0), U.4 (D1), U.5 (D2)
- net PU: now also U.11 (A2), U.5 (A1), U.6 (D0)
- net Q2~.B0: now also U.11 (CLK)
- net READ_DIAG_BUS: now also U.12 (Y3_)
- net SCAN_CONTROL~: now also U.15 (Y0_)
- net SCAN_UIR~: now also U.11 (Y4_)
- net SCAN_WDR~: now also U.13 (Y2_)
- net STATE_MSB~: now also U.2 (Q), U.3 (B0)
- net T.T_DIAG_MODE: now also U.1, U.2 (Q)
- net TADR.DIAG_ON~: now also U.12 (Q4)
- net TRIGGER_SCOPE~: now also U.7 (Y7_)
- net TYPE.DIAG_ON~: now also U.9 (Q3)
- net UIR.DIAG_OFF: now also U.16 (Q6)
- net UIR.DIAG_ON~: now also U.19 (Q7)
- net UIR.SEL0~: now also U.15 (Q5)
- net WCS.DIAG.WE~: now also U.14 (Y1_)
- new net: U.1 (D0), U.19 (Q7), U.2 (D1)
- new net: U.11 (Y3), U.8 (D3) (x7)
- new net: U.12 (Y2), U.7 (D2) (x7)
- new net: U.13 (Y1), U.4 (D1) (x7)
- new net: U.14 (Y0), U.3 (D0) (x7)
- new net: U.18 (D7), U.6 (Y7) (x7)
- new net: U.17 (D6), U.7 (Y6) (x7)
- new net: U.14 (D5), U.8 (Y5) (x7)
- new net: U.13 (D4), U.9 (Y4) (x7)
- new net: U.1 (D0), U.4 (Q)
- new net: U.1 (S2), U.19 (Q7)
- new net: U.16 (Q6), U.2 (S1)
- new net: U.15 (Q5), U.3 (S0)

Commit message: Signal dedup, megacomp WCS, DRAM, ERAM
Connections:
- net CLK.2X.B0 renamed CLK.2X
- net Q2~.B0 renamed Q2~

Commit message: TYP+VAL RF and DFSM
Parts:
- removed U (x7): (no value), symbol r1000:PAxxx
- removed U (x7): (no value), symbol r1000:F374
- added U (x7): XPAXXXL, symbol r1000:XPAXXXL
Connections:
- net ACS.DIAG_OFF~: now also U.8 (Y5)
- net ADR.DIAG_OFF~: now also U.7 (Y6)
- net A_L.DIAG_OFF~: now also U.13 (Y1)
- net A_O.DIAG_ON~: now also U.11 (Y3)
- net BANK_SELECT~: now also U.12 (Y2)
- net BCS.DIAG_OFF~: now also U.7 (Y6)
- net B_L.DIAG_OFF~: now also U.11 (Y3)
- net B_O.DIAG_ON: now also U.14 (Y0)
- net CLK.2X: now also U.15 (CLK), U.15 (CLK), U.15 (CLK), U.15 (CLK), U.15 (CLK), U.15 (CLK)
- net CM.DIAG_ON~: now also U.14 (Y0)
- net COND.DIAG.EN~: now also U.8 (Y5)
- net CSA.DIAG.EN~: now also U.13 (Y1)
- net CSA.DIAG0: now also U.12 (Y2)
- net CSA.DIAG1: now also U.11 (Y3)
- net CSA.DIAG2: now also U.9 (Y4)
- net C_B.DIAG_ON~: now also U.13 (Y1)
- net DIAG.CMD0: now also U.19 (A0)
- net DIAG.CMD1: now also U.18 (A1)
- net DIAG.CMD2: now also U.17 (A2)
- net DIAG.CMD3: now also U.16 (A3)
- net DIAG.CMD4: now also U.5 (A4)
- net DIAG.CMD5: now also U.4 (A5), U.4 (A5), U.4 (A5), U.4 (A5), U.4 (A5), U.4 (A5)
- net DIAG.CMD6: now also U.3 (A6), U.3 (A6), U.3 (A6), U.3 (A6), U.3 (A6), U.3 (A6)
- net DIAG.CMD7: now also U.2 (A7), U.2 (A7), U.2 (A7), U.2 (A7), U.2 (A7), U.2 (A7)
- net DIAG.HUA0: now also U.14 (Y0), U.19 (A0), U.19 (A0), U.19 (A0), U.19 (A0), U.19 (A0), U.19 (A0)
- net DIAG.HUA1: now also U.13 (Y1), U.18 (A1), U.18 (A1), U.18 (A1), U.18 (A1), U.18 (A1), U.18 (A1)
- net DIAG.HUA2: now also U.12 (Y2), U.17 (A2), U.17 (A2), U.17 (A2), U.17 (A2), U.17 (A2), U.17 (A2)
- net DIAG.HUA3: now also U.11 (Y3), U.16 (A3), U.16 (A3), U.16 (A3), U.16 (A3), U.16 (A3), U.16 (A3)
- net DIAG.HUA4: now also U.5 (A4), U.5 (A4), U.5 (A4), U.5 (A4), U.5 (A4), U.5 (A4), U.9 (Y4)
- net DIAG.NO_STOP: now also U.9 (Y4)
- net DIAG.NSTATE0: now also U.4 (A5)
- net DIAG.NSTATE1: now also U.3 (A6)
- net DIAG.NSTATE2: now also U.2 (A7)
- net DIAG.NSTATE3: now also U.1 (A8)
- net DIAG.STATE1: now also U.8 (Y5)
- net DIAG.STATE2: now also U.7 (Y6)
- net DIAG.STATE3: now also U.6 (Y7)
- net DIAG.WDR.EN: now also U.6 (Y7)
- net DIAG.WDR.S0~: now also U.6 (Y7)
- net DIAG.WDR.S1~: now also U.7 (Y6)
- net DIAG_CNTR.EN~: now also U.11 (Y3)
- net DIAG_CNTR.LD~: now also U.9 (Y4)
- net DIAG_MODE: now also U.9 (Y4)
- net DIAG_STOP: now also U.14 (Y0)
- net DIAG_WRITE0: now also U.14 (Y0)
- net DIAG_WRITE1: now also U.13 (Y1)
- net FIU.DIAG_ON~: now also U.9 (Y4)
- net FORCE_SP_H1~: now also U.12 (Y2)
- net FREEZE.EN: now also U.8 (Y5)
- net FSM_DONE~: now also U.8 (Y5)
- net H1: now also U.1 (A8), U.1 (A8), U.1 (A8), U.1 (A8), U.1 (A8), U.1 (A8)
- net LOOP.DIAG.CT~: now also U.13 (Y1)
- net LOOP.DIAG.EN: now also U.12 (Y2)
- net LOOP.DIAG.LD~: now also U.14 (Y0)
- net NOVRAM.CS~: now also U.11 (Y3)
- net PAREG.SEL0: now also U.7 (Y6)
- net PAREG.SEL1: now also U.6 (Y7)
- net Q2~: now also U.15 (CLK)
- net TADR.DIAG_ON~: now also U.9 (Y4)
- net TYPE.DIAG_ON~: now also U.11 (Y3)
- net UIR.DIAG_OFF: now also U.7 (Y6)
- net UIR.DIAG_ON~: now also U.6 (Y7)
- net UIR.SEL0~: now also U.8 (Y5)
- net at U.1 (D0), U.2 (D1): now also U.6 (Y7)
- net at U.1 (S2): now also U.6 (Y7)
- net at U.2 (S1): now also U.7 (Y6)
- net at U.3 (S0): now also U.8 (Y5)
