File: Schematics/TYP/pg_47.kicad_sch (KiCad schematic)
At the start: 14 parts, among them U4901 F175, U4902 F02, U4903 F02, U4904 PA012, U4905 F157, U4906 F157, U4907 F157, U4908 F381, U4909 F157, U4910 F158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

Commit message: Update symbols from library
Parts:
- removed GB11, GB8: GB, symbol r1000:GB
- removed U4901: F175, symbol r1000:F175
- removed U4902, U4903, U4911, U4912: F02, symbol r1000:F02
- removed U4904: PA012, symbol r1000:PAxxx
- removed U4905, U4906, U4907, U4909: F157, symbol r1000:F157
- removed U4908: F381, symbol r1000:F381
- removed U4910: F158, symbol r1000:F158
- added U (x4): (no value), symbol r1000:F157
- added U: (no value), symbol r1000:F381
- added U: (no value), symbol r1000:F158
- added U: (no value), symbol r1000:F175
- added U (x4): (no value), symbol r1000:F02
- added U (x2): (no value), symbol r1000:GB
- added U: (no value), symbol r1000:PAxxx
Connections:
- net A_WRITE~: now also U.14 (Y0)
- net BOT_REG0: now also U.3 (B0)
- net BOT_REG1: now also U.6 (B1)
- net BOT_REG2: now also U.10 (B2)
- net BOT_REG3: now also U.13 (B3)
- net B_WRITE~: now also U.13 (Y1)
- net C.ALU.SEL0: now also U.12 (Y2), U.7 (S0)
- net C.ALU.SEL1: now also U.11 (Y3), U.6 (S1)
- net C.ALU.SEL2: now also U.15 (E), U.9 (Y4)
- net C.ALU.SUM0: now also U.12 (F0), U.2 (A0)
- net C.ALU.SUM1: now also U.11 (F1), U.5 (A1)
- net C.ALU.SUM2: now also U.11 (A2), U.9 (F2)
- net C.ALU.SUM3: now also U.14 (A3), U.8 (F3)
- net C.CSA.SEL: now also U.1 (S), U.1 (S), U.8 (Y5)
- net C.LOOP.SEL: now also U.1 (S), U.1 (S), U.1 (S), U.7 (Y6)
- net C.ZERO.SEL: now also U.1 (D0), U.15 (E), U.6 (Y7)
- net CSA_OFFSET0: now also U.3 (B0)
- net CSA_OFFSET1: now also U.6 (B1)
- net CSA_OFFSET2: now also U.10 (B2)
- net CSA_OFFSET3: now also U.13 (B3)
- net CSA_WRITE.EN~: now also U.3 (Q)
- net C_ADDR0: now also U.4 (Y0)
- net C_ADDR1: now also U.7 (Y1)
- net C_ADDR2: now also U.9 (Y2)
- net C_ADDR3: now also U.12 (Y3)
- net C_ADDR4: now also U.3 (Q)
- net C_ADDR5: now also U.3 (Q)
- net C_ADDR6: now also U.4 (Y0)
- net C_ADDR7: now also U.7 (Y1)
- net C_ADDR8: now also U.9 (Y2)
- net C_ADDR9: now also U.12 (Y3)
- net DIAG_WRITE0: now also U.18 (A1)
- net DIAG_WRITE1: now also U.17 (A2)
- net LOOP_CNT0: now also U.3 (B0)
- net LOOP_CNT1: now also U.6 (B1)
- net LOOP_CNT2: now also U.10 (B2)
- net LOOP_CNT3: now also U.13 (B3)
- net LOOP_CNT4: now also U.3 (B0)
- net LOOP_CNT5: now also U.6 (B1)
- net LOOP_CNT6: now also U.3 (B0)
- net LOOP_CNT7: now also U.6 (B1)
- net LOOP_CNT8: now also U.10 (B2)
- net LOOP_CNT9: now also U.13 (B3)
- net PD: now also U.15 (E), U.15 (E), U.15 (E), U.15 (OE)
- net PU: now also U.1 (CLR), U.15 (CI), U.5 (S2)
- net Q3~.B0: now also U.1 (D0)
- net T.CSA_HIT~: now also U.1, U.4 (D0)
- net T.CSA_WRITE~: now also U.1, U.5 (D1)
- net TOP_REG0: now also U.2 (A0)
- net TOP_REG1: now also U.5 (A1)
- net TOP_REG2: now also U.11 (A2)
- net TOP_REG3: now also U.14 (A3)
- net UIR.C0: now also U.16 (A3)
- net UIR.C1: now also U.5 (A1), U.5 (A4)
- net UIR.C2: now also U.2 (A0), U.4 (A5)
- net UIR.C3: now also U.3 (A6), U.5 (A1)
- net UIR.C4: now also U.11 (A2), U.2 (A7)
- net UIR.C5: now also U.1 (A8), U.14 (A3)
- net UIR.FRAME0: now also U.2 (A0)
- net UIR.FRAME1: now also U.5 (A1)
- net UIR.FRAME2: now also U.11 (A2)
- net UIR.FRAME3: now also U.14 (A3)
- net UIR.FRAME4: now also U.2 (A0)
- net UIR~.SCLK.B2: now also U.9 (CLK)
- new net: U.12 (Y3), U.4 (D3)
- new net: U.16 (D0), U.4 (Y0)
- new net: U.18 (D1), U.7 (Y1)
- new net: U.2 (D2), U.9 (Y2)
- new net: U.1 (A2), U.9 (Y2)
- new net: U.17 (A0), U.4 (Y0)
- new net: U.19 (A1), U.7 (Y1)
- new net: U.12 (Y3), U.3 (A3)
- new net: U.2 (D1), U.4 (Y0)
- new net: U.1 (D0), U.2 (D1), U.7 (Y1)
- new net: U.1 (D0), U.2 (Q0)
- new net: U.2 (D1), U.7 (Q1)
- new net: U.19 (A0), U.2 (D1), U.3 (Q)

Commit message: Signal dedup, megacomp WCS, DRAM, ERAM
Connections:
- net Q3~.B0 renamed Q3~
Changed lines of the file:
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@@
     (effects (font (size 2.54 2.54)) (justify left bottom))
   )
-  (label "Q3~.B0" (at 276.86 264.16 0) (fields_autoplaced)
+  (label "Q3~" (at 276.86 264.16 0) (fields_autoplaced)
     (effects (font (size 2.54 2.54)) (justify left bottom))
   )
@@
     )
   )
-  (global_label "Q3~.B0" (shape input) (at 53.34 264.16 180) (fields_autoplaced)
+  (global_label "Q3~" (shape input) (at 53.34 264.16 180) (fields_autoplaced)
     (effects (font (size 2.54 2.54)) (justify right))
     (property "Intersheet References" "${INTERSHEET_REFS}" (id 0) (at 35.4511 264.0013 0)

Commit message: Tested until uDiag @12.2s and fru_phase2 until 10.3s
Connections:
- net UIR~.SCLK.B2 renamed UIR.SCLK~
Changed lines of the file:
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@@
     (effects (font (size 2.54 2.54)) (justify left bottom))
   )
-  (label "UIR~.SCLK.B2" (at 200.66 269.24 0) (fields_autoplaced)
+  (label "UIR.SCLK~" (at 200.66 269.24 0) (fields_autoplaced)
     (effects (font (size 2.54 2.54)) (justify left bottom))
   )
@@
     )
   )
-  (global_label "UIR~.SCLK.B2" (shape input) (at 48.26 347.98 180) (fields_autoplaced)
+  (global_label "UIR.SCLK~" (shape input) (at 48.26 347.98 180) (fields_autoplaced)
     (effects (font (size 2.54 2.54)) (justify right))
     (property "Intersheet References" "${INTERSHEET_REFS}" (id 0) (at 18.2759 347.8213 0)
