File: Schematics/FIU/pg_58.kicad_sch (KiCad schematic)
At the start: 16 parts, among them U5901 F280, U5902 F280, U5903 F280, U5904 F280, U5905 F280, U5906 F280, U5907 F280, U5908 93S48, U5909 F280, U5910 F86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

Commit message: KiCad 6
Parts:
- U5901, U5902, U5903, U5904, U5905, U5906, U5907, U5909: value F280 -> (none)
- U5908: value 93S48 -> (none)
- U5910, U5911, U5913: value F86 -> (none)
- U5912: value F521 -> (none)
- U5914, U5915: value F04 -> (none)
- U5916: value F02 -> (none)

Commit message: Recover from KiCad-6 munging
Parts:
- U5901, U5902, U5903, U5904, U5905, U5906, U5907, U5909: value (none) -> F280
- U5908: value (none) -> 93S48
- U5910, U5911, U5913: value (none) -> F86
- U5912: value (none) -> F521
- U5914, U5915: value (none) -> F04
- U5916: value (none) -> F02
