File: Schematics/FIU/FIU.kicad_sch (KiCad schematic)
At the start: 2 parts

Commit message: More megacomp'in
Parts:
- U101, U102: value (none) -> ~
Changed lines of the file:
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@@
   (wire (pts (xy 566.42 259.08) (xy 566.42 261.62) ) (stroke (width 0) (type default) ) )
   (wire (pts (xy 566.42 243.84) (xy 566.42 246.38) ) (stroke (width 0) (type default) ) )
-  (symbol (lib_id "r1000:PD") (at 566.42 261.62 0) (unit 1) (in_bom no) (on_board yes) (property "Reference" "#PWR0102" (id 0) (at 566.42 261.62 0) (effects (font (size 1.27 1.27) ) hide ) ) (property "Value" "" (id 1) (at 566.42 261.62 0) (effects (font (size 1.27 1.27) ) hide ) ) (property "Footprint" "" (id 2) (at 566.42 261.62 0) (effects (font (size 1.27 1.27) ) hide ) ) (property "Datasheet" "" (id 3) (at 566.42 261.62 0) (effects (font (size 1.27 1.27) ) hide ) ) (pin "1" ) )
-  (symbol (lib_id "r1000:PU") (at 566.42 243.84 0) (unit 1) (in_bom yes) (on_board yes) (property "Reference" "#PWR0101" (id 0) (at 566.42 243.84 0) (effects (font (size 1.27 1.27) ) hide ) ) (property "Value" "" (id 1) (at 566.42 243.84 0) (effects (font (size 1.27 1.27) ) hide ) ) (property "Footprint" "" (id 2) (at 566.42 243.84 0) (effects (font (size 1.27 1.27) ) hide ) ) (property "Datasheet" "" (id 3) (at 566.42 243.84 0) (effects (font (size 1.27 1.27) ) hide ) ) (pin "1" ) )
-  (symbol (lib_id "r1000:Pull_Down") (at 566.42 259.08 0) (unit 1) (in_bom yes) (on_board yes) (property "Reference" "U102" (id 0) (at 566.42 259.08 0) (effects (font (size 1.27 1.27) ) ) ) (property "Value" "" (id 1) (at 566.42 255.27 0) (effects (font (size 2.54 2.54) ) ) ) (property "Footprint" "" (id 2) (at 566.42 259.08 0) (effects (font (size 1.27 1.27) ) hide ) ) (property "Datasheet" "" (id 3) (at 566.42 259.08 0) (effects (font (size 1.27 1.27) ) hide ) ) (pin "1" ) )
-  (symbol (lib_id "r1000:Pull_Up") (at 566.42 246.38 0) (unit 1) (in_bom yes) (on_board yes) (property "Reference" "U101" (id 0) (at 566.42 246.38 0) (effects (font (size 1.27 1.27) ) ) ) (property "Value" "" (id 1) (at 566.42 250.19 0) (effects (font (size 2.54 2.54) ) ) ) (property "Footprint" "" (id 2) (at 566.42 246.38 0) (effects (font (size 1.27 1.27) ) hide ) ) (property "Datasheet" "" (id 3) (at 566.42 246.38 0) (effects (font (size 1.27 1.27) ) hide ) ) (pin "1" ) )
+  (symbol (lib_id "r1000:PD") (at 566.42 261.62 0) (unit 1) (in_bom no) (on_board yes) (property "Reference" "#PWR0102" (id 0) (at 566.42 261.62 0) (effects (font (size 1.27 1.27) ) hide ) ) (property "Value" "~" (id 1) (at 566.42 261.62 0) (effects (font (size 1.27 1.27) ) hide ) ) (property "Footprint" "" (id 2) (at 566.42 261.62 0) (effects (font (size 1.27 1.27) ) hide ) ) (property "Datasheet" "" (id 3) (at 566.42 261.62 0) (effects (font (size 1.27 1.27) ) hide ) ) (pin "1" ) )
+  (symbol (lib_id "r1000:PU") (at 566.42 243.84 0) (unit 1) (in_bom yes) (on_board yes) (property "Reference" "#PWR0101" (id 0) (at 566.42 243.84 0) (effects (font (size 1.27 1.27) ) hide ) ) (property "Value" "~" (id 1) (at 566.42 243.84 0) (effects (font (size 1.27 1.27) ) hide ) ) (property "Footprint" "" (id 2) (at 566.42 243.84 0) (effects (font (size 1.27 1.27) ) hide ) ) (property "Datasheet" "" (id 3) (at 566.42 243.84 0) (effects (font (size 1.27 1.27) ) hide ) ) (pin "1" ) )
+  (symbol (lib_id "r1000:Pull_Down") (at 566.42 259.08 0) (unit 1) (in_bom yes) (on_board yes) (property "Reference" "U102" (id 0) (at 566.42 259.08 0) (effects (font (size 1.27 1.27) ) ) ) (property "Value" "~" (id 1) (at 566.42 255.27 0) (effects (font (size 2.54 2.54) ) ) ) (property "Footprint" "" (id 2) (at 566.42 259.08 0) (effects (font (size 1.27 1.27) ) hide ) ) (property "Datasheet" "" (id 3) (at 566.42 259.08 0) (effects (font (size 1.27 1.27) ) hide ) ) (pin "1" ) )
+  (symbol (lib_id "r1000:Pull_Up") (at 566.42 246.38 0) (unit 1) (in_bom yes) (on_board yes) (property "Reference" "U101" (id 0) (at 566.42 246.38 0) (effects (font (size 1.27 1.27) ) ) ) (property "Value" "~" (id 1) (at 566.42 250.19 0) (effects (font (size 2.54 2.54) ) ) ) (property "Footprint" "" (id 2) (at 566.42 246.38 0) (effects (font (size 1.27 1.27) ) hide ) ) (property "Datasheet" "" (id 3) (at 566.42 246.38 0) (effects (font (size 1.27 1.27) ) hide ) ) (pin "1" ) )
   (text "Board: FIU Branch: megacomp2" (at 7.62 370.84 0) (effects (font (size 7.62 7.62) (thickness 1.27) bold ) (justify left bottom) ) )
   (sheet_instances

Commit message: Megacomp F299X8
Parts:
- U101, U102: value ~ -> (none)
Changed lines of the file:
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@@
   (wire (pts (xy 566.42 259.08) (xy 566.42 261.62) ) (stroke (width 0) (type default) ) )
   (wire (pts (xy 566.42 243.84) (xy 566.42 246.38) ) (stroke (width 0) (type default) ) )
-  (symbol (lib_id "r1000:PD") (at 566.42 261.62 0) (unit 1) (in_bom no) (on_board yes) (property "Reference" "#PWR0102" (id 0) (at 566.42 261.62 0) (effects (font (size 1.27 1.27) ) hide ) ) (property "Value" "~" (id 1) (at 566.42 261.62 0) (effects (font (size 1.27 1.27) ) hide ) ) (property "Footprint" "" (id 2) (at 566.42 261.62 0) (effects (font (size 1.27 1.27) ) hide ) ) (property "Datasheet" "" (id 3) (at 566.42 261.62 0) (effects (font (size 1.27 1.27) ) hide ) ) (pin "1" ) )
-  (symbol (lib_id "r1000:PU") (at 566.42 243.84 0) (unit 1) (in_bom yes) (on_board yes) (property "Reference" "#PWR0101" (id 0) (at 566.42 243.84 0) (effects (font (size 1.27 1.27) ) hide ) ) (property "Value" "~" (id 1) (at 566.42 243.84 0) (effects (font (size 1.27 1.27) ) hide ) ) (property "Footprint" "" (id 2) (at 566.42 243.84 0) (effects (font (size 1.27 1.27) ) hide ) ) (property "Datasheet" "" (id 3) (at 566.42 243.84 0) (effects (font (size 1.27 1.27) ) hide ) ) (pin "1" ) )
-  (symbol (lib_id "r1000:Pull_Down") (at 566.42 259.08 0) (unit 1) (in_bom yes) (on_board yes) (property "Reference" "U102" (id 0) (at 566.42 259.08 0) (effects (font (size 1.27 1.27) ) ) ) (property "Value" "~" (id 1) (at 566.42 255.27 0) (effects (font (size 2.54 2.54) ) ) ) (property "Footprint" "" (id 2) (at 566.42 259.08 0) (effects (font (size 1.27 1.27) ) hide ) ) (property "Datasheet" "" (id 3) (at 566.42 259.08 0) (effects (font (size 1.27 1.27) ) hide ) ) (pin "1" ) )
-  (symbol (lib_id "r1000:Pull_Up") (at 566.42 246.38 0) (unit 1) (in_bom yes) (on_board yes) (property "Reference" "U101" (id 0) (at 566.42 246.38 0) (effects (font (size 1.27 1.27) ) ) ) (property "Value" "~" (id 1) (at 566.42 250.19 0) (effects (font (size 2.54 2.54) ) ) ) (property "Footprint" "" (id 2) (at 566.42 246.38 0) (effects (font (size 1.27 1.27) ) hide ) ) (property "Datasheet" "" (id 3) (at 566.42 246.38 0) (effects (font (size 1.27 1.27) ) hide ) ) (pin "1" ) )
+  (symbol (lib_id "r1000:PD") (at 566.42 261.62 0) (unit 1) (in_bom no) (on_board yes) (property "Reference" "#PWR0102" (id 0) (at 566.42 261.62 0) (effects (font (size 1.27 1.27) ) hide ) ) (property "Value" "" (id 1) (at 566.42 261.62 0) (effects (font (size 1.27 1.27) ) hide ) ) (property "Footprint" "" (id 2) (at 566.42 261.62 0) (effects (font (size 1.27 1.27) ) hide ) ) (property "Datasheet" "" (id 3) (at 566.42 261.62 0) (effects (font (size 1.27 1.27) ) hide ) ) (pin "1" ) )
+  (symbol (lib_id "r1000:PU") (at 566.42 243.84 0) (unit 1) (in_bom yes) (on_board yes) (property "Reference" "#PWR0101" (id 0) (at 566.42 243.84 0) (effects (font (size 1.27 1.27) ) hide ) ) (property "Value" "" (id 1) (at 566.42 243.84 0) (effects (font (size 1.27 1.27) ) hide ) ) (property "Footprint" "" (id 2) (at 566.42 243.84 0) (effects (font (size 1.27 1.27) ) hide ) ) (property "Datasheet" "" (id 3) (at 566.42 243.84 0) (effects (font (size 1.27 1.27) ) hide ) ) (pin "1" ) )
+  (symbol (lib_id "r1000:Pull_Down") (at 566.42 259.08 0) (unit 1) (in_bom yes) (on_board yes) (property "Reference" "U102" (id 0) (at 566.42 259.08 0) (effects (font (size 1.27 1.27) ) ) ) (property "Value" "" (id 1) (at 566.42 255.27 0) (effects (font (size 2.54 2.54) ) ) ) (property "Footprint" "" (id 2) (at 566.42 259.08 0) (effects (font (size 1.27 1.27) ) hide ) ) (property "Datasheet" "" (id 3) (at 566.42 259.08 0) (effects (font (size 1.27 1.27) ) hide ) ) (pin "1" ) )
+  (symbol (lib_id "r1000:Pull_Up") (at 566.42 246.38 0) (unit 1) (in_bom yes) (on_board yes) (property "Reference" "U101" (id 0) (at 566.42 246.38 0) (effects (font (size 1.27 1.27) ) ) ) (property "Value" "" (id 1) (at 566.42 250.19 0) (effects (font (size 2.54 2.54) ) ) ) (property "Footprint" "" (id 2) (at 566.42 246.38 0) (effects (font (size 1.27 1.27) ) hide ) ) (property "Datasheet" "" (id 3) (at 566.42 246.38 0) (effects (font (size 1.27 1.27) ) hide ) ) (pin "1" ) )
   (text "Board: FIU Branch: megacomp2" (at 7.62 370.84 0) (effects (font (size 7.62 7.62) (thickness 1.27) bold ) (justify left bottom) ) )
   (sheet_instances

Commit message: Megacomp the rotator
Other:
- note added: "ROTATOR TIER 2 <6>"
- note added: "ROTATOR TIER1/VALUE HALF <6>"
- note removed: "ROTATOR TIER 2"
- note removed: "ROTATOR TIER1/VALUE HALF"
Changed lines of the file:
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@@
   (sheet (at 12.70 134.62) (size 20.32 5.08) (property "Sheet name" "Page 17" (id 0) (at 35.56 139.70 0) (effects (font (size 2.54 2.54) ) (justify left bottom) ) ) (property "Sheet file" "pg_17.kicad_sch" (id 1) (at 35.56 137.16 0) (effects (justify left bottom) hide ) ) )
   (text "ROTATOR TIER1/TYPE HALF" (at 53.34 139.70 0) (effects (font (size 2.54 2.54) ) (justify left bottom) ) )
-  (sheet (at 12.70 142.24) (size 20.32 5.08) (property "Sheet name" "Page 18" (id 0) (at 35.56 147.32 0) (effects (font (size 2.54 2.54) ) (justify left bottom) ) ) (property "Sheet file" "pg_18.kicad_sch" (id 1) (at 35.56 144.78 0) (effects (justify left bottom) hide ) ) )
-  (text "ROTATOR TIER1/VALUE HALF" (at 53.34 147.32 0) (effects (font (size 2.54 2.54) ) (justify left bottom) ) )
-  (sheet (at 12.70 149.86) (size 20.32 5.08) (property "Sheet name" "Page 19" (id 0) (at 35.56 154.94 0) (effects (font (size 2.54 2.54) ) (justify left bottom) ) ) (property "Sheet file" "pg_19.kicad_sch" (id 1) (at 35.56 152.40 0) (effects (justify left bottom) hide ) ) )
-  (text "ROTATOR TIER 2" (at 53.34 154.94 0) (effects (font (size 2.54 2.54) ) (justify left bottom) ) )
+  (sheet (at 12.70 142.24) (size 20.32 5.08) (property "Sheet name" "Page 18" (id 0) (at 35.56 147.32 0) (effects (font (size 2.54 2.54) ) (justify left bottom) ) ) (property "Sheet file" "pg_18.kicad_sch" (id 1) (at 35.56 144.78 0) (effects (justify left bottom) hide ) ) (fill (color 192 192 192 1.0) ) )
+  (text "ROTATOR TIER1/VALUE HALF <6>" (at 53.34 147.32 0) (effects (font (size 2.54 2.54) ) (justify left bottom) ) )
+  (sheet (at 12.70 149.86) (size 20.32 5.08) (property "Sheet name" "Page 19" (id 0) (at 35.56 154.94 0) (effects (font (size 2.54 2.54) ) (justify left bottom) ) ) (property "Sheet file" "pg_19.kicad_sch" (id 1) (at 35.56 152.40 0) (effects (justify left bottom) hide ) ) (fill (color 192 192 192 1.0) ) )
+  (text "ROTATOR TIER 2 <6>" (at 53.34 154.94 0) (effects (font (size 2.54 2.54) ) (justify left bottom) ) )
   (sheet (at 12.70 157.48) (size 20.32 5.08) (property "Sheet name" "Page 20" (id 0) (at 35.56 162.56 0) (effects (font (size 2.54 2.54) ) (justify left bottom) ) ) (property "Sheet file" "pg_20.kicad_sch" (id 1) (at 35.56 160.02 0) (effects (justify left bottom) hide ) ) )
   (text "ROTATOR TIER 3" (at 53.34 162.56 0) (effects (font (size 2.54 2.54) ) (justify left bottom) ) )

Commit message: Snapshot.
Parts:
- renumbered U102 to U, U101 to U
