File: Schematics/FIU/pg_55.kicad_sch (KiCad schematic)
At the start: 12 parts, among them U5601 XBUF48, U5604 F245, U5608 F86, U5609 F86, U5610 F86, U5611 F86, U5612 2149, U5613 2149, U5614 F151

Commit message: KiCad 6
Parts:
- GB222, GB272, GB273: value GB -> (none)
- U5601: value XBUF48 -> (none)
- U5604: value F245 -> (none)
- U5608, U5609, U5610, U5611: value F86 -> (none)
- U5612, U5613: value 2149 -> (none)
- U5614: value F151 -> (none)

Commit message: Recover from KiCad-6 munging
Parts:
- GB222, GB272, GB273: value (none) -> GB
- U5601: value (none) -> XBUF48
- U5604: value (none) -> F245
- U5608, U5609, U5610, U5611: value (none) -> F86
- U5612, U5613: value (none) -> 2149
- U5614: value (none) -> F151

Commit message: F245 work
Connections:
- net LINE2: now also U5604.4 (B0); no longer U5604.18 (B0)
- net LINE3: now also U5604.6 (B1); no longer U5604.17 (B1)
- net LINE4: now also U5604.8 (B2); no longer U5604.16 (B2)
- net LINE5: now also U5604.10 (B3); no longer U5604.15 (B3)
- net LINE6: now also U5604.12 (B4); no longer U5604.14 (B4)
- net LINE7: now also U5604.14 (B5); no longer U5604.13 (B5)
- net LINE8: now also U5604.16 (B6); no longer U5604.12 (B6)
- net LINE9: now also U5604.18 (B7); no longer U5604.11 (B7)
- net PD: now also U5604.2 (OE); no longer U5604.19 (OE)
- net VI.D14: now also U5604.3 (A0); no longer U5604.2 (A0)
- net VI.D15: now also U5604.5 (A1); no longer U5604.3 (A1)
- net VI.D16: now also U5604.7 (A2); no longer U5604.4 (A2)
- net VI.D17: now also U5604.9 (A3); no longer U5604.5 (A3)
- net VI.D18: now also U5604.11 (A4); no longer U5604.6 (A4)
- net VI.D19: now also U5604.13 (A5); no longer U5604.7 (A5)
- net VI.D20: now also U5604.15 (A6); no longer U5604.8 (A6)
- net VI.D21: now also U5604.17 (A7); no longer U5604.9 (A7)
Changed lines of the file:
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@@
   (label "VI.D21" (at 480.06 114.3 0) (effects (font (size 2.54 2.54) ) (justify left bottom) ) )
   (global_label "VI.D[0..63]" (shape bidirectional) (at 505.46 20.32 0) (fields_autoplaced) (effects (font (size 2.54 2.54) ) (justify left) ) (property "Intersheet References" "${INTERSHEET_REFS}" (id 0) (at 530.485 20.1613 0) (effects (font (size 1.905 1.905) ) (justify left) ) ) )
-  (symbol (lib_id "r1000:F245") (at 508 111.76 0) (unit 1) (in_bom yes) (on_board yes) (property "Reference" "U5604" (id 0) (at 510.54 106.68 0) (effects (font (size 1.27 1.27) ) ) ) (property "Value" "F245" (id 1) (at 504.19 119.38 0) (effects (font (size 2.54 2.54) ) (justify left) ) ) (property "Footprint" "" (id 2) (at 509.27 113.03 0) (effects (font (size 1.27 1.27) ) hide ) ) (property "Datasheet" "" (id 3) (at 509.27 113.03 0) (effects (font (size 1.27 1.27) ) hide ) ) (property "Location" "K30" (id 4) (at 506.73 111.76 0) (effects (font (size 2.54 2.54) ) (justify left) ) ) (property "Name" "FRDRV2" (id 5) (at 511.81 127 0) (effects (font (size 2.54 2.54) ) (justify bottom) ) ) (pin "1") (pin "11") (pin "12") (pin "13") (pin "14") (pin "15") (pin "16") (pin "17") (pin "18") (pin "19") (pin "2") (pin "3") (pin "4") (pin "5") (pin "6") (pin "7") (pin "8") (pin "9") )
+  (symbol (lib_id "r1000:F245") (at 508 111.76 0) (unit 1) (in_bom yes) (on_board yes) (property "Reference" "U5604" (id 0) (at 510.54 106.68 0) (effects (font (size 1.27 1.27) ) ) ) (property "Value" "F245" (id 1) (at 504.19 119.38 0) (effects (font (size 2.54 2.54) ) (justify left) ) ) (property "Footprint" "" (id 2) (at 509.27 113.03 0) (effects (font (size 1.27 1.27) ) hide ) ) (property "Datasheet" "" (id 3) (at 509.27 113.03 0) (effects (font (size 1.27 1.27) ) hide ) ) (property "Location" "K30" (id 4) (at 506.73 111.76 0) (effects (font (size 2.54 2.54) ) (justify left) ) ) (property "Name" "FRDRV2" (id 5) (at 511.81 127 0) (effects (font (size 2.54 2.54) ) (justify bottom) ) ) (pin "1") (pin "10") (pin "11") (pin "12") (pin "13") (pin "14") (pin "15") (pin "16") (pin "17") (pin "18") (pin "2") (pin "3") (pin "4") (pin "5") (pin "6") (pin "7") (pin "8") (pin "9") )
   (label "LINE2" (at 530.86 78.74 0) (effects (font (size 2.54 2.54) ) (justify left bottom) ) )
   (label "LINE3" (at 530.86 83.82 0) (effects (font (size 2.54 2.54) ) (justify left bottom) ) )

Commit message: Polish
Changed lines of the file:
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@@
   (bus (pts (xy 472.44 96.52) (xy 472.44 101.6) ) )
   (bus (pts (xy 53.34 27.94) (xy 53.34 35.56) ) )
-  (bus (pts (xy 53.34 297.18) (xy 53.34 304.8) ) )
   (bus (pts (xy 53.34 35.56) (xy 53.34 53.34) ) )
   (bus (pts (xy 53.34 53.34) (xy 53.34 297.18) ) )
@@
   (bus (pts (xy 60.96 271.78) (xy 60.96 276.86) ) )
   (bus (pts (xy 60.96 276.86) (xy 60.96 287.02) ) )
-  (bus (pts (xy 60.96 287.02) (xy 60.96 304.8) ) )
   (bus (pts (xy 60.96 40.64) (xy 60.96 58.42) ) )
   (bus (pts (xy 60.96 58.42) (xy 60.96 71.12) ) )
@@
   (bus (pts (xy 68.58 241.3) (xy 68.58 246.38) ) )
   (bus (pts (xy 68.58 246.38) (xy 68.58 292.1) ) )
-  (bus (pts (xy 68.58 292.1) (xy 68.58 304.8) ) )
   (bus (pts (xy 68.58 76.2) (xy 68.58 137.16) ) )
   (wire (pts (xy 101.6 299.72) (xy 55.88 299.72) ) )

Commit message: Snapshot.
Parts:
- removed GB222, GB272, GB273: GB, symbol r1000:GB
- removed U5601: XBUF48, symbol r1000:XBUF48
- removed U5604: F245, symbol r1000:F245
- removed U5608, U5609, U5610, U5611: F86, symbol r1000:F86
- removed U5612, U5613: 2149, symbol r1000:2149
- removed U5614: F151, symbol r1000:F151
- added U (x2): (no value), symbol r1000:2149
- added U (x3): (no value), symbol r1000:GB
- added U (x4): (no value), symbol r1000:F86
- added U: (no value), symbol r1000:F245
- added U: (no value), symbol r1000:F151
- added U: (no value), symbol r1000:XBUF48
Connections:
- net B_MEM32_BOARD~: now also U.1, U.7 (E~)
- net CSA_OOR: now also U.87 (I42)
- net DIAG_HASH.CS: now also U.1 (D0)
- net DIAG_HASH.WE~: now also U.10 (WE), U.10 (WE)
- net F.CSA_HIT~: now also U.89 (I43)
- net F.HIT_OFFS0: now also U.91 (I44)
- net F.HIT_OFFS1: now also U.93 (I45)
- net F.HIT_OFFS2: now also U.95 (I46)
- net F.HIT_OFFS3: now also U.97 (I47)
- net F.MCOND_TRUE~: now also U.5 (I1)
- net F.MEM_COND~: now also U.7 (I2)
- net F.MEM_EXCEPTION~: now also U.41 (I19)
- net F.PAGE_XING~: now also U.35 (I16)
- net F.REF_MACRO.BP~: now also U.39 (I18)
- net F.RESTORE_RDR~: now also U.37 (I17)
- net F.SET2: now also U.1, U.23 (I10)
- net F.SET3: now also U.1, U.25 (I11)
- net FRAME_ADR.OE~: now also U.1 (DIR), U.2 (D1), U.2 (OE)
- net IN_RANGE~: now also U.85 (I41)
- net LINE0: now also U.11 (I4), U.5 (Y)
- net LINE1: now also U.13 (I5), U.3 (Q)
- net LINE10: now also U.15 (I6), U.3 (Q), U.71 (I34)
- net LINE11: now also U.17 (I7), U.3 (Q), U.67 (I32)
- net LINE2: now also U.14 (DQ0), U.4 (B0)
- net LINE3: now also U.13 (DQ1), U.6 (B1)
- net LINE4: now also U.12 (DQ2), U.8 (B2)
- net LINE5: now also U.10 (B3), U.11 (DQ3)
- net LINE6: now also U.12 (B4), U.14 (DQ0)
- net LINE7: now also U.13 (DQ1), U.14 (B5)
- net LINE8: now also U.12 (DQ2), U.16 (B6)
- net LINE9: now also U.11 (DQ3), U.18 (B7)
- net MAR.NAME12: now also U.10 (S1)
- net MAR.NAME13: now also U.2 (D1)
- net MAR.NAME14: now also U.5 (A0)
- net MAR.NAME15: now also U.6 (A1)
- net MAR.NAME16: now also U.7 (A2)
- net MAR.NAME17: now also U.4 (A3)
- net MAR.NAME18: now also U.5 (A0)
- net MAR.NAME19: now also U.6 (A1)
- net MAR.NAME20: now also U.7 (A2)
- net MAR.NAME21: now also U.4 (A3)
- net MAR.OFFS10: now also U.2 (A5), U.3 (A4)
- net MAR.OFFS11: now also U.1 (A6), U.2 (A5)
- net MAR.OFFS12: now also U.1 (A6)
- net MAR.OFFS13: now also U.17 (A7)
- net MAR.OFFS14: now also U.16 (A8)
- net MAR.OFFS15: now also U.15 (A9)
- net MAR.OFFS16: now also U.2 (D1)
- net MAR.OFFS17: now also U.11 (S2), U.16 (A8)
- net MAR.OFFS18: now also U.15 (A9), U.2 (D1)
- net MAR.OFFS7: now also U.17 (A7)
- net MAR.OFFS8: now also U.1 (D0)
- net MAR.OFFS9: now also U.3 (A4)
- net MAR.SPACE0: now also U.1 (D0)
- net MAR.SPACE1: now also U.9 (S0)
- net MAR.SPACE2: now also U.1 (D0)
- net MRU0: now also U.27 (I12)
- net MRU1: now also U.29 (I13)
- net NAME_MATCH~: now also U.83 (I40)
- net PD: now also U.1 (D), U.1 (INV), U.13 (G), U.14 (F), U.2 (OE), U.3 (I0), U.4 (A), U.43 (I20), U.45 (I21), U.47 (I22), U.49 (I23), U.51 (I24), U.53 (I25), U.55 (I26), U.57 (I27), U.59 (I28), U.61 (I29), U.63 (I30), U.65 (I31), U.69 (I33), U.73 (I35), U.75 (I36), U.77 (I37), U.79 (I38), U.81 (I39), U.9 (I3)
- net PU: now also U.12 (H), U.15 (E), U.2 (C), U.3 (B), U.31 (I14), U.33 (I15)
- net SET0: now also U.19 (I8)
- net SET1: now also U.21 (I9)
- net VI.D10: now also U.8 (Y2)
- net VI.D11: now also U.10 (Y3)
- net VI.D12: now also U.12 (Y4)
- net VI.D13: now also U.14 (Y5)
- net VI.D14: now also U.3 (A0)
- net VI.D15: now also U.5 (A1)
- net VI.D16: now also U.7 (A2)
- net VI.D17: now also U.9 (A3)
- net VI.D18: now also U.11 (A4)
- net VI.D19: now also U.13 (A5)
- net VI.D20: now also U.15 (A6)
- net VI.D21: now also U.17 (A7)
- net VI.D22: now also U.16 (Y6)
- net VI.D23: now also U.18 (Y7)
- net VI.D24: now also U.20 (Y8)
- net VI.D25: now also U.22 (Y9)
- net VI.D26: now also U.24 (Y10)
- net VI.D27: now also U.26 (Y11)
- net VI.D28: now also U.28 (Y12)
- net VI.D29: now also U.30 (Y13)
- net VI.D30: now also U.32 (Y14)
- net VI.D31: now also U.34 (Y15)
- net VI.D32: now also U.36 (Y16)
- net VI.D33: now also U.38 (Y17)
- net VI.D34: now also U.40 (Y18)
- net VI.D35: now also U.42 (Y19)
- net VI.D36: now also U.44 (Y20)
- net VI.D37: now also U.46 (Y21)
- net VI.D38: now also U.48 (Y22)
- net VI.D39: now also U.50 (Y23)
- net VI.D40: now also U.52 (Y24)
- net VI.D41: now also U.54 (Y25)
- net VI.D42: now also U.56 (Y26)
- net VI.D43: now also U.58 (Y27)
- net VI.D44: now also U.60 (Y28)
- net VI.D45: now also U.62 (Y29)
- net VI.D46: now also U.64 (Y30)
- net VI.D47: now also U.66 (Y31)
- net VI.D48: now also U.68 (Y32)
- net VI.D49: now also U.70 (Y33)
- net VI.D50: now also U.72 (Y34)
- net VI.D51: now also U.74 (Y35)
- net VI.D52: now also U.76 (Y36)
- net VI.D53: now also U.78 (Y37)
- net VI.D54: now also U.80 (Y38)
- net VI.D55: now also U.82 (Y39)
- net VI.D56: now also U.84 (Y40)
- net VI.D57: now also U.86 (Y41)
- net VI.D58: now also U.88 (Y42)
- net VI.D59: now also U.90 (Y43)
- net VI.D60: now also U.92 (Y44)
- net VI.D61: now also U.94 (Y45)
- net VI.D62: now also U.96 (Y46)
- net VI.D63: now also U.98 (Y47)
- net VI.D8: now also U.4 (Y0)
- net VI.D9: now also U.6 (Y1)
- new net: U.3 (Q), U.8 (CS), U.8 (CS)
