File: Schematics/IOC/pg_53.kicad_sch (KiCad schematic)
At the start: 38 parts, among them U5301 F244, U5302 F02, U5303 F64, U5304 F244, U5305 F64, U5306 F244, U5307 F64, U5308 F139, U5309 F74, U5310 F74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

Commit message: KiCad 6
Parts:
- GB243, GB261, GB262, GB264, GB267, GB268: value GB -> (none)
- GF148, GF150, GF181, GF189, GF197, GF295, GF296, GF297, GF298: value GF -> (none)
- U5301, U5304, U5306, U5322: value F244 -> (none)
- U5302: value F02 -> (none)
- U5303, U5305, U5307: value F64 -> (none)
- U5308, U5311: value F139 -> (none)
- U5309, U5310: value F74 -> (none)
- U5312, U5313, U5314, U5319: value F40 -> (none)
- U5315, U5316, U5317, U5318: value F04 -> (none)
- U5320: value F37 -> (none)
- U5321: value F20 -> (none)
- U5323: value F374 -> (none)

Commit message: Recover from KiCad-6 munging
Parts:
- GB243, GB261, GB262, GB264, GB267, GB268: value (none) -> GB
- GF148, GF150, GF181, GF189, GF197, GF295, GF296, GF297, GF298: value (none) -> GF
- U5301, U5304, U5306, U5322: value (none) -> F244
- U5302: value (none) -> F02
- U5303, U5305, U5307: value (none) -> F64
- U5308, U5311: value (none) -> F139
- U5309, U5310: value (none) -> F74
- U5312, U5313, U5314, U5319: value (none) -> F40
- U5315, U5316, U5317, U5318: value (none) -> F04
- U5320: value (none) -> F37
- U5321: value (none) -> F20
- U5323: value (none) -> F374
