File: Schematics/IOC/pg_43.kicad_sch (KiCad schematic)
At the start: 9 parts, among them U4301 F299, U4302 F299, U4303 F299, U4304 F299, U4305 F240, U4306 F299, U4307 F299, U4308 F299, U4309 F299

Commit message: KiCad 6
Parts:
- U4301, U4302, U4303, U4304, U4306, U4307, U4308, U4309: value F299 -> (none)
- U4305: value F240 -> (none)

Commit message: Recover from KiCad-6 munging
Parts:
- U4301, U4302, U4303, U4304, U4306, U4307, U4308, U4309: value (none) -> F299
- U4305: value (none) -> F240

Commit message: Snapshot, much IOC polishing
Connections:
- net IOC_TV.EN~B2 is gone; now on net IOC_TV.EN~: U4301.2 (G1), U4301.3 (G2), U4303.2 (G1), U4303.3 (G2), U4306.2 (G1), U4306.3 (G2), U4308.2 (G1), U4308.3 (G2)
- net IOC_TV.EN~B0 renamed IOC_TV.EN~

Commit message: Polish
Changed lines of the file:
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@@
   (bus (pts (xy 160.02 218.44) (xy 160.02 223.52) ) )
   (bus (pts (xy 160.02 223.52) (xy 160.02 228.6) ) )
-  (bus (pts (xy 160.02 228.6) (xy 160.02 233.68) ) )
   (bus (pts (xy 160.02 66.04) (xy 160.02 71.12) ) )
   (bus (pts (xy 160.02 71.12) (xy 160.02 76.2) ) )
@@
   (bus (pts (xy 266.7 218.44) (xy 266.7 223.52) ) )
   (bus (pts (xy 266.7 223.52) (xy 266.7 228.6) ) )
-  (bus (pts (xy 266.7 228.6) (xy 266.7 233.68) ) )
   (bus (pts (xy 266.7 66.04) (xy 266.7 71.12) ) )
   (bus (pts (xy 266.7 71.12) (xy 266.7 76.2) ) )
@@
   (bus (pts (xy 373.38 218.44) (xy 373.38 223.52) ) )
   (bus (pts (xy 373.38 223.52) (xy 373.38 228.6) ) )
-  (bus (pts (xy 373.38 228.6) (xy 373.38 233.68) ) )
   (bus (pts (xy 373.38 66.04) (xy 373.38 71.12) ) )
   (bus (pts (xy 373.38 71.12) (xy 373.38 76.2) ) )

Commit message: Megacomp DUMSC
Parts:
- removed U4301, U4302, U4303, U4304, U4306, U4307, U4308, U4309: F299, symbol r1000:F299
- removed U4305: F240, symbol r1000:F240
Connections:
- no-connect marks 25 -> 0
