File: Schematics/IOC/pg_49.kicad_sch (KiCad schematic)
At the start: 18 parts, among them U4901 F04, U4902 F10, U4903 F20, U4904 F02, U4905 F04, U4906 F158, U4907 F00, U4908 F40, U4909 F37, U4910 F74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

Commit message: KiCad 6
Parts:
- GB127, GB217, GB226: value GB -> (none)
- U4901, U4905: value F04 -> (none)
- U4902: value F10 -> (none)
- U4903: value F20 -> (none)
- U4904: value F02 -> (none)
- U4906: value F158 -> (none)
- U4907: value F00 -> (none)
- U4908: value F40 -> (none)
- U4909: value F37 -> (none)
- U4910, U4914: value F74 -> (none)
- U4911, U4915: value F374 -> (none)
- U4912, U4913: value F244 -> (none)

Commit message: Recover from KiCad-6 munging
Parts:
- GB127, GB217, GB226: value (none) -> GB
- U4901, U4905: value (none) -> F04
- U4902: value (none) -> F10
- U4903: value (none) -> F20
- U4904: value (none) -> F02
- U4906: value (none) -> F158
- U4907: value (none) -> F00
- U4908: value (none) -> F40
- U4909: value (none) -> F37
- U4910, U4914: value (none) -> F74
- U4911, U4915: value (none) -> F374
- U4912, U4913: value (none) -> F244

Commit message: Snapshot, much IOC polishing
Connections:
- net MEM_TV.DRV~ renamed I.MEM_TV.EN~

Commit message: Polish IOC
Parts:
- removed U4910, U4914: F74, symbol r1000:F74
- removed U4911, U4915: F374, symbol r1000:F374
- removed U4912, U4913: F244, symbol r1000:F244
- added U5021, U5022: XREG9, symbol r1000:XREG9
Connections:
- net CHECKBIT.CLK: now also U5022.1 (CLK)
- net DIAG_CB.DRV~: now also U5021.3 (OE)
- net DRIVE_TYP_INFO~: now also U5022.3 (OE)
- net I.CB0: now also U5021.7 (Q0)
- net I.CB1: now also U5021.9 (Q1)
- net I.CB2: now also U5021.11 (Q2)
- net I.CB3: now also U5021.13 (Q3)
- net I.CB4: now also U5021.15 (Q4)
- net I.CB5: now also U5021.17 (Q5)
- net I.CB6: now also U5021.19 (Q6)
- net I.CB7: now also U5021.21 (Q7)
- net I.CB8: now also U5021.23 (Q8)
- net ICB0~: now also U5022.6 (D0)
- net ICB1~: now also U5022.8 (D1)
- net ICB2~: now also U5022.10 (D2)
- net ICB3~: now also U5022.12 (D3)
- net ICB4~: now also U5022.14 (D4)
- net ICB5~: now also U5022.16 (D5)
- net ICB6~: now also U5022.18 (D6)
- net ICB7~: now also U5022.20 (D7)
- net ICB8~: now also U5022.22 (D8)
- net ITYP.48: now also U5021.6 (D0), U5022.7 (Q0)
- net ITYP.49: now also U5021.8 (D1), U5022.9 (Q1)
- net ITYP.50: now also U5021.10 (D2), U5022.11 (Q2)
- net ITYP.51: now also U5021.12 (D3), U5022.13 (Q3)
- net ITYP.52: now also U5021.14 (D4), U5022.15 (Q4)
- net ITYP.53: now also U5021.16 (D5), U5022.17 (Q5)
- net ITYP.54: now also U5021.18 (D6), U5022.19 (Q6)
- net ITYP.55: now also U5021.20 (D7), U5022.21 (Q7)
- net ITYP.56: now also U5021.22 (D8)
- net LOAD_DIAG_CB.S~: now also U5021.1 (CLK)
- net TCB8~: now also U5022.23 (Q8)
- no-connect marks 17 -> 2

Commit message: Polish
Parts:
- removed U5021, U5022: XREG9, symbol r1000:XREG9
Connections:
- no-connect marks 2 -> 0

Commit message: Snapshot
Connections:
- net I.BUZZ_OFF~ renamed Q1~
Other:
- note added: "I.BUZZ_OFF~"
Changed lines of the file:
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@@
   (label "DRIVE_OTHER_CB~" (at 106.68 355.6 0) (effects (font (size 2.54 2.54) ) (justify left bottom) ) )
   (symbol (lib_id "r1000:F04") (at 162.56 355.6 0) (unit 1) (in_bom yes) (on_board yes) (property "Reference" "U4901" (id 0) (at 162.56 355.6 0) (effects (font (size 1.27 1.27) ) ) ) (property "Value" "F04" (id 1) (at 163.83 360.68 0) (effects (font (size 2.54 2.54) ) (justify left) ) ) (property "Footprint" "" (id 2) (at 162.56 355.6 0) (effects (font (size 1.27 1.27) ) hide ) ) (property "Datasheet" "" (id 3) (at 162.56 355.6 0) (effects (font (size 1.27 1.27) ) hide ) ) (property "Location" "D23" (id 4) (at 149.86 360.68 0) (effects (font (size 2.54 2.54) ) (justify left) ) ) (property "Name" "ECINV0A" (id 5) (at 162.56 350.52 0) (effects (font (size 2.54 2.54) ) (justify bottom) ) ) (pin "1") (pin "2") )
-  (global_label "I.BUZZ_OFF~" (shape input) (at 187.96 292.1 180) (fields_autoplaced) (effects (font (size 2.54 2.54) ) (justify right) ) (property "Intersheet References" "${INTERSHEET_REFS}" (id 0) (at 153.7426 291.9413 0) (effects (font (size 1.905 1.905) ) (justify right) ) ) )
+  (global_label "Q1~" (shape input) (at 187.96 292.1 180) (fields_autoplaced) (effects (font (size 2.54 2.54) ) (justify right) ) (property "Intersheetrefs" "${INTERSHEET_REFS}" (id 0) (at 175.3823 292.1 0) (effects (font (size 1.27 1.27) ) (justify right) ) ) )
   (global_label "I.MEM_TV.EN~" (shape input) (at 187.96 307.34 180) (fields_autoplaced) (effects (font (size 2.54 2.54) ) (justify right) ) (property "Intersheet References" "${INTERSHEET_REFS}" (id 0) (at 158.7016 307.1813 0) (effects (font (size 1.905 1.905) ) (justify right) ) ) )
   (global_label "UIR.LOAD_WDR" (shape input) (at 190.5 297.18 180) (fields_autoplaced) (effects (font (size 2.54 2.54) ) (justify right) ) (property "Intersheet References" "${INTERSHEET_REFS}" (id 0) (at 158.7016 297.0213 0) (effects (font (size 1.905 1.905) ) (justify right) ) ) )
   (global_label "DRIVE_OTHER_CB~" (shape input) (at 190.5 302.26 180) (fields_autoplaced) (effects (font (size 2.54 2.54) ) (justify right) ) (property "Intersheet References" "${INTERSHEET_REFS}" (id 0) (at 152.0492 302.1013 0) (effects (font (size 1.905 1.905) ) (justify right) ) ) )
   (global_label "DISABLE_ECC" (shape input) (at 190.5 332.74 180) (fields_autoplaced) (effects (font (size 2.54 2.54) ) (justify right) ) (property "Intersheet References" "${INTERSHEET_REFS}" (id 0) (at 161.1207 332.5813 0) (effects (font (size 1.905 1.905) ) (justify right) ) ) )
-  (label "I.BUZZ_OFF~" (at 190.5 363.22 0) (effects (font (size 2.54 2.54) ) (justify left bottom) ) )
+  (global_label "Q1~" (shape input) (at 190.5 363.22 180) (fields_autoplaced) (effects (font (size 2.54 2.54) ) (justify right) ) (property "Intersheetrefs" "${INTERSHEET_REFS}" (id 0) (at 177.9223 363.22 0) (effects (font (size 1.27 1.27) ) (justify right) ) ) )
+  (text "I.BUZZ_OFF~" (at 198.12 292.1 0) (effects (font (size 2.54 2.54) ) (justify left bottom) ) )
+  (text "I.BUZZ_OFF~" (at 200.66 363.22 0) (effects (font (size 2.54 2.54) ) (justify left bottom) ) )
   (junction (at 228.6 355.6) (diameter 0) (color 0 0 0 0) )
   (junction (at 231.14 307.34) (diameter 0) (color 0 0 0 0) )

Commit message: Snapshot
Parts:
- removed GB127, GB217, GB226: GB, symbol r1000:GB
- removed U4901, U4905: F04, symbol r1000:F04
- removed U4902: F10, symbol r1000:F10
- removed U4903: F20, symbol r1000:F20
- removed U4904: F02, symbol r1000:F02
- removed U4906: F158, symbol r1000:F158
- removed U4907: F00, symbol r1000:F00
- removed U4908: F40, symbol r1000:F40
- removed U4909: F37, symbol r1000:F37
- added U: (no value), symbol r1000:F02
- added U (x3): (no value), symbol r1000:GB
- added U: (no value), symbol r1000:F37
- added U (x2): (no value), symbol r1000:F04
- added U: (no value), symbol r1000:F20
- added U: (no value), symbol r1000:F10
- added U: (no value), symbol r1000:F40
- added U: (no value), symbol r1000:F00
- added U: (no value), symbol r1000:F158
Connections:
- net CLOCKSTOP.EN: now also U.1 (D0)
- net DIAG.DSC_S0: now also U.2 (A0)
- net DIAG.DSC_S1: now also U.5 (A1)
- net DIAG.EID_S0: now also U.11 (A2)
- net DIAG.EID_S1: now also U.14 (A3)
- net DIAG.SC_CTL~: now also U.1 (S)
- net DIAG_CB.DRV~: now also U.4 (Q)
- net DISABLE_ECC: now also U.2 (D1)
- net DRIVE_OTHER_CB~: now also U.1 (D0), U.4 (D2)
- net DUMMY.S0: now also U.4 (Y0)
- net DUMMY.S1: now also U.7 (Y1)
- net ECC_ENABLE: now also U.3 (Q), U.4 (D4)
- net EID.S0: now also U.9 (Y2)
- net EID.S1: now also U.12 (Y3)
- net I.ECC_STOP.EN: now also U.1, U.3 (Q)
- net I.MEM_TV.EN~: now also U.1 (D0), U.10 (B2), U.13 (B3), U.5 (D3)
- net I.NO_PCHECK~: now also U.1, U.5 (D5)
- net I.RESTORE_RDR~: now also U.1, U.1 (D0)
- net LOAD_DUMMY~: now also U.3 (B0), U.3 (Q), U.6 (B1)
- net NORMAL_CB.EN~: now also U.6 (Q)
- net PD: now also U.15 (E)
- net Q1~: now also U.1 (D0), U.3 (D2)
- net READ_DUMMY~: now also U.1 (D0)
- net RESTORE_RDR: now also U.2 (D1), U.2 (Q)
- net SEQ.CKSTOP~: now also U.2 (D3)
- net UIR.LOAD_WDR: now also U.2 (D1)
- new net: U.1 (D0), U.2 (D1), U.6 (Q)
- new net: U.1 (D0), U.2 (D1), U.2 (Q)

Commit message: Snapshot.
Connections:
- net UIR.LOAD_WDR: now also U.1 (D0)
- net at U.1 (D0), U.2 (D1), U.2 (Q): now also U.3 (D2)
- removed net Q1~: U.1 (D0), U.3 (D2)
Other:
- note removed: "I.BUZZ_OFF~"
Changed lines of the file:
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@@
   (junction (at 431.8 236.22) (diameter 0) (color 0 0 0 0)
   )
+  (junction (at 228.6 358.14) (diameter 0) (color 0 0 0 0)
+  )
+  (junction (at 231.14 297.18) (diameter 0) (color 0 0 0 0)
+  )
   (junction (at 508 40.64) (diameter 0) (color 0 0 0 0)
   )
@@
     (stroke (width 0) (type default))
   )
-  (wire (pts (xy 190.5 297.18) (xy 236.22 297.18))
+  (wire (pts (xy 190.5 297.18) (xy 231.14 297.18))
+    (stroke (width 0) (type default))
+  )
+  (wire (pts (xy 231.14 297.18) (xy 236.22 297.18))
     (stroke (width 0) (type default))
   )
@@
     (stroke (width 0) (type default))
   )
+  (wire (pts (xy 231.14 292.1) (xy 231.14 297.18))
+    (stroke (width 0) (type default))
+  )
   (wire (pts (xy 347.98 236.22) (xy 350.52 236.22))
     (stroke (width 0) (type default))
@@
     (stroke (width 0) (type default))
   )
+  (wire (pts (xy 236.22 292.1) (xy 231.14 292.1))
+    (stroke (width 0) (type default))
+  )
   (wire (pts (xy 347.98 251.46) (xy 350.52 251.46))
     (stroke (width 0) (type default))
@@
     (stroke (width 0) (type default))
   )
-  (wire (pts (xy 190.5 363.22) (xy 238.76 363.22))
+  (wire (pts (xy 228.6 363.22) (xy 228.6 358.14))
     (stroke (width 0) (type default))
   )
@@
     (stroke (width 0) (type default))
   )
+  (wire (pts (xy 238.76 363.22) (xy 228.6 363.22))
+    (stroke (width 0) (type default))
+  )
   (wire (pts (xy 381 38.1) (xy 416.56 38.1))
     (stroke (width 0) (type default))
@@
     (stroke (width 0) (type default))
   )
-  (wire (pts (xy 187.96 292.1) (xy 236.22 292.1))
-    (stroke (width 0) (type default))
-  )
   (wire (pts (xy 482.6 40.64) (xy 508 40.64))
     (stroke (width 0) (type default))
@@
     (stroke (width 0) (type default))
   )
-  (text "I.BUZZ_OFF~" (at 200.66 363.22 0)
-    (effects (font (size 2.54 2.54)) (justify left bottom))
-  )
-  (text "I.BUZZ_OFF~" (at 198.12 292.1 0)
-    (effects (font (size 2.54 2.54)) (justify left bottom))
-  )
   (label "DIAG.EID_S1" (at 401.32 154.94 0) (fields_autoplaced)
     (effects (font (size 2.54 2.54)) (justify left bottom))
@@
   (label "I.MEM_TV.EN~" (at 401.32 170.18 0) (fields_autoplaced)
     (effects (font (size 2.54 2.54)) (justify left bottom))
-  )
-  (global_label "Q1~" (shape input) (at 190.5 363.22 180) (fields_autoplaced)
-    (effects (font (size 2.54 2.54)) (justify right))
-    (property "Intersheetrefs" "${INTERSHEET_REFS}" (id 0) (at 177.9223 363.22 0)
-      (effects (font (size 1.27 1.27)) (justify right))
-    )
   )
   (global_label "DISABLE_ECC" (shape input) (at 190.5 332.74 180) (fields_autoplaced)
@@
     )
   )
-  (global_label "Q1~" (shape input) (at 187.96 292.1 180) (fields_autoplaced)
-    (effects (font (size 2.54 2.54)) (justify right))
-    (property "Intersheetrefs" "${INTERSHEET_REFS}" (id 0) (at 175.3823 292.1 0)
-      (effects (font (size 1.27 1.27)) (justify right))
-    )
-  )
