File: Schematics/IOC/pg_41.kicad_sch (KiCad schematic)
At the start: 80 parts, among them U4101 F244, U4102 F244, U4103 F244, U4104 F244, U4105 F244, U4106 F244, U4107 F244, U4108 F244, U4109 F244, U4110 F244, U4111 F244, U4112 F244, U4113 F244, U4114 F244, U4115 F244, U4116 F244

Commit message: KiCad 6
Parts:
- GF10, GF100, GF102, GF104, GF106, GF116, GF118, GF120, GF122, GF168, GF170, GF172, GF174, GF184, GF186, GF188, GF190, GF20, GF200, GF202, GF204, GF206, GF216, GF218, GF22, GF220, GF222, GF232, GF234, GF236, GF238, GF24, GF248, GF250, GF252, GF254, GF26, GF264, GF266, GF268, GF270, GF280, GF282, GF284, GF286, GF36, GF38, GF4, GF40, GF42, GF52, GF54, GF56, GF58, GF6, GF68, GF70, GF72, GF74, GF8, GF84, GF86, GF88, GF90: value GF -> (none)
- U4101, U4102, U4103, U4104, U4105, U4106, U4107, U4108, U4109, U4110, U4111, U4112, U4113, U4114, U4115, U4116: value F244 -> (none)

Commit message: Recover from KiCad-6 munging
Parts:
- GF10, GF100, GF102, GF104, GF106, GF116, GF118, GF120, GF122, GF168, GF170, GF172, GF174, GF184, GF186, GF188, GF190, GF20, GF200, GF202, GF204, GF206, GF216, GF218, GF22, GF220, GF222, GF232, GF234, GF236, GF238, GF24, GF248, GF250, GF252, GF254, GF26, GF264, GF266, GF268, GF270, GF280, GF282, GF284, GF286, GF36, GF38, GF4, GF40, GF42, GF52, GF54, GF56, GF58, GF6, GF68, GF70, GF72, GF74, GF8, GF84, GF86, GF88, GF90: value (none) -> GF
- U4101, U4102, U4103, U4104, U4105, U4106, U4107, U4108, U4109, U4110, U4111, U4112, U4113, U4114, U4115, U4116: value (none) -> F244

Commit message: Align to grid
Parts:
- removed GF10, GF100, GF102, GF104, GF106, GF116, GF118, GF120, GF122, GF168, GF170, GF172, GF174, GF184, GF186, GF188, GF190, GF20, GF200, GF202, GF204, GF206, GF216, GF218, GF22, GF220, GF222, GF232, GF234, GF236, GF238, GF24, GF248, GF250, GF252, GF254, GF26, GF264, GF266, GF268, GF270, GF280, GF282, GF284, GF286, GF36, GF38, GF4, GF40, GF42, GF52, GF54, GF56, GF58, GF6, GF68, GF70, GF72, GF74, GF8, GF84, GF86, GF88, GF90: GF, symbol r1000:GF
- removed U4101, U4102, U4103, U4104, U4105, U4106, U4107, U4108, U4109, U4110, U4111, U4112, U4113, U4114, U4115, U4116: F244, symbol r1000:F244
- added U (x64): (no value), symbol r1000:GF
- added U (x16): (no value), symbol r1000:F244
Connections:
- net I.VAL.0: now also U.1, U.2 (I0), U.3 (Y7)
- net I.VAL.1: now also U.1, U.4 (I1), U.5 (Y6)
- net I.VAL.10: now also U.1, U.6 (I2), U.7 (Y5)
- net I.VAL.11: now also U.1, U.8 (I3), U.9 (Y4)
- net I.VAL.12: now also U.1, U.2 (I0), U.3 (Y7)
- net I.VAL.13: now also U.1, U.4 (I1), U.5 (Y6)
- net I.VAL.14: now also U.1, U.6 (I2), U.7 (Y5)
- net I.VAL.15: now also U.1, U.8 (I3), U.9 (Y4)
- net I.VAL.16: now also U.1, U.2 (I0), U.3 (Y7)
- net I.VAL.17: now also U.1, U.4 (I1), U.5 (Y6)
- net I.VAL.18: now also U.1, U.6 (I2), U.7 (Y5)
- net I.VAL.19: now also U.1, U.8 (I3), U.9 (Y4)
- net I.VAL.2: now also U.1, U.6 (I2), U.7 (Y5)
- net I.VAL.20: now also U.1, U.2 (I0), U.3 (Y7)
- net I.VAL.21: now also U.1, U.4 (I1), U.5 (Y6)
- net I.VAL.22: now also U.1, U.6 (I2), U.7 (Y5)
- net I.VAL.23: now also U.1, U.8 (I3), U.9 (Y4)
- net I.VAL.24: now also U.1, U.2 (I0), U.3 (Y7)
- net I.VAL.25: now also U.1, U.4 (I1), U.5 (Y6)
- net I.VAL.26: now also U.1, U.6 (I2), U.7 (Y5)
- net I.VAL.27: now also U.1, U.8 (I3), U.9 (Y4)
- net I.VAL.28: now also U.1, U.2 (I0), U.3 (Y7)
- net I.VAL.29: now also U.1, U.4 (I1), U.5 (Y6)
- net I.VAL.3: now also U.1, U.8 (I3), U.9 (Y4)
- net I.VAL.30: now also U.1, U.6 (I2), U.7 (Y5)
- net I.VAL.31: now also U.1, U.8 (I3), U.9 (Y4)
- net I.VAL.32: now also U.1, U.2 (I0), U.3 (Y7)
- net I.VAL.33: now also U.1, U.4 (I1), U.5 (Y6)
- net I.VAL.34: now also U.1, U.6 (I2), U.7 (Y5)
- net I.VAL.35: now also U.1, U.8 (I3), U.9 (Y4)
- net I.VAL.36: now also U.1, U.2 (I0), U.3 (Y7)
- net I.VAL.37: now also U.1, U.4 (I1), U.5 (Y6)
- net I.VAL.38: now also U.1, U.6 (I2), U.7 (Y5)
- net I.VAL.39: now also U.1, U.8 (I3), U.9 (Y4)
- net I.VAL.4: now also U.1, U.2 (I0), U.3 (Y7)
- net I.VAL.40: now also U.1, U.2 (I0), U.3 (Y7)
- net I.VAL.41: now also U.1, U.4 (I1), U.5 (Y6)
- net I.VAL.42: now also U.1, U.6 (I2), U.7 (Y5)
- net I.VAL.43: now also U.1, U.8 (I3), U.9 (Y4)
- net I.VAL.44: now also U.1, U.2 (I0), U.3 (Y7)
- net I.VAL.45: now also U.1, U.4 (I1), U.5 (Y6)
- net I.VAL.46: now also U.1, U.6 (I2), U.7 (Y5)
- net I.VAL.47: now also U.1, U.8 (I3), U.9 (Y4)
- net I.VAL.48: now also U.1, U.2 (I0), U.3 (Y7)
- net I.VAL.49: now also U.1, U.4 (I1), U.5 (Y6)
- net I.VAL.5: now also U.1, U.4 (I1), U.5 (Y6)
- net I.VAL.50: now also U.1, U.6 (I2), U.7 (Y5)
- net I.VAL.51: now also U.1, U.8 (I3), U.9 (Y4)
- net I.VAL.52: now also U.1, U.2 (I0), U.3 (Y7)
- net I.VAL.53: now also U.1, U.4 (I1), U.5 (Y6)
- net I.VAL.54: now also U.1, U.6 (I2), U.7 (Y5)
- net I.VAL.55: now also U.1, U.8 (I3), U.9 (Y4)
- net I.VAL.56: now also U.1, U.2 (I0), U.3 (Y7)
- net I.VAL.57: now also U.1, U.4 (I1), U.5 (Y6)
- net I.VAL.58: now also U.1, U.6 (I2), U.7 (Y5)
- net I.VAL.59: now also U.1, U.8 (I3), U.9 (Y4)
- net I.VAL.6: now also U.1, U.6 (I2), U.7 (Y5)
- net I.VAL.60: now also U.1, U.2 (I0), U.3 (Y7)
- net I.VAL.61: now also U.1, U.4 (I1), U.5 (Y6)
- net I.VAL.62: now also U.1, U.6 (I2), U.7 (Y5)
- net I.VAL.63: now also U.1, U.8 (I3), U.9 (Y4)
- net I.VAL.7: now also U.1, U.8 (I3), U.9 (Y4)
- net I.VAL.8: now also U.1, U.2 (I0), U.3 (Y7)
- net I.VAL.9: now also U.1, U.4 (I1), U.5 (Y6)
- net IVAL.0: now also U.17 (I7), U.18 (Y0)
- net IVAL.1: now also U.15 (I6), U.16 (Y1)
- net IVAL.10: now also U.13 (I5), U.14 (Y2)
- net IVAL.11: now also U.11 (I4), U.12 (Y3)
- net IVAL.12: now also U.17 (I7), U.18 (Y0)
- net IVAL.13: now also U.15 (I6), U.16 (Y1)
- net IVAL.14: now also U.13 (I5), U.14 (Y2)
- net IVAL.15: now also U.11 (I4), U.12 (Y3)
- net IVAL.16: now also U.17 (I7), U.18 (Y0)
- net IVAL.17: now also U.15 (I6), U.16 (Y1)
- net IVAL.18: now also U.13 (I5), U.14 (Y2)
- net IVAL.19: now also U.11 (I4), U.12 (Y3)
- net IVAL.2: now also U.13 (I5), U.14 (Y2)
- net IVAL.20: now also U.17 (I7), U.18 (Y0)
- net IVAL.21: now also U.15 (I6), U.16 (Y1)
- net IVAL.22: now also U.13 (I5), U.14 (Y2)
- net IVAL.23: now also U.11 (I4), U.12 (Y3)
- net IVAL.24: now also U.17 (I7), U.18 (Y0)
- net IVAL.25: now also U.15 (I6), U.16 (Y1)
- net IVAL.26: now also U.13 (I5), U.14 (Y2)
- net IVAL.27: now also U.11 (I4), U.12 (Y3)
- net IVAL.28: now also U.17 (I7), U.18 (Y0)
- net IVAL.29: now also U.15 (I6), U.16 (Y1)
- net IVAL.3: now also U.11 (I4), U.12 (Y3)
- net IVAL.30: now also U.13 (I5), U.14 (Y2)
- net IVAL.31: now also U.11 (I4), U.12 (Y3)
- net IVAL.32: now also U.17 (I7), U.18 (Y0)
- net IVAL.33: now also U.15 (I6), U.16 (Y1)
- net IVAL.34: now also U.13 (I5), U.14 (Y2)
- net IVAL.35: now also U.11 (I4), U.12 (Y3)
- net IVAL.36: now also U.17 (I7), U.18 (Y0)
- net IVAL.37: now also U.15 (I6), U.16 (Y1)
- net IVAL.38: now also U.13 (I5), U.14 (Y2)
- net IVAL.39: now also U.11 (I4), U.12 (Y3)
- net IVAL.4: now also U.17 (I7), U.18 (Y0)
- net IVAL.40: now also U.17 (I7), U.18 (Y0)
- net IVAL.41: now also U.15 (I6), U.16 (Y1)
- net IVAL.42: now also U.13 (I5), U.14 (Y2)
- net IVAL.43: now also U.11 (I4), U.12 (Y3)
- net IVAL.44: now also U.17 (I7), U.18 (Y0)
- net IVAL.45: now also U.15 (I6), U.16 (Y1)
- net IVAL.46: now also U.13 (I5), U.14 (Y2)
- net IVAL.47: now also U.11 (I4), U.12 (Y3)
- net IVAL.48: now also U.17 (I7), U.18 (Y0)
- net IVAL.49: now also U.15 (I6), U.16 (Y1)
- net IVAL.5: now also U.15 (I6), U.16 (Y1)
- net IVAL.50: now also U.13 (I5), U.14 (Y2)
- net IVAL.51: now also U.11 (I4), U.12 (Y3)
- net IVAL.52: now also U.17 (I7), U.18 (Y0)
- net IVAL.53: now also U.15 (I6), U.16 (Y1)
- net IVAL.54: now also U.13 (I5), U.14 (Y2)
- net IVAL.55: now also U.11 (I4), U.12 (Y3)
- net IVAL.56: now also U.17 (I7), U.18 (Y0)
- net IVAL.57: now also U.15 (I6), U.16 (Y1)
- net IVAL.58: now also U.13 (I5), U.14 (Y2)
- net IVAL.59: now also U.11 (I4), U.12 (Y3)
- net IVAL.6: now also U.13 (I5), U.14 (Y2)
- net IVAL.60: now also U.17 (I7), U.18 (Y0)
- net IVAL.61: now also U.15 (I6), U.16 (Y1)
- net IVAL.62: now also U.13 (I5), U.14 (Y2)
- net IVAL.63: now also U.11 (I4), U.12 (Y3)
- net IVAL.7: now also U.11 (I4), U.12 (Y3)
- net IVAL.8: now also U.17 (I7), U.18 (Y0)
- net IVAL.9: now also U.15 (I6), U.16 (Y1)
- net TV.DRV~: now also U.19 (OE1), U.19 (OE1), U.19 (OE1), U.19 (OE1), U.19 (OE1), U.19 (OE1), U.19 (OE1), U.19 (OE1), U.19 (OE1), U.19 (OE1), U.19 (OE1), U.19 (OE1), U.19 (OE1), U.19 (OE1), U.19 (OE1), U.19 (OE1)
- net VAL.RCV~: now also U.1 (OE0), U.1 (OE0), U.1 (OE0), U.1 (OE0), U.1 (OE0), U.1 (OE0), U.1 (OE0), U.1 (OE0), U.1 (OE0), U.1 (OE0), U.1 (OE0), U.1 (OE0), U.1 (OE0), U.1 (OE0), U.1 (OE0), U.1 (OE0)

Commit message: Bussing planes
Parts:
- removed U (x16): (no value), symbol r1000:F244
- added U (x2): XBUF64, symbol r1000:XBUF64
Connections:
- net I.VAL.0: now also U.3 (I0), U.4 (Y0)
- net I.VAL.1: now also U.5 (I1), U.6 (Y1)
- net I.VAL.10: now also U.23 (I10), U.24 (Y10)
- net I.VAL.11: now also U.25 (I11), U.26 (Y11)
- net I.VAL.12: now also U.27 (I12), U.28 (Y12)
- net I.VAL.13: now also U.29 (I13), U.30 (Y13)
- net I.VAL.14: now also U.31 (I14), U.32 (Y14)
- net I.VAL.15: now also U.33 (I15), U.34 (Y15)
- net I.VAL.16: now also U.35 (I16), U.36 (Y16)
- net I.VAL.17: now also U.37 (I17), U.38 (Y17)
- net I.VAL.18: now also U.39 (I18), U.40 (Y18)
- net I.VAL.19: now also U.41 (I19), U.42 (Y19)
- net I.VAL.2: now also U.7 (I2), U.8 (Y2)
- net I.VAL.20: now also U.43 (I20), U.44 (Y20)
- net I.VAL.21: now also U.45 (I21), U.46 (Y21)
- net I.VAL.22: now also U.47 (I22), U.48 (Y22)
- net I.VAL.23: now also U.49 (I23), U.50 (Y23)
- net I.VAL.24: now also U.51 (I24), U.52 (Y24)
- net I.VAL.25: now also U.53 (I25), U.54 (Y25)
- net I.VAL.26: now also U.55 (I26), U.56 (Y26)
- net I.VAL.27: now also U.57 (I27), U.58 (Y27)
- net I.VAL.28: now also U.59 (I28), U.60 (Y28)
- net I.VAL.29: now also U.61 (I29), U.62 (Y29)
- net I.VAL.3: now also U.10 (Y3), U.9 (I3)
- net I.VAL.30: now also U.63 (I30), U.64 (Y30)
- net I.VAL.31: now also U.65 (I31), U.66 (Y31)
- net I.VAL.32: now also U.67 (I32), U.68 (Y32)
- net I.VAL.33: now also U.69 (I33), U.70 (Y33)
- net I.VAL.34: now also U.71 (I34), U.72 (Y34)
- net I.VAL.35: now also U.73 (I35), U.74 (Y35)
- net I.VAL.36: now also U.75 (I36), U.76 (Y36)
- net I.VAL.37: now also U.77 (I37), U.78 (Y37)
- net I.VAL.38: now also U.79 (I38), U.80 (Y38)
- net I.VAL.39: now also U.81 (I39), U.82 (Y39)
- net I.VAL.4: now also U.11 (I4), U.12 (Y4)
- net I.VAL.40: now also U.83 (I40), U.84 (Y40)
- net I.VAL.41: now also U.85 (I41), U.86 (Y41)
- net I.VAL.42: now also U.87 (I42), U.88 (Y42)
- net I.VAL.43: now also U.89 (I43), U.90 (Y43)
- net I.VAL.44: now also U.91 (I44), U.92 (Y44)
- net I.VAL.45: now also U.93 (I45), U.94 (Y45)
- net I.VAL.46: now also U.95 (I46), U.96 (Y46)
- net I.VAL.47: now also U.97 (I47), U.98 (Y47)
- net I.VAL.48: now also U.100 (Y48), U.99 (I48)
- net I.VAL.49: now also U.101 (I49), U.102 (Y49)
- net I.VAL.5: now also U.13 (I5), U.14 (Y5)
- net I.VAL.50: now also U.103 (I50), U.104 (Y50)
- net I.VAL.51: now also U.105 (I51), U.106 (Y51)
- net I.VAL.52: now also U.107 (I52), U.108 (Y52)
- net I.VAL.53: now also U.109 (I53), U.110 (Y53)
- net I.VAL.54: now also U.111 (I54), U.112 (Y54)
- net I.VAL.55: now also U.113 (I55), U.114 (Y55)
- net I.VAL.56: now also U.115 (I56), U.116 (Y56)
- net I.VAL.57: now also U.117 (I57), U.118 (Y57)
- net I.VAL.58: now also U.119 (I58), U.120 (Y58)
- net I.VAL.59: now also U.121 (I59), U.122 (Y59)
- net I.VAL.6: now also U.15 (I6), U.16 (Y6)
- net I.VAL.60: now also U.123 (I60), U.124 (Y60)
- net I.VAL.61: now also U.125 (I61), U.126 (Y61)
- net I.VAL.62: now also U.127 (I62), U.128 (Y62)
- net I.VAL.63: now also U.129 (I63), U.130 (Y63)
- net I.VAL.7: now also U.17 (I7), U.18 (Y7)
- net I.VAL.8: now also U.19 (I8), U.20 (Y8)
- net I.VAL.9: now also U.21 (I9), U.22 (Y9)
- net IVAL.0: now also U.3 (I0), U.4 (Y0)
- net IVAL.1: now also U.5 (I1), U.6 (Y1)
- net IVAL.10: now also U.23 (I10), U.24 (Y10)
- net IVAL.11: now also U.25 (I11), U.26 (Y11)
- net IVAL.12: now also U.27 (I12), U.28 (Y12)
- net IVAL.13: now also U.29 (I13), U.30 (Y13)
- net IVAL.14: now also U.31 (I14), U.32 (Y14)
- net IVAL.15: now also U.33 (I15), U.34 (Y15)
- net IVAL.16: now also U.35 (I16), U.36 (Y16)
- net IVAL.17: now also U.37 (I17), U.38 (Y17)
- net IVAL.18: now also U.39 (I18), U.40 (Y18)
- net IVAL.19: now also U.41 (I19), U.42 (Y19)
- net IVAL.2: now also U.7 (I2), U.8 (Y2)
- net IVAL.20: now also U.43 (I20), U.44 (Y20)
- net IVAL.21: now also U.45 (I21), U.46 (Y21)
- net IVAL.22: now also U.47 (I22), U.48 (Y22)
- net IVAL.23: now also U.49 (I23), U.50 (Y23)
- net IVAL.24: now also U.51 (I24), U.52 (Y24)
- net IVAL.25: now also U.53 (I25), U.54 (Y25)
- net IVAL.26: now also U.55 (I26), U.56 (Y26)
- net IVAL.27: now also U.57 (I27), U.58 (Y27)
- net IVAL.28: now also U.59 (I28), U.60 (Y28)
- net IVAL.29: now also U.61 (I29), U.62 (Y29)
- net IVAL.3: now also U.10 (Y3), U.9 (I3)
- net IVAL.30: now also U.63 (I30), U.64 (Y30)
- net IVAL.31: now also U.65 (I31), U.66 (Y31)
- net IVAL.32: now also U.67 (I32), U.68 (Y32)
- net IVAL.33: now also U.69 (I33), U.70 (Y33)
- net IVAL.34: now also U.71 (I34), U.72 (Y34)
- net IVAL.35: now also U.73 (I35), U.74 (Y35)
- net IVAL.36: now also U.75 (I36), U.76 (Y36)
- net IVAL.37: now also U.77 (I37), U.78 (Y37)
- net IVAL.38: now also U.79 (I38), U.80 (Y38)
- net IVAL.39: now also U.81 (I39), U.82 (Y39)
- net IVAL.4: now also U.11 (I4), U.12 (Y4)
- net IVAL.40: now also U.83 (I40), U.84 (Y40)
- net IVAL.41: now also U.85 (I41), U.86 (Y41)
- net IVAL.42: now also U.87 (I42), U.88 (Y42)
- net IVAL.43: now also U.89 (I43), U.90 (Y43)
- net IVAL.44: now also U.91 (I44), U.92 (Y44)
- net IVAL.45: now also U.93 (I45), U.94 (Y45)
- net IVAL.46: now also U.95 (I46), U.96 (Y46)
- net IVAL.47: now also U.97 (I47), U.98 (Y47)
- net IVAL.48: now also U.100 (Y48), U.99 (I48)
- net IVAL.49: now also U.101 (I49), U.102 (Y49)
- net IVAL.5: now also U.13 (I5), U.14 (Y5)
- net IVAL.50: now also U.103 (I50), U.104 (Y50)
- net IVAL.51: now also U.105 (I51), U.106 (Y51)
- net IVAL.52: now also U.107 (I52), U.108 (Y52)
- net IVAL.53: now also U.109 (I53), U.110 (Y53)
- net IVAL.54: now also U.111 (I54), U.112 (Y54)
- net IVAL.55: now also U.113 (I55), U.114 (Y55)
- net IVAL.56: now also U.115 (I56), U.116 (Y56)
- net IVAL.57: now also U.117 (I57), U.118 (Y57)
- net IVAL.58: now also U.119 (I58), U.120 (Y58)
- net IVAL.59: now also U.121 (I59), U.122 (Y59)
- net IVAL.6: now also U.15 (I6), U.16 (Y6)
- net IVAL.60: now also U.123 (I60), U.124 (Y60)
- net IVAL.61: now also U.125 (I61), U.126 (Y61)
- net IVAL.62: now also U.127 (I62), U.128 (Y62)
- net IVAL.63: now also U.129 (I63), U.130 (Y63)
- net IVAL.7: now also U.17 (I7), U.18 (Y7)
- net IVAL.8: now also U.19 (I8), U.20 (Y8)
- net IVAL.9: now also U.21 (I9), U.22 (Y9)
- net TV.DRV~: now also U.2 (OE)
- net VAL.RCV~: now also U.2 (OE)
- no-connect marks 0 -> 2
