File: Schematics/IOC/pg_28.kicad_sch (KiCad schematic)
At the start: 4 parts, among them U2919 F280, U2920 F280, U2921 F280, U2922 F280

Commit message: KiCad 6
Parts:
- U2919, U2920, U2921, U2922: value F280 -> (none)
Changed lines of the file:
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@@
   (global_label "RAM.DI30" (shape input) (at 114.3 317.5 180) (fields_autoplaced) (effects (font (size 2.54 2.54) ) (justify right) ) (property "Intersheet References" "${INTERSHEET_REFS}" (id 0) (at 91.6759 317.3413 0) (effects (font (size 2.54 2.54) ) (justify right) ) ) )
   (global_label "RAM.DI31" (shape input) (at 114.3 322.58 180) (fields_autoplaced) (effects (font (size 2.54 2.54) ) (justify right) ) (property "Intersheet References" "${INTERSHEET_REFS}" (id 0) (at 91.6759 322.4213 0) (effects (font (size 2.54 2.54) ) (justify right) ) ) )
-  (symbol (lib_id "r1000:F280") (at 142.24 99.06 0) (unit 1) (in_bom yes) (on_board yes) (property "Reference" "U2920" (id 0) (at 144.78 93.98 0) ) (property "Value" "F280" (id 1) (at 135.89 104.14 0) (effects (font (size 2.54 2.54) ) (justify left) ) ) (property "Footprint" "" (id 2) (at 143.51 100.33 0) (effects (font (size 1.27 1.27) ) hide ) ) (property "Datasheet" "" (id 3) (at 143.51 100.33 0) (effects (font (size 1.27 1.27) ) hide ) ) (property "Location" "I30" (id 4) (at 140.97 99.06 0) (effects (font (size 2.54 2.54) ) (justify left) ) ) (property "Name" "MPGEN0" (id 5) (at 143.51 111.76 0) (effects (font (size 2.54 2.54) ) (justify bottom) ) ) (pin "1") (pin "10") (pin "11") (pin "12") (pin "13") (pin "2") (pin "4") (pin "5") (pin "6") (pin "8") (pin "9") )
-  (symbol (lib_id "r1000:F280") (at 142.24 175.26 0) (unit 1) (in_bom yes) (on_board yes) (property "Reference" "U2922" (id 0) (at 144.78 170.18 0) ) (property "Value" "F280" (id 1) (at 135.89 180.34 0) (effects (font (size 2.54 2.54) ) (justify left) ) ) (property "Footprint" "" (id 2) (at 143.51 176.53 0) (effects (font (size 1.27 1.27) ) hide ) ) (property "Datasheet" "" (id 3) (at 143.51 176.53 0) (effects (font (size 1.27 1.27) ) hide ) ) (property "Location" "I32" (id 4) (at 140.97 175.26 0) (effects (font (size 2.54 2.54) ) (justify left) ) ) (property "Name" "MPGEN1" (id 5) (at 143.51 187.96 0) (effects (font (size 2.54 2.54) ) (justify bottom) ) ) (pin "1") (pin "10") (pin "11") (pin "12") (pin "13") (pin "2") (pin "4") (pin "5") (pin "6") (pin "8") (pin "9") )
-  (symbol (lib_id "r1000:F280") (at 142.24 251.46 0) (unit 1) (in_bom yes) (on_board yes) (property "Reference" "U2921" (id 0) (at 144.78 246.38 0) ) (property "Value" "F280" (id 1) (at 135.89 256.54 0) (effects (font (size 2.54 2.54) ) (justify left) ) ) (property "Footprint" "" (id 2) (at 143.51 252.73 0) (effects (font (size 1.27 1.27) ) hide ) ) (property "Datasheet" "" (id 3) (at 143.51 252.73 0) (effects (font (size 1.27 1.27) ) hide ) ) (property "Location" "I17" (id 4) (at 140.97 251.46 0) (effects (font (size 2.54 2.54) ) (justify left) ) ) (property "Name" "MPGEN2" (id 5) (at 143.51 264.16 0) (effects (font (size 2.54 2.54) ) (justify bottom) ) ) (pin "1") (pin "10") (pin "11") (pin "12") (pin "13") (pin "2") (pin "4") (pin "5") (pin "6") (pin "8") (pin "9") )
-  (symbol (lib_id "r1000:F280") (at 142.24 327.66 0) (unit 1) (in_bom yes) (on_board yes) (property "Reference" "U2919" (id 0) (at 144.78 322.58 0) ) (property "Value" "F280" (id 1) (at 135.89 332.74 0) (effects (font (size 2.54 2.54) ) (justify left) ) ) (property "Footprint" "" (id 2) (at 143.51 328.93 0) (effects (font (size 1.27 1.27) ) hide ) ) (property "Datasheet" "" (id 3) (at 143.51 328.93 0) (effects (font (size 1.27 1.27) ) hide ) ) (property "Location" "I15" (id 4) (at 140.97 327.66 0) (effects (font (size 2.54 2.54) ) (justify left) ) ) (property "Name" "MPGEN3" (id 5) (at 143.51 340.36 0) (effects (font (size 2.54 2.54) ) (justify bottom) ) ) (pin "1") (pin "10") (pin "11") (pin "12") (pin "13") (pin "2") (pin "4") (pin "5") (pin "6") (pin "8") (pin "9") )
+  (symbol (lib_id "r1000:F280") (at 142.24 99.06 0) (unit 1) (in_bom yes) (on_board yes) (property "Reference" "U2920" (id 0) (at 144.78 93.98 0) ) (property "Value" "" (id 1) (at 135.89 104.14 0) (effects (font (size 2.54 2.54) ) (justify left) ) ) (property "Footprint" "" (id 2) (at 143.51 100.33 0) (effects (font (size 1.27 1.27) ) hide ) ) (property "Datasheet" "" (id 3) (at 143.51 100.33 0) (effects (font (size 1.27 1.27) ) hide ) ) (property "Location" "I30" (id 4) (at 140.97 99.06 0) (effects (font (size 2.54 2.54) ) (justify left) ) ) (property "Name" "MPGEN0" (id 5) (at 143.51 111.76 0) (effects (font (size 2.54 2.54) ) (justify bottom) ) ) (pin "1") (pin "10") (pin "11") (pin "12") (pin "13") (pin "2") (pin "4") (pin "5") (pin "6") (pin "8") (pin "9") )
+  (symbol (lib_id "r1000:F280") (at 142.24 175.26 0) (unit 1) (in_bom yes) (on_board yes) (property "Reference" "U2922" (id 0) (at 144.78 170.18 0) ) (property "Value" "" (id 1) (at 135.89 180.34 0) (effects (font (size 2.54 2.54) ) (justify left) ) ) (property "Footprint" "" (id 2) (at 143.51 176.53 0) (effects (font (size 1.27 1.27) ) hide ) ) (property "Datasheet" "" (id 3) (at 143.51 176.53 0) (effects (font (size 1.27 1.27) ) hide ) ) (property "Location" "I32" (id 4) (at 140.97 175.26 0) (effects (font (size 2.54 2.54) ) (justify left) ) ) (property "Name" "MPGEN1" (id 5) (at 143.51 187.96 0) (effects (font (size 2.54 2.54) ) (justify bottom) ) ) (pin "1") (pin "10") (pin "11") (pin "12") (pin "13") (pin "2") (pin "4") (pin "5") (pin "6") (pin "8") (pin "9") )
+  (symbol (lib_id "r1000:F280") (at 142.24 251.46 0) (unit 1) (in_bom yes) (on_board yes) (property "Reference" "U2921" (id 0) (at 144.78 246.38 0) ) (property "Value" "" (id 1) (at 135.89 256.54 0) (effects (font (size 2.54 2.54) ) (justify left) ) ) (property "Footprint" "" (id 2) (at 143.51 252.73 0) (effects (font (size 1.27 1.27) ) hide ) ) (property "Datasheet" "" (id 3) (at 143.51 252.73 0) (effects (font (size 1.27 1.27) ) hide ) ) (property "Location" "I17" (id 4) (at 140.97 251.46 0) (effects (font (size 2.54 2.54) ) (justify left) ) ) (property "Name" "MPGEN2" (id 5) (at 143.51 264.16 0) (effects (font (size 2.54 2.54) ) (justify bottom) ) ) (pin "1") (pin "10") (pin "11") (pin "12") (pin "13") (pin "2") (pin "4") (pin "5") (pin "6") (pin "8") (pin "9") )
+  (symbol (lib_id "r1000:F280") (at 142.24 327.66 0) (unit 1) (in_bom yes) (on_board yes) (property "Reference" "U2919" (id 0) (at 144.78 322.58 0) ) (property "Value" "" (id 1) (at 135.89 332.74 0) (effects (font (size 2.54 2.54) ) (justify left) ) ) (property "Footprint" "" (id 2) (at 143.51 328.93 0) (effects (font (size 1.27 1.27) ) hide ) ) (property "Datasheet" "" (id 3) (at 143.51 328.93 0) (effects (font (size 1.27 1.27) ) hide ) ) (property "Location" "I15" (id 4) (at 140.97 327.66 0) (effects (font (size 2.54 2.54) ) (justify left) ) ) (property "Name" "MPGEN3" (id 5) (at 143.51 340.36 0) (effects (font (size 2.54 2.54) ) (justify bottom) ) ) (pin "1") (pin "10") (pin "11") (pin "12") (pin "13") (pin "2") (pin "4") (pin "5") (pin "6") (pin "8") (pin "9") )
   (no_connect (at 157.48 68.58) )
   (no_connect (at 157.48 144.78) )

Commit message: Recover from KiCad-6 munging
Parts:
- U2919, U2920, U2921, U2922: value (none) -> F280
Changed lines of the file:
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@@
 (kicad_sch
-  (version 20211123)
+  (version 20220126)
   (generator eeschema)
   (paper "User" 584.2 378.46)
@@
   (global_label "RAM.DI30" (shape input) (at 114.3 317.5 180) (fields_autoplaced) (effects (font (size 2.54 2.54) ) (justify right) ) (property "Intersheet References" "${INTERSHEET_REFS}" (id 0) (at 91.6759 317.3413 0) (effects (font (size 2.54 2.54) ) (justify right) ) ) )
   (global_label "RAM.DI31" (shape input) (at 114.3 322.58 180) (fields_autoplaced) (effects (font (size 2.54 2.54) ) (justify right) ) (property "Intersheet References" "${INTERSHEET_REFS}" (id 0) (at 91.6759 322.4213 0) (effects (font (size 2.54 2.54) ) (justify right) ) ) )
-  (symbol (lib_id "r1000:F280") (at 142.24 99.06 0) (unit 1) (in_bom yes) (on_board yes) (property "Reference" "U2920" (id 0) (at 144.78 93.98 0) ) (property "Value" "" (id 1) (at 135.89 104.14 0) (effects (font (size 2.54 2.54) ) (justify left) ) ) (property "Footprint" "" (id 2) (at 143.51 100.33 0) (effects (font (size 1.27 1.27) ) hide ) ) (property "Datasheet" "" (id 3) (at 143.51 100.33 0) (effects (font (size 1.27 1.27) ) hide ) ) (property "Location" "I30" (id 4) (at 140.97 99.06 0) (effects (font (size 2.54 2.54) ) (justify left) ) ) (property "Name" "MPGEN0" (id 5) (at 143.51 111.76 0) (effects (font (size 2.54 2.54) ) (justify bottom) ) ) (pin "1") (pin "10") (pin "11") (pin "12") (pin "13") (pin "2") (pin "4") (pin "5") (pin "6") (pin "8") (pin "9") )
-  (symbol (lib_id "r1000:F280") (at 142.24 175.26 0) (unit 1) (in_bom yes) (on_board yes) (property "Reference" "U2922" (id 0) (at 144.78 170.18 0) ) (property "Value" "" (id 1) (at 135.89 180.34 0) (effects (font (size 2.54 2.54) ) (justify left) ) ) (property "Footprint" "" (id 2) (at 143.51 176.53 0) (effects (font (size 1.27 1.27) ) hide ) ) (property "Datasheet" "" (id 3) (at 143.51 176.53 0) (effects (font (size 1.27 1.27) ) hide ) ) (property "Location" "I32" (id 4) (at 140.97 175.26 0) (effects (font (size 2.54 2.54) ) (justify left) ) ) (property "Name" "MPGEN1" (id 5) (at 143.51 187.96 0) (effects (font (size 2.54 2.54) ) (justify bottom) ) ) (pin "1") (pin "10") (pin "11") (pin "12") (pin "13") (pin "2") (pin "4") (pin "5") (pin "6") (pin "8") (pin "9") )
-  (symbol (lib_id "r1000:F280") (at 142.24 251.46 0) (unit 1) (in_bom yes) (on_board yes) (property "Reference" "U2921" (id 0) (at 144.78 246.38 0) ) (property "Value" "" (id 1) (at 135.89 256.54 0) (effects (font (size 2.54 2.54) ) (justify left) ) ) (property "Footprint" "" (id 2) (at 143.51 252.73 0) (effects (font (size 1.27 1.27) ) hide ) ) (property "Datasheet" "" (id 3) (at 143.51 252.73 0) (effects (font (size 1.27 1.27) ) hide ) ) (property "Location" "I17" (id 4) (at 140.97 251.46 0) (effects (font (size 2.54 2.54) ) (justify left) ) ) (property "Name" "MPGEN2" (id 5) (at 143.51 264.16 0) (effects (font (size 2.54 2.54) ) (justify bottom) ) ) (pin "1") (pin "10") (pin "11") (pin "12") (pin "13") (pin "2") (pin "4") (pin "5") (pin "6") (pin "8") (pin "9") )
-  (symbol (lib_id "r1000:F280") (at 142.24 327.66 0) (unit 1) (in_bom yes) (on_board yes) (property "Reference" "U2919" (id 0) (at 144.78 322.58 0) ) (property "Value" "" (id 1) (at 135.89 332.74 0) (effects (font (size 2.54 2.54) ) (justify left) ) ) (property "Footprint" "" (id 2) (at 143.51 328.93 0) (effects (font (size 1.27 1.27) ) hide ) ) (property "Datasheet" "" (id 3) (at 143.51 328.93 0) (effects (font (size 1.27 1.27) ) hide ) ) (property "Location" "I15" (id 4) (at 140.97 327.66 0) (effects (font (size 2.54 2.54) ) (justify left) ) ) (property "Name" "MPGEN3" (id 5) (at 143.51 340.36 0) (effects (font (size 2.54 2.54) ) (justify bottom) ) ) (pin "1") (pin "10") (pin "11") (pin "12") (pin "13") (pin "2") (pin "4") (pin "5") (pin "6") (pin "8") (pin "9") )
+  (symbol (lib_id "r1000:F280") (at 142.24 99.06 0) (unit 1) (in_bom yes) (on_board yes) (property "Reference" "U2920" (id 0) (at 144.78 93.98 0) (effects (font (size 1.27 1.27) ) ) ) (property "Value" "F280" (id 1) (at 135.89 104.14 0) (effects (font (size 2.54 2.54) ) (justify left) ) ) (property "Footprint" "" (id 2) (at 143.51 100.33 0) (effects (font (size 1.27 1.27) ) hide ) ) (property "Datasheet" "" (id 3) (at 143.51 100.33 0) (effects (font (size 1.27 1.27) ) hide ) ) (property "Location" "I30" (id 4) (at 140.97 99.06 0) (effects (font (size 2.54 2.54) ) (justify left) ) ) (property "Name" "MPGEN0" (id 5) (at 143.51 111.76 0) (effects (font (size 2.54 2.54) ) (justify bottom) ) ) (pin "1") (pin "10") (pin "11") (pin "12") (pin "13") (pin "2") (pin "4") (pin "5") (pin "6") (pin "8") (pin "9") )
+  (symbol (lib_id "r1000:F280") (at 142.24 175.26 0) (unit 1) (in_bom yes) (on_board yes) (property "Reference" "U2922" (id 0) (at 144.78 170.18 0) (effects (font (size 1.27 1.27) ) ) ) (property "Value" "F280" (id 1) (at 135.89 180.34 0) (effects (font (size 2.54 2.54) ) (justify left) ) ) (property "Footprint" "" (id 2) (at 143.51 176.53 0) (effects (font (size 1.27 1.27) ) hide ) ) (property "Datasheet" "" (id 3) (at 143.51 176.53 0) (effects (font (size 1.27 1.27) ) hide ) ) (property "Location" "I32" (id 4) (at 140.97 175.26 0) (effects (font (size 2.54 2.54) ) (justify left) ) ) (property "Name" "MPGEN1" (id 5) (at 143.51 187.96 0) (effects (font (size 2.54 2.54) ) (justify bottom) ) ) (pin "1") (pin "10") (pin "11") (pin "12") (pin "13") (pin "2") (pin "4") (pin "5") (pin "6") (pin "8") (pin "9") )
+  (symbol (lib_id "r1000:F280") (at 142.24 251.46 0) (unit 1) (in_bom yes) (on_board yes) (property "Reference" "U2921" (id 0) (at 144.78 246.38 0) (effects (font (size 1.27 1.27) ) ) ) (property "Value" "F280" (id 1) (at 135.89 256.54 0) (effects (font (size 2.54 2.54) ) (justify left) ) ) (property "Footprint" "" (id 2) (at 143.51 252.73 0) (effects (font (size 1.27 1.27) ) hide ) ) (property "Datasheet" "" (id 3) (at 143.51 252.73 0) (effects (font (size 1.27 1.27) ) hide ) ) (property "Location" "I17" (id 4) (at 140.97 251.46 0) (effects (font (size 2.54 2.54) ) (justify left) ) ) (property "Name" "MPGEN2" (id 5) (at 143.51 264.16 0) (effects (font (size 2.54 2.54) ) (justify bottom) ) ) (pin "1") (pin "10") (pin "11") (pin "12") (pin "13") (pin "2") (pin "4") (pin "5") (pin "6") (pin "8") (pin "9") )
+  (symbol (lib_id "r1000:F280") (at 142.24 327.66 0) (unit 1) (in_bom yes) (on_board yes) (property "Reference" "U2919" (id 0) (at 144.78 322.58 0) (effects (font (size 1.27 1.27) ) ) ) (property "Value" "F280" (id 1) (at 135.89 332.74 0) (effects (font (size 2.54 2.54) ) (justify left) ) ) (property "Footprint" "" (id 2) (at 143.51 328.93 0) (effects (font (size 1.27 1.27) ) hide ) ) (property "Datasheet" "" (id 3) (at 143.51 328.93 0) (effects (font (size 1.27 1.27) ) hide ) ) (property "Location" "I15" (id 4) (at 140.97 327.66 0) (effects (font (size 2.54 2.54) ) (justify left) ) ) (property "Name" "MPGEN3" (id 5) (at 143.51 340.36 0) (effects (font (size 2.54 2.54) ) (justify bottom) ) ) (pin "1") (pin "10") (pin "11") (pin "12") (pin "13") (pin "2") (pin "4") (pin "5") (pin "6") (pin "8") (pin "9") )
   (no_connect (at 157.48 68.58) )
   (no_connect (at 157.48 144.78) )

Commit message: Align to grid
Parts:
- removed U2919, U2920, U2921, U2922: F280, symbol r1000:F280
- added U (x4): (no value), symbol r1000:F280
Connections:
- net GOOD_PARITY: now also U.4 (I8), U.4 (I8), U.4 (I8), U.4 (I8)
- net RAM.DI0: now also U.8 (I0)
- net RAM.DI1: now also U.9 (I1)
- net RAM.DI10: now also U.10 (I2)
- net RAM.DI11: now also U.11 (I3)
- net RAM.DI12: now also U.12 (I4)
- net RAM.DI13: now also U.13 (I5)
- net RAM.DI14: now also U.1 (I6)
- net RAM.DI15: now also U.2 (I7)
- net RAM.DI16: now also U.8 (I0)
- net RAM.DI17: now also U.9 (I1)
- net RAM.DI18: now also U.10 (I2)
- net RAM.DI19: now also U.11 (I3)
- net RAM.DI2: now also U.10 (I2)
- net RAM.DI20: now also U.12 (I4)
- net RAM.DI21: now also U.13 (I5)
- net RAM.DI22: now also U.1 (I6)
- net RAM.DI23: now also U.2 (I7)
- net RAM.DI24: now also U.8 (I0)
- net RAM.DI25: now also U.9 (I1)
- net RAM.DI26: now also U.10 (I2)
- net RAM.DI27: now also U.11 (I3)
- net RAM.DI28: now also U.12 (I4)
- net RAM.DI29: now also U.13 (I5)
- net RAM.DI3: now also U.11 (I3)
- net RAM.DI30: now also U.1 (I6)
- net RAM.DI31: now also U.2 (I7)
- net RAM.DI4: now also U.12 (I4)
- net RAM.DI5: now also U.13 (I5)
- net RAM.DI6: now also U.1 (I6)
- net RAM.DI7: now also U.2 (I7)
- net RAM.DI8: now also U.8 (I0)
- net RAM.DI9: now also U.9 (I1)
- net RAM.DIP0: now also U.6 (POD)
- net RAM.DIP1: now also U.6 (POD)
- net RAM.DIP2: now also U.6 (POD)
- net RAM.DIP3: now also U.6 (POD)

Commit message: Polish
Parts:
- U2919, U2920, U2921, U2922: renamed from U; value (none) -> F280
