File: Schematics/IOC/pg_04.kicad_sch (KiCad schematic)
At the start: 2 parts, among them U501 F257, U502 F257

Commit message: KiCad 6
Parts:
- U501, U502: value F257 -> (none)
Changed lines of the file:
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@@
   (junction (at 347.98 162.56) (diameter 0) (color 0 0 0 0) )
   (junction (at 353.06 154.94) (diameter 0) (color 0 0 0 0) )
-  (symbol (lib_id "r1000:F257") (at 370.84 218.44 0) (unit 1) (in_bom yes) (on_board yes) (property "Reference" "U501" (id 0) (at 373.38 213.36 0) ) (property "Value" "F257" (id 1) (at 367.03 223.52 0) (effects (font (size 2.54 2.54) ) (justify left) ) ) (property "Footprint" "" (id 2) (at 372.11 219.71 0) (effects (font (size 1.27 1.27) ) hide ) ) (property "Datasheet" "" (id 3) (at 372.11 219.71 0) (effects (font (size 1.27 1.27) ) hide ) ) (property "Location" "L13" (id 4) (at 369.57 218.44 0) (effects (font (size 2.54 2.54) ) (justify left) ) ) (property "Name" "ATUMUX0" (id 5) (at 372.11 231.14 0) (effects (font (size 2.54 2.54) ) (justify bottom) ) ) (pin "1") (pin "10") (pin "11") (pin "12") (pin "13") (pin "14") (pin "15") (pin "2") (pin "3") (pin "4") (pin "5") (pin "6") (pin "7") (pin "9") )
-  (symbol (lib_id "r1000:F257") (at 370.84 327.66 0) (unit 1) (in_bom yes) (on_board yes) (property "Reference" "U502" (id 0) (at 373.38 322.58 0) ) (property "Value" "F257" (id 1) (at 367.03 332.74 0) (effects (font (size 2.54 2.54) ) (justify left) ) ) (property "Footprint" "" (id 2) (at 372.11 328.93 0) (effects (font (size 1.27 1.27) ) hide ) ) (property "Datasheet" "" (id 3) (at 372.11 328.93 0) (effects (font (size 1.27 1.27) ) hide ) ) (property "Location" "K13" (id 4) (at 369.57 327.66 0) (effects (font (size 2.54 2.54) ) (justify left) ) ) (property "Name" "ATUMUX1" (id 5) (at 372.11 340.36 0) (effects (font (size 2.54 2.54) ) (justify bottom) ) ) (pin "1") (pin "10") (pin "11") (pin "12") (pin "13") (pin "14") (pin "15") (pin "2") (pin "3") (pin "4") (pin "5") (pin "6") (pin "7") (pin "9") )
+  (symbol (lib_id "r1000:F257") (at 370.84 218.44 0) (unit 1) (in_bom yes) (on_board yes) (property "Reference" "U501" (id 0) (at 373.38 213.36 0) ) (property "Value" "" (id 1) (at 367.03 223.52 0) (effects (font (size 2.54 2.54) ) (justify left) ) ) (property "Footprint" "" (id 2) (at 372.11 219.71 0) (effects (font (size 1.27 1.27) ) hide ) ) (property "Datasheet" "" (id 3) (at 372.11 219.71 0) (effects (font (size 1.27 1.27) ) hide ) ) (property "Location" "L13" (id 4) (at 369.57 218.44 0) (effects (font (size 2.54 2.54) ) (justify left) ) ) (property "Name" "ATUMUX0" (id 5) (at 372.11 231.14 0) (effects (font (size 2.54 2.54) ) (justify bottom) ) ) (pin "1") (pin "10") (pin "11") (pin "12") (pin "13") (pin "14") (pin "15") (pin "2") (pin "3") (pin "4") (pin "5") (pin "6") (pin "7") (pin "9") )
+  (symbol (lib_id "r1000:F257") (at 370.84 327.66 0) (unit 1) (in_bom yes) (on_board yes) (property "Reference" "U502" (id 0) (at 373.38 322.58 0) ) (property "Value" "" (id 1) (at 367.03 332.74 0) (effects (font (size 2.54 2.54) ) (justify left) ) ) (property "Footprint" "" (id 2) (at 372.11 328.93 0) (effects (font (size 1.27 1.27) ) hide ) ) (property "Datasheet" "" (id 3) (at 372.11 328.93 0) (effects (font (size 1.27 1.27) ) hide ) ) (property "Location" "K13" (id 4) (at 369.57 327.66 0) (effects (font (size 2.54 2.54) ) (justify left) ) ) (property "Name" "ATUMUX1" (id 5) (at 372.11 340.36 0) (effects (font (size 2.54 2.54) ) (justify bottom) ) ) (pin "1") (pin "10") (pin "11") (pin "12") (pin "13") (pin "14") (pin "15") (pin "2") (pin "3") (pin "4") (pin "5") (pin "6") (pin "7") (pin "9") )
   (label "RAM.A14" (at 396.24 185.42 0) (effects (font (size 2.54 2.54) ) (justify left bottom) ) )
   (label "RAM.A15" (at 396.24 195.58 0) (effects (font (size 2.54 2.54) ) (justify left bottom) ) )

Commit message: Recover from KiCad-6 munging
Parts:
- U501, U502: value (none) -> F257
Changed lines of the file:
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@@
 (kicad_sch
-  (version 20211123)
+  (version 20220126)
   (generator eeschema)
   (paper "User" 584.2 378.46)
@@
   (junction (at 347.98 162.56) (diameter 0) (color 0 0 0 0) )
   (junction (at 353.06 154.94) (diameter 0) (color 0 0 0 0) )
-  (symbol (lib_id "r1000:F257") (at 370.84 218.44 0) (unit 1) (in_bom yes) (on_board yes) (property "Reference" "U501" (id 0) (at 373.38 213.36 0) ) (property "Value" "" (id 1) (at 367.03 223.52 0) (effects (font (size 2.54 2.54) ) (justify left) ) ) (property "Footprint" "" (id 2) (at 372.11 219.71 0) (effects (font (size 1.27 1.27) ) hide ) ) (property "Datasheet" "" (id 3) (at 372.11 219.71 0) (effects (font (size 1.27 1.27) ) hide ) ) (property "Location" "L13" (id 4) (at 369.57 218.44 0) (effects (font (size 2.54 2.54) ) (justify left) ) ) (property "Name" "ATUMUX0" (id 5) (at 372.11 231.14 0) (effects (font (size 2.54 2.54) ) (justify bottom) ) ) (pin "1") (pin "10") (pin "11") (pin "12") (pin "13") (pin "14") (pin "15") (pin "2") (pin "3") (pin "4") (pin "5") (pin "6") (pin "7") (pin "9") )
-  (symbol (lib_id "r1000:F257") (at 370.84 327.66 0) (unit 1) (in_bom yes) (on_board yes) (property "Reference" "U502" (id 0) (at 373.38 322.58 0) ) (property "Value" "" (id 1) (at 367.03 332.74 0) (effects (font (size 2.54 2.54) ) (justify left) ) ) (property "Footprint" "" (id 2) (at 372.11 328.93 0) (effects (font (size 1.27 1.27) ) hide ) ) (property "Datasheet" "" (id 3) (at 372.11 328.93 0) (effects (font (size 1.27 1.27) ) hide ) ) (property "Location" "K13" (id 4) (at 369.57 327.66 0) (effects (font (size 2.54 2.54) ) (justify left) ) ) (property "Name" "ATUMUX1" (id 5) (at 372.11 340.36 0) (effects (font (size 2.54 2.54) ) (justify bottom) ) ) (pin "1") (pin "10") (pin "11") (pin "12") (pin "13") (pin "14") (pin "15") (pin "2") (pin "3") (pin "4") (pin "5") (pin "6") (pin "7") (pin "9") )
+  (symbol (lib_id "r1000:F257") (at 370.84 218.44 0) (unit 1) (in_bom yes) (on_board yes) (property "Reference" "U501" (id 0) (at 373.38 213.36 0) (effects (font (size 1.27 1.27) ) ) ) (property "Value" "F257" (id 1) (at 367.03 223.52 0) (effects (font (size 2.54 2.54) ) (justify left) ) ) (property "Footprint" "" (id 2) (at 372.11 219.71 0) (effects (font (size 1.27 1.27) ) hide ) ) (property "Datasheet" "" (id 3) (at 372.11 219.71 0) (effects (font (size 1.27 1.27) ) hide ) ) (property "Location" "L13" (id 4) (at 369.57 218.44 0) (effects (font (size 2.54 2.54) ) (justify left) ) ) (property "Name" "ATUMUX0" (id 5) (at 372.11 231.14 0) (effects (font (size 2.54 2.54) ) (justify bottom) ) ) (pin "1") (pin "10") (pin "11") (pin "12") (pin "13") (pin "14") (pin "15") (pin "2") (pin "3") (pin "4") (pin "5") (pin "6") (pin "7") (pin "9") )
+  (symbol (lib_id "r1000:F257") (at 370.84 327.66 0) (unit 1) (in_bom yes) (on_board yes) (property "Reference" "U502" (id 0) (at 373.38 322.58 0) (effects (font (size 1.27 1.27) ) ) ) (property "Value" "F257" (id 1) (at 367.03 332.74 0) (effects (font (size 2.54 2.54) ) (justify left) ) ) (property "Footprint" "" (id 2) (at 372.11 328.93 0) (effects (font (size 1.27 1.27) ) hide ) ) (property "Datasheet" "" (id 3) (at 372.11 328.93 0) (effects (font (size 1.27 1.27) ) hide ) ) (property "Location" "K13" (id 4) (at 369.57 327.66 0) (effects (font (size 2.54 2.54) ) (justify left) ) ) (property "Name" "ATUMUX1" (id 5) (at 372.11 340.36 0) (effects (font (size 2.54 2.54) ) (justify bottom) ) ) (pin "1") (pin "10") (pin "11") (pin "12") (pin "13") (pin "14") (pin "15") (pin "2") (pin "3") (pin "4") (pin "5") (pin "6") (pin "7") (pin "9") )
   (label "RAM.A14" (at 396.24 185.42 0) (effects (font (size 2.54 2.54) ) (justify left bottom) ) )
   (label "RAM.A15" (at 396.24 195.58 0) (effects (font (size 2.54 2.54) ) (justify left bottom) ) )

Commit message: Snapshot, much IOC polishing
Changed lines of the file:
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@@
   (wire (pts (xy 388.62 314.96) (xy 424.18 314.96) ) )
   (wire (pts (xy 388.62 325.12) (xy 424.18 325.12) ) )
-  (global_label "RAM.IOP_GRANT~" (shape input) (at 302.26 154.94 180) (fields_autoplaced) (effects (font (size 2.54 2.54) ) (justify right) ) (property "Intersheet References" "${INTERSHEET_REFS}" (id 0) (at 266.2101 154.7813 0) (effects (font (size 2.54 2.54) ) (justify right) ) ) )
-  (global_label "USER_REF" (shape input) (at 304.8 162.56 180) (fields_autoplaced) (effects (font (size 2.54 2.54) ) (justify right) ) (property "Intersheet References" "${INTERSHEET_REFS}" (id 0) (at 280.7244 162.4013 0) (effects (font (size 2.54 2.54) ) (justify right) ) ) )
-  (global_label "IOP.A[14..21]" (shape input) (at 304.8 175.26 180) (fields_autoplaced) (effects (font (size 2.54 2.54) ) (justify right) ) (property "Intersheet References" "${INTERSHEET_REFS}" (id 0) (at 274.314 175.1013 0) (effects (font (size 2.54 2.54) ) (justify right) ) ) )
+  (global_label "RAM.IOP_GRANT~" (shape input) (at 302.26 154.94 180) (fields_autoplaced) (effects (font (size 2.54 2.54) ) (justify right) ) (property "Intersheet References" "${INTERSHEET_REFS}" (id 0) (at 266.2101 154.7813 0) (effects (font (size 1.905 1.905) ) (justify right) ) ) )
+  (global_label "USER_REF" (shape input) (at 304.8 162.56 180) (fields_autoplaced) (effects (font (size 2.54 2.54) ) (justify right) ) (property "Intersheet References" "${INTERSHEET_REFS}" (id 0) (at 280.7244 162.4013 0) (effects (font (size 1.905 1.905) ) (justify right) ) ) )
+  (global_label "IOP.A[1..31]" (shape input) (at 304.8 175.26 180) (fields_autoplaced) (effects (font (size 2.54 2.54) ) (justify right) ) (property "Intersheet References" "${INTERSHEET_REFS}" (id 0) (at 276.2569 175.26 0) (effects (font (size 1.905 1.905) ) (justify right) ) ) )
   (bus_entry (at 312.42 180.34) (size 2.54 2.54) )
   (bus_entry (at 312.42 185.42) (size 2.54 2.54) )
@@
   (bus_entry (at 426.72 312.42) (size -2.54 2.54) )
   (bus_entry (at 426.72 322.58) (size -2.54 2.54) )
-  (global_label "RAM.A[14..21]" (shape output) (at 431.8 182.88 0) (fields_autoplaced) (effects (font (size 2.54 2.54) ) (justify left) ) (property "Intersheet References" "${INTERSHEET_REFS}" (id 0) (at 463.4956 182.7213 0) (effects (font (size 2.54 2.54) ) (justify left) ) ) )
+  (global_label "RAM.A[14..29]" (shape output) (at 431.8 182.88 0) (fields_autoplaced) (effects (font (size 2.54 2.54) ) (justify left) ) (property "Intersheet References" "${INTERSHEET_REFS}" (id 0) (at 463.9716 182.88 0) (effects (font (size 1.905 1.905) ) (justify left) ) ) )
 )

Commit message: F245 work
Changed lines of the file:
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@@
   (global_label "RAM.IOP_GRANT~" (shape input) (at 302.26 154.94 180) (fields_autoplaced) (effects (font (size 2.54 2.54) ) (justify right) ) (property "Intersheet References" "${INTERSHEET_REFS}" (id 0) (at 266.2101 154.7813 0) (effects (font (size 1.905 1.905) ) (justify right) ) ) )
   (global_label "USER_REF" (shape input) (at 304.8 162.56 180) (fields_autoplaced) (effects (font (size 2.54 2.54) ) (justify right) ) (property "Intersheet References" "${INTERSHEET_REFS}" (id 0) (at 280.7244 162.4013 0) (effects (font (size 1.905 1.905) ) (justify right) ) ) )
-  (global_label "IOP.A[1..31]" (shape input) (at 304.8 175.26 180) (fields_autoplaced) (effects (font (size 2.54 2.54) ) (justify right) ) (property "Intersheet References" "${INTERSHEET_REFS}" (id 0) (at 276.2569 175.26 0) (effects (font (size 1.905 1.905) ) (justify right) ) ) )
+  (global_label "IOP.A[0..31]" (shape input) (at 304.8 175.26 180) (fields_autoplaced) (effects (font (size 2.54 2.54) ) (justify right) ) (property "Intersheet References" "${INTERSHEET_REFS}" (id 0) (at 276.2569 175.26 0) (effects (font (size 1.905 1.905) ) (justify right) ) ) )
   (bus_entry (at 312.42 180.34) (size 2.54 2.54) )
   (bus_entry (at 312.42 185.42) (size 2.54 2.54) )

Commit message: Snapshot
Parts:
- removed U501, U502: F257, symbol r1000:F257
