File: Schematics/IOC/pg_31.kicad_sch (KiCad schematic)
At the start: 32 parts, among them U3101 F04, U3102 F04, U3103 F04, U3104 F04, U3105 F04, U3106 F04, U3107 F04, U3108 F04, U3109 F04, U3110 F04, U3111 F04, U3112 F04, U3113 F04, U3114 F04, U3115 F04, U3116 F04, U3117 F04, U3118 F04, U3119 F04, U3120 F04, U3121 F04, U3122 F04, U3123 F04, U3124 F04, U3125 F04, U3126 F04, U3127 F04, U3128 F04, U3129 F04, U3130 F04, U3131 F04, U3132 F04

Commit message: Align to grid
Parts:
- removed U3101, U3102, U3103, U3104, U3105, U3106, U3107, U3108, U3109, U3110, U3111, U3112, U3113, U3114, U3115, U3116, U3117, U3118, U3119, U3120, U3121, U3122, U3123, U3124, U3125, U3126, U3127, U3128, U3129, U3130, U3131, U3132: F04, symbol r1000:F04
- added U (x32): (no value), symbol r1000:F04
Connections:
- net A14.B2~: now also U.2 (Q)
- net A14.B3~: now also U.2 (Q)
- net A15.B2~: now also U.2 (Q)
- net A15.B3~: now also U.2 (Q)
- net A16.B2~: now also U.2 (Q)
- net A16.B3~: now also U.2 (Q)
- net A17.B2~: now also U.2 (Q)
- net A17.B3~: now also U.2 (Q)
- net A18.B2~: now also U.2 (Q)
- net A18.B3~: now also U.2 (Q)
- net A19.B2~: now also U.2 (Q)
- net A19.B3~: now also U.2 (Q)
- net A20.B2~: now also U.2 (Q)
- net A20.B3~: now also U.2 (Q)
- net A21.B2~: now also U.2 (Q)
- net A21.B3~: now also U.2 (Q)
- net A22.B2~: now also U.2 (Q)
- net A22.B3~: now also U.2 (Q)
- net A23.B2~: now also U.2 (Q)
- net A23.B3~: now also U.2 (Q)
- net A24.B2~: now also U.2 (Q)
- net A24.B3~: now also U.2 (Q)
- net A25.B2~: now also U.2 (Q)
- net A25.B3~: now also U.2 (Q)
- net A26.B2~: now also U.2 (Q)
- net A26.B3~: now also U.2 (Q)
- net A27.B2~: now also U.2 (Q)
- net A27.B3~: now also U.2 (Q)
- net A28.B2~: now also U.2 (Q)
- net A28.B3~: now also U.2 (Q)
- net A29.B2~: now also U.2 (Q)
- net A29.B3~: now also U.2 (Q)
- net RAM.A14: now also U.1 (D0), U.1 (D0)
- net RAM.A15: now also U.1 (D0), U.1 (D0)
- net RAM.A16: now also U.1 (D0), U.1 (D0)
- net RAM.A17: now also U.1 (D0), U.1 (D0)
- net RAM.A18: now also U.1 (D0), U.1 (D0)
- net RAM.A19: now also U.1 (D0), U.1 (D0)
- net RAM.A20: now also U.1 (D0), U.1 (D0)
- net RAM.A21: now also U.1 (D0), U.1 (D0)
- net RAM.A22: now also U.1 (D0), U.1 (D0)
- net RAM.A23: now also U.1 (D0), U.1 (D0)
- net RAM.A24: now also U.1 (D0), U.1 (D0)
- net RAM.A25: now also U.1 (D0), U.1 (D0)
- net RAM.A26: now also U.1 (D0), U.1 (D0)
- net RAM.A27: now also U.1 (D0), U.1 (D0)
- net RAM.A28: now also U.1 (D0), U.1 (D0)
- net RAM.A29: now also U.1 (D0), U.1 (D0)

Commit message: IOC: dedup, clocks, dfsm
Parts:
- removed U (x32): (no value), symbol r1000:F04
