File: Schematics/MEM32/pg_26.kicad_sch (KiCad schematic)
At the start: 52 parts, among them U2701 F00, U2702 F00, U2703 F00, U2704 F00, U2705 F00, U2706 F00, U2707 F00, U2708 F00, U2709 F00, U2710 F00, U2711 F00, U2712 F00, U2713 F374, U2714 F00, U2715 F00, U2716 F00, U2717 F00, U2718 F00, U2719 F00, U2720 F00, U2721 F00, U2722 F00, U2723 F00, U2724 F00, U2725 F00, U2726 F374, U2727 F00, U2728 F00, U2729 F00, U2730 F00, U2731 F00, U2732 F00, U2733 F00, U2734 F00, U2735 F00, U2736 F00, U2737 F00, U2738 F00, U2739 F374, U2740 F00, U2741 F00, U2742 F00, U2743 F00, U2744 F00, U2745 F00, U2746 F00, U2747 F00, U2748 F00, U2749 F00, U2750 F00, U2751 F00, U2752 F374

Commit message: Deduplicate signals
Parts:
- removed U2714, U2715, U2716, U2717, U2718, U2719, U2720, U2721, U2722, U2723, U2724, U2725, U2727, U2728, U2729, U2730, U2731, U2732, U2733, U2734, U2735, U2736, U2737, U2738, U2740, U2741, U2742, U2743, U2744, U2745, U2746, U2747, U2748, U2749, U2750, U2751: F00, symbol r1000:F00
- removed U2752: F374, symbol r1000:F374
Connections:
- net TAGA13_Y: now also U2739.13 (D4)
- net TAGA13: now reaches U2739.12 (Q4)
- net TAGA0A0 renamed TAGA0
- net TAGA0A1 renamed TAGA1
- net TAGA0A10 renamed TAGA10
- net TAGA0A11 renamed TAGA11
- net TAGA0A12 renamed TAGA12
- net TAGA0A2 renamed TAGA2
- net TAGA0A3 renamed TAGA3
- net TAGA0A4 renamed TAGA4
- net TAGA0A5 renamed TAGA5
- net TAGA0A6 renamed TAGA6
- net TAGA0A7 renamed TAGA7
- net TAGA0A8 renamed TAGA8
- net TAGA0A9 renamed TAGA9
- net TAGA1A12: no longer names the net of U2739.5 (Q1)
- net TAGB0A12: no longer names the net of U2739.6 (Q2)
- net TAGB1A12: no longer names the net of U2739.9 (Q3)
- no-connect marks 16 -> 9

Commit message: Remove buffer suffixes
Connections:
- net CLK2X_B0 renamed CLK2X
Changed lines of the file:
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@@
   (global_label "TAGA12_Y" (shape input) (at 281.94 317.5 180) (fields_autoplaced) (effects (font (size 2.54 2.54) ) (justify right) ) (property "Intersheet References" "${INTERSHEET_REFS}" (id 0) (at 259.334 317.3413 0) (effects (font (size 2.54 2.54) ) (justify right) ) ) )
   (global_label "TAGA13_Y" (shape input) (at 281.94 322.58 180) (fields_autoplaced) (effects (font (size 2.54 2.54) ) (justify right) ) (property "Intersheet References" "${INTERSHEET_REFS}" (id 0) (at 259.334 322.4213 0) (effects (font (size 2.54 2.54) ) (justify right) ) ) )
-  (global_label "CLK2X_B0" (shape input) (at 299.72 297.18 180) (fields_autoplaced) (effects (font (size 2.54 2.54) ) (justify right) ) (property "Intersheet References" "${INTERSHEET_REFS}" (id 0) (at 276.0254 297.0213 0) (effects (font (size 2.54 2.54) ) (justify right) ) ) )
+  (global_label "CLK2X" (shape input) (at 299.72 297.18 180) (fields_autoplaced) (effects (font (size 2.54 2.54) ) (justify right) ) (property "Intersheet References" "${INTERSHEET_REFS}" (id 0) (at 276.0254 297.0213 0) (effects (font (size 2.54 2.54) ) (justify right) ) ) )
   (junction (at 309.88 317.5) (diameter 0) (color 0 0 0 0) )
   (junction (at 309.88 322.58) (diameter 0) (color 0 0 0 0) )

Commit message: Revert illegal optimization
Parts:
- added U2714: F374, symbol r1000:F374
Connections:
- net PD: now also U2714.1 (OE)
- net TAGA13: now also U2714.2 (Q0); no longer U2739.12 (Q4)
- net TAGA13_Y: now also U2714.3 (D0); no longer U2739.13 (D4)
- new net CLK2X~: U2714.11 (CLK)
- no-connect marks 9 -> 25
Changed lines of the file:
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@@
   (wire (pts (xy 205.74 350.52) (xy 238.76 350.52) ) )
   (wire (pts (xy 281.94 317.5) (xy 309.88 317.5) ) )
-  (wire (pts (xy 281.94 322.58) (xy 299.72 322.58) ) )
   (wire (pts (xy 299.72 297.18) (xy 327.66 297.18) ) )
-  (wire (pts (xy 299.72 322.58) (xy 299.72 337.82) ) )
-  (wire (pts (xy 299.72 337.82) (xy 314.96 337.82) ) )
   (wire (pts (xy 309.88 317.5) (xy 314.96 317.5) ) )
   (wire (pts (xy 309.88 322.58) (xy 309.88 317.5) ) )
@@
   (wire (pts (xy 335.28 299.72) (xy 335.28 302.26) ) )
   (wire (pts (xy 340.36 299.72) (xy 335.28 299.72) ) )
-  (wire (pts (xy 347.98 317.5) (xy 375.92 317.5) ) )
-  (wire (pts (xy 347.98 337.82) (xy 375.92 337.82) ) )
+  (wire (pts (xy 347.98 317.5) (xy 368.3 317.5) ) )
   (wire (pts (xy 38.1 314.96) (xy 71.12 314.96) ) )
   (wire (pts (xy 38.1 320.04) (xy 71.12 320.04) ) )
@@
   (wire (pts (xy 38.1 345.44) (xy 71.12 345.44) ) )
   (wire (pts (xy 38.1 350.52) (xy 71.12 350.52) ) )
+  (wire (pts (xy 388.62 304.8) (xy 396.24 304.8) ) )
+  (wire (pts (xy 396.24 304.8) (xy 396.24 317.5) ) )
+  (wire (pts (xy 396.24 317.5) (xy 401.32 317.5) ) )
   (wire (pts (xy 40.64 119.38) (xy 66.04 119.38) ) )
   (wire (pts (xy 40.64 139.7) (xy 66.04 139.7) ) )
@@
   (wire (pts (xy 40.64 78.74) (xy 66.04 78.74) ) )
   (wire (pts (xy 40.64 99.06) (xy 66.04 99.06) ) )
+  (wire (pts (xy 408.94 289.56) (xy 414.02 289.56) ) )
+  (wire (pts (xy 414.02 289.56) (xy 414.02 302.26) ) )
+  (wire (pts (xy 421.64 299.72) (xy 421.64 302.26) ) )
+  (wire (pts (xy 426.72 299.72) (xy 421.64 299.72) ) )
+  (wire (pts (xy 434.34 317.5) (xy 452.12 317.5) ) )
   (wire (pts (xy 60.96 297.18) (xy 83.82 297.18) ) )
   (wire (pts (xy 83.82 297.18) (xy 185.42 297.18) ) )
@@
   (global_label "TS_TRADR13L" (shape output) (at 238.76 350.52 0) (fields_autoplaced) (effects (font (size 2.54 2.54) ) (justify left) ) (property "Intersheet References" "${INTERSHEET_REFS}" (id 0) (at 268.5022 350.3613 0) (effects (font (size 2.54 2.54) ) (justify left) ) ) )
   (global_label "TAGA12_Y" (shape input) (at 281.94 317.5 180) (fields_autoplaced) (effects (font (size 2.54 2.54) ) (justify right) ) (property "Intersheet References" "${INTERSHEET_REFS}" (id 0) (at 259.334 317.3413 0) (effects (font (size 2.54 2.54) ) (justify right) ) ) )
-  (global_label "TAGA13_Y" (shape input) (at 281.94 322.58 180) (fields_autoplaced) (effects (font (size 2.54 2.54) ) (justify right) ) (property "Intersheet References" "${INTERSHEET_REFS}" (id 0) (at 259.334 322.4213 0) (effects (font (size 2.54 2.54) ) (justify right) ) ) )
   (global_label "CLK2X" (shape input) (at 299.72 297.18 180) (fields_autoplaced) (effects (font (size 2.54 2.54) ) (justify right) ) (property "Intersheet References" "${INTERSHEET_REFS}" (id 0) (at 276.0254 297.0213 0) (effects (font (size 2.54 2.54) ) (justify right) ) ) )
   (junction (at 309.88 317.5) (diameter 0) (color 0 0 0 0) )
   (junction (at 309.88 322.58) (diameter 0) (color 0 0 0 0) )
   (junction (at 309.88 327.66) (diameter 0) (color 0 0 0 0) )
+  (no_connect (at 314.96 337.82) )
   (no_connect (at 314.96 342.9) )
   (no_connect (at 314.96 347.98) )
@@
   (no_connect (at 347.98 327.66) )
   (no_connect (at 347.98 332.74) )
+  (no_connect (at 347.98 337.82) )
   (no_connect (at 347.98 342.9) )
   (no_connect (at 347.98 347.98) )
   (no_connect (at 347.98 353.06) )
   (label "TAGA12" (at 353.06 317.5 0) (effects (font (size 2.54 2.54) ) (justify left bottom) ) )
-  (label "TAGA13" (at 353.06 337.82 0) (effects (font (size 2.54 2.54) ) (justify left bottom) ) )
+  (global_label "TAGA13_Y" (shape input) (at 388.62 304.8 180) (fields_autoplaced) (effects (font (size 2.54 2.54) ) (justify right) ) (property "Intersheet References" "${INTERSHEET_REFS}" (id 0) (at 366.014 304.6413 0) (effects (font (size 2.54 2.54) ) (justify right) ) ) )
+  (no_connect (at 401.32 322.58) )
+  (no_connect (at 401.32 327.66) )
+  (no_connect (at 401.32 332.74) )
+  (no_connect (at 401.32 337.82) )
+  (no_connect (at 401.32 342.9) )
+  (no_connect (at 401.32 347.98) )
+  (no_connect (at 401.32 353.06) )
+  (global_label "CLK2X~" (shape input) (at 408.94 289.56 180) (fields_autoplaced) (effects (font (size 2.54 2.54) ) (justify right) ) (property "Intersheet References" "${INTERSHEET_REFS}" (id 0) (at 390.3254 289.4013 0) (effects (font (size 2.54 2.54) ) (justify right) ) ) )
+  (symbol (lib_id "r1000:F374") (at 416.56 350.52 0) (unit 1) (in_bom yes) (on_board yes) (property "Reference" "U2714" (id 0) (at 419.1 345.44 0) ) (property "Value" "F374" (id 1) (at 412.75 358.14 0) (effects (font (size 2.54 2.54) ) (justify left) ) ) (property "Footprint" "" (id 2) (at 417.83 351.79 0) (effects (font (size 1.27 1.27) ) hide ) ) (property "Datasheet" "" (id 3) (at 417.83 351.79 0) (effects (font (size 1.27 1.27) ) hide ) ) (property "Location" "L22" (id 4) (at 415.29 350.52 0) (effects (font (size 2.54 2.54) ) (justify left) ) ) (property "Name" "TSAREG1" (id 5) (at 417.83 365.76 0) (effects (font (size 2.54 2.54) ) (justify bottom) ) ) (pin "1") (pin "11") (pin "12") (pin "13") (pin "14") (pin "15") (pin "16") (pin "17") (pin "18") (pin "19") (pin "2") (pin "3") (pin "4") (pin "5") (pin "6") (pin "7") (pin "8") (pin "9") )
+  (symbol (lib_id "r1000:PD") (at 426.72 299.72 0) (unit 1) (in_bom no) (on_board yes) (property "Reference" "#PWR02703" (id 0) (at 426.72 299.72 0) (effects (font (size 1.27 1.27) ) hide ) ) (property "Value" "PD" (id 1) (at 426.72 299.72 0) (effects (font (size 1.27 1.27) ) hide ) ) (property "Footprint" "" (id 2) (at 426.72 299.72 0) (effects (font (size 1.27 1.27) ) hide ) ) (property "Datasheet" "" (id 3) (at 426.72 299.72 0) (effects (font (size 1.27 1.27) ) hide ) ) (pin "1") )
+  (no_connect (at 434.34 322.58) )
+  (no_connect (at 434.34 327.66) )
+  (no_connect (at 434.34 332.74) )
+  (no_connect (at 434.34 337.82) )
+  (no_connect (at 434.34 342.9) )
+  (no_connect (at 434.34 347.98) )
+  (no_connect (at 434.34 353.06) )
+  (label "TAGA13" (at 436.88 317.5 0) (effects (font (size 2.54 2.54) ) (justify left bottom) ) )
 )

Commit message: KiCad 6
Parts:
- U2701, U2702, U2703, U2704, U2705, U2706, U2707, U2708, U2709, U2710, U2711, U2712: value F00 -> (none)
- U2713, U2714, U2726, U2739: value F374 -> (none)

Commit message: Recover from KiCad-6 munging
Parts:
- U2701, U2702, U2703, U2704, U2705, U2706, U2707, U2708, U2709, U2710, U2711, U2712: value (none) -> F00
- U2713, U2714, U2726, U2739: value (none) -> F374
