File: Schematics/MEM32/pg_18.kicad_sch (KiCad schematic)
At the start: 16 parts, among them U1901 F280, U1902 F280, U1903 F280, U1904 F280, U1905 F280, U1906 F280, U1907 F280, U1908 F280, U1909 F280, U1910 F374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

Commit message: KiCad 6
Parts:
- U1901, U1902, U1903, U1904, U1905, U1906, U1907, U1908, U1909: value F280 -> (none)
- U1910, U1911, U1912, U1913: value F374 -> (none)
- U1914: value F521 -> (none)
- U1915, U1916: value F299 -> (none)

Commit message: Recover from KiCad-6 munging
Parts:
- U1901, U1902, U1903, U1904, U1905, U1906, U1907, U1908, U1909: value (none) -> F280
- U1910, U1911, U1912, U1913: value (none) -> F374
- U1914: value (none) -> F521
- U1915, U1916: value (none) -> F299

Commit message: polish
Parts:
- removed U1903, U1904, U1905, U1907, U1908, U1909: F280, symbol r1000:F280
- U1901: value F280 -> XPAR64; symbol r1000:F280 -> r1000:XPAR64; Location M14 -> x99; Name TSBPG7 -> TSBPG
Connections:
- net PD: no longer U1901.8 (I0)
- net TAGB_0: now also U1901.2 (I0)
- net TAGB_1: now also U1901.3 (I1)
- net TAGB_10: now also U1901.12 (I10)
- net TAGB_11: now also U1901.13 (I11)
- net TAGB_12: now also U1901.14 (I12)
- net TAGB_13: now also U1901.15 (I13)
- net TAGB_14: now also U1901.16 (I14)
- net TAGB_15: now also U1901.17 (I15)
- net TAGB_16: now also U1901.18 (I16)
- net TAGB_17: now also U1901.19 (I17)
- net TAGB_18: now also U1901.20 (I18)
- net TAGB_19: now also U1901.21 (I19)
- net TAGB_2: now also U1901.4 (I2)
- net TAGB_20: now also U1901.22 (I20)
- net TAGB_21: now also U1901.23 (I21)
- net TAGB_22: now also U1901.24 (I22)
- net TAGB_23: now also U1901.25 (I23)
- net TAGB_24: now also U1901.26 (I24)
- net TAGB_25: now also U1901.27 (I25)
- net TAGB_26: now also U1901.28 (I26)
- net TAGB_27: now also U1901.29 (I27)
- net TAGB_28: now also U1901.30 (I28)
- net TAGB_29: now also U1901.31 (I29)
- net TAGB_3: now also U1901.5 (I3)
- net TAGB_30: now also U1901.32 (I30)
- net TAGB_31: now also U1901.33 (I31)
- net TAGB_32: now also U1901.34 (I32)
- net TAGB_33: now also U1901.35 (I33)
- net TAGB_34: now also U1901.36 (I34)
- net TAGB_35: now also U1901.37 (I35)
- net TAGB_36: now also U1901.38 (I36)
- net TAGB_37: now also U1901.39 (I37)
- net TAGB_38: now also U1901.40 (I38)
- net TAGB_39: now also U1901.41 (I39)
- net TAGB_4: now also U1901.6 (I4)
- net TAGB_40: now also U1901.42 (I40)
- net TAGB_41: now also U1901.43 (I41)
- net TAGB_42: now also U1901.44 (I42)
- net TAGB_43: now also U1901.45 (I43)
- net TAGB_44: now also U1901.46 (I44)
- net TAGB_45: now also U1901.47 (I45)
- net TAGB_46: now also U1901.48 (I46)
- net TAGB_47: now also U1901.49 (I47)
- net TAGB_5: now also U1901.7 (I5)
- net TAGB_56: now also U1901.58 (I56); no longer U1901.4 (I8)
- net TAGB_57: now also U1901.59 (I57); no longer U1901.2 (I7)
- net TAGB_58: now also U1901.60 (I58); no longer U1901.1 (I6)
- net TAGB_59: now also U1901.61 (I59); no longer U1901.13 (I5)
- net TAGB_6: now also U1901.8 (I6)
- net TAGB_60: now also U1901.62 (I60); no longer U1901.12 (I4)
- net TAGB_61: now also U1901.63 (I61); no longer U1901.11 (I3)
- net TAGB_62: now also U1901.64 (I62); no longer U1901.10 (I2)
- net TAGB_63: now also U1901.65 (I63); no longer U1901.9 (I1)
- net TAGB_7: now also U1901.9 (I7)
- net TAGB_8: now also U1901.10 (I8)
- net TAGB_9: now also U1901.11 (I9)
- net TAGB_G7: now reaches U1910.3 (D0), U1911.3 (D0)
- net TAGB_G7: now also U1901.73 (P7); no longer U1901.6 (POD)
- net TAGB_G4: now reaches U1910.8 (D3), U1911.8 (D3)
- net TAGB_G4: now also U1901.70 (P4)
- net TAGB_G2: now reaches U1910.14 (D5), U1911.14 (D5)
- net TAGB_G2: now also U1901.68 (P2)
- net TAGB_G0: now reaches U1910.18 (D7), U1911.18 (D7)
- net TAGB_G0: now also U1901.66 (P0)
- net TAGB_G5: now reaches U1910.7 (D2), U1911.7 (D2)
- net TAGB_G5: now also U1901.71 (P5)
- net TAGB_G3: now reaches U1910.13 (D4), U1911.13 (D4)
- net TAGB_G3: now also U1901.69 (P3)
- net TAGB_G1: now reaches U1910.17 (D6), U1911.17 (D6)
- net TAGB_G1: now also U1901.67 (P1)
- no-connect marks 11 -> 15
Other:
- moved on the sheet: U1902, U1906, U1914

Commit message: Fix parity sense
Connections:
- net PD: now also U1901.1 (ODD)
- no-connect marks 15 -> 14
Changed lines of the file:
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@@
   (wire (pts (xy 561.34 48.26) (xy 561.34 137.16) ) )
   (wire (pts (xy 68.58 17.78) (xy 198.12 17.78) ) )
+  (wire (pts (xy 78.74 22.86) (xy 78.74 25.4) ) )
+  (wire (pts (xy 83.82 22.86) (xy 78.74 22.86) ) )
+  (wire (pts (xy 83.82 25.4) (xy 83.82 22.86) ) )
   (wire (pts (xy 99.06 35.56) (xy 121.92 35.56) ) )
   (wire (pts (xy 99.06 40.64) (xy 121.92 40.64) ) )
@@
   (label "TAGB_48" (at 73.66 17.78 0) (effects (font (size 2.54 2.54) ) (justify left bottom) ) )
   (symbol (lib_id "r1000:XPAR64") (at 76.2 353.06 0) (unit 1) (in_bom yes) (on_board yes) (property "Reference" "U1901" (id 0) (at 78.74 347.98 0) (effects (font (size 1.27 1.27) ) ) ) (property "Value" "XPAR64" (id 1) (at 67.31 360.68 0) (effects (font (size 2.54 2.54) ) (justify left) ) ) (property "Footprint" "" (id 2) (at 77.47 354.33 0) (effects (font (size 1.27 1.27) ) hide ) ) (property "Datasheet" "" (id 3) (at 77.47 354.33 0) (effects (font (size 1.27 1.27) ) hide ) ) (property "Location" "x99" (id 4) (at 74.93 353.06 0) (effects (font (size 2.54 2.54) ) (justify left) ) ) (property "Name" "TSBPG" (id 5) (at 80.01 368.3 0) (effects (font (size 2.54 2.54) ) (justify bottom) ) ) (pin "1") (pin "10") (pin "11") (pin "12") (pin "13") (pin "14") (pin "15") (pin "16") (pin "17") (pin "18") (pin "19") (pin "2") (pin "20") (pin "21") (pin "22") (pin "23") (pin "24") (pin "25") (pin "26") (pin "27") (pin "28") (pin "29") (pin "3") (pin "30") (pin "31") (pin "32") (pin "33") (pin "34") (pin "35") (pin "36") (pin "37") (pin "38") (pin "39") (pin "4") (pin "40") (pin "41") (pin "42") (pin "43") (pin "44") (pin "45") (pin "46") (pin "47") (pin "48") (pin "49") (pin "5") (pin "50") (pin "51") (pin "52") (pin "53") (pin "54") (pin "55") (pin "56") (pin "57") (pin "58") (pin "59") (pin "6") (pin "60") (pin "61") (pin "62") (pin "63") (pin "64") (pin "65") (pin "66") (pin "67") (pin "68") (pin "69") (pin "7") (pin "70") (pin "71") (pin "72") (pin "73") (pin "74") (pin "8") (pin "9") )
-  (no_connect (at 78.74 25.4) )
+  (symbol (lib_id "r1000:PD") (at 83.82 25.4 0) (unit 1) (in_bom no) (on_board yes) (property "Reference" "#PWR01901" (id 0) (at 83.82 25.4 0) (effects (font (size 1.27 1.27) ) hide ) ) (property "Value" "PD" (id 1) (at 83.82 25.4 0) (effects (font (size 1.27 1.27) ) hide ) ) (property "Footprint" "" (id 2) (at 83.82 25.4 0) (effects (font (size 1.27 1.27) ) hide ) ) (property "Datasheet" "" (id 3) (at 83.82 25.4 0) (effects (font (size 1.27 1.27) ) hide ) ) (pin "1") )
   (no_connect (at 99.06 66.04) )
   (no_connect (at 99.06 81.28) )

Commit message: Snapshot
Connections:
- net TAGBE_49: now also U1906.10 (I2); no longer U1906.4 (I8)
- net TAGBE_50: now also U1906.11 (I3); no longer U1906.2 (I7)
- net TAGBE_51: now also U1906.12 (I4); no longer U1906.1 (I6)
- net TAGBE_53: now also U1906.1 (I6); no longer U1906.12 (I4)
- net TAGBE_54: now also U1906.2 (I7); no longer U1906.11 (I3)
- net TAGBE_55: now also U1906.4 (I8); no longer U1906.10 (I2)
- net TAGBL_49: now also U1902.10 (I2); no longer U1902.4 (I8)
- net TAGBL_50: now also U1902.11 (I3); no longer U1902.2 (I7)
- net TAGBL_51: now also U1902.12 (I4); no longer U1902.1 (I6)
- net TAGBL_53: now also U1902.1 (I6); no longer U1902.12 (I4)
- net TAGBL_54: now also U1902.2 (I7); no longer U1902.11 (I3)
- net TAGBL_55: now also U1902.4 (I8); no longer U1902.10 (I2)
Changed lines of the file:
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@@
   (bus_entry (at 193.04 142.24) (size 2.54 2.54) )
   (junction (at 198.12 33.02) (diameter 0) (color 0 0 0 0) )
-  (label "TAGBE_55" (at 200.66 38.1 0) (effects (font (size 2.54 2.54) ) (justify left bottom) ) )
-  (label "TAGBE_54" (at 200.66 43.18 0) (effects (font (size 2.54 2.54) ) (justify left bottom) ) )
-  (label "TAGBE_53" (at 200.66 48.26 0) (effects (font (size 2.54 2.54) ) (justify left bottom) ) )
+  (label "TAGBE_49" (at 200.66 38.1 0) (effects (font (size 2.54 2.54) ) (justify left bottom) ) )
+  (label "TAGBE_50" (at 200.66 43.18 0) (effects (font (size 2.54 2.54) ) (justify left bottom) ) )
+  (label "TAGBE_51" (at 200.66 48.26 0) (effects (font (size 2.54 2.54) ) (justify left bottom) ) )
   (label "TAGBE_52" (at 200.66 53.34 0) (effects (font (size 2.54 2.54) ) (justify left bottom) ) )
-  (label "TAGBE_51" (at 200.66 58.42 0) (effects (font (size 2.54 2.54) ) (justify left bottom) ) )
-  (label "TAGBE_50" (at 200.66 63.5 0) (effects (font (size 2.54 2.54) ) (justify left bottom) ) )
-  (label "TAGBE_49" (at 200.66 68.58 0) (effects (font (size 2.54 2.54) ) (justify left bottom) ) )
-  (label "TAGBL_55" (at 200.66 114.3 0) (effects (font (size 2.54 2.54) ) (justify left bottom) ) )
-  (label "TAGBL_54" (at 200.66 119.38 0) (effects (font (size 2.54 2.54) ) (justify left bottom) ) )
-  (label "TAGBL_53" (at 200.66 124.46 0) (effects (font (size 2.54 2.54) ) (justify left bottom) ) )
+  (label "TAGBE_53" (at 200.66 58.42 0) (effects (font (size 2.54 2.54) ) (justify left bottom) ) )
+  (label "TAGBE_54" (at 200.66 63.5 0) (effects (font (size 2.54 2.54) ) (justify left bottom) ) )
+  (label "TAGBE_55" (at 200.66 68.58 0) (effects (font (size 2.54 2.54) ) (justify left bottom) ) )
+  (label "TAGBL_49" (at 200.66 114.3 0) (effects (font (size 2.54 2.54) ) (justify left bottom) ) )
+  (label "TAGBL_50" (at 200.66 119.38 0) (effects (font (size 2.54 2.54) ) (justify left bottom) ) )
+  (label "TAGBL_51" (at 200.66 124.46 0) (effects (font (size 2.54 2.54) ) (justify left bottom) ) )
   (label "TAGBL_52" (at 200.66 129.54 0) (effects (font (size 2.54 2.54) ) (justify left bottom) ) )
-  (label "TAGBL_51" (at 200.66 134.62 0) (effects (font (size 2.54 2.54) ) (justify left bottom) ) )
-  (label "TAGBL_50" (at 200.66 139.7 0) (effects (font (size 2.54 2.54) ) (justify left bottom) ) )
-  (label "TAGBL_49" (at 200.66 144.78 0) (effects (font (size 2.54 2.54) ) (justify left bottom) ) )
+  (label "TAGBL_53" (at 200.66 134.62 0) (effects (font (size 2.54 2.54) ) (justify left bottom) ) )
+  (label "TAGBL_54" (at 200.66 139.7 0) (effects (font (size 2.54 2.54) ) (justify left bottom) ) )
+  (label "TAGBL_55" (at 200.66 144.78 0) (effects (font (size 2.54 2.54) ) (justify left bottom) ) )
   (symbol (lib_id "r1000:PD") (at 220.98 27.94 0) (unit 1) (in_bom no) (on_board yes) (property "Reference" "#PWR0132" (id 0) (at 220.98 27.94 0) (effects (font (size 1.27 1.27) ) hide ) ) (property "Value" "PD" (id 1) (at 220.98 27.94 0) (effects (font (size 1.27 1.27) ) hide ) ) (property "Footprint" "" (id 2) (at 220.98 27.94 0) (effects (font (size 1.27 1.27) ) hide ) ) (property "Datasheet" "" (id 3) (at 220.98 27.94 0) (effects (font (size 1.27 1.27) ) hide ) ) (pin "1") )
   (symbol (lib_id "r1000:PD") (at 220.98 104.14 0) (unit 1) (in_bom no) (on_board yes) (property "Reference" "#PWR0140" (id 0) (at 220.98 104.14 0) (effects (font (size 1.27 1.27) ) hide ) ) (property "Value" "PD" (id 1) (at 220.98 104.14 0) (effects (font (size 1.27 1.27) ) hide ) ) (property "Footprint" "" (id 2) (at 220.98 104.14 0) (effects (font (size 1.27 1.27) ) hide ) ) (property "Datasheet" "" (id 3) (at 220.98 104.14 0) (effects (font (size 1.27 1.27) ) hide ) ) (pin "1") )
   (symbol (lib_id "r1000:F280") (at 238.76 68.58 0) (unit 1) (in_bom yes) (on_board yes) (property "Reference" "U1906" (id 0) (at 241.3 63.5 0) (effects (font (size 1.27 1.27) ) ) ) (property "Value" "F280" (id 1) (at 232.41 73.66 0) (effects (font (size 2.54 2.54) ) (justify left) ) ) (property "Footprint" "" (id 2) (at 240.03 69.85 0) (effects (font (size 1.27 1.27) ) hide ) ) (property "Datasheet" "" (id 3) (at 240.03 69.85 0) (effects (font (size 1.27 1.27) ) hide ) ) (property "Location" "N7" (id 4) (at 237.49 68.58 0) (effects (font (size 2.54 2.54) ) (justify left) ) ) (property "Name" "TSBEPG6" (id 5) (at 240.03 81.28 0) (effects (font (size 2.54 2.54) ) (justify bottom) ) ) (pin "1") (pin "10") (pin "11") (pin "12") (pin "13") (pin "2") (pin "4") (pin "5") (pin "6") (pin "8") (pin "9") )
   (symbol (lib_id "r1000:F280") (at 238.76 144.78 0) (unit 1) (in_bom yes) (on_board yes) (property "Reference" "U1902" (id 0) (at 241.3 139.7 0) (effects (font (size 1.27 1.27) ) ) ) (property "Value" "F280" (id 1) (at 232.41 149.86 0) (effects (font (size 2.54 2.54) ) (justify left) ) ) (property "Footprint" "" (id 2) (at 240.03 146.05 0) (effects (font (size 1.27 1.27) ) hide ) ) (property "Datasheet" "" (id 3) (at 240.03 146.05 0) (effects (font (size 1.27 1.27) ) hide ) ) (property "Location" "N4" (id 4) (at 237.49 144.78 0) (effects (font (size 2.54 2.54) ) (justify left) ) ) (property "Name" "TSBLPG6" (id 5) (at 240.03 157.48 0) (effects (font (size 2.54 2.54) ) (justify bottom) ) ) (pin "1") (pin "10") (pin "11") (pin "12") (pin "13") (pin "2") (pin "4") (pin "5") (pin "6") (pin "8") (pin "9") )
-  (global_label "CLK2X" (shape input) (at 251.46 355.6 180) (fields_autoplaced) (effects (font (size 2.54 2.54) ) (justify right) ) (property "Intersheet References" "${INTERSHEET_REFS}" (id 0) (at 227.7654 355.4413 0) (effects (font (size 1.905 1.905) ) (justify right) ) ) )
-  (global_label "CLK2X~" (shape input) (at 251.46 363.22 180) (fields_autoplaced) (effects (font (size 2.54 2.54) ) (justify right) ) (property "Intersheet References" "${INTERSHEET_REFS}" (id 0) (at 227.8864 363.0613 0) (effects (font (size 1.905 1.905) ) (justify right) ) ) )
+  (global_label "CLK2X" (shape input) (at 251.46 355.6 180) (fields_autoplaced) (effects (font (size 2.54 2.54) ) (justify right) ) (property "Intersheet References" "${INTERSHEET_REFS}" (id 0) (at 233.9929 355.6 0) (effects (font (size 1.905 1.905) ) (justify right) ) ) )
+  (global_label "CLK2X~" (shape input) (at 251.46 363.22 180) (fields_autoplaced) (effects (font (size 2.54 2.54) ) (justify right) ) (property "Intersheet References" "${INTERSHEET_REFS}" (id 0) (at 232.1786 363.22 0) (effects (font (size 1.905 1.905) ) (justify right) ) ) )
   (no_connect (at 254 38.1) )
   (no_connect (at 254 114.3) )

Commit message: Snapshot
Parts:
- removed U1901: XPAR64, symbol r1000:XPAR64
- removed U1902, U1906: F280, symbol r1000:F280
- removed U1910, U1911, U1912, U1913: F374, symbol r1000:F374
- removed U1914: F521, symbol r1000:F521
- removed U1915, U1916: F299, symbol r1000:F299
- added U (x4): (no value), symbol r1000:F374
- added U (x2): (no value), symbol r1000:F280
- added U: (no value), symbol r1000:F521
- added U: (no value), symbol r1000:XPAR64
- added U (x2): (no value), symbol r1000:F299
Connections:
- net CLK2X: now also U.11 (CLK), U.11 (CLK), U.12 (CLK), U.12 (CLK)
- net CLK2X~: now also U.11 (CLK), U.11 (CLK)
- net DIAG_1: now also U.18 (LSI)
- net PD: now also U.1 (E), U.1 (ODD), U.11 (RSI), U.11 (RSI), U.8 (I0), U.8 (I0)
- net PU: now also U.9 (CLR), U.9 (CLR)
- net TAGBE_49: now also U.10 (I2)
- net TAGBE_50: now also U.11 (I3)
- net TAGBE_51: now also U.12 (I4)
- net TAGBE_52: now also U.13 (I5)
- net TAGBE_53: now also U.1 (I6)
- net TAGBE_54: now also U.2 (I7)
- net TAGBE_55: now also U.4 (I8)
- net TAGBE_P6: now also U.4 (D1)
- net TAGBL_49: now also U.10 (I2)
- net TAGBL_50: now also U.11 (I3)
- net TAGBL_51: now also U.12 (I4)
- net TAGBL_52: now also U.13 (I5)
- net TAGBL_53: now also U.1 (I6)
- net TAGBL_54: now also U.2 (I7)
- net TAGBL_55: now also U.4 (I8)
- net TAGBL_P6: now also U.4 (D1)
- net TAGB_0: now also U.2 (I0)
- net TAGB_1: now also U.3 (I1)
- net TAGB_10: now also U.12 (I10)
- net TAGB_11: now also U.13 (I11)
- net TAGB_12: now also U.14 (I12)
- net TAGB_13: now also U.15 (I13)
- net TAGB_14: now also U.16 (I14)
- net TAGB_15: now also U.17 (I15)
- net TAGB_16: now also U.18 (I16)
- net TAGB_17: now also U.19 (I17)
- net TAGB_18: now also U.20 (I18)
- net TAGB_19: now also U.21 (I19)
- net TAGB_2: now also U.4 (I2)
- net TAGB_20: now also U.22 (I20)
- net TAGB_21: now also U.23 (I21)
- net TAGB_22: now also U.24 (I22)
- net TAGB_23: now also U.25 (I23)
- net TAGB_24: now also U.26 (I24)
- net TAGB_25: now also U.27 (I25)
- net TAGB_26: now also U.28 (I26)
- net TAGB_27: now also U.29 (I27)
- net TAGB_28: now also U.30 (I28)
- net TAGB_29: now also U.31 (I29)
- net TAGB_3: now also U.5 (I3)
- net TAGB_30: now also U.32 (I30)
- net TAGB_31: now also U.33 (I31)
- net TAGB_32: now also U.34 (I32)
- net TAGB_33: now also U.35 (I33)
- net TAGB_34: now also U.36 (I34)
- net TAGB_35: now also U.37 (I35)
- net TAGB_36: now also U.38 (I36)
- net TAGB_37: now also U.39 (I37)
- net TAGB_38: now also U.40 (I38)
- net TAGB_39: now also U.41 (I39)
- net TAGB_4: now also U.6 (I4)
- net TAGB_40: now also U.42 (I40)
- net TAGB_41: now also U.43 (I41)
- net TAGB_42: now also U.44 (I42)
- net TAGB_43: now also U.45 (I43)
- net TAGB_44: now also U.46 (I44)
- net TAGB_45: now also U.47 (I45)
- net TAGB_46: now also U.48 (I46)
- net TAGB_47: now also U.49 (I47)
- net TAGB_48: now also U.9 (I1), U.9 (I1)
- net TAGB_5: now also U.7 (I5)
- net TAGB_56: now also U.58 (I56)
- net TAGB_57: now also U.59 (I57)
- net TAGB_58: now also U.60 (I58)
- net TAGB_59: now also U.61 (I59)
- net TAGB_6: now also U.8 (I6)
- net TAGB_60: now also U.62 (I60)
- net TAGB_61: now also U.63 (I61)
- net TAGB_62: now also U.64 (I62)
- net TAGB_63: now also U.65 (I63)
- net TAGB_7: now also U.9 (I7)
- net TAGB_8: now also U.10 (I8)
- net TAGB_9: now also U.11 (I9)
- net TAGB_G0: now also U.18 (D7), U.18 (D7), U.66 (P0)
- net TAGB_G1: now also U.17 (D6), U.17 (D6), U.67 (P1)
- net TAGB_G2: now also U.14 (D5), U.14 (D5), U.68 (P2)
- net TAGB_G3: now also U.13 (D4), U.13 (D4), U.69 (P3)
- net TAGB_G4: now also U.70 (P4), U.8 (D3), U.8 (D3)
- net TAGB_G5: now also U.7 (D2), U.7 (D2), U.71 (P5)
- net TAGB_G7: now also U.3 (D0), U.3 (D0), U.73 (P7)
- net TAGB_P0: now also U.18 (D7), U.18 (D7)
- net TAGB_P1: now also U.17 (D6), U.17 (D6)
- net TAGB_P2: now also U.14 (D5), U.14 (D5)
- net TAGB_P3: now also U.13 (D4), U.13 (D4)
- net TAGB_P4: now also U.8 (D3), U.8 (D3)
- net TAGB_P5: now also U.7 (D2), U.7 (D2)
- net TAGB_P7: now also U.3 (D0), U.3 (D0)
- net TSB_PAR_OUT: now also U.8 (Q0)
- net TSB_PERR: now also U.19 (A=B)
- net TS_EPAR_OE~: now also U.1 (OE), U.1 (OE)
- net TS_LPAR_OE~: now also U.1 (OE), U.1 (OE)
- net TS_PAR_MODE0: now also U.2 (G1), U.2 (G1), U.3 (G2), U.3 (G2)
- net TS_PAR_S0: now also U.19 (S0), U.19 (S0)
- net TS_PAR_S1: now also U.1 (S1), U.1 (S1)
- new net: U.12 (B4), U.12 (Q4), U.12 (Q4), U.5 (DQ4)
- new net: U.14 (B5), U.15 (DQ5), U.15 (Q5), U.15 (Q5)
- new net: U.16 (B6), U.16 (Q6), U.16 (Q6), U.4 (DQ6)
- new net: U.16 (DQ7), U.18 (B7), U.19 (Q7), U.19 (Q7)
- new net: U.2 (Q0), U.2 (Q0), U.3 (B0), U.7 (DQ0)
- new net: U.13 (DQ1), U.5 (B1), U.5 (Q1), U.5 (Q1)
- new net: U.6 (DQ2), U.6 (Q2), U.6 (Q2), U.7 (B2)
- new net: U.14 (DQ3), U.9 (B3), U.9 (Q3), U.9 (Q3)
- new net: U.4 (D1), U.6 (POD) (x2)
- new net: U.11 (A4), U.12 (Q4), U.12 (Q4), U.5 (DQ4)
- new net: U.13 (A5), U.15 (DQ5), U.15 (Q5), U.15 (Q5)
- new net: U.15 (A6), U.16 (Q6), U.16 (Q6), U.4 (DQ6)
- new net: U.16 (DQ7), U.17 (A7), U.19 (Q7), U.19 (Q7)
- new net: U.2 (A0), U.2 (Q0), U.2 (Q0), U.7 (DQ0)
- new net: U.13 (DQ1), U.4 (A1), U.5 (Q1), U.5 (Q1)
- new net: U.6 (A2), U.6 (DQ2), U.6 (Q2), U.6 (Q2)
- new net: U.14 (DQ3), U.8 (A3), U.9 (Q3), U.9 (Q3)
- new net: U.18 (LSI), U.8 (Q0)
