File: Schematics/MEM32/pg_46.kicad_sch (KiCad schematic)
At the start: 3 parts, among them U4701 F00, U4702 F00, U4703 F00

Commit message: Collect DRAM planes on a single page with megacomps
Parts:
- removed U4701, U4702, U4703: F00, symbol r1000:F00
Changed lines of the file:
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@@
   (paper "User" 584.2 378.46)
   (title_block (title "PLANEB\\nRAS, CAS, WE GENERATION") (date "08-MAR-90") (rev "0.0") (comment 1 "MEM32 BOARD") (comment 2 "232-003066") (comment 3 "S400") (comment 4 "RELEASED") )
-  (wire (pts (xy 198.12 193.04) (xy 226.06 193.04) ) )
-  (wire (pts (xy 223.52 20.32) (xy 223.52 17.78) ) )
-  (wire (pts (xy 223.52 20.32) (xy 307.34 20.32) ) )
-  (wire (pts (xy 223.52 35.56) (xy 223.52 20.32) ) )
-  (wire (pts (xy 226.06 193.04) (xy 226.06 40.64) ) )
-  (wire (pts (xy 226.06 40.64) (xy 228.6 40.64) ) )
-  (wire (pts (xy 228.6 35.56) (xy 223.52 35.56) ) )
-  (wire (pts (xy 251.46 38.1) (xy 269.24 38.1) ) )
-  (wire (pts (xy 292.1 193.04) (xy 309.88 193.04) ) )
-  (wire (pts (xy 307.34 20.32) (xy 307.34 35.56) ) )
-  (wire (pts (xy 307.34 20.32) (xy 391.16 20.32) ) )
-  (wire (pts (xy 309.88 193.04) (xy 309.88 40.64) ) )
-  (wire (pts (xy 309.88 40.64) (xy 312.42 40.64) ) )
-  (wire (pts (xy 312.42 35.56) (xy 307.34 35.56) ) )
-  (wire (pts (xy 335.28 38.1) (xy 350.52 38.1) ) )
-  (wire (pts (xy 370.84 193.04) (xy 393.7 193.04) ) )
-  (wire (pts (xy 391.16 35.56) (xy 391.16 20.32) ) )
-  (wire (pts (xy 393.7 193.04) (xy 393.7 40.64) ) )
-  (wire (pts (xy 393.7 40.64) (xy 396.24 40.64) ) )
-  (wire (pts (xy 396.24 35.56) (xy 391.16 35.56) ) )
-  (wire (pts (xy 419.1 38.1) (xy 439.42 38.1) ) )
-  (global_label "DR_RASB" (shape input) (at 198.12 193.04 180) (fields_autoplaced) (effects (font (size 2.54 2.54) ) (justify right) ) (property "Intersheet References" "${INTERSHEET_REFS}" (id 0) (at 176.6026 192.8813 0) (effects (font (size 2.54 2.54) ) (justify right) ) ) )
-  (symbol (lib_id "r1000:PU") (at 223.52 17.78 0) (unit 1) (in_bom yes) (on_board yes) (property "Reference" "#PWR04701" (id 0) (at 223.52 17.78 0) (effects (font (size 1.27 1.27) ) hide ) ) (property "Value" "PU" (id 1) (at 223.52 17.78 0) (effects (font (size 1.27 1.27) ) hide ) ) (property "Footprint" "" (id 2) (at 223.52 17.78 0) (effects (font (size 1.27 1.27) ) hide ) ) (property "Datasheet" "" (id 3) (at 223.52 17.78 0) (effects (font (size 1.27 1.27) ) hide ) ) (pin "1") )
-  (junction (at 223.52 20.32) (diameter 0) (color 0 0 0 0) )
-  (symbol (lib_id "r1000:F00") (at 236.22 35.56 0) (unit 1) (in_bom yes) (on_board yes) (property "Reference" "U4701" (id 0) (at 251.46 35.56 0) ) (property "Value" "F00" (id 1) (at 238.125 40.64 0) (effects (font (size 2.54 2.54) ) ) ) (property "Footprint" "" (id 2) (at 236.22 22.86 0) (effects (font (size 1.27 1.27) ) hide ) ) (property "Datasheet" "" (id 3) (at 236.22 22.86 0) (effects (font (size 1.27 1.27) ) hide ) ) (property "Location" "F20" (id 4) (at 238.125 35.56 0) (effects (font (size 2.54 2.54) ) ) ) (property "Name" "BCDAB" (id 5) (at 238.76 48.26 0) (effects (font (size 2.54 2.54) ) (justify bottom) ) ) (pin "1") (pin "2") (pin "3") )
-  (global_label "BARAS~" (shape output) (at 269.24 38.1 0) (fields_autoplaced) (effects (font (size 2.54 2.54) ) (justify left) ) (property "Intersheet References" "${INTERSHEET_REFS}" (id 0) (at 287.7336 37.9413 0) (effects (font (size 2.54 2.54) ) (justify left) ) ) )
-  (global_label "DR_CASB" (shape input) (at 292.1 193.04 180) (fields_autoplaced) (effects (font (size 2.54 2.54) ) (justify right) ) (property "Intersheet References" "${INTERSHEET_REFS}" (id 0) (at 270.5826 192.8813 0) (effects (font (size 2.54 2.54) ) (justify right) ) ) )
-  (junction (at 307.34 20.32) (diameter 0) (color 0 0 0 0) )
-  (symbol (lib_id "r1000:F00") (at 320.04 35.56 0) (unit 1) (in_bom yes) (on_board yes) (property "Reference" "U4702" (id 0) (at 335.28 35.56 0) ) (property "Value" "F00" (id 1) (at 321.945 40.64 0) (effects (font (size 2.54 2.54) ) ) ) (property "Footprint" "" (id 2) (at 320.04 22.86 0) (effects (font (size 1.27 1.27) ) hide ) ) (property "Datasheet" "" (id 3) (at 320.04 22.86 0) (effects (font (size 1.27 1.27) ) hide ) ) (property "Location" "F20" (id 4) (at 321.945 35.56 0) (effects (font (size 2.54 2.54) ) ) ) (property "Name" "BCDAD" (id 5) (at 322.58 48.26 0) (effects (font (size 2.54 2.54) ) (justify bottom) ) ) (pin "1") (pin "2") (pin "3") )
-  (global_label "BACAS~" (shape output) (at 350.52 38.1 0) (fields_autoplaced) (effects (font (size 2.54 2.54) ) (justify left) ) (property "Intersheet References" "${INTERSHEET_REFS}" (id 0) (at 369.0136 37.9413 0) (effects (font (size 2.54 2.54) ) (justify left) ) ) )
-  (global_label "DR_WEB" (shape input) (at 370.84 193.04 180) (fields_autoplaced) (effects (font (size 2.54 2.54) ) (justify right) ) (property "Intersheet References" "${INTERSHEET_REFS}" (id 0) (at 351.2578 192.8813 0) (effects (font (size 2.54 2.54) ) (justify right) ) ) )
-  (symbol (lib_id "r1000:F00") (at 403.86 35.56 0) (unit 1) (in_bom yes) (on_board yes) (property "Reference" "U4703" (id 0) (at 419.1 35.56 0) ) (property "Value" "F00" (id 1) (at 405.765 40.64 0) (effects (font (size 2.54 2.54) ) ) ) (property "Footprint" "" (id 2) (at 403.86 22.86 0) (effects (font (size 1.27 1.27) ) hide ) ) (property "Datasheet" "" (id 3) (at 403.86 22.86 0) (effects (font (size 1.27 1.27) ) hide ) ) (property "Location" "F20" (id 4) (at 405.765 35.56 0) (effects (font (size 2.54 2.54) ) ) ) (property "Name" "BCDAA" (id 5) (at 406.4 48.26 0) (effects (font (size 2.54 2.54) ) (justify bottom) ) ) (pin "1") (pin "2") (pin "3") )
-  (global_label "BAWE~" (shape output) (at 439.42 38.1 0) (fields_autoplaced) (effects (font (size 2.54 2.54) ) (justify left) ) (property "Intersheet References" "${INTERSHEET_REFS}" (id 0) (at 455.9784 37.9413 0) (effects (font (size 2.54 2.54) ) (justify left) ) ) )
 )
