File: Schematics/SEQ/pg_15.kicad_sch (KiCad schematic)
At the start: 19 parts, among them U1601 PA040-02, U1602 F158, U1603 F158, U1604 F37, U1605 F37, U1606 F04, U1607 F37, U1608 F373, U1609 F37, U1610 F37, U1611 F04, U1612 F04, U1613 F00, U1614 F00, U1615 F64

Commit message: KiCad 6
Parts:
- GB241, GB242, GB246, GB252: value GB -> (none)
- U1601: value PA040-02 -> (none)
- U1602, U1603: value F158 -> (none)
- U1604, U1605, U1607, U1609, U1610: value F37 -> (none)
- U1606, U1611, U1612: value F04 -> (none)
- U1608: value F373 -> (none)
- U1613, U1614: value F00 -> (none)
- U1615: value F64 -> (none)

Commit message: Recover from KiCad-6 munging
Parts:
- GB241, GB242, GB246, GB252: value (none) -> GB
- U1601: value (none) -> PA040-02
- U1602, U1603: value (none) -> F158
- U1604, U1605, U1607, U1609, U1610: value (none) -> F37
- U1606, U1611, U1612: value (none) -> F04
- U1608: value (none) -> F373
- U1613, U1614: value (none) -> F00
- U1615: value (none) -> F64

Commit message: Fix polarity of unused part of driven FIU bus.
Parts:
- removed GB241, GB242, GB246, GB252: GB, symbol r1000:GB
- removed U1601: PA040-02, symbol r1000:PAxxx
- removed U1602, U1603: F158, symbol r1000:F158
- removed U1604, U1605, U1607, U1609, U1610: F37, symbol r1000:F37
- removed U1606, U1611, U1612: F04, symbol r1000:F04
- removed U1608: F373, symbol r1000:F373
- removed U1613, U1614: F00, symbol r1000:F00
- removed U1615: F64, symbol r1000:F64
- added U (x4): (no value), symbol r1000:GB
- added U (x5): (no value), symbol r1000:F37
- added U: (no value), symbol r1000:F373
- added U (x2): (no value), symbol r1000:F00
- added U (x3): (no value), symbol r1000:F04
- added U (x2): (no value), symbol r1000:F158
- added U: (no value), symbol r1000:F64
- added U: (no value), symbol r1000:PAxxx
Connections:
- net ADR.SPACE_PEV: now also U.12 (Y3)
- net ADR.SPACE~0: now also U.4 (Y0)
- net ADR.SPACE~1: now also U.7 (Y1)
- net ADR.SPACE~2: now also U.9 (Y2)
- net ADR_IS_CODE: now also U.3 (Q)
- net ADR_SEL.RND: now also U.5 (A4)
- net BAD_HINT: now also U.1 (A8)
- net BAD_HINT.DISP: now also U.1 (D0)
- net DISP_COND0: now also U.14 (Y0)
- net H2E: now also U.11 (LE)
- net IMPORT.COND~: now also U.4 (A5)
- net LOC_STOP.DIAG2~: now also U.1 (D0), U.1 (D0)
- net L_ABRT.RND: now also U.1 (D0)
- net MACRO.IBUFF~: now also U.2 (A0)
- net MACRO_EVENT~: now also U.1 (D0), U.1 (S), U.1 (S)
- net MAYBE_DISPATCH~: now also U.2 (A7)
- net MEM_STRT.DEC0: now also U.19 (A0)
- net MEM_STRT.DEC1: now also U.18 (A1)
- net MEM_STRT.DEC2: now also U.17 (A2)
- net PD: now also U.1 (OE), U.10 (B1), U.11 (A2), U.13 (D4), U.14 (D5), U.15 (E), U.15 (E), U.15 (OE), U.17 (D6), U.18 (D7), U.2 (A0), U.3 (A1), U.5 (A1), U.7 (D2), U.8 (D3), U.9 (B0)
- net PU: now also U.14 (A3), U.2 (A0), U.5 (A1)
- net Q.COND_TRUE~: now also U.1, U.1 (D0), U.2 (D1)
- net Q.E_ABORT~: now also U.1, U.3 (Q)
- net Q.L_ABORT~: now also U.1, U.3 (Q)
- net Q.MEM_COND~: now also U.1, U.1 (D0)
- net Q3_COND: now also U.6 (C2)
- net Q3_COND~: now also U.13 (D3)
- net RESOLVE_DRIVE~: now also U.7 (Y1)
- net RES_DRIVE: now also U.13 (Y1), U.6 (B1)
- net SEQ_STOP: now also U.3 (A6)
- net SEQ_STOP~: now also U.2 (D1)
- net WANNA_DISPATCH~: now also U.16 (A3)
- new net: U.1 (D0), U.2 (Q)
- new net: U.2 (D1), U.3 (Q)
- new net: U.3 (Q), U.4 (D1)
- new net: U.12 (D2), U.2 (Q0), U.5 (C1)
- new net: U.3 (D0), U.4 (Y0)
- new net: U.2 (D1), U.5 (Q1)
- new net: U.1 (D0), U.1 (D0), U.2 (Q)
- new net: U.2 (D1), U.2 (Q)
- new net: U.1 (D0), U.11 (D1), U.3 (Q)
- new net: U.2 (D1), U.6 (Y7)
- new net: U.3 (Q), U.4 (C0)
- new net: U.10 (B2), U.9 (Y4)
- new net: U.13 (B3), U.8 (Y5)
- new net: U.12 (Y2), U.3 (B0)
- new net: U.11 (Y3), U.6 (B1)
- new net: U.2 (D1), U.8 (Q)
- new net: U.3 (B0), U.7 (Y6)
