File: Schematics/SEQ/pg_26.kicad_sch (KiCad schematic)
At the start: 4 parts, among them U2701 F374, U2702 F374, U2703 F374, U2704 F20

Commit message: Much work on SEQ
Parts:
- removed U2702, U2703: F374, symbol r1000:F374
- U2701: value F374 -> XREG24; symbol r1000:F374 -> r1000:XREG24; Location K14 -> x99; Name SAVRG0 -> SAVRG
Connections:
- net EN_MICROS: now also U2704.2 (D1), U2704.4 (D2); no longer U2704.5 (D3)
- net OFFSET_BUS37: now also U2701.15 (Q4); no longer U2701.12 (Q4)
- net OFFSET_BUS38: now also U2701.17 (Q5); no longer U2701.15 (Q5)
- net OFFSET_BUS39: now also U2701.19 (Q6); no longer U2701.16 (Q6)
- net OFFSET_BUS40: now also U2701.21 (Q7); no longer U2701.19 (Q7)
- net OFFSET_BUS41: now also U2701.23 (Q8)
- net OFFSET_BUS42: now also U2701.25 (Q9)
- net OFFSET_BUS43: now also U2701.27 (Q10)
- net OFFSET_BUS44: now also U2701.29 (Q11)
- net OFFSET_BUS45: now also U2701.31 (Q12)
- net OFFSET_BUS46: now also U2701.33 (Q13)
- net OFFSET_BUS47: now also U2701.35 (Q14)
- net OFFSET_BUS48: now also U2701.37 (Q15)
- net OFFSET_BUS49: now also U2701.39 (Q16)
- net OFFSET_BUS50: now also U2701.41 (Q17)
- net OFFSET_BUS51: now also U2701.43 (Q18)
- net OFFSET_BUS52: now also U2701.45 (Q19)
- net OFFSET_BUS53: now also U2701.47 (Q20)
- net OFFSET_BUS54: now also U2701.49 (Q21)
- net OFFSET_BUS55: now also U2701.51 (Q22)
- net OFFSET_BUS56: now also U2701.53 (Q23)
- net RESOLVE_OFFS37: now also U2701.14 (D4); no longer U2701.13 (D4)
- net RESOLVE_OFFS38: now also U2701.16 (D5); no longer U2701.14 (D5)
- net RESOLVE_OFFS39: now also U2701.18 (D6); no longer U2701.17 (D6)
- net RESOLVE_OFFS40: now also U2701.20 (D7); no longer U2701.18 (D7)
- net RESOLVE_OFFS41: now also U2701.22 (D8)
- net RESOLVE_OFFS42: now also U2701.24 (D9)
- net RESOLVE_OFFS43: now also U2701.26 (D10)
- net RESOLVE_OFFS44: now also U2701.28 (D11)
- net RESOLVE_OFFS45: now also U2701.30 (D12)
- net RESOLVE_OFFS46: now also U2701.32 (D13)
- net RESOLVE_OFFS47: now also U2701.34 (D14)
- net RESOLVE_OFFS48: now also U2701.36 (D15)
- net RESOLVE_OFFS49: now also U2701.38 (D16)
- net RESOLVE_OFFS50: now also U2701.40 (D17)
- net RESOLVE_OFFS51: now also U2701.42 (D18)
- net RESOLVE_OFFS52: now also U2701.44 (D19)
- net RESOLVE_OFFS53: now also U2701.46 (D20)
- net RESOLVE_OFFS54: now also U2701.48 (D21)
- net RESOLVE_OFFS55: now also U2701.50 (D22)
- net RESOLVE_OFFS56: now also U2701.52 (D23)
- net RES_ALU.COUT: now also U2701.6 (D0); no longer U2701.3 (D0)
- net SAVE.CLK~: now also U2701.1 (CLK); no longer U2701.11 (CLK)
- net SAVE.OE~: now also U2701.3 (OE); no longer U2701.1 (OE)
- net at U2701.7 (Q0): now also U2704.5 (D3)
- now unconnected: U2701.2 (Q0)
- no-connect marks 6 -> 7
Other:
- moved on the sheet: U2704

Commit message: KiCad 6
Parts:
- U2701: value XREG24 -> (none)
- U2704: value F20 -> (none)
Changed lines of the file:
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@@
   (no_connect (at 246.38 142.24) )
   (global_label "SAVE.CLK~" (shape input) (at 254 109.22 180) (fields_autoplaced) (effects (font (size 2.54 2.54) ) (justify right) ) (property "Intersheet References" "${INTERSHEET_REFS}" (id 0) (at 229.9426 109.0613 0) (effects (font (size 2.54 2.54) ) (justify right) ) ) )
-  (symbol (lib_id "r1000:XREG24") (at 264.16 241.3 0) (unit 1) (in_bom yes) (on_board yes) (property "Reference" "U2701" (id 0) (at 266.7 236.22 0) ) (property "Value" "XREG24" (id 1) (at 262.89 246.38 0) (effects (font (size 2.54 2.54) ) (justify left) ) ) (property "Footprint" "" (id 2) (at 265.43 242.57 0) (effects (font (size 1.27 1.27) ) hide ) ) (property "Datasheet" "" (id 3) (at 265.43 242.57 0) (effects (font (size 1.27 1.27) ) hide ) ) (property "Location" "x99" (id 4) (at 262.89 241.3 0) (effects (font (size 2.54 2.54) ) (justify left) ) ) (property "Name" "SAVRG" (id 5) (at 267.97 254 0) (effects (font (size 2.54 2.54) ) (justify bottom) ) ) (pin "1") (pin "10") (pin "11") (pin "12") (pin "13") (pin "14") (pin "15") (pin "16") (pin "17") (pin "18") (pin "19") (pin "2") (pin "20") (pin "21") (pin "22") (pin "23") (pin "24") (pin "25") (pin "26") (pin "27") (pin "28") (pin "29") (pin "3") (pin "30") (pin "31") (pin "32") (pin "33") (pin "34") (pin "35") (pin "36") (pin "37") (pin "38") (pin "39") (pin "40") (pin "41") (pin "42") (pin "43") (pin "44") (pin "45") (pin "46") (pin "47") (pin "48") (pin "49") (pin "50") (pin "51") (pin "52") (pin "53") (pin "6") (pin "7") (pin "8") (pin "9") )
+  (symbol (lib_id "r1000:XREG24") (at 264.16 241.3 0) (unit 1) (in_bom yes) (on_board yes) (property "Reference" "U2701" (id 0) (at 266.7 236.22 0) ) (property "Value" "" (id 1) (at 262.89 246.38 0) (effects (font (size 2.54 2.54) ) (justify left) ) ) (property "Footprint" "" (id 2) (at 265.43 242.57 0) (effects (font (size 1.27 1.27) ) hide ) ) (property "Datasheet" "" (id 3) (at 265.43 242.57 0) (effects (font (size 1.27 1.27) ) hide ) ) (property "Location" "x99" (id 4) (at 262.89 241.3 0) (effects (font (size 2.54 2.54) ) (justify left) ) ) (property "Name" "SAVRG" (id 5) (at 267.97 254 0) (effects (font (size 2.54 2.54) ) (justify bottom) ) ) (pin "1") (pin "10") (pin "11") (pin "12") (pin "13") (pin "14") (pin "15") (pin "16") (pin "17") (pin "18") (pin "19") (pin "2") (pin "20") (pin "21") (pin "22") (pin "23") (pin "24") (pin "25") (pin "26") (pin "27") (pin "28") (pin "29") (pin "3") (pin "30") (pin "31") (pin "32") (pin "33") (pin "34") (pin "35") (pin "36") (pin "37") (pin "38") (pin "39") (pin "40") (pin "41") (pin "42") (pin "43") (pin "44") (pin "45") (pin "46") (pin "47") (pin "48") (pin "49") (pin "50") (pin "51") (pin "52") (pin "53") (pin "6") (pin "7") (pin "8") (pin "9") )
   (no_connect (at 266.7 111.76) )
   (global_label "SAVE.OE~" (shape input) (at 279.4 109.22 0) (fields_autoplaced) (effects (font (size 2.54 2.54) ) (justify left) ) (property "Intersheet References" "${INTERSHEET_REFS}" (id 0) (at 301.2803 109.0613 0) (effects (font (size 2.54 2.54) ) (justify left) ) ) )
@@
   (global_label "EN_MICROS" (shape input) (at 360.68 121.92 180) (fields_autoplaced) (effects (font (size 2.54 2.54) ) (justify right) ) (property "Intersheet References" "${INTERSHEET_REFS}" (id 0) (at 334.6873 121.7613 0) (effects (font (size 2.54 2.54) ) (justify right) ) ) )
   (junction (at 370.84 121.92) (diameter 0) (color 0 0 0 0) )
-  (symbol (lib_id "r1000:F20") (at 396.24 119.38 0) (unit 1) (in_bom yes) (on_board yes) (property "Reference" "U2704" (id 0) (at 404.495 116.84 0) ) (property "Value" "F20" (id 1) (at 395.605 121.92 0) (effects (font (size 2.54 2.54) ) ) ) (property "Footprint" "" (id 2) (at 394.97 119.38 0) (effects (font (size 1.27 1.27) ) hide ) ) (property "Datasheet" "" (id 3) (at 394.97 119.38 0) (effects (font (size 1.27 1.27) ) hide ) ) (property "Location" "K03" (id 4) (at 395.605 116.84 0) (effects (font (size 2.54 2.54) ) ) ) (property "Name" "LMACNB" (id 5) (at 401.32 130.175 0) (effects (font (size 2.54 2.54) ) (justify bottom) ) ) (pin "1") (pin "2") (pin "4") (pin "5") (pin "6") )
+  (symbol (lib_id "r1000:F20") (at 396.24 119.38 0) (unit 1) (in_bom yes) (on_board yes) (property "Reference" "U2704" (id 0) (at 404.495 116.84 0) ) (property "Value" "" (id 1) (at 395.605 121.92 0) (effects (font (size 2.54 2.54) ) ) ) (property "Footprint" "" (id 2) (at 394.97 119.38 0) (effects (font (size 1.27 1.27) ) hide ) ) (property "Datasheet" "" (id 3) (at 394.97 119.38 0) (effects (font (size 1.27 1.27) ) hide ) ) (property "Location" "K03" (id 4) (at 395.605 116.84 0) (effects (font (size 2.54 2.54) ) ) ) (property "Name" "LMACNB" (id 5) (at 401.32 130.175 0) (effects (font (size 2.54 2.54) ) (justify bottom) ) ) (pin "1") (pin "2") (pin "4") (pin "5") (pin "6") )
   (global_label "CHK_EXIT.UE~" (shape output) (at 421.64 119.38 0) (fields_autoplaced) (effects (font (size 2.54 2.54) ) (justify left) ) (property "Intersheet References" "${INTERSHEET_REFS}" (id 0) (at 451.987 119.2213 0) (effects (font (size 2.54 2.54) ) (justify left) ) ) )
 )

Commit message: Recover from KiCad-6 munging
Parts:
- U2701: value (none) -> XREG24
- U2704: value (none) -> F20

Commit message: Fix polarity of unused part of driven FIU bus.
Parts:
- removed U2701: XREG24, symbol r1000:XREG24
- removed U2704: F20, symbol r1000:F20
- added U: (no value), symbol r1000:F20
- added U: (no value), symbol r1000:XREG24
Connections:
- net CHK_EXIT.RND: now also U.1 (D0)
- net CHK_EXIT.UE~: now also U.6 (Q)
- net EN_MICROS: now also U.2 (D1), U.4 (D2)
- net OFFSET_BUS37: now also U.15 (Q4)
- net OFFSET_BUS38: now also U.17 (Q5)
- net OFFSET_BUS39: now also U.19 (Q6)
- net OFFSET_BUS40: now also U.21 (Q7)
- net OFFSET_BUS41: now also U.23 (Q8)
- net OFFSET_BUS42: now also U.25 (Q9)
- net OFFSET_BUS43: now also U.27 (Q10)
- net OFFSET_BUS44: now also U.29 (Q11)
- net OFFSET_BUS45: now also U.31 (Q12)
- net OFFSET_BUS46: now also U.33 (Q13)
- net OFFSET_BUS47: now also U.35 (Q14)
- net OFFSET_BUS48: now also U.37 (Q15)
- net OFFSET_BUS49: now also U.39 (Q16)
- net OFFSET_BUS50: now also U.41 (Q17)
- net OFFSET_BUS51: now also U.43 (Q18)
- net OFFSET_BUS52: now also U.45 (Q19)
- net OFFSET_BUS53: now also U.47 (Q20)
- net OFFSET_BUS54: now also U.49 (Q21)
- net OFFSET_BUS55: now also U.51 (Q22)
- net OFFSET_BUS56: now also U.53 (Q23)
- net RESOLVE_OFFS37: now also U.14 (D4)
- net RESOLVE_OFFS38: now also U.16 (D5)
- net RESOLVE_OFFS39: now also U.18 (D6)
- net RESOLVE_OFFS40: now also U.20 (D7)
- net RESOLVE_OFFS41: now also U.22 (D8)
- net RESOLVE_OFFS42: now also U.24 (D9)
- net RESOLVE_OFFS43: now also U.26 (D10)
- net RESOLVE_OFFS44: now also U.28 (D11)
- net RESOLVE_OFFS45: now also U.30 (D12)
- net RESOLVE_OFFS46: now also U.32 (D13)
- net RESOLVE_OFFS47: now also U.34 (D14)
- net RESOLVE_OFFS48: now also U.36 (D15)
- net RESOLVE_OFFS49: now also U.38 (D16)
- net RESOLVE_OFFS50: now also U.40 (D17)
- net RESOLVE_OFFS51: now also U.42 (D18)
- net RESOLVE_OFFS52: now also U.44 (D19)
- net RESOLVE_OFFS53: now also U.46 (D20)
- net RESOLVE_OFFS54: now also U.48 (D21)
- net RESOLVE_OFFS55: now also U.50 (D22)
- net RESOLVE_OFFS56: now also U.52 (D23)
- net RES_ALU.COUT: now also U.6 (D0)
- net SAVE.CLK~: now also U.1 (CLK)
- net SAVE.OE~: now also U.3 (OE)
- new net: U.5 (D3), U.7 (Q0)
