File: Schematics/SEQ/pg_38.kicad_sch (KiCad schematic)
At the start: 80 parts, among them U3901 F240, U3902 F240, U3903 F240, U3904 F240, U3905 F240, U3906 F240, U3907 F240, U3908 F240, U3909 F240, U3910 F240, U3911 F240, U3912 F240, U3913 F240, U3914 F240, U3915 F240, U3916 F240

Commit message: Use XBUF64 for Type bus
Parts:
- removed U3903, U3904, U3905, U3906, U3907, U3908, U3909, U3910, U3911, U3912, U3913, U3914, U3915, U3916: F240, symbol r1000:F240
- U3901: value F240 -> XBUF64; symbol r1000:F240 -> r1000:XBUF64; Location A45 -> x99; Name TXCVR0 -> TDRV
- U3902: value F240 -> XBUF64; symbol r1000:F240 -> r1000:XBUF64; Location A43 -> x99; Name TXCVR1 -> TRCV
Connections:
- net Q.TYPE.D0: now also U3901.4 (Y0), U3902.3 (I0); no longer U3901.2 (I0), U3901.9 (Y4)
- net Q.TYPE.D1: now also U3901.6 (Y1), U3902.5 (I1); no longer U3901.4 (I1), U3901.7 (Y5)
- net Q.TYPE.D10: now also U3901.24 (Y10), U3902.23 (I10)
- net Q.TYPE.D11: now also U3901.26 (Y11), U3902.25 (I11)
- net Q.TYPE.D12: now also U3901.28 (Y12), U3902.27 (I12)
- net Q.TYPE.D13: now also U3901.30 (Y13), U3902.29 (I13)
- net Q.TYPE.D14: now also U3901.32 (Y14), U3902.31 (I14)
- net Q.TYPE.D15: now also U3901.34 (Y15), U3902.33 (I15)
- net Q.TYPE.D16: now also U3901.36 (Y16), U3902.35 (I16)
- net Q.TYPE.D17: now also U3901.38 (Y17), U3902.37 (I17)
- net Q.TYPE.D18: now also U3901.40 (Y18), U3902.39 (I18)
- net Q.TYPE.D19: now also U3901.42 (Y19), U3902.41 (I19)
- net Q.TYPE.D2: now also U3901.8 (Y2), U3902.7 (I2); no longer U3901.5 (Y6), U3901.6 (I2)
- net Q.TYPE.D20: now also U3901.44 (Y20), U3902.43 (I20)
- net Q.TYPE.D21: now also U3901.46 (Y21), U3902.45 (I21)
- net Q.TYPE.D22: now also U3901.48 (Y22), U3902.47 (I22)
- net Q.TYPE.D23: now also U3901.50 (Y23), U3902.49 (I23)
- net Q.TYPE.D24: now also U3901.52 (Y24), U3902.51 (I24)
- net Q.TYPE.D25: now also U3901.54 (Y25), U3902.53 (I25)
- net Q.TYPE.D26: now also U3901.56 (Y26), U3902.55 (I26)
- net Q.TYPE.D27: now also U3901.58 (Y27), U3902.57 (I27)
- net Q.TYPE.D28: now also U3901.60 (Y28), U3902.59 (I28)
- net Q.TYPE.D29: now also U3901.62 (Y29), U3902.61 (I29)
- net Q.TYPE.D3: now also U3901.10 (Y3), U3902.9 (I3); no longer U3901.3 (Y7), U3901.8 (I3)
- net Q.TYPE.D30: now also U3901.64 (Y30), U3902.63 (I30)
- net Q.TYPE.D31: now also U3901.66 (Y31), U3902.65 (I31)
- net Q.TYPE.D32: now also U3901.68 (Y32), U3902.67 (I32)
- net Q.TYPE.D33: now also U3901.70 (Y33), U3902.69 (I33)
- net Q.TYPE.D34: now also U3901.72 (Y34), U3902.71 (I34)
- net Q.TYPE.D35: now also U3901.74 (Y35), U3902.73 (I35)
- net Q.TYPE.D36: now also U3901.76 (Y36), U3902.75 (I36)
- net Q.TYPE.D37: now also U3901.78 (Y37), U3902.77 (I37)
- net Q.TYPE.D38: now also U3901.80 (Y38), U3902.79 (I38)
- net Q.TYPE.D39: now also U3901.82 (Y39), U3902.81 (I39)
- net Q.TYPE.D4: now also U3901.12 (Y4), U3902.11 (I4); no longer U3902.2 (I0), U3902.9 (Y4)
- net Q.TYPE.D40: now also U3901.84 (Y40), U3902.83 (I40)
- net Q.TYPE.D41: now also U3901.86 (Y41), U3902.85 (I41)
- net Q.TYPE.D42: now also U3901.88 (Y42), U3902.87 (I42)
- net Q.TYPE.D43: now also U3901.90 (Y43), U3902.89 (I43)
- net Q.TYPE.D44: now also U3901.92 (Y44), U3902.91 (I44)
- net Q.TYPE.D45: now also U3901.94 (Y45), U3902.93 (I45)
- net Q.TYPE.D46: now also U3901.96 (Y46), U3902.95 (I46)
- net Q.TYPE.D47: now also U3901.98 (Y47), U3902.97 (I47)
- net Q.TYPE.D48: now also U3901.100 (Y48), U3902.99 (I48)
- net Q.TYPE.D49: now also U3901.102 (Y49), U3902.101 (I49)
- net Q.TYPE.D5: now also U3901.14 (Y5), U3902.13 (I5); no longer U3902.4 (I1), U3902.7 (Y5)
- net Q.TYPE.D50: now also U3901.104 (Y50), U3902.103 (I50)
- net Q.TYPE.D51: now also U3901.106 (Y51), U3902.105 (I51)
- net Q.TYPE.D52: now also U3901.108 (Y52), U3902.107 (I52)
- net Q.TYPE.D53: now also U3901.110 (Y53), U3902.109 (I53)
- net Q.TYPE.D54: now also U3901.112 (Y54), U3902.111 (I54)
- net Q.TYPE.D55: now also U3901.114 (Y55), U3902.113 (I55)
- net Q.TYPE.D56: now also U3901.116 (Y56), U3902.115 (I56)
- net Q.TYPE.D57: now also U3901.118 (Y57), U3902.117 (I57)
- net Q.TYPE.D58: now also U3901.120 (Y58), U3902.119 (I58)
- net Q.TYPE.D59: now also U3901.122 (Y59), U3902.121 (I59)
- net Q.TYPE.D6: now also U3901.16 (Y6), U3902.15 (I6); no longer U3902.5 (Y6), U3902.6 (I2)
- net Q.TYPE.D60: now also U3901.124 (Y60), U3902.123 (I60)
- net Q.TYPE.D61: now also U3901.126 (Y61), U3902.125 (I61)
- net Q.TYPE.D62: now also U3901.128 (Y62), U3902.127 (I62)
- net Q.TYPE.D63: now also U3901.130 (Y63), U3902.129 (I63)
- net Q.TYPE.D7: now also U3901.18 (Y7), U3902.17 (I7); no longer U3902.3 (Y7), U3902.8 (I3)
- net Q.TYPE.D8: now also U3901.20 (Y8), U3902.19 (I8)
- net Q.TYPE.D9: now also U3901.22 (Y9), U3902.21 (I9)
- net TYPE_DRV~: now also U3901.2 (OE); no longer U3901.19 (OE1), U3902.19 (OE1)
- net TYPE_VAL.OE~0: now also U3902.2 (OE); no longer U3901.1 (OE0), U3902.1 (OE0)
- net TYPE~0: now also U3901.3 (I0), U3902.4 (Y0); no longer U3901.11 (I4), U3901.18 (Y0)
- net TYPE~1: now also U3901.5 (I1), U3902.6 (Y1); no longer U3901.13 (I5), U3901.16 (Y1)
- net TYPE~10: now also U3901.23 (I10), U3902.24 (Y10)
- net TYPE~11: now also U3901.25 (I11), U3902.26 (Y11)
- net TYPE~12: now also U3901.27 (I12), U3902.28 (Y12)
- net TYPE~13: now also U3901.29 (I13), U3902.30 (Y13)
- net TYPE~14: now also U3901.31 (I14), U3902.32 (Y14)
- net TYPE~15: now also U3901.33 (I15), U3902.34 (Y15)
- net TYPE~16: now also U3901.35 (I16), U3902.36 (Y16)
- net TYPE~17: now also U3901.37 (I17), U3902.38 (Y17)
- net TYPE~18: now also U3901.39 (I18), U3902.40 (Y18)
- net TYPE~19: now also U3901.41 (I19), U3902.42 (Y19)
- net TYPE~2: now also U3901.7 (I2), U3902.8 (Y2); no longer U3901.14 (Y2), U3901.15 (I6)
- net TYPE~20: now also U3901.43 (I20), U3902.44 (Y20)
- net TYPE~21: now also U3901.45 (I21), U3902.46 (Y21)
- net TYPE~22: now also U3901.47 (I22), U3902.48 (Y22)
- net TYPE~23: now also U3901.49 (I23), U3902.50 (Y23)
- net TYPE~24: now also U3901.51 (I24), U3902.52 (Y24)
- net TYPE~25: now also U3901.53 (I25), U3902.54 (Y25)
- net TYPE~26: now also U3901.55 (I26), U3902.56 (Y26)
- net TYPE~27: now also U3901.57 (I27), U3902.58 (Y27)
- net TYPE~28: now also U3901.59 (I28), U3902.60 (Y28)
- net TYPE~29: now also U3901.61 (I29), U3902.62 (Y29)
- net TYPE~3: now also U3901.9 (I3), U3902.10 (Y3); no longer U3901.12 (Y3), U3901.17 (I7)
- net TYPE~30: now also U3901.63 (I30), U3902.64 (Y30)
- net TYPE~31: now also U3901.65 (I31), U3902.66 (Y31)
- net TYPE~32: now also U3901.67 (I32), U3902.68 (Y32)
- net TYPE~33: now also U3901.69 (I33), U3902.70 (Y33)
- net TYPE~34: now also U3901.71 (I34), U3902.72 (Y34)
- net TYPE~35: now also U3901.73 (I35), U3902.74 (Y35)
- net TYPE~36: now also U3901.75 (I36), U3902.76 (Y36)
- net TYPE~37: now also U3901.77 (I37), U3902.78 (Y37)
- net TYPE~38: now also U3901.79 (I38), U3902.80 (Y38)
- net TYPE~39: now also U3901.81 (I39), U3902.82 (Y39)
- net TYPE~4: now also U3901.11 (I4), U3902.12 (Y4); no longer U3902.11 (I4), U3902.18 (Y0)
- net TYPE~40: now also U3901.83 (I40), U3902.84 (Y40)
- net TYPE~41: now also U3901.85 (I41), U3902.86 (Y41)
- net TYPE~42: now also U3901.87 (I42), U3902.88 (Y42)
- net TYPE~43: now also U3901.89 (I43), U3902.90 (Y43)
- net TYPE~44: now also U3901.91 (I44), U3902.92 (Y44)
- net TYPE~45: now also U3901.93 (I45), U3902.94 (Y45)
- net TYPE~46: now also U3901.95 (I46), U3902.96 (Y46)
- net TYPE~47: now also U3901.97 (I47), U3902.98 (Y47)
- net TYPE~48: now also U3901.99 (I48), U3902.100 (Y48)
- net TYPE~49: now also U3901.101 (I49), U3902.102 (Y49)
- net TYPE~5: now also U3901.13 (I5), U3902.14 (Y5); no longer U3902.13 (I5), U3902.16 (Y1)
- net TYPE~50: now also U3901.103 (I50), U3902.104 (Y50)
- net TYPE~51: now also U3901.105 (I51), U3902.106 (Y51)
- net TYPE~52: now also U3901.107 (I52), U3902.108 (Y52)
- net TYPE~53: now also U3901.109 (I53), U3902.110 (Y53)
- net TYPE~54: now also U3901.111 (I54), U3902.112 (Y54)
- net TYPE~55: now also U3901.113 (I55), U3902.114 (Y55)
- net TYPE~56: now also U3901.115 (I56), U3902.116 (Y56)
- net TYPE~57: now also U3901.117 (I57), U3902.118 (Y57)
- net TYPE~58: now also U3901.119 (I58), U3902.120 (Y58)
- net TYPE~59: now also U3901.121 (I59), U3902.122 (Y59)
- net TYPE~6: now also U3901.15 (I6), U3902.16 (Y6); no longer U3902.14 (Y2), U3902.15 (I6)
- net TYPE~60: now also U3901.123 (I60), U3902.124 (Y60)
- net TYPE~61: now also U3901.125 (I61), U3902.126 (Y61)
- net TYPE~62: now also U3901.127 (I62), U3902.128 (Y62)
- net TYPE~63: now also U3901.129 (I63), U3902.130 (Y63)
- net TYPE~7: now also U3901.17 (I7), U3902.18 (Y7); no longer U3902.12 (Y3), U3902.17 (I7)
- net TYPE~8: now also U3901.19 (I8), U3902.20 (Y8)
- net TYPE~9: now also U3901.21 (I9), U3902.22 (Y9)
- new net PU: U3901.1 (INV), U3902.1 (INV)

Commit message: KiCad 6
Parts:
- GF108, GF110, GF112, GF114, GF12, GF124, GF126, GF128, GF130, GF14, GF16, GF176, GF178, GF18, GF180, GF182, GF192, GF194, GF196, GF198, GF208, GF210, GF212, GF214, GF224, GF226, GF228, GF230, GF240, GF242, GF244, GF246, GF256, GF258, GF260, GF262, GF272, GF274, GF276, GF278, GF28, GF288, GF290, GF292, GF294, GF30, GF32, GF34, GF44, GF46, GF48, GF50, GF60, GF62, GF64, GF66, GF76, GF78, GF80, GF82, GF92, GF94, GF96, GF98: value GF -> (none)
- U3901, U3902: value XBUF64 -> (none)

Commit message: Recover from KiCad-6 munging
Parts:
- GF108, GF110, GF112, GF114, GF12, GF124, GF126, GF128, GF130, GF14, GF16, GF176, GF178, GF18, GF180, GF182, GF192, GF194, GF196, GF198, GF208, GF210, GF212, GF214, GF224, GF226, GF228, GF230, GF240, GF242, GF244, GF246, GF256, GF258, GF260, GF262, GF272, GF274, GF276, GF278, GF28, GF288, GF290, GF292, GF294, GF30, GF32, GF34, GF44, GF46, GF48, GF50, GF60, GF62, GF64, GF66, GF76, GF78, GF80, GF82, GF92, GF94, GF96, GF98: value (none) -> GF
- U3901, U3902: value (none) -> XBUF64

Commit message: Fix 0/8 misreading
Connections:
- net PU renamed PD
Changed lines of the file:
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@@
   (wire (pts (xy 111.76 91.44) (xy 86.36 91.44) ) )
   (wire (pts (xy 111.76 96.52) (xy 86.36 96.52) ) )
+  (wire (pts (xy 119.38 17.78) (xy 124.46 17.78) ) )
   (wire (pts (xy 124.46 17.78) (xy 124.46 20.32) ) )
   (wire (pts (xy 134.62 17.78) (xy 134.62 20.32) ) )
@@
   (wire (pts (xy 233.68 91.44) (xy 264.16 91.44) ) )
   (wire (pts (xy 233.68 96.52) (xy 264.16 96.52) ) )
+  (wire (pts (xy 271.78 17.78) (xy 276.86 17.78) ) )
   (wire (pts (xy 276.86 17.78) (xy 276.86 20.32) ) )
   (wire (pts (xy 287.02 17.78) (xy 287.02 20.32) ) )
@@
   (label "TYPE~62" (at 91.44 350.52 0) (effects (font (size 2.54 2.54) ) (justify left bottom) ) )
   (label "TYPE~63" (at 91.44 355.6 0) (effects (font (size 2.54 2.54) ) (justify left bottom) ) )
-  (symbol (lib_id "r1000:PU") (at 124.46 17.78 0) (unit 1) (in_bom yes) (on_board yes) (property "Reference" "#PWR03901" (id 0) (at 124.46 17.78 0) (effects (font (size 1.27 1.27) ) hide ) ) (property "Value" "PU" (id 1) (at 124.46 17.78 0) (effects (font (size 1.27 1.27) ) hide ) ) (property "Footprint" "" (id 2) (at 124.46 17.78 0) (effects (font (size 1.27 1.27) ) hide ) ) (property "Datasheet" "" (id 3) (at 124.46 17.78 0) (effects (font (size 1.27 1.27) ) hide ) ) (pin "1") )
+  (symbol (lib_id "r1000:PD") (at 119.38 17.78 0) (unit 1) (in_bom no) (on_board yes) (property "Reference" "#PWR03901" (id 0) (at 119.38 17.78 0) (effects (font (size 1.27 1.27) ) hide ) ) (property "Value" "PD" (id 1) (at 119.38 17.78 0) (effects (font (size 1.27 1.27) ) hide ) ) (property "Footprint" "" (id 2) (at 119.38 17.78 0) (effects (font (size 1.27 1.27) ) hide ) ) (property "Datasheet" "" (id 3) (at 119.38 17.78 0) (effects (font (size 1.27 1.27) ) hide ) ) (pin "1") )
   (symbol (lib_id "r1000:XBUF64") (at 127 353.06 0) (unit 1) (in_bom yes) (on_board yes) (property "Reference" "U3901" (id 0) (at 129.54 347.98 0) (effects (font (size 1.27 1.27) ) ) ) (property "Value" "XBUF64" (id 1) (at 123.19 358.14 0) (effects (font (size 2.54 2.54) ) (justify left) ) ) (property "Footprint" "" (id 2) (at 128.27 354.33 0) (effects (font (size 1.27 1.27) ) hide ) ) (property "Datasheet" "" (id 3) (at 128.27 354.33 0) (effects (font (size 1.27 1.27) ) hide ) ) (property "Location" "x99" (id 4) (at 125.73 353.06 0) (effects (font (size 2.54 2.54) ) (justify left) ) ) (property "Name" "TDRV" (id 5) (at 130.81 365.76 0) (effects (font (size 2.54 2.54) ) (justify bottom) ) ) (pin "1") (pin "10") (pin "100") (pin "101") (pin "102") (pin "103") (pin "104") (pin "105") (pin "106") (pin "107") (pin "108") (pin "109") (pin "11") (pin "110") (pin "111") (pin "112") (pin "113") (pin "114") (pin "115") (pin "116") (pin "117") (pin "118") (pin "119") (pin "12") (pin "120") (pin "121") (pin "122") (pin "123") (pin "124") (pin "125") (pin "126") (pin "127") (pin "128") (pin "129") (pin "13") (pin "130") (pin "14") (pin "15") (pin "16") (pin "17") (pin "18") (pin "19") (pin "2") (pin "20") (pin "21") (pin "22") (pin "23") (pin "24") (pin "25") (pin "26") (pin "27") (pin "28") (pin "29") (pin "3") (pin "30") (pin "31") (pin "32") (pin "33") (pin "34") (pin "35") (pin "36") (pin "37") (pin "38") (pin "39") (pin "4") (pin "40") (pin "41") (pin "42") (pin "43") (pin "44") (pin "45") (pin "46") (pin "47") (pin "48") (pin "49") (pin "5") (pin "50") (pin "51") (pin "52") (pin "53") (pin "54") (pin "55") (pin "56") (pin "57") (pin "58") (pin "59") (pin "6") (pin "60") (pin "61") (pin "62") (pin "63") (pin "64") (pin "65") (pin "66") (pin "67") (pin "68") (pin "69") (pin "7") (pin "70") (pin "71") (pin "72") (pin "73") (pin "74") (pin "75") (pin "76") (pin "77") (pin "78") (pin "79") (pin "8") (pin "80") (pin "81") (pin "82") (pin "83") (pin "84") (pin "85") (pin "86") (pin "87") (pin "88") (pin "89") (pin "9") (pin "90") (pin "91") (pin "92") (pin "93") (pin "94") (pin "95") (pin "96") (pin "97") (pin "98") (pin "99") )
   (global_label "TYPE_DRV~" (shape input) (at 139.7 17.78 0) (fields_autoplaced) (effects (font (size 2.54 2.54) ) (justify left) ) (property "Intersheet References" "${INTERSHEET_REFS}" (id 0) (at 164.4831 17.6213 0) (effects (font (size 1.905 1.905) ) (justify left) ) ) )
@@
   (label "Q.TYPE.D62" (at 238.76 350.52 0) (effects (font (size 2.54 2.54) ) (justify left bottom) ) )
   (label "Q.TYPE.D63" (at 238.76 355.6 0) (effects (font (size 2.54 2.54) ) (justify left bottom) ) )
-  (symbol (lib_id "r1000:PU") (at 276.86 17.78 0) (unit 1) (in_bom yes) (on_board yes) (property "Reference" "#PWR03902" (id 0) (at 276.86 17.78 0) (effects (font (size 1.27 1.27) ) hide ) ) (property "Value" "PU" (id 1) (at 276.86 17.78 0) (effects (font (size 1.27 1.27) ) hide ) ) (property "Footprint" "" (id 2) (at 276.86 17.78 0) (effects (font (size 1.27 1.27) ) hide ) ) (property "Datasheet" "" (id 3) (at 276.86 17.78 0) (effects (font (size 1.27 1.27) ) hide ) ) (pin "1") )
+  (symbol (lib_id "r1000:PD") (at 271.78 17.78 0) (unit 1) (in_bom no) (on_board yes) (property "Reference" "#PWR03902" (id 0) (at 271.78 17.78 0) (effects (font (size 1.27 1.27) ) hide ) ) (property "Value" "PD" (id 1) (at 271.78 17.78 0) (effects (font (size 1.27 1.27) ) hide ) ) (property "Footprint" "" (id 2) (at 271.78 17.78 0) (effects (font (size 1.27 1.27) ) hide ) ) (property "Datasheet" "" (id 3) (at 271.78 17.78 0) (effects (font (size 1.27 1.27) ) hide ) ) (pin "1") )
   (symbol (lib_id "r1000:XBUF64") (at 279.4 353.06 0) (unit 1) (in_bom yes) (on_board yes) (property "Reference" "U3902" (id 0) (at 281.94 347.98 0) (effects (font (size 1.27 1.27) ) ) ) (property "Value" "XBUF64" (id 1) (at 275.59 358.14 0) (effects (font (size 2.54 2.54) ) (justify left) ) ) (property "Footprint" "" (id 2) (at 280.67 354.33 0) (effects (font (size 1.27 1.27) ) hide ) ) (property "Datasheet" "" (id 3) (at 280.67 354.33 0) (effects (font (size 1.27 1.27) ) hide ) ) (property "Location" "x99" (id 4) (at 278.13 353.06 0) (effects (font (size 2.54 2.54) ) (justify left) ) ) (property "Name" "TRCV" (id 5) (at 283.21 365.76 0) (effects (font (size 2.54 2.54) ) (justify bottom) ) ) (pin "1") (pin "10") (pin "100") (pin "101") (pin "102") (pin "103") (pin "104") (pin "105") (pin "106") (pin "107") (pin "108") (pin "109") (pin "11") (pin "110") (pin "111") (pin "112") (pin "113") (pin "114") (pin "115") (pin "116") (pin "117") (pin "118") (pin "119") (pin "12") (pin "120") (pin "121") (pin "122") (pin "123") (pin "124") (pin "125") (pin "126") (pin "127") (pin "128") (pin "129") (pin "13") (pin "130") (pin "14") (pin "15") (pin "16") (pin "17") (pin "18") (pin "19") (pin "2") (pin "20") (pin "21") (pin "22") (pin "23") (pin "24") (pin "25") (pin "26") (pin "27") (pin "28") (pin "29") (pin "3") (pin "30") (pin "31") (pin "32") (pin "33") (pin "34") (pin "35") (pin "36") (pin "37") (pin "38") (pin "39") (pin "4") (pin "40") (pin "41") (pin "42") (pin "43") (pin "44") (pin "45") (pin "46") (pin "47") (pin "48") (pin "49") (pin "5") (pin "50") (pin "51") (pin "52") (pin "53") (pin "54") (pin "55") (pin "56") (pin "57") (pin "58") (pin "59") (pin "6") (pin "60") (pin "61") (pin "62") (pin "63") (pin "64") (pin "65") (pin "66") (pin "67") (pin "68") (pin "69") (pin "7") (pin "70") (pin "71") (pin "72") (pin "73") (pin "74") (pin "75") (pin "76") (pin "77") (pin "78") (pin "79") (pin "8") (pin "80") (pin "81") (pin "82") (pin "83") (pin "84") (pin "85") (pin "86") (pin "87") (pin "88") (pin "89") (pin "9") (pin "90") (pin "91") (pin "92") (pin "93") (pin "94") (pin "95") (pin "96") (pin "97") (pin "98") (pin "99") )
   (global_label "TYPE_VAL.OE~0" (shape input) (at 292.1 17.78 0) (fields_autoplaced) (effects (font (size 2.54 2.54) ) (justify left) ) (property "Intersheet References" "${INTERSHEET_REFS}" (id 0) (at 324.6241 17.6213 0) (effects (font (size 1.905 1.905) ) (justify left) ) ) )

Commit message: Fix polarity of unused part of driven FIU bus.
Parts:
- removed GF108, GF110, GF112, GF114, GF12, GF124, GF126, GF128, GF130, GF14, GF16, GF176, GF178, GF18, GF180, GF182, GF192, GF194, GF196, GF198, GF208, GF210, GF212, GF214, GF224, GF226, GF228, GF230, GF240, GF242, GF244, GF246, GF256, GF258, GF260, GF262, GF272, GF274, GF276, GF278, GF28, GF288, GF290, GF292, GF294, GF30, GF32, GF34, GF44, GF46, GF48, GF50, GF60, GF62, GF64, GF66, GF76, GF78, GF80, GF82, GF92, GF94, GF96, GF98: GF, symbol r1000:GF
- removed U3901, U3902: XBUF64, symbol r1000:XBUF64
- added U (x64): (no value), symbol r1000:GF
- added U (x2): (no value), symbol r1000:XBUF64
Connections:
- net PD: now also U.1 (INV), U.1 (INV)
- net Q.TYPE.D0: now also U.1, U.3 (I0), U.4 (Y0)
- net Q.TYPE.D1: now also U.1, U.5 (I1), U.6 (Y1)
- net Q.TYPE.D10: now also U.1, U.23 (I10), U.24 (Y10)
- net Q.TYPE.D11: now also U.1, U.25 (I11), U.26 (Y11)
- net Q.TYPE.D12: now also U.1, U.27 (I12), U.28 (Y12)
- net Q.TYPE.D13: now also U.1, U.29 (I13), U.30 (Y13)
- net Q.TYPE.D14: now also U.1, U.31 (I14), U.32 (Y14)
- net Q.TYPE.D15: now also U.1, U.33 (I15), U.34 (Y15)
- net Q.TYPE.D16: now also U.1, U.35 (I16), U.36 (Y16)
- net Q.TYPE.D17: now also U.1, U.37 (I17), U.38 (Y17)
- net Q.TYPE.D18: now also U.1, U.39 (I18), U.40 (Y18)
- net Q.TYPE.D19: now also U.1, U.41 (I19), U.42 (Y19)
- net Q.TYPE.D2: now also U.1, U.7 (I2), U.8 (Y2)
- net Q.TYPE.D20: now also U.1, U.43 (I20), U.44 (Y20)
- net Q.TYPE.D21: now also U.1, U.45 (I21), U.46 (Y21)
- net Q.TYPE.D22: now also U.1, U.47 (I22), U.48 (Y22)
- net Q.TYPE.D23: now also U.1, U.49 (I23), U.50 (Y23)
- net Q.TYPE.D24: now also U.1, U.51 (I24), U.52 (Y24)
- net Q.TYPE.D25: now also U.1, U.53 (I25), U.54 (Y25)
- net Q.TYPE.D26: now also U.1, U.55 (I26), U.56 (Y26)
- net Q.TYPE.D27: now also U.1, U.57 (I27), U.58 (Y27)
- net Q.TYPE.D28: now also U.1, U.59 (I28), U.60 (Y28)
- net Q.TYPE.D29: now also U.1, U.61 (I29), U.62 (Y29)
- net Q.TYPE.D3: now also U.1, U.10 (Y3), U.9 (I3)
- net Q.TYPE.D30: now also U.1, U.63 (I30), U.64 (Y30)
- net Q.TYPE.D31: now also U.1, U.65 (I31), U.66 (Y31)
- net Q.TYPE.D32: now also U.1, U.67 (I32), U.68 (Y32)
- net Q.TYPE.D33: now also U.1, U.69 (I33), U.70 (Y33)
- net Q.TYPE.D34: now also U.1, U.71 (I34), U.72 (Y34)
- net Q.TYPE.D35: now also U.1, U.73 (I35), U.74 (Y35)
- net Q.TYPE.D36: now also U.1, U.75 (I36), U.76 (Y36)
- net Q.TYPE.D37: now also U.1, U.77 (I37), U.78 (Y37)
- net Q.TYPE.D38: now also U.1, U.79 (I38), U.80 (Y38)
- net Q.TYPE.D39: now also U.1, U.81 (I39), U.82 (Y39)
- net Q.TYPE.D4: now also U.1, U.11 (I4), U.12 (Y4)
- net Q.TYPE.D40: now also U.1, U.83 (I40), U.84 (Y40)
- net Q.TYPE.D41: now also U.1, U.85 (I41), U.86 (Y41)
- net Q.TYPE.D42: now also U.1, U.87 (I42), U.88 (Y42)
- net Q.TYPE.D43: now also U.1, U.89 (I43), U.90 (Y43)
- net Q.TYPE.D44: now also U.1, U.91 (I44), U.92 (Y44)
- net Q.TYPE.D45: now also U.1, U.93 (I45), U.94 (Y45)
- net Q.TYPE.D46: now also U.1, U.95 (I46), U.96 (Y46)
- net Q.TYPE.D47: now also U.1, U.97 (I47), U.98 (Y47)
- net Q.TYPE.D48: now also U.1, U.100 (Y48), U.99 (I48)
- net Q.TYPE.D49: now also U.1, U.101 (I49), U.102 (Y49)
- net Q.TYPE.D5: now also U.1, U.13 (I5), U.14 (Y5)
- net Q.TYPE.D50: now also U.1, U.103 (I50), U.104 (Y50)
- net Q.TYPE.D51: now also U.1, U.105 (I51), U.106 (Y51)
- net Q.TYPE.D52: now also U.1, U.107 (I52), U.108 (Y52)
- net Q.TYPE.D53: now also U.1, U.109 (I53), U.110 (Y53)
- net Q.TYPE.D54: now also U.1, U.111 (I54), U.112 (Y54)
- net Q.TYPE.D55: now also U.1, U.113 (I55), U.114 (Y55)
- net Q.TYPE.D56: now also U.1, U.115 (I56), U.116 (Y56)
- net Q.TYPE.D57: now also U.1, U.117 (I57), U.118 (Y57)
- net Q.TYPE.D58: now also U.1, U.119 (I58), U.120 (Y58)
- net Q.TYPE.D59: now also U.1, U.121 (I59), U.122 (Y59)
- net Q.TYPE.D6: now also U.1, U.15 (I6), U.16 (Y6)
- net Q.TYPE.D60: now also U.1, U.123 (I60), U.124 (Y60)
- net Q.TYPE.D61: now also U.1, U.125 (I61), U.126 (Y61)
- net Q.TYPE.D62: now also U.1, U.127 (I62), U.128 (Y62)
- net Q.TYPE.D63: now also U.1, U.129 (I63), U.130 (Y63)
- net Q.TYPE.D7: now also U.1, U.17 (I7), U.18 (Y7)
- net Q.TYPE.D8: now also U.1, U.19 (I8), U.20 (Y8)
- net Q.TYPE.D9: now also U.1, U.21 (I9), U.22 (Y9)
- net TYPE_DRV~: now also U.2 (OE)
- net TYPE_VAL.OE~0: now also U.2 (OE)
- net TYPE~0: now also U.3 (I0), U.4 (Y0)
- net TYPE~1: now also U.5 (I1), U.6 (Y1)
- net TYPE~10: now also U.23 (I10), U.24 (Y10)
- net TYPE~11: now also U.25 (I11), U.26 (Y11)
- net TYPE~12: now also U.27 (I12), U.28 (Y12)
- net TYPE~13: now also U.29 (I13), U.30 (Y13)
- net TYPE~14: now also U.31 (I14), U.32 (Y14)
- net TYPE~15: now also U.33 (I15), U.34 (Y15)
- net TYPE~16: now also U.35 (I16), U.36 (Y16)
- net TYPE~17: now also U.37 (I17), U.38 (Y17)
- net TYPE~18: now also U.39 (I18), U.40 (Y18)
- net TYPE~19: now also U.41 (I19), U.42 (Y19)
- net TYPE~2: now also U.7 (I2), U.8 (Y2)
- net TYPE~20: now also U.43 (I20), U.44 (Y20)
- net TYPE~21: now also U.45 (I21), U.46 (Y21)
- net TYPE~22: now also U.47 (I22), U.48 (Y22)
- net TYPE~23: now also U.49 (I23), U.50 (Y23)
- net TYPE~24: now also U.51 (I24), U.52 (Y24)
- net TYPE~25: now also U.53 (I25), U.54 (Y25)
- net TYPE~26: now also U.55 (I26), U.56 (Y26)
- net TYPE~27: now also U.57 (I27), U.58 (Y27)
- net TYPE~28: now also U.59 (I28), U.60 (Y28)
- net TYPE~29: now also U.61 (I29), U.62 (Y29)
- net TYPE~3: now also U.10 (Y3), U.9 (I3)
- net TYPE~30: now also U.63 (I30), U.64 (Y30)
- net TYPE~31: now also U.65 (I31), U.66 (Y31)
- net TYPE~32: now also U.67 (I32), U.68 (Y32)
- net TYPE~33: now also U.69 (I33), U.70 (Y33)
- net TYPE~34: now also U.71 (I34), U.72 (Y34)
- net TYPE~35: now also U.73 (I35), U.74 (Y35)
- net TYPE~36: now also U.75 (I36), U.76 (Y36)
- net TYPE~37: now also U.77 (I37), U.78 (Y37)
- net TYPE~38: now also U.79 (I38), U.80 (Y38)
- net TYPE~39: now also U.81 (I39), U.82 (Y39)
- net TYPE~4: now also U.11 (I4), U.12 (Y4)
- net TYPE~40: now also U.83 (I40), U.84 (Y40)
- net TYPE~41: now also U.85 (I41), U.86 (Y41)
- net TYPE~42: now also U.87 (I42), U.88 (Y42)
- net TYPE~43: now also U.89 (I43), U.90 (Y43)
- net TYPE~44: now also U.91 (I44), U.92 (Y44)
- net TYPE~45: now also U.93 (I45), U.94 (Y45)
- net TYPE~46: now also U.95 (I46), U.96 (Y46)
- net TYPE~47: now also U.97 (I47), U.98 (Y47)
- net TYPE~48: now also U.100 (Y48), U.99 (I48)
- net TYPE~49: now also U.101 (I49), U.102 (Y49)
- net TYPE~5: now also U.13 (I5), U.14 (Y5)
- net TYPE~50: now also U.103 (I50), U.104 (Y50)
- net TYPE~51: now also U.105 (I51), U.106 (Y51)
- net TYPE~52: now also U.107 (I52), U.108 (Y52)
- net TYPE~53: now also U.109 (I53), U.110 (Y53)
- net TYPE~54: now also U.111 (I54), U.112 (Y54)
- net TYPE~55: now also U.113 (I55), U.114 (Y55)
- net TYPE~56: now also U.115 (I56), U.116 (Y56)
- net TYPE~57: now also U.117 (I57), U.118 (Y57)
- net TYPE~58: now also U.119 (I58), U.120 (Y58)
- net TYPE~59: now also U.121 (I59), U.122 (Y59)
- net TYPE~6: now also U.15 (I6), U.16 (Y6)
- net TYPE~60: now also U.123 (I60), U.124 (Y60)
- net TYPE~61: now also U.125 (I61), U.126 (Y61)
- net TYPE~62: now also U.127 (I62), U.128 (Y62)
- net TYPE~63: now also U.129 (I63), U.130 (Y63)
- net TYPE~7: now also U.17 (I7), U.18 (Y7)
- net TYPE~8: now also U.19 (I8), U.20 (Y8)
- net TYPE~9: now also U.21 (I9), U.22 (Y9)
