File: Schematics/SEQ/pg_61.kicad_sch (KiCad schematic)
At the start: 18 parts, among them U6201 F04, U6202 F51, U6203 XREG16, U6204 F258, U6205 F258, U6208 F258, U6209 F258, U6212 F258, U6213 F258, U6216 F258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

Commit message: Much SEQ polishing
Parts:
- added U6206: F138, symbol r1000:F138
- added U6207, U6210, U6211, U6214: XBUF16, symbol r1000:XBUF16
- U6203: Name TOS -> TOPSTK
Connections:
- net BRNCH_ADR.UIR0: now also U6210.7 (I2)
- net BRNCH_ADR.UIR1: now also U6210.9 (I3)
- net BRNCH_ADR.UIR10: now also U6210.27 (I12)
- net BRNCH_ADR.UIR11: now also U6210.29 (I13)
- net BRNCH_ADR.UIR12: now also U6210.31 (I14)
- net BRNCH_ADR.UIR13: now also U6210.33 (I15)
- net BRNCH_ADR.UIR2: now also U6210.11 (I4)
- net BRNCH_ADR.UIR3: now also U6210.13 (I5)
- net BRNCH_ADR.UIR4: now also U6210.15 (I6)
- net BRNCH_ADR.UIR5: now also U6210.17 (I7)
- net BRNCH_ADR.UIR6: now also U6210.19 (I8)
- net BRNCH_ADR.UIR7: now also U6210.21 (I9)
- net BRNCH_ADR.UIR8: now also U6210.23 (I10)
- net BRNCH_ADR.UIR9: now also U6210.25 (I11)
- net CUR_UADR0: now also U6211.7 (I2)
- net CUR_UADR1: now also U6211.9 (I3)
- net CUR_UADR10: now also U6211.27 (I12)
- net CUR_UADR11: now also U6211.29 (I13)
- net CUR_UADR12: now also U6211.31 (I14)
- net CUR_UADR13: now also U6211.33 (I15)
- net CUR_UADR2: now also U6211.11 (I4)
- net CUR_UADR3: now also U6211.13 (I5)
- net CUR_UADR4: now also U6211.15 (I6)
- net CUR_UADR5: now also U6211.17 (I7)
- net CUR_UADR6: now also U6211.19 (I8)
- net CUR_UADR7: now also U6211.21 (I9)
- net CUR_UADR8: now also U6211.23 (I10)
- net CUR_UADR9: now also U6211.25 (I11)
- net C_UADR_ONE0: now also U6214.7 (I2)
- net C_UADR_ONE1: now also U6214.9 (I3)
- net C_UADR_ONE10: now also U6214.27 (I12)
- net C_UADR_ONE11: now also U6214.29 (I13)
- net C_UADR_ONE12: now also U6214.31 (I14)
- net C_UADR_ONE13: now also U6214.33 (I15)
- net C_UADR_ONE2: now also U6214.11 (I4)
- net C_UADR_ONE3: now also U6214.13 (I5)
- net C_UADR_ONE4: now also U6214.15 (I6)
- net C_UADR_ONE5: now also U6214.17 (I7)
- net C_UADR_ONE6: now also U6214.19 (I8)
- net C_UADR_ONE7: now also U6214.21 (I9)
- net C_UADR_ONE8: now also U6214.23 (I10)
- net C_UADR_ONE9: now also U6214.25 (I11)
- net FIU.IN~48: now also U6207.3 (I0)
- net FIU.IN~49: now also U6207.5 (I1)
- net FIU.IN~50: now also U6207.7 (I2)
- net FIU.IN~51: now also U6207.9 (I3)
- net FIU.IN~52: now also U6207.11 (I4)
- net FIU.IN~53: now also U6207.13 (I5)
- net FIU.IN~54: now also U6207.15 (I6)
- net FIU.IN~55: now also U6207.17 (I7)
- net FIU.IN~56: now also U6207.19 (I8)
- net FIU.IN~57: now also U6207.21 (I9)
- net FIU.IN~58: now also U6207.23 (I10)
- net FIU.IN~59: now also U6207.25 (I11)
- net FIU.IN~60: now also U6207.27 (I12)
- net FIU.IN~61: now also U6207.29 (I13)
- net FIU.IN~62: now also U6207.31 (I14)
- net FIU.IN~63: now also U6207.33 (I15)
- net H2: now also U6206.6 (D0); no longer U6222.1 (D0), U6224.1 (D0)
- net LATCHED_COND: now also U6210.5 (I1), U6211.5 (I1), U6214.5 (I1)
- net PD: now also U6222.1 (D0), U6224.1 (D0), U6206.3 (S0), U6206.5 (D2), U6207.1 (INV), U6210.1 (INV), U6211.1 (INV), U6214.1 (INV)
- net Q3_COND: now also U6210.3 (I0), U6211.3 (I0), U6214.3 (I0)
- net STACK_INP.SEL0: now also U6206.2 (S1)
- net STACK_INP.SEL1: now also U6206.1 (S2)
- net STKD0: now also U6207.4 (Y0), U6210.4 (Y0), U6211.4 (Y0), U6214.4 (Y0)
- net STKD1: now also U6207.6 (Y1), U6210.6 (Y1), U6211.6 (Y1), U6214.6 (Y1)
- net STKD10: now also U6207.24 (Y10), U6210.24 (Y10), U6211.24 (Y10), U6214.24 (Y10)
- net STKD11: now also U6207.26 (Y11), U6210.26 (Y11), U6211.26 (Y11), U6214.26 (Y11)
- net STKD12: now also U6207.28 (Y12), U6210.28 (Y12), U6211.28 (Y12), U6214.28 (Y12)
- net STKD13: now also U6207.30 (Y13), U6210.30 (Y13), U6211.30 (Y13), U6214.30 (Y13)
- net STKD14: now also U6207.32 (Y14), U6210.32 (Y14), U6211.32 (Y14), U6214.32 (Y14)
- net STKD15: now also U6207.34 (Y15), U6210.34 (Y15), U6211.34 (Y15), U6214.34 (Y15)
- net STKD2: now also U6207.8 (Y2), U6210.8 (Y2), U6211.8 (Y2), U6214.8 (Y2)
- net STKD3: now also U6207.10 (Y3), U6210.10 (Y3), U6211.10 (Y3), U6214.10 (Y3)
- net STKD4: now also U6207.12 (Y4), U6210.12 (Y4), U6211.12 (Y4), U6214.12 (Y4)
- net STKD5: now also U6207.14 (Y5), U6210.14 (Y5), U6211.14 (Y5), U6214.14 (Y5)
- net STKD6: now also U6207.16 (Y6), U6210.16 (Y6), U6211.16 (Y6), U6214.16 (Y6)
- net STKD7: now also U6207.18 (Y7), U6210.18 (Y7), U6211.18 (Y7), U6214.18 (Y7)
- net STKD8: now also U6207.20 (Y8), U6210.20 (Y8), U6211.20 (Y8), U6214.20 (Y8)
- net STKD9: now also U6207.22 (Y9), U6210.22 (Y9), U6211.22 (Y9), U6214.22 (Y9)
- net WRITE~: now also U6206.4 (D1)
- new net STIN.0: U6206.15 (Y0_), U6210.2 (OE)
- new net STIN.1: U6206.14 (Y1_), U6207.2 (OE)
- new net STIN.2: U6206.13 (Y2_), U6214.2 (OE)
- new net STIN.3: U6206.12 (Y3_), U6211.2 (OE)
- no-connect marks 0 -> 4
Other:
- moved on the sheet: U6201, U6202, U6203, U6204, U6205, U6208, U6209, U6212, U6213, U6216, U6217, U6219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

Commit message: Much work on SEQ
Parts:
- removed U6204, U6205, U6208, U6209, U6212, U6213, U6216, U6217: F258, symbol r1000:F258
- removed U6219, U6220: F04, symbol r1000:F04
- removed U6221, U6223: F02, symbol r1000:F02
- removed U6222, U6224: F00, symbol r1000:F00

Commit message: KiCad 6
Parts:
- U6201: value F04 -> (none)
- U6202: value F51 -> (none)
- U6203: value XREG16 -> (none)
- U6206: value F138 -> (none)
- U6207, U6210, U6211, U6214: value XBUF16 -> (none)
- U6225: value XSTKRAM -> (none)

Commit message: Recover from KiCad-6 munging
Parts:
- U6201: value (none) -> F04
- U6202: value (none) -> F51
- U6203: value (none) -> XREG16
- U6206: value (none) -> F138
- U6207, U6210, U6211, U6214: value (none) -> XBUF16
- U6225: value (none) -> XSTKRAM

Commit message: Snapshot, much IOC polishing
Connections:
- net Q2~: now also U6225.1 (WE); no longer U6225.33 (WE)
- net SAVED_LATCHED: now also U6225.5 (D1); no longer U6225.2 (D1)
- net STACK_OUT.SPARE: now also U6225.3 (D0); no longer U6225.1 (D0)
- net STKD0: now also U6225.4 (Q0); no longer U6225.17 (Q0)
- net STKD1: now also U6225.6 (Q1); no longer U6225.18 (Q1)
- net STKD10: now also U6225.24 (Q10); no longer U6225.27 (Q10)
- net STKD11: now also U6225.26 (Q11); no longer U6225.28 (Q11)
- net STKD12: now also U6225.28 (Q12); no longer U6225.29 (Q12)
- net STKD14: now also U6225.32 (Q14); no longer U6225.31 (Q14)
- net STKD15: now also U6225.34 (Q15); no longer U6225.32 (Q15)
- net STKD2: now also U6225.8 (Q2); no longer U6225.19 (Q2)
- net STKD3: now also U6225.10 (Q3); no longer U6225.20 (Q3)
- net STKD4: now also U6225.12 (Q4); no longer U6225.21 (Q4)
- net STKD5: now also U6225.14 (Q5); no longer U6225.22 (Q5)
- net STKD6: now also U6225.16 (Q6); no longer U6225.23 (Q6)
- net STKD7: now also U6225.18 (Q7); no longer U6225.24 (Q7)
- net STKD8: now also U6225.20 (Q8); no longer U6225.25 (Q8)
- net STKD9: now also U6225.22 (Q9); no longer U6225.26 (Q9)
- net TOP_USTACK0: now also U6225.7 (D2); no longer U6225.3 (D2)
- net TOP_USTACK1: now also U6225.9 (D3); no longer U6225.4 (D3)
- net TOP_USTACK10: now also U6225.27 (D12); no longer U6225.13 (D12)
- net TOP_USTACK11: now also U6225.29 (D13); no longer U6225.14 (D13)
- net TOP_USTACK12: now also U6225.31 (D14); no longer U6225.15 (D14)
- net TOP_USTACK13: now also U6225.33 (D15); no longer U6225.16 (D15)
- net TOP_USTACK2: now also U6225.11 (D4); no longer U6225.5 (D4)
- net TOP_USTACK3: now also U6225.13 (D5); no longer U6225.6 (D5)
- net TOP_USTACK4: now also U6225.15 (D6); no longer U6225.7 (D6)
- net TOP_USTACK5: now also U6225.17 (D7); no longer U6225.8 (D7)
- net TOP_USTACK6: now also U6225.19 (D8); no longer U6225.9 (D8)
- net TOP_USTACK7: now also U6225.21 (D9); no longer U6225.10 (D9)
- net TOP_USTACK8: now also U6225.23 (D10); no longer U6225.11 (D10)
- net TOP_USTACK9: now also U6225.25 (D11); no longer U6225.12 (D11)
- net at U6202.7 (Q): now also U6225.2 (CS); no longer U6225.34 (CS)

Commit message: Fix polarity of unused part of driven FIU bus.
Parts:
- removed U6201: F04, symbol r1000:F04
- removed U6202: F51, symbol r1000:F51
- removed U6203: XREG16, symbol r1000:XREG16
- removed U6206: F138, symbol r1000:F138
- removed U6207, U6210, U6211, U6214: XBUF16, symbol r1000:XBUF16
- removed U6225: XSTKRAM, symbol r1000:XSTKRAM
- added U (x4): (no value), symbol r1000:XBUF16
- added U: (no value), symbol r1000:F04
- added U: (no value), symbol r1000:XSTKRAM
- added U: (no value), symbol r1000:XREG16
- added U: (no value), symbol r1000:F51
- added U: (no value), symbol r1000:F138
Connections:
- net BRNCH_ADR.UIR0: now also U.7 (I2)
- net BRNCH_ADR.UIR1: now also U.9 (I3)
- net BRNCH_ADR.UIR10: now also U.27 (I12)
- net BRNCH_ADR.UIR11: now also U.29 (I13)
- net BRNCH_ADR.UIR12: now also U.31 (I14)
- net BRNCH_ADR.UIR13: now also U.33 (I15)
- net BRNCH_ADR.UIR2: now also U.11 (I4)
- net BRNCH_ADR.UIR3: now also U.13 (I5)
- net BRNCH_ADR.UIR4: now also U.15 (I6)
- net BRNCH_ADR.UIR5: now also U.17 (I7)
- net BRNCH_ADR.UIR6: now also U.19 (I8)
- net BRNCH_ADR.UIR7: now also U.21 (I9)
- net BRNCH_ADR.UIR8: now also U.23 (I10)
- net BRNCH_ADR.UIR9: now also U.25 (I11)
- net CUR_UADR0: now also U.7 (I2)
- net CUR_UADR1: now also U.9 (I3)
- net CUR_UADR10: now also U.27 (I12)
- net CUR_UADR11: now also U.29 (I13)
- net CUR_UADR12: now also U.31 (I14)
- net CUR_UADR13: now also U.33 (I15)
- net CUR_UADR2: now also U.11 (I4)
- net CUR_UADR3: now also U.13 (I5)
- net CUR_UADR4: now also U.15 (I6)
- net CUR_UADR5: now also U.17 (I7)
- net CUR_UADR6: now also U.19 (I8)
- net CUR_UADR7: now also U.21 (I9)
- net CUR_UADR8: now also U.23 (I10)
- net CUR_UADR9: now also U.25 (I11)
- net C_UADR_ONE0: now also U.7 (I2)
- net C_UADR_ONE1: now also U.9 (I3)
- net C_UADR_ONE10: now also U.27 (I12)
- net C_UADR_ONE11: now also U.29 (I13)
- net C_UADR_ONE12: now also U.31 (I14)
- net C_UADR_ONE13: now also U.33 (I15)
- net C_UADR_ONE2: now also U.11 (I4)
- net C_UADR_ONE3: now also U.13 (I5)
- net C_UADR_ONE4: now also U.15 (I6)
- net C_UADR_ONE5: now also U.17 (I7)
- net C_UADR_ONE6: now also U.19 (I8)
- net C_UADR_ONE7: now also U.21 (I9)
- net C_UADR_ONE8: now also U.23 (I10)
- net C_UADR_ONE9: now also U.25 (I11)
- net FIU.IN~48: now also U.3 (I0)
- net FIU.IN~49: now also U.5 (I1)
- net FIU.IN~50: now also U.7 (I2)
- net FIU.IN~51: now also U.9 (I3)
- net FIU.IN~52: now also U.11 (I4)
- net FIU.IN~53: now also U.13 (I5)
- net FIU.IN~54: now also U.15 (I6)
- net FIU.IN~55: now also U.17 (I7)
- net FIU.IN~56: now also U.19 (I8)
- net FIU.IN~57: now also U.21 (I9)
- net FIU.IN~58: now also U.23 (I10)
- net FIU.IN~59: now also U.25 (I11)
- net FIU.IN~60: now also U.27 (I12)
- net FIU.IN~61: now also U.29 (I13)
- net FIU.IN~62: now also U.31 (I14)
- net FIU.IN~63: now also U.33 (I15)
- net H2: now also U.4 (B1), U.6 (D0)
- net LATCHED_COND: now also U.5 (I1), U.5 (I1), U.5 (I1)
- net PD: now also U.1 (INV), U.1 (INV), U.1 (INV), U.1 (INV), U.2 (INV), U.3 (OE), U.3 (S0), U.5 (D2)
- net PU: now also U.1 (A1), U.3 (A3), U.5 (B2)
- net Q2~: now also U.1 (D0), U.1 (WE)
- net Q3_COND: now also U.3 (I0), U.3 (I0), U.3 (I0)
- net SAVED_LATCHED: now also U.5 (D1), U.9 (Q1)
- net SRA0: now also U.35 (A0)
- net SRA1: now also U.36 (A1)
- net SRA2: now also U.37 (A2)
- net SRA3: now also U.38 (A3)
- net STACK_INP.SEL0: now also U.2 (S1)
- net STACK_INP.SEL1: now also U.1 (S2)
- net STACK_OUT.SPARE: now also U.3 (D0), U.7 (Q0)
- net STIN.0: now also U.15 (Y0_), U.2 (OE)
- net STIN.1: now also U.14 (Y1_), U.2 (OE)
- net STIN.2: now also U.13 (Y2_), U.2 (OE)
- net STIN.3: now also U.12 (Y3_), U.2 (OE)
- net STKD0: now also U.4 (Q0), U.4 (Y0), U.4 (Y0), U.4 (Y0), U.4 (Y0), U.6 (D0)
- net STKD1: now also U.6 (Q1), U.6 (Y1), U.6 (Y1), U.6 (Y1), U.6 (Y1), U.8 (D1)
- net STKD10: now also U.24 (Q10), U.24 (Y10), U.24 (Y10), U.24 (Y10), U.24 (Y10), U.26 (D10)
- net STKD11: now also U.26 (Q11), U.26 (Y11), U.26 (Y11), U.26 (Y11), U.26 (Y11), U.28 (D11)
- net STKD12: now also U.28 (Q12), U.28 (Y12), U.28 (Y12), U.28 (Y12), U.28 (Y12), U.30 (D12)
- net STKD13: now also U.30 (Q13), U.30 (Y13), U.30 (Y13), U.30 (Y13), U.30 (Y13), U.32 (D13)
- net STKD14: now also U.32 (Q14), U.32 (Y14), U.32 (Y14), U.32 (Y14), U.32 (Y14), U.34 (D14)
- net STKD15: now also U.34 (Q15), U.34 (Y15), U.34 (Y15), U.34 (Y15), U.34 (Y15), U.36 (D15)
- net STKD2: now also U.10 (D2), U.8 (Q2), U.8 (Y2), U.8 (Y2), U.8 (Y2), U.8 (Y2)
- net STKD3: now also U.10 (Q3), U.10 (Y3), U.10 (Y3), U.10 (Y3), U.10 (Y3), U.12 (D3)
- net STKD4: now also U.12 (Q4), U.12 (Y4), U.12 (Y4), U.12 (Y4), U.12 (Y4), U.14 (D4)
- net STKD5: now also U.14 (Q5), U.14 (Y5), U.14 (Y5), U.14 (Y5), U.14 (Y5), U.16 (D5)
- net STKD6: now also U.16 (Q6), U.16 (Y6), U.16 (Y6), U.16 (Y6), U.16 (Y6), U.18 (D6)
- net STKD7: now also U.18 (Q7), U.18 (Y7), U.18 (Y7), U.18 (Y7), U.18 (Y7), U.20 (D7)
- net STKD8: now also U.20 (Q8), U.20 (Y8), U.20 (Y8), U.20 (Y8), U.20 (Y8), U.22 (D8)
- net STKD9: now also U.22 (Q9), U.22 (Y9), U.22 (Y9), U.22 (Y9), U.22 (Y9), U.24 (D9)
- net TOP_USTACK0: now also U.11 (Q2), U.7 (D2)
- net TOP_USTACK1: now also U.13 (Q3), U.9 (D3)
- net TOP_USTACK10: now also U.27 (D12), U.31 (Q12)
- net TOP_USTACK11: now also U.29 (D13), U.33 (Q13)
- net TOP_USTACK12: now also U.31 (D14), U.35 (Q14)
- net TOP_USTACK13: now also U.33 (D15), U.37 (Q15)
- net TOP_USTACK2: now also U.11 (D4), U.15 (Q4)
- net TOP_USTACK3: now also U.13 (D5), U.17 (Q5)
- net TOP_USTACK4: now also U.15 (D6), U.19 (Q6)
- net TOP_USTACK5: now also U.17 (D7), U.21 (Q7)
- net TOP_USTACK6: now also U.19 (D8), U.23 (Q8)
- net TOP_USTACK7: now also U.21 (D9), U.25 (Q9)
- net TOP_USTACK8: now also U.23 (D10), U.27 (Q10)
- net TOP_USTACK9: now also U.25 (D11), U.29 (Q11)
- net TOS.WE~: now also U.1 (CLK)
- net WRITE~: now also U.4 (D1), U.6 (B3)
- new net: U.2 (A2), U.2 (Q)
- new net: U.2 (CS), U.7 (Q)
