File: Schematics/SEQ/pg_63.kicad_sch (KiCad schematic)
At the start: 7 parts, among them U6401 F251, U6402 F251, U6403 F251, U6404 F251, U6405 F251, U6406 F251, U6407 F251

Commit message: Much SEQ polishing
Parts:
- removed U6401, U6402, U6403, U6404, U6405, U6406, U6407: F251, symbol r1000:F251
- added U6408: F138, symbol r1000:F138
- added U6409, U6410, U6411, U6412, U6413, U6414, U6416, U6417: XBUF16, symbol r1000:XBUF16
Connections:
- net BRNCH_ADR.UIR0: now also U6412.7 (I2), U6414.7 (I2), U6417.7 (I2)
- net BRNCH_ADR.UIR1: now also U6412.9 (I3), U6414.9 (I3), U6417.9 (I3)
- net BRNCH_ADR.UIR2: now also U6412.11 (I4), U6414.11 (I4), U6417.11 (I4)
- net BRNCH_ADR.UIR3: now also U6412.13 (I5), U6414.13 (I5), U6417.13 (I5)
- net BRNCH_ADR.UIR4: now also U6412.15 (I6), U6414.15 (I6), U6417.15 (I6)
- net BRNCH_ADR.UIR5: now also U6412.17 (I7), U6414.17 (I7), U6417.17 (I7)
- net BRNCH_ADR.UIR6: now also U6412.19 (I8), U6414.19 (I8), U6417.19 (I8)
- net CASE_UADR0: now also U6409.7 (I2)
- net CASE_UADR1: now also U6409.9 (I3)
- net CASE_UADR2: now also U6409.11 (I4)
- net CASE_UADR3: now also U6409.13 (I5)
- net CASE_UADR4: now also U6409.15 (I6)
- net CASE_UADR5: now also U6409.17 (I7)
- net CASE_UADR6: now also U6409.19 (I8)
- net C_UADR_ONE0: now also U6410.7 (I2), U6416.7 (I2)
- net C_UADR_ONE1: now also U6410.9 (I3), U6416.9 (I3)
- net C_UADR_ONE2: now also U6410.11 (I4), U6416.11 (I4)
- net C_UADR_ONE3: now also U6410.13 (I5), U6416.13 (I5)
- net C_UADR_ONE4: now also U6410.15 (I6), U6416.15 (I6)
- net C_UADR_ONE5: now also U6410.17 (I7), U6416.17 (I7)
- net C_UADR_ONE6: now also U6410.19 (I8), U6416.19 (I8)
- net GROUP_SEL0: now also U6408.2 (S1)
- net GROUP_SEL1: now also U6408.1 (S2)
- net TOP_USTACK0: now also U6413.7 (I2)
- net TOP_USTACK1: now also U6413.9 (I3)
- net TOP_USTACK2: now also U6413.11 (I4)
- net TOP_USTACK3: now also U6413.13 (I5)
- net TOP_USTACK4: now also U6413.15 (I6)
- net TOP_USTACK5: now also U6413.17 (I7)
- net TOP_USTACK6: now also U6413.19 (I8)
- net UADR.DEC0: now also U6411.7 (I2)
- net UADR.DEC1: now also U6411.9 (I3)
- net UADR.DEC2: now also U6411.11 (I4)
- net UADR.DEC3: now also U6411.13 (I5)
- net UADR.DEC4: now also U6411.15 (I6)
- net UADR.DEC5: now also U6411.17 (I7)
- net UADR.DEC6: now also U6411.19 (I8)
- net UADR_MUX.OE~: now also U6408.4 (D1)
- net UADR_MUX.SEL: now also U6408.3 (S0)
- net UADR~0: now also U6409.8 (Y2), U6410.8 (Y2), U6411.8 (Y2), U6412.8 (Y2), U6413.8 (Y2), U6414.8 (Y2), U6416.8 (Y2), U6417.8 (Y2)
- net UADR~1: now also U6409.10 (Y3), U6410.10 (Y3), U6411.10 (Y3), U6412.10 (Y3), U6413.10 (Y3), U6414.10 (Y3), U6416.10 (Y3), U6417.10 (Y3)
- net UADR~2: now also U6409.12 (Y4), U6410.12 (Y4), U6411.12 (Y4), U6412.12 (Y4), U6413.12 (Y4), U6414.12 (Y4), U6416.12 (Y4), U6417.12 (Y4)
- net UADR~3: now also U6409.14 (Y5), U6410.14 (Y5), U6411.14 (Y5), U6412.14 (Y5), U6413.14 (Y5), U6414.14 (Y5), U6416.14 (Y5), U6417.14 (Y5)
- net UADR~4: now also U6409.16 (Y6), U6410.16 (Y6), U6411.16 (Y6), U6412.16 (Y6), U6413.16 (Y6), U6414.16 (Y6), U6416.16 (Y6), U6417.16 (Y6)
- net UADR~5: now also U6409.18 (Y7), U6410.18 (Y7), U6411.18 (Y7), U6412.18 (Y7), U6413.18 (Y7), U6414.18 (Y7), U6416.18 (Y7), U6417.18 (Y7)
- net UADR~6: now also U6409.20 (Y8), U6410.20 (Y8), U6411.20 (Y8), U6412.20 (Y8), U6413.20 (Y8), U6414.20 (Y8), U6416.20 (Y8), U6417.20 (Y8)
- new net BRNCH_ADR.UIR10: U6412.27 (I12), U6414.27 (I12), U6417.27 (I12)
- new net BRNCH_ADR.UIR11: U6412.29 (I13), U6414.29 (I13), U6417.29 (I13)
- new net BRNCH_ADR.UIR12: U6412.31 (I14), U6414.31 (I14), U6417.31 (I14)
- new net BRNCH_ADR.UIR13: U6412.33 (I15), U6414.33 (I15), U6417.33 (I15)
- new net BRNCH_ADR.UIR7: U6412.21 (I9), U6414.21 (I9), U6417.21 (I9)
- new net BRNCH_ADR.UIR8: U6412.23 (I10), U6414.23 (I10), U6417.23 (I10)
- new net BRNCH_ADR.UIR9: U6412.25 (I11), U6414.25 (I11), U6417.25 (I11)
- new net CASE_UADR10: U6409.27 (I12)
- new net CASE_UADR11: U6409.29 (I13)
- new net CASE_UADR12: U6409.31 (I14)
- new net CASE_UADR13: U6409.33 (I15)
- new net CASE_UADR7: U6409.21 (I9)
- new net CASE_UADR8: U6409.23 (I10)
- new net CASE_UADR9: U6409.25 (I11)
- new net C_UADR_ONE10: U6410.27 (I12), U6416.27 (I12)
- new net C_UADR_ONE11: U6410.29 (I13), U6416.29 (I13)
- new net C_UADR_ONE12: U6410.31 (I14), U6416.31 (I14)
- new net C_UADR_ONE13: U6410.33 (I15), U6416.33 (I15)
- new net C_UADR_ONE7: U6410.21 (I9), U6416.21 (I9)
- new net C_UADR_ONE8: U6410.23 (I10), U6416.23 (I10)
- new net C_UADR_ONE9: U6410.25 (I11), U6416.25 (I11)
- new net PD: U6408.5 (D2), U6409.1 (INV), U6409.3 (I0), U6409.5 (I1), U6410.1 (INV), U6410.3 (I0), U6410.5 (I1), U6411.1 (INV), U6411.3 (I0), U6411.33 (I15), U6411.5 (I1), U6412.1 (INV), U6412.3 (I0), U6412.5 (I1), U6413.1 (INV), U6413.3 (I0), U6413.5 (I1), U6414.1 (INV), U6414.3 (I0), U6414.5 (I1), U6416.1 (INV), U6416.3 (I0), U6416.5 (I1), U6417.1 (INV), U6417.3 (I0), U6417.5 (I1)
- new net PU: U6408.6 (D0)
- new net TOP_USTACK10: U6413.27 (I12)
- new net TOP_USTACK11: U6413.29 (I13)
- new net TOP_USTACK12: U6413.31 (I14)
- new net TOP_USTACK13: U6413.33 (I15)
- new net TOP_USTACK7: U6413.21 (I9)
- new net TOP_USTACK8: U6413.23 (I10)
- new net TOP_USTACK9: U6413.25 (I11)
- new net UADR.DEC10: U6411.27 (I12)
- new net UADR.DEC11: U6411.29 (I13)
- new net UADR.DEC12: U6411.31 (I14)
- new net UADR.DEC7: U6411.21 (I9)
- new net UADR.DEC8: U6411.23 (I10)
- new net UADR.DEC9: U6411.25 (I11)
- new net UADR~10: U6409.28 (Y12), U6410.28 (Y12), U6411.28 (Y12), U6412.28 (Y12), U6413.28 (Y12), U6414.28 (Y12), U6416.28 (Y12), U6417.28 (Y12)
- new net UADR~11: U6409.30 (Y13), U6410.30 (Y13), U6411.30 (Y13), U6412.30 (Y13), U6413.30 (Y13), U6414.30 (Y13), U6416.30 (Y13), U6417.30 (Y13)
- new net UADR~12: U6409.32 (Y14), U6410.32 (Y14), U6411.32 (Y14), U6412.32 (Y14), U6413.32 (Y14), U6414.32 (Y14), U6416.32 (Y14), U6417.32 (Y14)
- new net UADR~13: U6409.34 (Y15), U6410.34 (Y15), U6411.34 (Y15), U6412.34 (Y15), U6413.34 (Y15), U6414.34 (Y15), U6416.34 (Y15), U6417.34 (Y15)
- new net UADR~7: U6409.22 (Y9), U6410.22 (Y9), U6411.22 (Y9), U6412.22 (Y9), U6413.22 (Y9), U6414.22 (Y9), U6416.22 (Y9), U6417.22 (Y9)
- new net UADR~8: U6409.24 (Y10), U6410.24 (Y10), U6411.24 (Y10), U6412.24 (Y10), U6413.24 (Y10), U6414.24 (Y10), U6416.24 (Y10), U6417.24 (Y10)
- new net UADR~9: U6409.26 (Y11), U6410.26 (Y11), U6411.26 (Y11), U6412.26 (Y11), U6413.26 (Y11), U6414.26 (Y11), U6416.26 (Y11), U6417.26 (Y11)
- new net UASEL~0: U6408.15 (Y0_), U6409.2 (OE)
- new net UASEL~1: U6408.14 (Y1_), U6411.2 (OE)
- new net UASEL~2: U6408.13 (Y2_), U6413.2 (OE)
- new net UASEL~3: U6408.12 (Y3_), U6416.2 (OE)
- new net UASEL~4: U6408.11 (Y4_), U6410.2 (OE)
- new net UASEL~5: U6408.10 (Y5_), U6412.2 (OE)
- new net UASEL~6: U6408.9 (Y6_), U6414.2 (OE)
- new net UASEL~7: U6408.7 (Y7_), U6417.2 (OE)
- no-connect marks 7 -> 16

Commit message: KiCad 6
Parts:
- U6408: value F138 -> (none)
- U6409, U6410, U6411, U6412, U6413, U6414, U6416, U6417: value XBUF16 -> (none)

Commit message: Recover from KiCad-6 munging
Parts:
- U6408: value (none) -> F138
- U6409, U6410, U6411, U6412, U6413, U6414, U6416, U6417: value (none) -> XBUF16

Commit message: Fix polarity of unused part of driven FIU bus.
Parts:
- removed U6408: F138, symbol r1000:F138
- removed U6409, U6410, U6411, U6412, U6413, U6414, U6416, U6417: XBUF16, symbol r1000:XBUF16
- added U (x8): (no value), symbol r1000:XBUF16
- added U: (no value), symbol r1000:F138
Connections:
- net BRNCH_ADR.UIR0: now also U.7 (I2), U.7 (I2), U.7 (I2)
- net BRNCH_ADR.UIR1: now also U.9 (I3), U.9 (I3), U.9 (I3)
- net BRNCH_ADR.UIR10: now also U.27 (I12), U.27 (I12), U.27 (I12)
- net BRNCH_ADR.UIR11: now also U.29 (I13), U.29 (I13), U.29 (I13)
- net BRNCH_ADR.UIR12: now also U.31 (I14), U.31 (I14), U.31 (I14)
- net BRNCH_ADR.UIR13: now also U.33 (I15), U.33 (I15), U.33 (I15)
- net BRNCH_ADR.UIR2: now also U.11 (I4), U.11 (I4), U.11 (I4)
- net BRNCH_ADR.UIR3: now also U.13 (I5), U.13 (I5), U.13 (I5)
- net BRNCH_ADR.UIR4: now also U.15 (I6), U.15 (I6), U.15 (I6)
- net BRNCH_ADR.UIR5: now also U.17 (I7), U.17 (I7), U.17 (I7)
- net BRNCH_ADR.UIR6: now also U.19 (I8), U.19 (I8), U.19 (I8)
- net BRNCH_ADR.UIR7: now also U.21 (I9), U.21 (I9), U.21 (I9)
- net BRNCH_ADR.UIR8: now also U.23 (I10), U.23 (I10), U.23 (I10)
- net BRNCH_ADR.UIR9: now also U.25 (I11), U.25 (I11), U.25 (I11)
- net CASE_UADR0: now also U.7 (I2)
- net CASE_UADR1: now also U.9 (I3)
- net CASE_UADR10: now also U.27 (I12)
- net CASE_UADR11: now also U.29 (I13)
- net CASE_UADR12: now also U.31 (I14)
- net CASE_UADR13: now also U.33 (I15)
- net CASE_UADR2: now also U.11 (I4)
- net CASE_UADR3: now also U.13 (I5)
- net CASE_UADR4: now also U.15 (I6)
- net CASE_UADR5: now also U.17 (I7)
- net CASE_UADR6: now also U.19 (I8)
- net CASE_UADR7: now also U.21 (I9)
- net CASE_UADR8: now also U.23 (I10)
- net CASE_UADR9: now also U.25 (I11)
- net C_UADR_ONE0: now also U.7 (I2), U.7 (I2)
- net C_UADR_ONE1: now also U.9 (I3), U.9 (I3)
- net C_UADR_ONE10: now also U.27 (I12), U.27 (I12)
- net C_UADR_ONE11: now also U.29 (I13), U.29 (I13)
- net C_UADR_ONE12: now also U.31 (I14), U.31 (I14)
- net C_UADR_ONE13: now also U.33 (I15), U.33 (I15)
- net C_UADR_ONE2: now also U.11 (I4), U.11 (I4)
- net C_UADR_ONE3: now also U.13 (I5), U.13 (I5)
- net C_UADR_ONE4: now also U.15 (I6), U.15 (I6)
- net C_UADR_ONE5: now also U.17 (I7), U.17 (I7)
- net C_UADR_ONE6: now also U.19 (I8), U.19 (I8)
- net C_UADR_ONE7: now also U.21 (I9), U.21 (I9)
- net C_UADR_ONE8: now also U.23 (I10), U.23 (I10)
- net C_UADR_ONE9: now also U.25 (I11), U.25 (I11)
- net GROUP_SEL0: now also U.2 (S1)
- net GROUP_SEL1: now also U.1 (S2)
- net PD: now also U.1 (INV), U.1 (INV), U.1 (INV), U.1 (INV), U.1 (INV), U.1 (INV), U.1 (INV), U.1 (INV), U.3 (I0), U.3 (I0), U.3 (I0), U.3 (I0), U.3 (I0), U.3 (I0), U.3 (I0), U.3 (I0), U.33 (I15), U.5 (D2), U.5 (I1), U.5 (I1), U.5 (I1), U.5 (I1), U.5 (I1), U.5 (I1), U.5 (I1), U.5 (I1)
- net PU: now also U.6 (D0)
- net TOP_USTACK0: now also U.7 (I2)
- net TOP_USTACK1: now also U.9 (I3)
- net TOP_USTACK10: now also U.27 (I12)
- net TOP_USTACK11: now also U.29 (I13)
- net TOP_USTACK12: now also U.31 (I14)
- net TOP_USTACK13: now also U.33 (I15)
- net TOP_USTACK2: now also U.11 (I4)
- net TOP_USTACK3: now also U.13 (I5)
- net TOP_USTACK4: now also U.15 (I6)
- net TOP_USTACK5: now also U.17 (I7)
- net TOP_USTACK6: now also U.19 (I8)
- net TOP_USTACK7: now also U.21 (I9)
- net TOP_USTACK8: now also U.23 (I10)
- net TOP_USTACK9: now also U.25 (I11)
- net UADR.DEC0: now also U.7 (I2)
- net UADR.DEC1: now also U.9 (I3)
- net UADR.DEC10: now also U.27 (I12)
- net UADR.DEC11: now also U.29 (I13)
- net UADR.DEC12: now also U.31 (I14)
- net UADR.DEC2: now also U.11 (I4)
- net UADR.DEC3: now also U.13 (I5)
- net UADR.DEC4: now also U.15 (I6)
- net UADR.DEC5: now also U.17 (I7)
- net UADR.DEC6: now also U.19 (I8)
- net UADR.DEC7: now also U.21 (I9)
- net UADR.DEC8: now also U.23 (I10)
- net UADR.DEC9: now also U.25 (I11)
- net UADR_MUX.OE~: now also U.4 (D1)
- net UADR_MUX.SEL: now also U.3 (S0)
- net UADR~0: now also U.8 (Y2), U.8 (Y2), U.8 (Y2), U.8 (Y2), U.8 (Y2), U.8 (Y2), U.8 (Y2), U.8 (Y2)
- net UADR~1: now also U.10 (Y3), U.10 (Y3), U.10 (Y3), U.10 (Y3), U.10 (Y3), U.10 (Y3), U.10 (Y3), U.10 (Y3)
- net UADR~10: now also U.28 (Y12), U.28 (Y12), U.28 (Y12), U.28 (Y12), U.28 (Y12), U.28 (Y12), U.28 (Y12), U.28 (Y12)
- net UADR~11: now also U.30 (Y13), U.30 (Y13), U.30 (Y13), U.30 (Y13), U.30 (Y13), U.30 (Y13), U.30 (Y13), U.30 (Y13)
- net UADR~12: now also U.32 (Y14), U.32 (Y14), U.32 (Y14), U.32 (Y14), U.32 (Y14), U.32 (Y14), U.32 (Y14), U.32 (Y14)
- net UADR~13: now also U.34 (Y15), U.34 (Y15), U.34 (Y15), U.34 (Y15), U.34 (Y15), U.34 (Y15), U.34 (Y15), U.34 (Y15)
- net UADR~2: now also U.12 (Y4), U.12 (Y4), U.12 (Y4), U.12 (Y4), U.12 (Y4), U.12 (Y4), U.12 (Y4), U.12 (Y4)
- net UADR~3: now also U.14 (Y5), U.14 (Y5), U.14 (Y5), U.14 (Y5), U.14 (Y5), U.14 (Y5), U.14 (Y5), U.14 (Y5)
- net UADR~4: now also U.16 (Y6), U.16 (Y6), U.16 (Y6), U.16 (Y6), U.16 (Y6), U.16 (Y6), U.16 (Y6), U.16 (Y6)
- net UADR~5: now also U.18 (Y7), U.18 (Y7), U.18 (Y7), U.18 (Y7), U.18 (Y7), U.18 (Y7), U.18 (Y7), U.18 (Y7)
- net UADR~6: now also U.20 (Y8), U.20 (Y8), U.20 (Y8), U.20 (Y8), U.20 (Y8), U.20 (Y8), U.20 (Y8), U.20 (Y8)
- net UADR~7: now also U.22 (Y9), U.22 (Y9), U.22 (Y9), U.22 (Y9), U.22 (Y9), U.22 (Y9), U.22 (Y9), U.22 (Y9)
- net UADR~8: now also U.24 (Y10), U.24 (Y10), U.24 (Y10), U.24 (Y10), U.24 (Y10), U.24 (Y10), U.24 (Y10), U.24 (Y10)
- net UADR~9: now also U.26 (Y11), U.26 (Y11), U.26 (Y11), U.26 (Y11), U.26 (Y11), U.26 (Y11), U.26 (Y11), U.26 (Y11)
- net UASEL~0: now also U.15 (Y0_), U.2 (OE)
- net UASEL~1: now also U.14 (Y1_), U.2 (OE)
- net UASEL~2: now also U.13 (Y2_), U.2 (OE)
- net UASEL~3: now also U.12 (Y3_), U.2 (OE)
- net UASEL~4: now also U.11 (Y4_), U.2 (OE)
- net UASEL~5: now also U.10 (Y5_), U.2 (OE)
- net UASEL~6: now also U.2 (OE), U.9 (Y6_)
- net UASEL~7: now also U.2 (OE), U.7 (Y7_)
