File: Schematics/SEQ/pg_09.kicad_sch (KiCad schematic)
At the start: 0 parts

Commit message: Add page titles
Other:
- title: SEQ 9 -> MACRO SEQUENCING LOGIC
Changed lines of the file:
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@@
   (paper "User" 584.2 378.46)
   (title_block
-    (title "SEQ 9")
+    (title "MACRO SEQUENCING LOGIC")
     (date "22-MAY-90")
     (rev "1.0")
