File: Schematics/SEQ/pg_85.kicad_sch (KiCad schematic)
At the start: 8 parts, among them U8601 F299, U8602 F299, U8603 F299, U8604 F299, U8605 F299, U8606 F299, U8607 F299, U8608 F299

Commit message: Fix 0/8 typo
Parts:
- removed U8601, U8602, U8603, U8604, U8605, U8606, U8607, U8608: F299, symbol r1000:F299
- added U (x8): (no value), symbol r1000:F299
Connections:
- net ALWAYS.B1.CLK~: now also U.12 (CLK), U.12 (CLK), U.12 (CLK), U.12 (CLK), U.12 (CLK), U.12 (CLK), U.12 (CLK), U.12 (CLK)
- net DGRG_VAL.OE~: now also U.2 (G1), U.2 (G1), U.2 (G1), U.2 (G1), U.2 (G1), U.2 (G1), U.2 (G1), U.2 (G1)
- net DG_SEQ_V.MODE0: now also U.19 (S0), U.19 (S0), U.19 (S0), U.19 (S0), U.19 (S0), U.19 (S0), U.19 (S0), U.19 (S0)
- net DG_SEQ_V.MODE1: now also U.1 (S1), U.1 (S1), U.1 (S1), U.1 (S1), U.1 (S1), U.1 (S1), U.1 (S1), U.1 (S1)
- net DIAG.D0: now also U.11 (RSI)
- net DIAG.D1: now also U.11 (RSI)
- net DIAG.D2: now also U.11 (RSI)
- net DIAG.D3: now also U.11 (RSI)
- net DIAG.D4: now also U.11 (RSI)
- net DIAG.D5: now also U.11 (RSI)
- net DIAG.D6: now also U.11 (RSI)
- net DIAG.D7: now also U.11 (RSI)
- net L_VAL~15: now also U.17 (Q7)
- net L_VAL~23: now also U.17 (Q7)
- net L_VAL~31: now also U.17 (Q7)
- net L_VAL~39: now also U.17 (Q7)
- net L_VAL~47: now also U.17 (Q7)
- net L_VAL~55: now also U.17 (Q7)
- net L_VAL~63: now also U.17 (Q7)
- net L_VAL~7: now also U.17 (Q7)
- net PD: now also U.3 (G2), U.3 (G2), U.3 (G2), U.3 (G2), U.3 (G2), U.3 (G2), U.3 (G2), U.3 (G2)
- net PU: now also U.9 (CLR), U.9 (CLR), U.9 (CLR), U.9 (CLR), U.9 (CLR), U.9 (CLR), U.9 (CLR), U.9 (CLR)
- net VAL~0: now also U.7 (DQ0)
- net VAL~1: now also U.13 (DQ1)
- net VAL~10: now also U.6 (DQ2)
- net VAL~11: now also U.14 (DQ3)
- net VAL~12: now also U.5 (DQ4)
- net VAL~13: now also U.15 (DQ5)
- net VAL~14: now also U.4 (DQ6)
- net VAL~15: now also U.16 (DQ7)
- net VAL~16: now also U.7 (DQ0)
- net VAL~17: now also U.13 (DQ1)
- net VAL~18: now also U.6 (DQ2)
- net VAL~19: now also U.14 (DQ3)
- net VAL~2: now also U.6 (DQ2)
- net VAL~20: now also U.5 (DQ4)
- net VAL~21: now also U.15 (DQ5)
- net VAL~22: now also U.4 (DQ6)
- net VAL~23: now also U.16 (DQ7)
- net VAL~24: now also U.7 (DQ0)
- net VAL~25: now also U.13 (DQ1)
- net VAL~26: now also U.6 (DQ2)
- net VAL~27: now also U.14 (DQ3)
- net VAL~28: now also U.5 (DQ4)
- net VAL~29: now also U.15 (DQ5)
- net VAL~3: now also U.14 (DQ3)
- net VAL~30: now also U.4 (DQ6)
- net VAL~31: now also U.16 (DQ7)
- net VAL~32: now also U.7 (DQ0)
- net VAL~33: now also U.13 (DQ1)
- net VAL~34: now also U.6 (DQ2)
- net VAL~35: now also U.14 (DQ3)
- net VAL~36: now also U.5 (DQ4)
- net VAL~37: now also U.15 (DQ5)
- net VAL~38: now also U.4 (DQ6)
- net VAL~39: now also U.16 (DQ7)
- net VAL~4: now also U.5 (DQ4)
- net VAL~40: now also U.7 (DQ0)
- net VAL~41: now also U.13 (DQ1)
- net VAL~42: now also U.6 (DQ2)
- net VAL~43: now also U.14 (DQ3)
- net VAL~44: now also U.5 (DQ4)
- net VAL~45: now also U.15 (DQ5)
- net VAL~46: now also U.4 (DQ6)
- net VAL~47: now also U.16 (DQ7)
- net VAL~48: now also U.7 (DQ0)
- net VAL~49: now also U.13 (DQ1)
- net VAL~5: now also U.15 (DQ5)
- net VAL~50: now also U.6 (DQ2)
- net VAL~51: now also U.14 (DQ3)
- net VAL~52: now also U.5 (DQ4)
- net VAL~53: now also U.15 (DQ5)
- net VAL~54: now also U.4 (DQ6)
- net VAL~55: now also U.16 (DQ7)
- net VAL~56: now also U.7 (DQ0)
- net VAL~57: now also U.13 (DQ1)
- net VAL~58: now also U.6 (DQ2)
- net VAL~59: now also U.14 (DQ3)
- net VAL~6: now also U.4 (DQ6)
- net VAL~60: now also U.5 (DQ4)
- net VAL~61: now also U.15 (DQ5)
- net VAL~62: now also U.4 (DQ6)
- net VAL~63: now also U.16 (DQ7)
- net VAL~7: now also U.16 (DQ7)
- net VAL~8: now also U.7 (DQ0)
- net VAL~9: now also U.13 (DQ1)

Commit message: SEQ: dedup, clocks, dfsm
Connections:
- net ALWAYS.B1.CLK~ renamed ALWAYS.CLK~
Changed lines of the file:
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@@
     )
   )
-  (global_label "ALWAYS.B1.CLK~" (shape input) (at 93.98 43.18 180) (fields_autoplaced)
+  (global_label "ALWAYS.CLK~" (shape input) (at 93.98 43.18 180) (fields_autoplaced)
     (effects (font (size 2.54 2.54)) (justify right))
     (property "Intersheet References" "${INTERSHEET_REFS}" (id 0) (at 58.9159 43.0213 0)

Commit message: Tested to 5.82 seconds (rm031)
Parts:
- removed U (x8): (no value), symbol r1000:F299
- added U: F299X8, symbol r1000:F299X8
Connections:
- net ALWAYS.CLK~: now also U.4 (CLK)
- net DGRG_VAL.OE~: now also U.12 (G1)
- net DG_SEQ_V.MODE0: now also U.7 (S0)
- net DG_SEQ_V.MODE1: now also U.9 (S1)
- net DIAG.D0: now also U.19 (RI0)
- net DIAG.D1: now also U.21 (RI1)
- net DIAG.D2: now also U.23 (RI2)
- net DIAG.D3: now also U.25 (RI3)
- net DIAG.D4: now also U.27 (RI4)
- net DIAG.D5: now also U.29 (RI5)
- net DIAG.D6: now also U.31 (RI6)
- net DIAG.D7: now also U.33 (RI7)
- net L_VAL~15: now also U.38 (Q1)
- net L_VAL~23: now also U.40 (Q2)
- net L_VAL~31: now also U.42 (Q3)
- net L_VAL~39: now also U.44 (Q4)
- net L_VAL~47: now also U.46 (Q5)
- net L_VAL~55: now also U.48 (Q6)
- net L_VAL~63: now also U.50 (Q7)
- net L_VAL~7: now also U.36 (Q0)
- net PD: now also U.14 (G2)
- net VAL~0: now also U.1 (DQ0)
- net VAL~1: now also U.3 (DQ1)
- net VAL~10: now also U.17 (DQ10)
- net VAL~11: now also U.18 (DQ11)
- net VAL~12: now also U.20 (DQ12)
- net VAL~13: now also U.22 (DQ13)
- net VAL~14: now also U.24 (DQ14)
- net VAL~15: now also U.26 (DQ15)
- net VAL~16: now also U.28 (DQ16)
- net VAL~17: now also U.30 (DQ17)
- net VAL~18: now also U.32 (DQ18)
- net VAL~19: now also U.34 (DQ19)
- net VAL~2: now also U.5 (DQ2)
- net VAL~20: now also U.35 (DQ20)
- net VAL~21: now also U.37 (DQ21)
- net VAL~22: now also U.39 (DQ22)
- net VAL~23: now also U.41 (DQ23)
- net VAL~24: now also U.43 (DQ24)
- net VAL~25: now also U.45 (DQ25)
- net VAL~26: now also U.47 (DQ26)
- net VAL~27: now also U.49 (DQ27)
- net VAL~28: now also U.51 (DQ28)
- net VAL~29: now also U.52 (DQ29)
- net VAL~3: now also U.6 (DQ3)
- net VAL~30: now also U.54 (DQ30)
- net VAL~31: now also U.56 (DQ31)
- net VAL~32: now also U.58 (DQ32)
- net VAL~33: now also U.60 (DQ33)
- net VAL~34: now also U.62 (DQ34)
- net VAL~35: now also U.64 (DQ35)
- net VAL~36: now also U.66 (DQ36)
- net VAL~37: now also U.68 (DQ37)
- net VAL~38: now also U.69 (DQ38)
- net VAL~39: now also U.70 (DQ39)
- net VAL~4: now also U.8 (DQ4)
- net VAL~40: now also U.71 (DQ40)
- net VAL~41: now also U.72 (DQ41)
- net VAL~42: now also U.73 (DQ42)
- net VAL~43: now also U.74 (DQ43)
- net VAL~44: now also U.75 (DQ44)
- net VAL~45: now also U.76 (DQ45)
- net VAL~46: now also U.77 (DQ46)
- net VAL~47: now also U.78 (DQ47)
- net VAL~48: now also U.79 (DQ48)
- net VAL~49: now also U.80 (DQ49)
- net VAL~5: now also U.10 (DQ5)
- net VAL~50: now also U.81 (DQ50)
- net VAL~51: now also U.82 (DQ51)
- net VAL~52: now also U.83 (DQ52)
- net VAL~53: now also U.84 (DQ53)
- net VAL~54: now also U.85 (DQ54)
- net VAL~55: now also U.86 (DQ55)
- net VAL~56: now also U.87 (DQ56)
- net VAL~57: now also U.88 (DQ57)
- net VAL~58: now also U.89 (DQ58)
- net VAL~59: now also U.90 (DQ59)
- net VAL~6: now also U.11 (DQ6)
- net VAL~60: now also U.91 (DQ60)
- net VAL~61: now also U.92 (DQ61)
- net VAL~62: now also U.93 (DQ62)
- net VAL~63: now also U.94 (DQ63)
- net VAL~7: now also U.13 (DQ7)
- net VAL~8: now also U.15 (DQ8)
- net VAL~9: now also U.16 (DQ9)
- no-connect marks 16 -> 9

Commit message: New kicad + MEM32 polish
Parts:
- renumbered U to U95
Changed lines of the file:
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@@
-(kicad_sch (version 20220404) (generator eeschema)
+(kicad_sch (version 20221206) (generator eeschema)
   (paper "User" 584.2 378.46)
   (title_block
@@
   (global_label "L_VAL~55" (shape output) (at 228.6 157.48 0) (fields_autoplaced)
     (effects (font (size 2.54 2.54)) (justify left))
-    (property "Intersheet References" "${INTERSHEET_REFS}" (id 0) (at 250.4803 157.3213 0)
+    (property "Intersheetrefs" "${INTERSHEET_REFS}" (at 250.4803 157.3213 0)
       (effects (font (size 1.905 1.905)) (justify left))
     )
@@
   (global_label "DIAG.D[0..7]" (shape input) (at 251.46 76.2 0) (fields_autoplaced)
     (effects (font (size 2.54 2.54)) (justify left))
-    (property "Intersheet References" "${INTERSHEET_REFS}" (id 0) (at 279.146 76.0413 0)
+    (property "Intersheetrefs" "${INTERSHEET_REFS}" (at 279.146 76.0413 0)
       (effects (font (size 1.905 1.905)) (justify left))
     )
@@
   (global_label "L_VAL~31" (shape output) (at 228.6 142.24 0) (fields_autoplaced)
     (effects (font (size 2.54 2.54)) (justify left))
-    (property "Intersheet References" "${INTERSHEET_REFS}" (id 0) (at 250.4803 142.0813 0)
+    (property "Intersheetrefs" "${INTERSHEET_REFS}" (at 250.4803 142.0813 0)
       (effects (font (size 1.905 1.905)) (justify left))
     )
@@
   (global_label "L_VAL~7" (shape output) (at 228.6 127 0) (fields_autoplaced)
     (effects (font (size 2.54 2.54)) (justify left))
-    (property "Intersheet References" "${INTERSHEET_REFS}" (id 0) (at 248.0612 126.8413 0)
+    (property "Intersheetrefs" "${INTERSHEET_REFS}" (at 248.0612 126.8413 0)
       (effects (font (size 1.905 1.905)) (justify left))
     )
@@
   (global_label "DGRG_VAL.OE~" (shape input) (at 228.6 55.88 0) (fields_autoplaced)
     (effects (font (size 2.54 2.54)) (justify left))
-    (property "Intersheet References" "${INTERSHEET_REFS}" (id 0) (at 259.9146 55.7213 0)
+    (property "Intersheetrefs" "${INTERSHEET_REFS}" (at 259.9146 55.7213 0)
       (effects (font (size 1.905 1.905)) (justify left))
     )
@@
   (global_label "DG_SEQ_V.MODE0" (shape input) (at 228.6 40.64 0) (fields_autoplaced)
     (effects (font (size 2.54 2.54)) (justify left))
-    (property "Intersheet References" "${INTERSHEET_REFS}" (id 0) (at 265.9622 40.4813 0)
+    (property "Intersheetrefs" "${INTERSHEET_REFS}" (at 265.9622 40.4813 0)
       (effects (font (size 1.905 1.905)) (justify left))
     )
@@
   (global_label "DG_SEQ_V.MODE1" (shape input) (at 228.6 45.72 0) (fields_autoplaced)
     (effects (font (size 2.54 2.54)) (justify left))
-    (property "Intersheet References" "${INTERSHEET_REFS}" (id 0) (at 265.9622 45.5613 0)
+    (property "Intersheetrefs" "${INTERSHEET_REFS}" (at 265.9622 45.5613 0)
       (effects (font (size 1.905 1.905)) (justify left))
     )
@@
   (global_label "L_VAL~23" (shape output) (at 228.6 137.16 0) (fields_autoplaced)
     (effects (font (size 2.54 2.54)) (justify left))
-    (property "Intersheet References" "${INTERSHEET_REFS}" (id 0) (at 250.4803 137.0013 0)
+    (property "Intersheetrefs" "${INTERSHEET_REFS}" (at 250.4803 137.0013 0)
       (effects (font (size 1.905 1.905)) (justify left))
     )
@@
   (global_label "VAL~[0..63]" (shape input) (at 154.94 20.32 180) (fields_autoplaced)
     (effects (font (size 2.54 2.54)) (justify right))
-    (property "Intersheet References" "${INTERSHEET_REFS}" (id 0) (at 125.4293 20.32 0)
+    (property "Intersheetrefs" "${INTERSHEET_REFS}" (at 125.4293 20.32 0)
       (effects (font (size 1.905 1.905)) (justify right))
     )
@@
   (global_label "L_VAL~63" (shape output) (at 228.6 162.56 0) (fields_autoplaced)
     (effects (font (size 2.54 2.54)) (justify left))
-    (property "Intersheet References" "${INTERSHEET_REFS}" (id 0) (at 250.4803 162.4013 0)
+    (property "Intersheetrefs" "${INTERSHEET_REFS}" (at 250.4803 162.4013 0)
       (effects (font (size 1.905 1.905)) (justify left))
     )
@@
   (global_label "L_VAL~15" (shape output) (at 228.6 132.08 0) (fields_autoplaced)
     (effects (font (size 2.54 2.54)) (justify left))
-    (property "Intersheet References" "${INTERSHEET_REFS}" (id 0) (at 250.4803 131.9213 0)
+    (property "Intersheetrefs" "${INTERSHEET_REFS}" (at 250.4803 131.9213 0)
       (effects (font (size 1.905 1.905)) (justify left))
     )
@@
   (global_label "ALWAYS.CLK~" (shape input) (at 228.6 30.48 0) (fields_autoplaced)
     (effects (font (size 2.54 2.54)) (justify left))
-    (property "Intersheet References" "${INTERSHEET_REFS}" (id 0) (at 263.6641 30.3213 0)
+    (property "Intersheetrefs" "${INTERSHEET_REFS}" (at 263.6641 30.3213 0)
       (effects (font (size 1.905 1.905)) (justify left))
     )
@@
   (global_label "L_VAL~47" (shape output) (at 228.6 152.4 0) (fields_autoplaced)
     (effects (font (size 2.54 2.54)) (justify left))
-    (property "Intersheet References" "${INTERSHEET_REFS}" (id 0) (at 250.4803 152.2413 0)
+    (property "Intersheetrefs" "${INTERSHEET_REFS}" (at 250.4803 152.2413 0)
       (effects (font (size 1.905 1.905)) (justify left))
     )
@@
   (global_label "L_VAL~39" (shape output) (at 228.6 147.32 0) (fields_autoplaced)
     (effects (font (size 2.54 2.54)) (justify left))
-    (property "Intersheet References" "${INTERSHEET_REFS}" (id 0) (at 250.4803 147.1613 0)
+    (property "Intersheetrefs" "${INTERSHEET_REFS}" (at 250.4803 147.1613 0)
       (effects (font (size 1.905 1.905)) (justify left))
     )
   )
   (symbol (lib_id "r1000:F299X8") (at 203.2 353.06 0) (unit 1)
-    (in_bom yes) (on_board yes)
-    (default_instance (reference "U") (unit 1) (value "F299X8") (footprint ""))
-    (property "Reference" "U" (id 0) (at 205.74 347.98 0)
+    (in_bom yes) (on_board yes) (dnp no)
+    (property "Reference" "U95" (at 205.74 347.98 0)
       (effects (font (size 1.27 1.27)))
     )
-    (property "Value" "F299X8" (id 1) (at 199.39 358.14 0)
+    (property "Value" "F299X8" (at 199.39 358.14 0)
       (effects (font (size 2.54 2.54)) (justify left))
     )
-    (property "Footprint" "" (id 2) (at 204.47 354.33 0)
+    (property "Footprint" "" (at 204.47 354.33 0)
       (effects (font (size 1.27 1.27)) hide)
     )
-    (property "Datasheet" "" (id 3) (at 204.47 354.33 0)
+    (property "Datasheet" "" (at 204.47 354.33 0)
       (effects (font (size 1.27 1.27)) hide)
     )
-    (property "Location" "x99" (id 4) (at 201.93 353.06 0)
+    (property "Location" "x99" (at 201.93 353.06 0)
       (effects (font (size 2.54 2.54)) (justify left))
     )
-    (property "Name" "SEQDGV" (id 5) (at 207.01 365.76 0)
+    (property "Name" "SEQDGV" (at 207.01 365.76 0)
       (effects (font (size 2.54 2.54)) (justify bottom))
     )
@@
     (pin "93")
     (pin "94")
+    (instances
+      (project "SEQ"
+        (path "/20011966-1ffc-24d7-1b4b-436a182362c4/20011966-045f-514b-3eab-565a48439a3a"
+          (reference "U95") (unit 1)
+        )
+      )
+    )
   )
   (symbol (lib_id "r1000:PD") (at 226.06 60.96 0) (unit 1)
-    (in_bom no) (on_board yes)
-    (default_instance (reference "U") (unit 1) (value "") (footprint ""))
-    (property "Reference" "U" (id 0) (at 226.06 60.96 0)
+    (in_bom no) (on_board yes) (dnp no)
+    (property "Reference" "#PWR08601" (at 226.06 60.96 0)
       (effects (font (size 1.27 1.27)) hide)
     )
-    (property "Value" "" (id 1) (at 226.06 60.96 0)
+    (property "Value" "PD" (at 226.06 60.96 0)
       (effects (font (size 1.27 1.27)) hide)
     )
-    (property "Footprint" "" (id 2) (at 226.06 60.96 0)
+    (property "Footprint" "" (at 226.06 60.96 0)
       (effects (font (size 1.27 1.27)) hide)
     )
-    (property "Datasheet" "" (id 3) (at 226.06 60.96 0)
+    (property "Datasheet" "" (at 226.06 60.96 0)
       (effects (font (size 1.27 1.27)) hide)
     )
     (pin "1")
+    (instances
+      (project "SEQ"
+        (path "/20011966-1ffc-24d7-1b4b-436a182362c4/20011966-045f-514b-3eab-565a48439a3a"
+          (reference "#PWR08601") (unit 1)
+        )
+      )
+    )
   )
 )
