File: Schematics/SEQ/pg_12.kicad_sch (KiCad schematic)
At the start: 26 parts

Commit message: SEQ: dedup, clocks, dfsm
Connections:
- net ALWAYS.B1.CLK~ renamed ALWAYS.CLK~
Changed lines of the file:
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@@
     )
   )
-  (global_label "ALWAYS.B1.CLK~" (shape input) (at 457.2 101.6 180) (fields_autoplaced)
+  (global_label "ALWAYS.CLK~" (shape input) (at 457.2 101.6 180) (fields_autoplaced)
     (effects (font (size 2.54 2.54)) (justify right))
     (property "Intersheet References" "${INTERSHEET_REFS}" (id 0) (at 422.1359 101.4413 0)

Commit message: New kicad + MEM32 polish
Parts:
- U1301, U1302, U1304, U1305, U1320, U1322, U1323: renamed from U; value (none) -> F02
- U1303, U1308: renamed from U; value (none) -> F158
- U1306, U1307, U1318, U1324: renamed from U; value (none) -> F04
- U1309, U1310: renamed from U; value (none) -> F139
- U1311, U1312, U1321, U1325: renamed from U; value (none) -> F00
- U1313, U1314, U1315, U1316, U1317: renamed from U; value (none) -> F37
- U1319: renamed from U; value (none) -> F74
- U1326: renamed from U; value (none) -> F194

Commit message: Integrate SEQ from mc4a
Connections:
- net PU: no longer U1319.1 (CL_), U1319.4 (PR_)
- no-connect marks 3 -> 5
Changed lines of the file:
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@@
   (junction (at 106.68 269.24) (diameter 0) (color 0 0 0 0)
   )
+  (no_connect (at 373.38 25.4))
+  (no_connect (at 373.38 60.96))
   (no_connect (at 386.08 38.1))
   (no_connect (at 281.94 86.36))
@@
     (stroke (width 0) (type default))
   )
-  (wire (pts (xy 373.38 20.32) (xy 373.38 25.4))
-    (stroke (width 0) (type default))
-  )
   (wire (pts (xy 264.16 284.48) (xy 264.16 302.26))
     (stroke (width 0) (type default))
@@
   )
   (wire (pts (xy 406.4 142.24) (xy 411.48 142.24))
-    (stroke (width 0) (type default))
-  )
-  (wire (pts (xy 365.76 60.96) (xy 373.38 60.96))
     (stroke (width 0) (type default))
   )
@@
         (path "/20011966-1ffc-24d7-1b4b-436a182362c4/20011966-6971-43fc-362b-5da89d8c67d5"
           (reference "U1314") (unit 1)
-        )
-      )
-    )
-  )
-  (symbol (lib_id "r1000:PU") (at 373.38 20.32 0) (unit 1)
-    (in_bom yes) (on_board yes) (dnp no)
-    (property "Reference" "#PWR01308" (at 373.38 20.32 0)
-      (effects (font (size 1.27 1.27)) hide)
-    )
-    (property "Value" "PU" (at 373.38 20.32 0)
-      (effects (font (size 1.27 1.27)) hide)
-    )
-    (property "Footprint" "" (at 373.38 20.32 0)
-      (effects (font (size 1.27 1.27)) hide)
-    )
-    (property "Datasheet" "" (at 373.38 20.32 0)
-      (effects (font (size 1.27 1.27)) hide)
-    )
-    (pin "1")
-    (instances
-      (project "SEQ"
-        (path "/20011966-1ffc-24d7-1b4b-436a182362c4/20011966-6971-43fc-362b-5da89d8c67d5"
-          (reference "#PWR01308") (unit 1)
         )
       )
@@
         )
       )
-    )
-  )
-  (symbol (lib_id "r1000:PU") (at 365.76 60.96 0) (unit 1)
-    (in_bom yes) (on_board yes) (dnp no)
-    (property "Reference" "#PWR01307" (at 365.76 60.96 0)
-      (effects (font (size 1.27 1.27)) hide)
-    )
-    (property "Value" "PU" (at 365.76 60.96 0)
-      (effects (font (size 1.27 1.27)) hide)
-    )
-    (property "Footprint" "" (at 365.76 60.96 0)
-      (effects (font (size 1.27 1.27)) hide)
-    )
-    (property "Datasheet" "" (at 365.76 60.96 0)
-      (effects (font (size 1.27 1.27)) hide)
-    )
-    (pin "1")
-    (instances
-      (project "SEQ"
-        (path "/20011966-1ffc-24d7-1b4b-436a182362c4/20011966-6971-43fc-362b-5da89d8c67d5"
-          (reference "#PWR01307") (unit 1)
-        )
-      )

Commit message: Schematics for run rr026
Connections:
- net DISP_TIME.B: no longer names the net of U1326.13 (Q2)
- net TSVLD_SIM0: no longer names the net of U1326.14 (Q1)
- no-connect marks 5 -> 7
Changed lines of the file:
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@@
   )
   (no_connect (at 373.38 25.4))
+  (no_connect (at 487.68 154.94))
   (no_connect (at 373.38 60.96))
   (no_connect (at 386.08 38.1))
+  (no_connect (at 487.68 160.02))
   (no_connect (at 281.94 86.36))
   (no_connect (at 454.66 170.18))
@@
     (stroke (width 0) (type default))
   )
-  (wire (pts (xy 487.68 160.02) (xy 523.24 160.02))
-    (stroke (width 0) (type default))
-  )
   (wire (pts (xy 454.66 165.1) (xy 452.12 165.1))
     (stroke (width 0) (type default))
@@
   )
   (wire (pts (xy 193.04 154.94) (xy 193.04 104.14))
-    (stroke (width 0) (type default))
-  )
-  (wire (pts (xy 487.68 154.94) (xy 523.24 154.94))
     (stroke (width 0) (type default))
   )
@@
     (effects (font (size 2.54 2.54)) (justify left bottom))
   )
-  (label "DISP_TIME.B" (at 500.38 160.02 0) (fields_autoplaced)
-    (effects (font (size 2.54 2.54)) (justify left bottom))
-  )
   (label "MEM_STRT.DEC~1" (at 66.04 144.78 0) (fields_autoplaced)
     (effects (font (size 2.54 2.54)) (justify left bottom))
@@
     (effects (font (size 2.54 2.54)) (justify left bottom))
   )
-  (label "TSVLD_SIM0" (at 500.38 154.94 0) (fields_autoplaced)
-    (effects (font (size 2.54 2.54)) (justify left bottom))
-  )
